File: Tester/ECAD/ControllerBoard/SignalInputOuput.sch (KiCad schematic (older format))
At the start: 10 parts

Commit message: Added the Manufacturer Part Number component field.
Parts:
- J? (x10): Manufacturer Part Number (none) -> tbd
Changed lines of the file:
@@
 F 2 "" H 1700 2850 50  0001 C CNN
 F 3 "~" H 1700 2850 50  0001 C CNN
+F 4 "tbd" H 1700 2850 50  0001 C CNN "Manufacturer Part Number"
 	1    1700 2850
 	1    0    0    -1
@@
 F 2 "" H 1700 3250 50  0001 C CNN
 F 3 "~" H 1700 3250 50  0001 C CNN
+F 4 "tbd" H 1700 3250 50  0001 C CNN "Manufacturer Part Number"
 	1    1700 3250
 	1    0    0    -1
@@
 F 2 "" H 1700 3650 50  0001 C CNN
 F 3 "~" H 1700 3650 50  0001 C CNN
+F 4 "tbd" H 1700 3650 50  0001 C CNN "Manufacturer Part Number"
 	1    1700 3650
 	1    0    0    -1
@@
 F 2 "" H 1700 4050 50  0001 C CNN
 F 3 "~" H 1700 4050 50  0001 C CNN
+F 4 "tbd" H 1700 4050 50  0001 C CNN "Manufacturer Part Number"
 	1    1700 4050
 	1    0    0    -1
@@
 F 2 "" H 1700 4450 50  0001 C CNN
 F 3 "~" H 1700 4450 50  0001 C CNN
+F 4 "tbd" H 1700 4450 50  0001 C CNN "Manufacturer Part Number"
 	1    1700 4450
 	1    0    0    -1
@@
 F 2 "" H 1700 4850 50  0001 C CNN
 F 3 "~" H 1700 4850 50  0001 C CNN
+F 4 "tbd" H 1700 4850 50  0001 C CNN "Manufacturer Part Number"
 	1    1700 4850
 	1    0    0    -1
@@
 F 2 "" H 10250 5800 50  0001 C CNN
 F 3 "~" H 10250 5800 50  0001 C CNN
+F 4 "tbd" H 10250 5800 50  0001 C CNN "Manufacturer Part Number"
 	1    10250 5800
 	-1   0    0    -1
@@
 F 2 "" H 10250 4400 50  0001 C CNN
 F 3 "~" H 10250 4400 50  0001 C CNN
+F 4 "tbd" H 10250 4400 50  0001 C CNN "Manufacturer Part Number"
 	1    10250 4400
 	-1   0    0    -1
@@
 F 2 "" H 10250 2750 50  0001 C CNN
 F 3 "~" H 10250 2750 50  0001 C CNN
+F 4 "tbd" H 10250 2750 50  0001 C CNN "Manufacturer Part Number"
 	1    10250 2750
 	-1   0    0    -1
@@
 F 2 "" H 10250 1200 50  0001 C CNN
 F 3 "~" H 10250 1200 50  0001 C CNN
+F 4 "tbd" H 10250 1200 50  0001 C CNN "Manufacturer Part Number"
 	1    10250 1200
 	-1   0    0    -1

Commit message: Progressed component assigment.
Parts:
- J10, J11, J6, J7, J8, J9: renamed from J?; Manufacturer Part Number tbd -> 0530480210
- J12, J13, J14: renamed from J?; Manufacturer Part Number tbd -> 0530480810
- J15: renamed from J?; Manufacturer Part Number tbd -> 0530480410
Changed lines of the file:
@@
 P 1700 2850
 AR Path="/5E5070AC/5E55B73E" Ref="J?"  Part="1"
-AR Path="/5E55806E/5E55B73E" Ref="J?"  Part="1"
-F 0 "J?" H 1808 3031 50  0000 C CNN
+AR Path="/5E55806E/5E55B73E" Ref="J6"  Part="1"
+F 0 "J6" H 1808 3031 50  0000 C CNN
 F 1 "Conn_01x02_Male" H 1808 2940 50  0000 C CNN
 F 2 "" H 1700 2850 50  0001 C CNN
 F 3 "~" H 1700 2850 50  0001 C CNN
-F 4 "tbd" H 1700 2850 50  0001 C CNN "Manufacturer Part Number"
+F 4 "0530480210" H 1700 2850 50  0001 C CNN "Manufacturer Part Number"
 	1    1700 2850
 	1    0    0    -1
@@
 P 1700 3250
 AR Path="/5E5070AC/5E55B744" Ref="J?"  Part="1"
-AR Path="/5E55806E/5E55B744" Ref="J?"  Part="1"
-F 0 "J?" H 1808 3431 50  0000 C CNN
+AR Path="/5E55806E/5E55B744" Ref="J7"  Part="1"
+F 0 "J7" H 1808 3431 50  0000 C CNN
 F 1 "Conn_01x02_Male" H 1808 3340 50  0000 C CNN
 F 2 "" H 1700 3250 50  0001 C CNN
 F 3 "~" H 1700 3250 50  0001 C CNN
-F 4 "tbd" H 1700 3250 50  0001 C CNN "Manufacturer Part Number"
+F 4 "0530480210" H 1700 3250 50  0001 C CNN "Manufacturer Part Number"
 	1    1700 3250
 	1    0    0    -1
@@
 P 1700 3650
 AR Path="/5E5070AC/5E55B74A" Ref="J?"  Part="1"
-AR Path="/5E55806E/5E55B74A" Ref="J?"  Part="1"
-F 0 "J?" H 1808 3831 50  0000 C CNN
+AR Path="/5E55806E/5E55B74A" Ref="J8"  Part="1"
+F 0 "J8" H 1808 3831 50  0000 C CNN
 F 1 "Conn_01x02_Male" H 1808 3740 50  0000 C CNN
 F 2 "" H 1700 3650 50  0001 C CNN
 F 3 "~" H 1700 3650 50  0001 C CNN
-F 4 "tbd" H 1700 3650 50  0001 C CNN "Manufacturer Part Number"
+F 4 "0530480210" H 1700 3650 50  0001 C CNN "Manufacturer Part Number"
 	1    1700 3650
 	1    0    0    -1
@@
 P 1700 4050
 AR Path="/5E5070AC/5E55B750" Ref="J?"  Part="1"
-AR Path="/5E55806E/5E55B750" Ref="J?"  Part="1"
-F 0 "J?" H 1808 4231 50  0000 C CNN
+AR Path="/5E55806E/5E55B750" Ref="J9"  Part="1"
+F 0 "J9" H 1808 4231 50  0000 C CNN
 F 1 "Conn_01x02_Male" H 1808 4140 50  0000 C CNN
 F 2 "" H 1700 4050 50  0001 C CNN
 F 3 "~" H 1700 4050 50  0001 C CNN
-F 4 "tbd" H 1700 4050 50  0001 C CNN "Manufacturer Part Number"
+F 4 "0530480210" H 1700 4050 50  0001 C CNN "Manufacturer Part Number"
 	1    1700 4050
 	1    0    0    -1
@@
 P 1700 4450
 AR Path="/5E5070AC/5E55B756" Ref="J?"  Part="1"
-AR Path="/5E55806E/5E55B756" Ref="J?"  Part="1"
-F 0 "J?" H 1808 4631 50  0000 C CNN
+AR Path="/5E55806E/5E55B756" Ref="J10"  Part="1"
+F 0 "J10" H 1808 4631 50  0000 C CNN
 F 1 "Conn_01x02_Male" H 1808 4540 50  0000 C CNN
 F 2 "" H 1700 4450 50  0001 C CNN
 F 3 "~" H 1700 4450 50  0001 C CNN
-F 4 "tbd" H 1700 4450 50  0001 C CNN "Manufacturer Part Number"
+F 4 "0530480210" H 1700 4450 50  0001 C CNN "Manufacturer Part Number"
 	1    1700 4450
 	1    0    0    -1
@@
 P 1700 4850
 AR Path="/5E5070AC/5E55B75C" Ref="J?"  Part="1"
-AR Path="/5E55806E/5E55B75C" Ref="J?"  Part="1"
-F 0 "J?" H 1808 5031 50  0000 C CNN
+AR Path="/5E55806E/5E55B75C" Ref="J11"  Part="1"
+F 0 "J11" H 1808 5031 50  0000 C CNN
 F 1 "Conn_01x02_Male" H 1808 4940 50  0000 C CNN
 F 2 "" H 1700 4850 50  0001 C CNN
 F 3 "~" H 1700 4850 50  0001 C CNN
-F 4 "tbd" H 1700 4850 50  0001 C CNN "Manufacturer Part Number"
+F 4 "0530480210" H 1700 4850 50  0001 C CNN "Manufacturer Part Number"
 	1    1700 4850
 	1    0    0    -1
@@
 P 10250 5800
 AR Path="/5E5070AC/5E560967" Ref="J?"  Part="1"
-AR Path="/5E55806E/5E560967" Ref="J?"  Part="1"
-F 0 "J?" H 10358 6081 50  0000 C CNN
+AR Path="/5E55806E/5E560967" Ref="J15"  Part="1"
+F 0 "J15" H 10358 6081 50  0000 C CNN
 F 1 "Conn_01x04_Male" H 10358 5990 50  0000 C CNN
 F 2 "" H 10250 5800 50  0001 C CNN
 F 3 "~" H 10250 5800 50  0001 C CNN
-F 4 "tbd" H 10250 5800 50  0001 C CNN "Manufacturer Part Number"
+F 4 "0530480410" H 10250 5800 50  0001 C CNN "Manufacturer Part Number"
 	1    10250 5800
 	-1   0    0    -1
@@
 P 10250 4400
 AR Path="/5E5070AC/5E56096D" Ref="J?"  Part="1"
-AR Path="/5E55806E/5E56096D" Ref="J?"  Part="1"
-F 0 "J?" H 10358 4881 50  0000 C CNN
+AR Path="/5E55806E/5E56096D" Ref="J14"  Part="1"
+F 0 "J14" H 10358 4881 50  0000 C CNN
 F 1 "Conn_01x08_Male" H 10358 4790 50  0000 C CNN
 F 2 "" H 10250 4400 50  0001 C CNN
 F 3 "~" H 10250 4400 50  0001 C CNN
-F 4 "tbd" H 10250 4400 50  0001 C CNN "Manufacturer Part Number"
+F 4 "0530480810" H 10250 4400 50  0001 C CNN "Manufacturer Part Number"
 	1    10250 4400
 	-1   0    0    -1
@@
 P 10250 2750
 AR Path="/5E5070AC/5E560973" Ref="J?"  Part="1"
-AR Path="/5E55806E/5E560973" Ref="J?"  Part="1"
-F 0 "J?" H 10358 3231 50  0000 C CNN
+AR Path="/5E55806E/5E560973" Ref="J13"  Part="1"
+F 0 "J13" H 10358 3231 50  0000 C CNN
 F 1 "Conn_01x08_Male" H 10358 3140 50  0000 C CNN
 F 2 "" H 10250 2750 50  0001 C CNN
 F 3 "~" H 10250 2750 50  0001 C CNN
-F 4 "tbd" H 10250 2750 50  0001 C CNN "Manufacturer Part Number"
+F 4 "0530480810" H 10250 2750 50  0001 C CNN "Manufacturer Part Number"
 	1    10250 2750
 	-1   0    0    -1
@@
 P 10250 1200
 AR Path="/5E5070AC/5E560979" Ref="J?"  Part="1"
-AR Path="/5E55806E/5E560979" Ref="J?"  Part="1"
-F 0 "J?" H 10358 1681 50  0000 C CNN
+AR Path="/5E55806E/5E560979" Ref="J12"  Part="1"
+F 0 "J12" H 10358 1681 50  0000 C CNN
 F 1 "Conn_01x08_Male" H 10358 1590 50  0000 C CNN
 F 2 "" H 10250 1200 50  0001 C CNN
 F 3 "~" H 10250 1200 50  0001 C CNN
-F 4 "tbd" H 10250 1200 50  0001 C CNN "Manufacturer Part Number"
+F 4 "0530480810" H 10250 1200 50  0001 C CNN "Manufacturer Part Number"
 	1    10250 1200
 	-1   0    0    -1

Commit message: Component assigment cont.
Parts:
- J10, J11, J6, J7, J8, J9: footprint (none) -> Connector_Molex:Molex_PicoBlade_53048-0210_1x02_P1.25mm_Horizontal
- J12, J13, J14: footprint (none) -> Connector_Molex:Molex_PicoBlade_53048-0810_1x08_P1.25mm_Horizontal
- J15: footprint (none) -> Connector_Molex:Molex_PicoBlade_53048-0410_1x04_P1.25mm_Horizontal
Changed lines of the file:
@@
 F 0 "J6" H 1808 3031 50  0000 C CNN
 F 1 "Conn_01x02_Male" H 1808 2940 50  0000 C CNN
-F 2 "" H 1700 2850 50  0001 C CNN
+F 2 "Connector_Molex:Molex_PicoBlade_53048-0210_1x02_P1.25mm_Horizontal" H 1700 2850 50  0001 C CNN
 F 3 "~" H 1700 2850 50  0001 C CNN
 F 4 "0530480210" H 1700 2850 50  0001 C CNN "Manufacturer Part Number"
@@
 F 0 "J7" H 1808 3431 50  0000 C CNN
 F 1 "Conn_01x02_Male" H 1808 3340 50  0000 C CNN
-F 2 "" H 1700 3250 50  0001 C CNN
+F 2 "Connector_Molex:Molex_PicoBlade_53048-0210_1x02_P1.25mm_Horizontal" H 1700 3250 50  0001 C CNN
 F 3 "~" H 1700 3250 50  0001 C CNN
 F 4 "0530480210" H 1700 3250 50  0001 C CNN "Manufacturer Part Number"
@@
 F 0 "J8" H 1808 3831 50  0000 C CNN
 F 1 "Conn_01x02_Male" H 1808 3740 50  0000 C CNN
-F 2 "" H 1700 3650 50  0001 C CNN
+F 2 "Connector_Molex:Molex_PicoBlade_53048-0210_1x02_P1.25mm_Horizontal" H 1700 3650 50  0001 C CNN
 F 3 "~" H 1700 3650 50  0001 C CNN
 F 4 "0530480210" H 1700 3650 50  0001 C CNN "Manufacturer Part Number"
@@
 F 0 "J9" H 1808 4231 50  0000 C CNN
 F 1 "Conn_01x02_Male" H 1808 4140 50  0000 C CNN
-F 2 "" H 1700 4050 50  0001 C CNN
+F 2 "Connector_Molex:Molex_PicoBlade_53048-0210_1x02_P1.25mm_Horizontal" H 1700 4050 50  0001 C CNN
 F 3 "~" H 1700 4050 50  0001 C CNN
 F 4 "0530480210" H 1700 4050 50  0001 C CNN "Manufacturer Part Number"
@@
 F 0 "J10" H 1808 4631 50  0000 C CNN
 F 1 "Conn_01x02_Male" H 1808 4540 50  0000 C CNN
-F 2 "" H 1700 4450 50  0001 C CNN
+F 2 "Connector_Molex:Molex_PicoBlade_53048-0210_1x02_P1.25mm_Horizontal" H 1700 4450 50  0001 C CNN
 F 3 "~" H 1700 4450 50  0001 C CNN
 F 4 "0530480210" H 1700 4450 50  0001 C CNN "Manufacturer Part Number"
@@
 F 0 "J11" H 1808 5031 50  0000 C CNN
 F 1 "Conn_01x02_Male" H 1808 4940 50  0000 C CNN
-F 2 "" H 1700 4850 50  0001 C CNN
+F 2 "Connector_Molex:Molex_PicoBlade_53048-0210_1x02_P1.25mm_Horizontal" H 1700 4850 50  0001 C CNN
 F 3 "~" H 1700 4850 50  0001 C CNN
 F 4 "0530480210" H 1700 4850 50  0001 C CNN "Manufacturer Part Number"
@@
 F 0 "J15" H 10358 6081 50  0000 C CNN
 F 1 "Conn_01x04_Male" H 10358 5990 50  0000 C CNN
-F 2 "" H 10250 5800 50  0001 C CNN
+F 2 "Connector_Molex:Molex_PicoBlade_53048-0410_1x04_P1.25mm_Horizontal" H 10250 5800 50  0001 C CNN
 F 3 "~" H 10250 5800 50  0001 C CNN
 F 4 "0530480410" H 10250 5800 50  0001 C CNN "Manufacturer Part Number"
@@
 F 0 "J14" H 10358 4881 50  0000 C CNN
 F 1 "Conn_01x08_Male" H 10358 4790 50  0000 C CNN
-F 2 "" H 10250 4400 50  0001 C CNN
+F 2 "Connector_Molex:Molex_PicoBlade_53048-0810_1x08_P1.25mm_Horizontal" H 10250 4400 50  0001 C CNN
 F 3 "~" H 10250 4400 50  0001 C CNN
 F 4 "0530480810" H 10250 4400 50  0001 C CNN "Manufacturer Part Number"
@@
 F 0 "J13" H 10358 3231 50  0000 C CNN
 F 1 "Conn_01x08_Male" H 10358 3140 50  0000 C CNN
-F 2 "" H 10250 2750 50  0001 C CNN
+F 2 "Connector_Molex:Molex_PicoBlade_53048-0810_1x08_P1.25mm_Horizontal" H 10250 2750 50  0001 C CNN
 F 3 "~" H 10250 2750 50  0001 C CNN
 F 4 "0530480810" H 10250 2750 50  0001 C CNN "Manufacturer Part Number"
@@
 F 0 "J12" H 10358 1681 50  0000 C CNN
 F 1 "Conn_01x08_Male" H 10358 1590 50  0000 C CNN
-F 2 "" H 10250 1200 50  0001 C CNN
+F 2 "Connector_Molex:Molex_PicoBlade_53048-0810_1x08_P1.25mm_Horizontal" H 10250 1200 50  0001 C CNN
 F 3 "~" H 10250 1200 50  0001 C CNN
 F 4 "0530480810" H 10250 1200 50  0001 C CNN "Manufacturer Part Number"

Commit message: Progressed circuit layout.
Connections:
- net labels added: END_STOP_X, END_STOP_Y, END_STOP_Z, VPOS_SENS_5V, V_LASER_5V
- net labels removed: VCC_5V
- wire segments 40 -> 12

Commit message: Progressed circuit layout.
Connections:
- net labels added: VPOS_SENS_3.3V
- net labels removed: END_STOP_X, END_STOP_Y, END_STOP_Z, LASER_SCL, LASER_SDA, VPOS_SENS_5V
- wire segments 12 -> 0
Other:
- note added: "1 5V\n2 ~NCS\n3 MISO\n4 MOSI\n5 SCLK\n6 MOTION\n7 ~NRESET\n8 GND"
- note added: "1 GND\n2 SDA\n3 SCL\n4 5V"
- moved on the sheet: J10, J11, J15, J6, J7, J8, J9

Commit message: Progressed circuit design.
Parts:
- added C18, C19, C20, C21, C22, C23: 0.1uC, Capacitor_SMD:C_0805_2012Metric_Pad1.15x1.40mm_HandSolder, symbol Device:C
- added R10, R11, R12, R13, R14, R15, R16, R17, R18, R7, R8, R9: 10kR, Resistor_SMD:R_0805_2012Metric_Pad1.15x1.40mm_HandSolder, symbol Device:R
- added U5: 74HC14, Package_SO:SOIC-14_3.9x8.7mm_P1.27mm, symbol 74xx:74HC14
Connections:
- net labels added: LASER_SCL, LASER_SDA, VMCU, VPOS_SENS_5V
- net labels removed: VPOS_SENS_3.3V
- wire segments 0 -> 95
Other:
- note added: "Level shifting logic"
- note added: "Switch debouncing logic."
- moved on the sheet: J10, J11, J15, J6, J7, J8, J9

Commit message: Update SignalInputOuput.sch
Parts:
- added Q1, Q2: BSS138, Package_TO_SOT_SMD:SOT-23, symbol Transistor_FET:BSS138
- added R19, R20, R21, R22: 10kR, Resistor_SMD:R_0805_2012Metric_Pad1.15x1.40mm_HandSolder, symbol Device:R
Connections:
- wire segments 95 -> 115
Changed lines of the file:
@@
 	5650 1750 5750 1750
-Wire Wire Line
-	5750 1750 5750 7450
 Wire Wire Line
 	5750 7450 2350 7450
@@
 Wire Wire Line
 	5750 1450 5650 1450
-Text HLabel 6300 1500 2    50   BiDi ~ 0
+Text HLabel 6900 1850 2    50   BiDi ~ 0
 LASER_SDA
-Text HLabel 6300 1650 2    50   Input ~ 0
+Text HLabel 6900 1200 2    50   Input ~ 0
 LASER_SCL
-Text Notes 5900 1250 0    50   ~ 0
+Text Notes 6000 700  0    50   ~ 0
 Level shifting logic
+$Comp
+L Transistor_FET:BSS138 Q1
+U 1 1 5E5993CA
+P 6350 1300
+F 0 "Q1" V 6692 1300 50  0000 C CNN
+F 1 "BSS138" V 6601 1300 50  0000 C CNN
+F 2 "Package_TO_SOT_SMD:SOT-23" H 6550 1225 50  0001 L CIN
+F 3 "https://www.fairchildsemi.com/datasheets/BS/BSS138.pdf" H 6350 1300 50  0001 L CNN
+	1    6350 1300
+	0    -1   -1   0
+$EndComp
+$Comp
+L Transistor_FET:BSS138 Q2
+U 1 1 5E59E66A
+P 6350 1950
+F 0 "Q2" V 6692 1950 50  0000 C CNN
+F 1 "BSS138" V 6601 1950 50  0000 C CNN
+F 2 "Package_TO_SOT_SMD:SOT-23" H 6550 1875 50  0001 L CIN
+F 3 "https://www.fairchildsemi.com/datasheets/BS/BSS138.pdf" H 6350 1950 50  0001 L CNN
+	1    6350 1950
+	0    -1   -1   0
+$EndComp
+$Comp
+L Device:R R21
+U 1 1 5E59FB6E
+P 6550 1350
+F 0 "R21" V 6343 1350 50  0000 C CNN
+F 1 "10kR" V 6434 1350 50  0000 C CNN
+F 2 "Resistor_SMD:R_0805_2012Metric_Pad1.15x1.40mm_HandSolder" V 6480 1350 50  0001 C CNN
+F 3 "~" H 6550 1350 50  0001 C CNN
+	1    6550 1350
+	-1   0    0    1
+$EndComp
+$Comp
+L Device:R R19
+U 1 1 5E5A00FF
+P 6150 1350
+F 0 "R19" V 5943 1350 50  0000 C CNN
+F 1 "10kR" V 6034 1350 50  0000 C CNN
+F 2 "Resistor_SMD:R_0805_2012Metric_Pad1.15x1.40mm_HandSolder" V 6080 1350 50  0001 C CNN
+F 3 "~" H 6150 1350 50  0001 C CNN
+	1    6150 1350
+	1    0    0    -1
+$EndComp
+$Comp
+L Device:R R22
+U 1 1 5E5A053C
+P 6550 2000
+F 0 "R22" V 6343 2000 50  0000 C CNN
+F 1 "10kR" V 6434 2000 50  0000 C CNN
+F 2 "Resistor_SMD:R_0805_2012Metric_Pad1.15x1.40mm_HandSolder" V 6480 2000 50  0001 C CNN
+F 3 "~" H 6550 2000 50  0001 C CNN
+	1    6550 2000
+	-1   0    0    1
+$EndComp
+Wire Wire Line
+	6350 1500 6550 1500
+Wire Wire Line
+	6350 2150 6550 2150
+Wire Wire Line
+	5850 1650 5650 1650
+Connection ~ 6550 1200
+Connection ~ 6550 1850
+Wire Wire Line
+	6150 1200 5850 1200
+Wire Wire Line
+	5850 1200 5850 1550
+Wire Wire Line
+	5850 1550 5650 1550
+Connection ~ 6150 1200
+Wire Wire Line
+	6150 1850 5850 1850
+Wire Wire Line
+	5850 1850 5850 1650
+Connection ~ 6150 1850
+Wire Wire Line
+	5750 1750 5750 7450
+Wire Wire Line
+	5750 1450 6000 1450
+Wire Wire Line
+	6000 1450 6000 1500
+Wire Wire Line
+	6000 2150 6150 2150
+Connection ~ 5750 1450
+Wire Wire Line
+	6150 1500 6000 1500
+Connection ~ 6000 1500
+Wire Wire Line
+	6000 1500 6000 2150
+$Comp
+L Device:R R20
+U 1 1 5E5A0381
+P 6150 2000
+F 0 "R20" V 5943 2000 50  0000 C CNN
+F 1 "10kR" V 6034 2000 50  0000 C CNN
+F 2 "Resistor_SMD:R_0805_2012Metric_Pad1.15x1.40mm_HandSolder" V 6080 2000 50  0001 C CNN
+F 3 "~" H 6150 2000 50  0001 C CNN
+	1    6150 2000
+	1    0    0    -1
+$EndComp
+Wire Wire Line
+	2350 800  6800 800
+Wire Wire Line
+	6800 800  6800 1500
+Wire Wire Line
+	6800 1500 6550 1500
+Connection ~ 2350 800
+Connection ~ 6550 1500
+Wire Wire Line
+	6800 1500 6800 2150
+Wire Wire Line
+	6800 2150 6550 2150
+Connection ~ 6800 1500
+Connection ~ 6550 2150
+Wire Wire Line
+	6550 1200 6900 1200
+Wire Wire Line
+	6550 1850 6900 1850
 $EndSCHEMATC
