File: Tester/ECAD/OpticPositionSensor/OpticPositionSensor.sch (KiCad schematic (older format))
At the start: 18 parts, among them J1 Conn_01x08_Male, U1 TLV70019_SOT23-5, U2 PMW3360DM-T2QU, U3 SN74LVC1T45DBV, U4 SN74LVC1T45DBV, U5 SN74LVC1T45DBV, U6 SN74LVC1T45DBV, U7 SN74LVC1T45DBV, U8 SN74LVC1T45DBV

Commit message: Added the Manufacturer Part Number component field.
Parts:
- C1, C2, C3, C4, H1, H2, H3, H4, J1, R1, U1, U2, U3, U4, U5, U6, U7, U8: Manufacturer Part Number (none) -> tbd
Changed lines of the file:
@@
 F 2 "PixArt:PMW3360DM-T2QU" H 2150 4200 50  0001 C CNN
 F 3 "" H 2150 4200 50  0001 C CNN
+F 4 "tbd" H 2150 4200 50  0001 C CNN "Manufacturer Part Number"
 	1    2150 4200
 	1    0    0    -1
@@
 F 2 "Capacitor_SMD:C_0805_2012Metric_Pad1.15x1.40mm_HandSolder" H 1238 6000 50  0001 C CNN
 F 3 "~" H 1200 6150 50  0001 C CNN
+F 4 "tbd" H 1200 6150 50  0001 C CNN "Manufacturer Part Number"
 	1    1200 6150
 	1    0    0    -1
@@
 F 2 "Capacitor_SMD:C_0805_2012Metric_Pad1.15x1.40mm_HandSolder" H 1688 6000 50  0001 C CNN
 F 3 "~" H 1650 6150 50  0001 C CNN
+F 4 "tbd" H 1650 6150 50  0001 C CNN "Manufacturer Part Number"
 	1    1650 6150
 	1    0    0    -1
@@
 F 2 "Package_TO_SOT_SMD:SOT-23-6_Handsoldering" H 4750 2100 50  0001 C CNN
 F 3 "http://www.ti.com/lit/ds/symlink/sn74lvc1t45.pdf" H 3850 1900 50  0001 C CNN
+F 4 "tbd" H 4750 2550 50  0001 C CNN "Manufacturer Part Number"
 	1    4750 2550
 	1    0    0    -1
@@
 F 2 "Package_TO_SOT_SMD:SOT-23-6_Handsoldering" H 4750 3150 50  0001 C CNN
 F 3 "http://www.ti.com/lit/ds/symlink/sn74lvc1t45.pdf" H 3850 2950 50  0001 C CNN
+F 4 "tbd" H 4750 3600 50  0001 C CNN "Manufacturer Part Number"
 	1    4750 3600
 	1    0    0    -1
@@
 F 2 "Package_TO_SOT_SMD:SOT-23-6_Handsoldering" H 4750 6250 50  0001 C CNN
 F 3 "http://www.ti.com/lit/ds/symlink/sn74lvc1t45.pdf" H 3850 6050 50  0001 C CNN
+F 4 "tbd" H 4750 6700 50  0001 C CNN "Manufacturer Part Number"
 	1    4750 6700
 	1    0    0    -1
@@
 F 2 "Package_TO_SOT_SMD:SOT-23-6_Handsoldering" H 4750 5150 50  0001 C CNN
 F 3 "http://www.ti.com/lit/ds/symlink/sn74lvc1t45.pdf" H 3850 4950 50  0001 C CNN
+F 4 "tbd" H 4750 5600 50  0001 C CNN "Manufacturer Part Number"
 	1    4750 5600
 	1    0    0    -1
@@
 F 2 "Package_TO_SOT_SMD:SOT-23-6_Handsoldering" H 4750 4150 50  0001 C CNN
 F 3 "http://www.ti.com/lit/ds/symlink/sn74lvc1t45.pdf" H 3850 3950 50  0001 C CNN
+F 4 "tbd" H 4750 4600 50  0001 C CNN "Manufacturer Part Number"
 	1    4750 4600
 	1    0    0    -1
@@
 F 2 "Package_TO_SOT_SMD:SOT-23-6_Handsoldering" H 4750 950 50  0001 C CNN
 F 3 "http://www.ti.com/lit/ds/symlink/sn74lvc1t45.pdf" H 3850 750 50  0001 C CNN
+F 4 "tbd" H 4750 1400 50  0001 C CNN "Manufacturer Part Number"
 	1    4750 1400
 	1    0    0    -1
@@
 F 2 "Package_TO_SOT_SMD:SOT-23-5_HandSoldering" H 2050 2025 50  0001 C CIN
 F 3 "http://www.ti.com/lit/ds/symlink/tlv700.pdf" H 2050 1750 50  0001 C CNN
+F 4 "tbd" H 2050 1700 50  0001 C CNN "Manufacturer Part Number"
 	1    2050 1700
 	1    0    0    -1
@@
 F 2 "Capacitor_SMD:C_0805_2012Metric_Pad1.15x1.40mm_HandSolder" H 2588 1700 50  0001 C CNN
 F 3 "~" H 2550 1850 50  0001 C CNN
+F 4 "tbd" H 2550 1850 50  0001 C CNN "Manufacturer Part Number"
 	1    2550 1850
 	1    0    0    -1
@@
 F 2 "Capacitor_SMD:C_0805_2012Metric_Pad1.15x1.40mm_HandSolder" H 1338 1700 50  0001 C CNN
 F 3 "~" H 1300 1850 50  0001 C CNN
+F 4 "tbd" H 1300 1850 50  0001 C CNN "Manufacturer Part Number"
 	1    1300 1850
 	1    0    0    -1
@@
 F 2 "Resistor_SMD:R_0805_2012Metric_Pad1.15x1.40mm_HandSolder" V 2830 3400 50  0001 C CNN
 F 3 "~" H 2900 3400 50  0001 C CNN
+F 4 "tbd" H 2900 3400 50  0001 C CNN "Manufacturer Part Number"
 	1    2900 3400
 	1    0    0    -1
@@
 F 2 "MountingHole:MountingHole_3.2mm_M3_Pad" H 9700 1650 50  0001 C CNN
 F 3 "~" H 9700 1650 50  0001 C CNN
+F 4 "tbd" H 9700 1650 50  0001 C CNN "Manufacturer Part Number"
 	1    9700 1650
 	1    0    0    -1
@@
 F 2 "MountingHole:MountingHole_3.2mm_M3_Pad" H 9700 1950 50  0001 C CNN
 F 3 "~" H 9700 1950 50  0001 C CNN
+F 4 "tbd" H 9700 1950 50  0001 C CNN "Manufacturer Part Number"
 	1    9700 1950
 	1    0    0    -1
@@
 F 2 "MountingHole:MountingHole_3.2mm_M3_Pad" H 9700 2250 50  0001 C CNN
 F 3 "~" H 9700 2250 50  0001 C CNN
+F 4 "tbd" H 9700 2250 50  0001 C CNN "Manufacturer Part Number"
 	1    9700 2250
 	1    0    0    -1
@@
 F 2 "MountingHole:MountingHole_3.2mm_M3_Pad" H 9700 2500 50  0001 C CNN
 F 3 "~" H 9700 2500 50  0001 C CNN
+F 4 "tbd" H 9700 2500 50  0001 C CNN "Manufacturer Part Number"
 	1    9700 2500
 	1    0    0    -1
@@
 F 2 "Connector_Molex:Molex_PicoBlade_53048-0810_1x08_P1.25mm_Horizontal" H 8500 3700 50  0001 C CNN
 F 3 "~" H 8500 3700 50  0001 C CNN
+F 4 "tbd" H 8500 3700 50  0001 C CNN "Manufacturer Part Number"
 	1    8500 3700
 	-1   0    0    1

Commit message: Progressed circuit layout.
Parts:
- U1: Manufacturer Part Number tbd -> TLV70019DDCT
- U3, U4, U5, U6, U7, U8: Manufacturer Part Number tbd -> SN74LVC1T45DBVR
Changed lines of the file:
@@
 F 2 "Package_TO_SOT_SMD:SOT-23-6_Handsoldering" H 4750 2100 50  0001 C CNN
 F 3 "http://www.ti.com/lit/ds/symlink/sn74lvc1t45.pdf" H 3850 1900 50  0001 C CNN
-F 4 "tbd" H 4750 2550 50  0001 C CNN "Manufacturer Part Number"
+F 4 "SN74LVC1T45DBVR" H 4750 2550 50  0001 C CNN "Manufacturer Part Number"
 	1    4750 2550
 	1    0    0    -1
@@
 F 2 "Package_TO_SOT_SMD:SOT-23-6_Handsoldering" H 4750 3150 50  0001 C CNN
 F 3 "http://www.ti.com/lit/ds/symlink/sn74lvc1t45.pdf" H 3850 2950 50  0001 C CNN
-F 4 "tbd" H 4750 3600 50  0001 C CNN "Manufacturer Part Number"
+F 4 "SN74LVC1T45DBVR" H 4750 3600 50  0001 C CNN "Manufacturer Part Number"
 	1    4750 3600
 	1    0    0    -1
@@
 F 2 "Package_TO_SOT_SMD:SOT-23-6_Handsoldering" H 4750 6250 50  0001 C CNN
 F 3 "http://www.ti.com/lit/ds/symlink/sn74lvc1t45.pdf" H 3850 6050 50  0001 C CNN
-F 4 "tbd" H 4750 6700 50  0001 C CNN "Manufacturer Part Number"
+F 4 "SN74LVC1T45DBVR" H 4750 6700 50  0001 C CNN "Manufacturer Part Number"
 	1    4750 6700
 	1    0    0    -1
@@
 F 2 "Package_TO_SOT_SMD:SOT-23-6_Handsoldering" H 4750 5150 50  0001 C CNN
 F 3 "http://www.ti.com/lit/ds/symlink/sn74lvc1t45.pdf" H 3850 4950 50  0001 C CNN
-F 4 "tbd" H 4750 5600 50  0001 C CNN "Manufacturer Part Number"
+F 4 "SN74LVC1T45DBVR" H 4750 5600 50  0001 C CNN "Manufacturer Part Number"
 	1    4750 5600
 	1    0    0    -1
@@
 F 2 "Package_TO_SOT_SMD:SOT-23-6_Handsoldering" H 4750 4150 50  0001 C CNN
 F 3 "http://www.ti.com/lit/ds/symlink/sn74lvc1t45.pdf" H 3850 3950 50  0001 C CNN
-F 4 "tbd" H 4750 4600 50  0001 C CNN "Manufacturer Part Number"
+F 4 "SN74LVC1T45DBVR" H 4750 4600 50  0001 C CNN "Manufacturer Part Number"
 	1    4750 4600
 	1    0    0    -1
@@
 F 2 "Package_TO_SOT_SMD:SOT-23-6_Handsoldering" H 4750 950 50  0001 C CNN
 F 3 "http://www.ti.com/lit/ds/symlink/sn74lvc1t45.pdf" H 3850 750 50  0001 C CNN
-F 4 "tbd" H 4750 1400 50  0001 C CNN "Manufacturer Part Number"
+F 4 "SN74LVC1T45DBVR" H 4750 1400 50  0001 C CNN "Manufacturer Part Number"
 	1    4750 1400
 	1    0    0    -1
@@
 F 2 "Package_TO_SOT_SMD:SOT-23-5_HandSoldering" H 2050 2025 50  0001 C CIN
 F 3 "http://www.ti.com/lit/ds/symlink/tlv700.pdf" H 2050 1750 50  0001 C CNN
-F 4 "tbd" H 2050 1700 50  0001 C CNN "Manufacturer Part Number"
+F 4 "TLV70019DDCT" H 2050 1700 50  0001 C CNN "Manufacturer Part Number"
 	1    2050 1700
 	1    0    0    -1

Commit message: Added BOM components.
Parts:
- J1: Manufacturer Part Number tbd -> 0530480810
- U2: Manufacturer Part Number tbd -> (none)
Changed lines of the file:
@@
 F 2 "PixArt:PMW3360DM-T2QU" H 2150 4200 50  0001 C CNN
 F 3 "" H 2150 4200 50  0001 C CNN
-F 4 "tbd" H 2150 4200 50  0001 C CNN "Manufacturer Part Number"
+F 4 "" H 2150 4200 50  0001 C CNN "Manufacturer Part Number"
 	1    2150 4200
 	1    0    0    -1
@@
 F 2 "Connector_Molex:Molex_PicoBlade_53048-0810_1x08_P1.25mm_Horizontal" H 8500 3700 50  0001 C CNN
 F 3 "~" H 8500 3700 50  0001 C CNN
-F 4 "tbd" H 8500 3700 50  0001 C CNN "Manufacturer Part Number"
+F 4 "0530480810" H 8500 3700 50  0001 C CNN "Manufacturer Part Number"
 	1    8500 3700
 	-1   0    0    1

Commit message: Added bom components.
Parts:
- C1: Manufacturer Part Number tbd -> C0805C475K9PACTU
- C2, C4: Manufacturer Part Number tbd -> CC0805MKX7R7BB105
- C3: Manufacturer Part Number tbd -> CC0805ZRY5V8BB104
- H1, H2, H3, H4: Manufacturer Part Number tbd -> (none)
- R1: Manufacturer Part Number tbd -> RC0805FR-0739RL
Changed lines of the file:
@@
 F 2 "Capacitor_SMD:C_0805_2012Metric_Pad1.15x1.40mm_HandSolder" H 1238 6000 50  0001 C CNN
 F 3 "~" H 1200 6150 50  0001 C CNN
-F 4 "tbd" H 1200 6150 50  0001 C CNN "Manufacturer Part Number"
+F 4 "C0805C475K9PACTU" H 1200 6150 50  0001 C CNN "Manufacturer Part Number"
 	1    1200 6150
 	1    0    0    -1
@@
 F 2 "Capacitor_SMD:C_0805_2012Metric_Pad1.15x1.40mm_HandSolder" H 1688 6000 50  0001 C CNN
 F 3 "~" H 1650 6150 50  0001 C CNN
-F 4 "tbd" H 1650 6150 50  0001 C CNN "Manufacturer Part Number"
+F 4 "CC0805ZRY5V8BB104" H 1650 6150 50  0001 C CNN "Manufacturer Part Number"
 	1    1650 6150
 	1    0    0    -1
@@
 F 2 "Capacitor_SMD:C_0805_2012Metric_Pad1.15x1.40mm_HandSolder" H 2588 1700 50  0001 C CNN
 F 3 "~" H 2550 1850 50  0001 C CNN
-F 4 "tbd" H 2550 1850 50  0001 C CNN "Manufacturer Part Number"
+F 4 "CC0805MKX7R7BB105" H 2550 1850 50  0001 C CNN "Manufacturer Part Number"
 	1    2550 1850
 	1    0    0    -1
@@
 F 2 "Capacitor_SMD:C_0805_2012Metric_Pad1.15x1.40mm_HandSolder" H 1338 1700 50  0001 C CNN
 F 3 "~" H 1300 1850 50  0001 C CNN
-F 4 "tbd" H 1300 1850 50  0001 C CNN "Manufacturer Part Number"
+F 4 "CC0805MKX7R7BB105" H 1300 1850 50  0001 C CNN "Manufacturer Part Number"
 	1    1300 1850
 	1    0    0    -1
@@
 F 2 "Resistor_SMD:R_0805_2012Metric_Pad1.15x1.40mm_HandSolder" V 2830 3400 50  0001 C CNN
 F 3 "~" H 2900 3400 50  0001 C CNN
-F 4 "tbd" H 2900 3400 50  0001 C CNN "Manufacturer Part Number"
+F 4 "RC0805FR-0739RL" H 2900 3400 50  0001 C CNN "Manufacturer Part Number"
 	1    2900 3400
 	1    0    0    -1
@@
 F 2 "MountingHole:MountingHole_3.2mm_M3_Pad" H 9700 1650 50  0001 C CNN
 F 3 "~" H 9700 1650 50  0001 C CNN
-F 4 "tbd" H 9700 1650 50  0001 C CNN "Manufacturer Part Number"
+F 4 "" H 9700 1650 50  0001 C CNN "Manufacturer Part Number"
 	1    9700 1650
 	1    0    0    -1
@@
 F 2 "MountingHole:MountingHole_3.2mm_M3_Pad" H 9700 1950 50  0001 C CNN
 F 3 "~" H 9700 1950 50  0001 C CNN
-F 4 "tbd" H 9700 1950 50  0001 C CNN "Manufacturer Part Number"
+F 4 "" H 9700 1950 50  0001 C CNN "Manufacturer Part Number"
 	1    9700 1950
 	1    0    0    -1
@@
 F 2 "MountingHole:MountingHole_3.2mm_M3_Pad" H 9700 2250 50  0001 C CNN
 F 3 "~" H 9700 2250 50  0001 C CNN
-F 4 "tbd" H 9700 2250 50  0001 C CNN "Manufacturer Part Number"
+F 4 "" H 9700 2250 50  0001 C CNN "Manufacturer Part Number"
 	1    9700 2250
 	1    0    0    -1
@@
 F 2 "MountingHole:MountingHole_3.2mm_M3_Pad" H 9700 2500 50  0001 C CNN
 F 3 "~" H 9700 2500 50  0001 C CNN
-F 4 "tbd" H 9700 2500 50  0001 C CNN "Manufacturer Part Number"
+F 4 "" H 9700 2500 50  0001 C CNN "Manufacturer Part Number"
 	1    9700 2500
 	1    0    0    -1
