File: Tester/ECAD/LightSource/LightSource.kicad_pcb (KiCad board)
At the start: 2 copper layers, 40 x 50 mm, 34 parts, among them J1 Barrel_Jack_Switch, Q1 FZT694BTA, U1 TL431, U2 LM321, U3 L78M09

Commit message: Update LightSource.kicad_pcb
Parts:
- moved TP5 59.5 mm to (112.2, 95.0)
- moved TP6 51.0 mm to (102.2, 90.0)
- moved R7 47.8 mm to (117.8, 85.2)
- moved C2 46.1 mm to (122.0, 85.3)
- moved R8 46.1 mm to (122.0, 83.0), turned to 180 degrees
- moved C3 45.4 mm to (122.0, 91.8), turned to 0 degrees
- moved TP2 43.8 mm to (103.2, 112.5)
- moved U2 43.1 mm to (122.0, 88.5), turned to 180 degrees
- moved R6 37.7 mm to (114.8, 78.5)
- moved R9 36.5 mm to (122.0, 80.8), turned to 0 degrees
- moved TP4 27.6 mm to (125.2, 93.5)
- moved TP1 23.7 mm to (108.5, 112.0)
- moved TP3 12.4 mm to (134.8, 88.5)
- moved C1 6.25 mm to (125.2, 88.5), turned to 90 degrees
- moved R1 3.00 mm to (128.2, 84.5)
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Routing:
- net /Vout: track 0.00 -> 29.1 mm
- net Net-(C1-Pad1): track 0.00 -> 20.4 mm
- net GND: track 0.00 -> 4.55 mm
- net Net-(R5-Pad2): track 0.00 -> 4.46 mm
- net Net-(R4-Pad2): track 0.00 -> 4.19 mm
- net /Vref: track 0.00 -> 4.02 mm
- net +9V: track 0.00 -> 2.31 mm
- net Net-(C2-Pad2): track 0.00 -> 2.28 mm
- net Net-(C2-Pad1): track 0.00 -> 2.28 mm

Commit message: Update LightSource.kicad_pcb
Parts:
- moved TP1 19.6 mm to (114.2, 93.2)
- moved TP5 8.51 mm to (117.8, 88.5)
- moved C4 5.30 mm to (122.0, 109.8), turned to 90 degrees
- moved C5 3.73 mm to (122.0, 105.0), turned to 270 degrees
- moved U3 1.96 mm to (114.8, 107.8)
- moved TP2 1.03 mm to (102.2, 112.8)
Routing:
- net GND: track 4.55 -> 37.3 mm, vias 0 -> 5
- net +12V: track 0.00 -> 7.97 mm
- net Net-(C2-Pad1): track 2.28 -> 8.05 mm
- net Net-(C2-Pad2): track 2.28 -> 6.84 mm
- net +9V: track 2.31 -> 5.97 mm
- added copper zone on B.Cu, net GND
- added copper zone on F.Cu, net GND

Commit message: Update LightSource.kicad_pcb
Parts:
- moved TP1 13.3 mm to (125.2, 100.8)
- moved C5 6.81 mm to (115.2, 104.5), turned to 180 degrees
- moved U3 2.70 mm to (113.2, 110.0)
- moved C4 1.37 mm to (121.0, 110.8)
Routing:
- net GND: track 37.3 -> 45.2 mm, vias 5 -> 9
- net +12V: track 7.97 -> 9.39 mm

Commit message: Update LightSource.kicad_pcb
Parts:
- added REF**: Polarity_Center_Positive_6mm_SilkScreen, Symbol:Polarity_Center_Positive_6mm_SilkScreen, B.Cu at (113.2, 104.5)
- added REF**: KiCad-Logo2_5mm_SilkScreen, Symbol:KiCad-Logo2_5mm_SilkScreen, B.Cu at (120.0, 90.0)
- JP1, JP2, JP3: moved to B.Cu
- moved TP6 22.4 mm to (121.0, 77.8)
- moved JP2 18.7 mm to (111.2, 83.2)
- moved JP3 17.7 mm to (103.2, 83.2)
- moved JP1 15.3 mm to (107.2, 83.2), turned to 90 degrees
- moved TP1 12.5 mm to (114.8, 94.0)
- moved Q1 4.72 mm to (108.5, 83.0)
- moved R6 2.21 mm to (115.7, 80.5)
Routing:
- net +9V: track 6.03 -> 35.1 mm, vias 0 -> 4
- net Net-(JP3-Pad2): track 3.85 -> 24.2 mm
- net Net-(JP2-Pad2): track 3.85 -> 21.2 mm
- net Net-(JP1-Pad2): track 3.75 -> 21.0 mm
- net Net-(Q1-Pad3): track 0.00 -> 14.9 mm
- net /Light Source/Cathode: track 0.00 -> 8.25 mm, vias 0 -> 12
- net Net-(Q1-Pad1): track 0.00 -> 5.12 mm
- net GND: track 45.2 -> 45.1 mm, vias 9 -> 13
- added copper zone on F.Cu, net +9V
- added copper zone on F.Cu, net /Light Source/Cathode
Other:
- board text added: "INPUT: +12 V, 500 mA"

Commit message: Update LightSource.kicad_pcb
Parts:
- moved TP5 0.71 mm to (118.2, 88.0)
Routing:
- net GND: track 45.1 -> 45.9 mm
- net Net-(C2-Pad1): track 8.05 -> 7.47 mm
- net +9V: track 35.1 -> 35.6 mm

Commit message: Update LightSource.kicad_pcb
Parts:
- removed REF**: Polarity_Center_Positive_6mm_SilkScreen, Symbol:Polarity_Center_Positive_6mm_SilkScreen
- removed REF**: KiCad-Logo2_5mm_SilkScreen, Symbol:KiCad-Logo2_5mm_SilkScreen
- RV1, RV2: footprint Potentiometer_THT:Potentiometer_Bourns_3386F_Vertical -> Potentiometer_THT_custom:Potentiometer_Bourns_3362P_Vertical
- moved TP1 20.8 mm to (125.5, 76.2)
- moved RV2 4.51 mm to (133.8, 79.5)
- moved RV1 4.14 mm to (133.8, 92.5)
Routing:
- net +9V: track 35.6 -> 28.2 mm
- net /Vout: track 29.1 -> 24.3 mm
- net Net-(R4-Pad2): track 4.19 -> 5.08 mm

Commit message: Update LightSource.kicad_pcb
Parts:
- added REF**: Polarity_Center_Positive_6mm_SilkScreen, Symbol:Polarity_Center_Positive_6mm_SilkScreen, F.Cu at (104.2, 100.0)
- added REF**: KiCad-Logo2_5mm_SilkScreen, Symbol:KiCad-Logo2_5mm_SilkScreen, B.Cu at (120.0, 105.0)
Other:
- board text added: "Coarse"
- board text added: "Fine"
- board text added: "Laser Diode driver 2021, Nuno Sousa"
