File: Tester/ECAD/LightSourceLED/LightSource.kicad_pcb (KiCad board)
At the start: 2 copper layers, 40 x 50 mm, 12 parts, among them J1 Barrel_Jack_Switch, U3 L78M09

Commit message: Update LightSource.kicad_pcb
Parts:
- REF**: moved to F.Cu
- moved REF** 17.5 mm to (120.0, 105.0)
- moved REF** 1.46 mm to (105.0, 90.0), turned to 90 degrees
Other:
- board text added: "LED driver 2021, Nuno Sousa"
