File: Tester/ECAD/TranslationStageControl/TranslationStageControl.kicad_pcb (KiCad board)
At the start: 2 copper layers, 51.5 x 79.5 mm, 0 parts

Commit message: Progressed CAD
Other:
- board outline removed
