File: Tester/ECAD/USB_RS232_Adapter/USB_RS232_Adapter.kicad_sch (KiCad schematic)
At the start: 4 parts

Commit message: Progressed ECAD.
Parts:
- removed U?: MAX3227, Package_SO:SSOP-16_5.3x6.2mm_P0.65mm, symbol Interface_UART:MAX3227
Other:
- moved on the sheet: J?
Changed lines of the file:
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@@
 (kicad_sch (version 20211123) (generator eeschema)
   (paper "A4")
-  (symbol (lib_id "Connector:DB9_Female_MountingHoles") (at 261.62 88.9 0) (unit 1)
+  (symbol (lib_id "Connector:DB9_Female_MountingHoles") (at 242.57 87.63 0) (unit 1)
     (in_bom yes) (on_board yes) (fields_autoplaced)
-    (property "Reference" "J?" (id 0) (at 266.7 87.6299 0)
+    (property "Reference" "J?" (id 0) (at 247.65 86.3599 0)
       (effects (font (size 1.27 1.27)) (justify left))
     )
-    (property "Value" "DB9_Female_MountingHoles" (id 1) (at 266.7 90.1699 0)
+    (property "Value" "DB9_Female_MountingHoles" (id 1) (at 247.65 88.8999 0)
       (effects (font (size 1.27 1.27)) (justify left))
     )
-    (property "Footprint" "" (id 2) (at 261.62 88.9 0)
+    (property "Footprint" "" (id 2) (at 242.57 87.63 0)
       (effects (font (size 1.27 1.27)) hide)
     )
-    (property "Datasheet" " ~" (id 3) (at 261.62 88.9 0)
+    (property "Datasheet" " ~" (id 3) (at 242.57 87.63 0)
       (effects (font (size 1.27 1.27)) hide)
     )
     (pin "0")
     (pin "1")
-    (pin "2")
-    (pin "3")
-    (pin "4")
-    (pin "5")
-    (pin "6")
-    (pin "7")
-    (pin "8")
-    (pin "9")
-  )
-  (symbol (lib_id "Interface_UART:MAX3227") (at 210.82 83.82 0) (unit 1)
-    (in_bom yes) (on_board yes) (fields_autoplaced)
-    (property "Reference" "U?" (id 0) (at 212.8394 53.34 0)
-      (effects (font (size 1.27 1.27)) (justify left))
-    )
-    (property "Value" "MAX3227" (id 1) (at 212.8394 55.88 0)
-      (effects (font (size 1.27 1.27)) (justify left))
-    )
-    (property "Footprint" "Package_SO:SSOP-16_5.3x6.2mm_P0.65mm" (id 2) (at 210.82 116.84 0)
-      (effects (font (size 1.27 1.27)) hide)
-    )
-    (property "Datasheet" "https://datasheets.maximintegrated.com/en/ds/MAX3224-MAX3245.pdf" (id 3) (at 210.82 81.28 0)
-      (effects (font (size 1.27 1.27)) hide)
-    )
-    (pin "1")
-    (pin "10")
-    (pin "11")
-    (pin "12")
-    (pin "13")
-    (pin "14")
-    (pin "15")
-    (pin "16")
     (pin "2")
     (pin "3")
@@
       (reference "J?") (unit 1) (value "USB_B") (footprint "")
     )
-    (path "/37c2e270-ade2-49f7-8b14-4c158a4bd5ad"
-      (reference "U?") (unit 1) (value "MAX3227") (footprint "Package_SO:SSOP-16_5.3x6.2mm_P0.65mm")
-    )
     (path "/e1de4777-bf27-4a74-bb99-7d2b1f61ea04"

Commit message: Progressed ECAD
Parts:
- removed J?: DB9_Female_MountingHoles, symbol Connector:DB9_Female_MountingHoles
- added J2: DB9_Male, Connector_Dsub:DSUB-9_Male_Horizontal_P2.77x2.84mm_EdgePinOffset7.70mm_Housed_MountingHolesOffset9.12mm, symbol Connector:DB9_Male
- added U2: SP213E, Package_SO:SSOP-28_5.3x10.2mm_P0.65mm, symbol Interface_UART_custom:MAX213
- J1: renamed from J?; footprint (none) -> Connector_USB:USB_B_OST_USB-B1HSxx_Horizontal; Manufacturer Part Number (none) -> U241-041N-1BR85-1
- U1: renamed from U?; Manufacturer Part Number (none) -> CH340T
Connections:
- new net CTS: J2.8, U2.4 (RIN2)
- new net DCD: J2.1, U2.18 (RIN5)
- new net DSR: J2.6, U2.27 (RIN3)
- new net DTR: J2.4, U2.3 (DOUT2)
- new net GND: J2.5
- new net RI: J2.9, U2.23 (RIN4)
- new net RTS: J2.7, U2.1 (DOUT3)
- new net RX: J2.2, U2.9 (RIN1)
- new net TX: J2.3, U2.2 (DOUT1)
Other:
- moved on the sheet: J1, U1

Commit message: Progressed ECAD
Parts:
- added C1, C11, C12, C2, C3, C6, C7: 0.1uC, Capacitor_SMD:C_0805_2012Metric_Pad1.18x1.45mm_HandSolder, symbol Device:C
- added C10, C9: 33pC, Capacitor_SMD:C_0805_2012Metric_Pad1.18x1.45mm_HandSolder, symbol Device:C
- added C4: 4.7nC, Capacitor_SMD:C_0805_2012Metric_Pad1.18x1.45mm_HandSolder, symbol Device:C
- added C8: 10uC, Capacitor_SMD:C_0805_2012Metric_Pad1.18x1.45mm_HandSolder, symbol Device:C
- added FB1: FerriteBead_Small, Inductor_SMD:L_0805_2012Metric_Pad1.15x1.40mm_HandSolder, symbol Device:FerriteBead_Small
- added R1: 1MR, Resistor_SMD:R_0805_2012Metric_Pad1.20x1.40mm_HandSolder, symbol Device:R
- added U3: USBLC6-2SC6, Package_TO_SOT_SMD:SOT-23-6, symbol Power_Protection:USBLC6-2SC6
- added Y1: 12MHz, symbol Device:Crystal
Connections:
- net GND: now also J1.4 (GND), U1.8 (GND), U2.10 (GND), C1.1, C10.2, C12.1, C4.2, C6.1, C7.1, C8.1, C9.2, R1.2, U3.2 (GND)
- net VBUS: now reaches U2.11 (VCC)
- net VBUS: now also U1.19 (VCC), C11.2, C12.2, C6.2, C8.2, FB1.1, U3.5 (VBUS)
- net C1+: now reaches U2.12 (C1+)
- net C1+: now also C2.2
- net V+: now reaches U2.13 (V+)
- net V+: now also C11.1
- net C1-: now reaches U2.14 (C1-)
- net C1-: now also C2.1
- net C2+: now reaches U2.15 (C2+)
- net C2+: now also C3.2
- net C2-: now reaches U2.16 (C2-)
- net C2-: now also C3.1
- net V-: now reaches U2.17 (V-)
- net V-: now also C1.2
- net at U2.19 (ROUT5): now also U1.14 (~{DCD})
- net at U2.20 (DIN3): now also U1.16 (~{RTS})
- net at U2.22 (ROUT4): now also U1.13 (~{RI})
- net at U2.26 (ROUT3): now also U1.12 (~{DSR})
- net at U2.5 (ROUT2): now also U1.11 (~{CTS})
- net at U2.6 (DIN2): now also U1.15 (~{DTR})
- net at U2.7 (DIN1): now also U1.3 (TXD)
- net at U2.8 (ROUT1): now also U1.4 (RXD)
- net at J1.1 (VBUS): now also FB1.2
- net at J1.2 (D-): now also U3.1 (I/O1)
- net at J1.3 (D+): now also U3.3 (I/O2)
- net at J1.5 (Shield): now also C4.1, R1.1
- net at U1.10 (XO): now also C10.1, Y1.2
- net V3: now reaches U1.5 (V3)
- net V3: now also C7.2
- net at U1.6 (UD+): now also U3.4 (I/O2)
- net at U1.7 (UD-): now also U3.6 (I/O1)
- net at U1.9 (XI): now also C9.1, Y1.1
- no-connect marks 0 -> 3
Other:
- note added: "RS232 Level Translator"
- note added: "USB interface"
- note added: "USB to RS232"
- moved on the sheet: J1, J2, U1, U2

Commit message: Update USB_RS232_Adapter.kicad_sch
Parts:
- added F1: Polyfuse, Fuse:Fuse_0805_2012Metric_Pad1.15x1.40mm_HandSolder, symbol Device:Polyfuse_Small
- C4: Manufacturer Part Number (none) -> CC0805KRX7R9BB472
- FB1: value FerriteBead_Small -> FerriteBead; Manufacturer Part Number (none) -> BLM21BB050SN1D
- R1: Manufacturer Part Number (none) -> RC0805FR-071ML
- U3: Manufacturer Part Number (none) -> USBLC6-2SC6
Connections:
- net at J1.1 (VBUS): now also F1.1; no longer FB1.2
- new net: F1.2, FB1.2
Other:
- moved on the sheet: FB1
Changed lines of the file:
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@@
     (stroke (width 0) (type default) (color 0 0 0 0))
   )
-  (wire (pts (xy 59.69 104.14) (xy 73.66 104.14))
+  (wire (pts (xy 64.77 104.14) (xy 73.66 104.14))
     (stroke (width 0) (type default) (color 0 0 0 0))
   )
@@
     (stroke (width 0) (type default) (color 0 0 0 0))
   )
+  (wire (pts (xy 73.66 102.87) (xy 73.66 104.14))
+    (stroke (width 0) (type default) (color 0 0 0 0))
+  )
   (wire (pts (xy 166.37 104.14) (xy 166.37 123.19))
     (stroke (width 0) (type default) (color 0 0 0 0))
@@
     (stroke (width 0) (type default) (color 0 0 0 0))
   )
+  (wire (pts (xy 52.07 104.14) (xy 59.69 104.14))
+    (stroke (width 0) (type default) (color 0 0 0 0))
+  )
   (wire (pts (xy 176.53 101.6) (xy 181.61 101.6))
     (stroke (width 0) (type default) (color 0 0 0 0))
   )
-  (wire (pts (xy 73.66 104.14) (xy 73.66 102.87))
-    (stroke (width 0) (type default) (color 0 0 0 0))
-  )
   (wire (pts (xy 88.9 120.65) (xy 88.9 109.22))
     (stroke (width 0) (type default) (color 0 0 0 0))
@@
     (stroke (width 0) (type default) (color 0 0 0 0))
   )
-  (wire (pts (xy 43.18 104.14) (xy 54.61 104.14))
+  (wire (pts (xy 43.18 104.14) (xy 46.99 104.14))
     (stroke (width 0) (type default) (color 0 0 0 0))
   )
@@
       (effects (font (size 1.27 1.27)) hide)
     )
-    (property "Datasheet" "https://www.st.com/resource/en/datasheet/usblc6-2.pdf" (id 3) (at 78.74 114.3 0)
+    (property "Datasheet" "https://datasheet.lcsc.com/lcsc/1811141711_STMicroelectronics-USBLC6-2SC6_C7519.pdf" (id 3) (at 78.74 114.3 0)
+      (effects (font (size 1.27 1.27)) hide)
+    )
+    (property "Manufacturer Part Number" "USBLC6-2SC6" (id 4) (at 73.66 123.19 0)
       (effects (font (size 1.27 1.27)) hide)
     )
@@
     (pin "2")
   )
+  (symbol (lib_id "Device:Polyfuse_Small") (at 49.53 104.14 90) (unit 1)
+    (in_bom yes) (on_board yes) (fields_autoplaced)
+    (property "Reference" "F1" (id 0) (at 49.53 97.79 90))
+    (property "Value" "Polyfuse" (id 1) (at 49.53 100.33 90))
+    (property "Footprint" "Fuse:Fuse_0805_2012Metric_Pad1.15x1.40mm_HandSolder" (id 2) (at 54.61 102.87 0)
+      (effects (font (size 1.27 1.27)) (justify left) hide)
+    )
+    (property "Datasheet" "https://datasheet.lcsc.com/lcsc/1810071612_RUILON-Shenzhen-Ruilongyuan-Elec-SMD0805P020TF_C20976.pdf" (id 3) (at 49.53 104.14 0)
+      (effects (font (size 1.27 1.27)) hide)
+    )
+    (property "Manufacturer Part Number" "SMD0805P020TF" (id 4) (at 49.53 104.14 0)
+      (effects (font (size 1.27 1.27)) hide)
+    )
+    (pin "1")
+    (pin "2")
+  )
   (symbol (lib_id "power:VBUS") (at 213.36 68.58 0) (unit 1)
     (in_bom yes) (on_board yes) (fields_autoplaced)
@@
       (effects (font (size 1.27 1.27)) hide)
     )
-    (property "Datasheet" "~" (id 3) (at 39.37 135.89 0)
-      (effects (font (size 1.27 1.27)) hide)
-    )
-    (pin "1")
-    (pin "2")
-  )
-  (symbol (lib_id "Device:FerriteBead_Small") (at 57.15 104.14 270) (unit 1)
-    (in_bom yes) (on_board yes) (fields_autoplaced)
-    (property "Reference" "FB1" (id 0) (at 57.1881 97.79 90))
-    (property "Value" "FerriteBead_Small" (id 1) (at 57.1881 100.33 90))
-    (property "Footprint" "Inductor_SMD:L_0805_2012Metric_Pad1.15x1.40mm_HandSolder" (id 2) (at 57.15 102.362 90)
-      (effects (font (size 1.27 1.27)) hide)
-    )
-    (property "Datasheet" "~" (id 3) (at 57.15 104.14 0)
+    (property "Datasheet" "https://datasheet.lcsc.com/lcsc/1810311431_YAGEO-RC0805FR-071ML_C107700.pdf" (id 3) (at 39.37 135.89 0)
+      (effects (font (size 1.27 1.27)) hide)
+    )
+    (property "Manufacturer Part Number" "RC0805FR-071ML" (id 4) (at 39.37 135.89 0)
+      (effects (font (size 1.27 1.27)) hide)
+    )
+    (pin "1")
+    (pin "2")
+  )
+  (symbol (lib_id "Device:FerriteBead_Small") (at 62.23 104.14 270) (unit 1)
+    (in_bom yes) (on_board yes) (fields_autoplaced)
+    (property "Reference" "FB1" (id 0) (at 62.2681 97.79 90))
+    (property "Value" "FerriteBead" (id 1) (at 62.2681 100.33 90))
+    (property "Footprint" "Inductor_SMD:L_0805_2012Metric_Pad1.15x1.40mm_HandSolder" (id 2) (at 62.23 102.362 90)
+      (effects (font (size 1.27 1.27)) hide)
+    )
+    (property "Datasheet" "https://datasheet.lcsc.com/lcsc/1810201231_Murata-Electronics-BLM21BB050SN1D_C113035.pdf" (id 3) (at 62.23 104.14 0)
+      (effects (font (size 1.27 1.27)) hide)
+    )
+    (property "Manufacturer Part Number" "BLM21BB050SN1D" (id 4) (at 62.23 104.14 0)
       (effects (font (size 1.27 1.27)) hide)
     )
@@
       (effects (font (size 1.27 1.27)) hide)
     )
-    (property "Datasheet" "~" (id 3) (at 26.67 135.89 0)
+    (property "Datasheet" "https://datasheet.lcsc.com/lcsc/1811061821_YAGEO-CC0805KRX7R9BB472_C107153.pdf" (id 3) (at 26.67 135.89 0)
+      (effects (font (size 1.27 1.27)) hide)
+    )
+    (property "Manufacturer Part Number" "CC0805KRX7R9BB472" (id 4) (at 26.67 135.89 0)
       (effects (font (size 1.27 1.27)) hide)
     )
@@
       (reference "C12") (unit 1) (value "0.1uC") (footprint "Capacitor_SMD:C_0805_2012Metric_Pad1.18x1.45mm_HandSolder")
     )
+    (path "/3c559a96-2c80-4f4c-b299-ee6165d1ac21"
+      (reference "F1") (unit 1) (value "Polyfuse") (footprint "Fuse:Fuse_0805_2012Metric_Pad1.15x1.40mm_HandSolder")
+    )
     (path "/d3eabcb2-dd57-404e-8549-62d4dedf74ad"
-      (reference "FB1") (unit 1) (value "FerriteBead_Small") (footprint "Inductor_SMD:L_0805_2012Metric_Pad1.15x1.40mm_HandSolder")
+      (reference "FB1") (unit 1) (value "FerriteBead") (footprint "Inductor_SMD:L_0805_2012Metric_Pad1.15x1.40mm_HandSolder")
     )
     (path "/9aefe026-a140-4f96-a0e9-b703b2910bed"

Commit message: Update USB_RS232_Adapter.kicad_sch
Parts:
- added C5: 0.1uC, Capacitor_SMD:C_0805_2012Metric_Pad1.18x1.45mm_HandSolder, symbol Device:C
- C1, C11, C12, C2, C3, C6, C7: Manufacturer Part Number (none) -> CC0805KRX7R8BB104
- C10, C9: Manufacturer Part Number (none) -> CC0805JRNPO9BN330
- C8: Manufacturer Part Number (none) -> LMK212ABJ106KG-T
- Y1: footprint (none) -> Crystal:Crystal_SMD_HC49-SD_HandSoldering; Manufacturer Part Number (none) -> SXMH12.000F2020F30
Connections:
- net GND: now also C5.1
- net VBUS: now also U2.24 (EN), U2.25 (~{SHDN}), C5.2
- no-connect marks 3 -> 5

Commit message: Progressed ECAD
Parts:
- removed U1: CH340T, Package_SO:SSOP-20_5.3x7.2mm_P0.65mm, symbol Interface_USB:CH340T
- added D1: LED, symbol Device:LED
- added H1, H2, H3, H4: MountingHole, MountingHole:MountingHole_3.2mm_M3_Pad, symbol Mechanical:MountingHole
- added Q1: BC846, Package_TO_SOT_SMD:SOT-23, symbol Transistor_BJT:BC846
- added R2, R3: R, symbol Device:R
- added U1: CH340T, Package_SO:SSOP-20_5.3x7.2mm_P0.65mm, symbol Interface_USB_custom:CH340T
Connections:
- net GND: now also Q1.2 (E), U1.8 (GND)
- net V3: now also U1.5 (V3)
- net VBUS: now also D1.2 (A), U1.19 (VCC)
- net at U3.4 (I/O2): now also U1.6 (UD+)
- net at U3.6 (I/O1): now also U1.7 (UD-)
- net at C9.1, Y1.1: now also U1.9 (XI)
- net at U2.19 (ROUT5): now also U1.14 (~{DCD})
- net at U2.20 (DIN3): now also U1.16 (~{RTS})
- net at U2.22 (ROUT4): now also U1.13 (~{RI})
- net at U2.26 (ROUT3): now also U1.12 (~{DSR})
- net at U2.5 (ROUT2): now also U1.11 (~{CTS})
- net at U2.6 (DIN2): now also U1.15 (~{DTR})
- net at U2.7 (DIN1): now also U1.3 (TXD)
- net at U2.8 (ROUT1): now also U1.4 (RXD)
- net at C10.1, Y1.2: now also U1.10 (XO)
- new net: Q1.1 (B), R2.2
- new net: Q1.3 (C), R3.2
- new net: D1.1 (K), R3.1
- new net TX_LED: R2.1, U1.17 (TNOW)
- no-connect marks 5 -> 6

Commit message: Progressed ECAD
Parts:
- D1: footprint (none) -> LED_SMD:LED_0805_2012Metric_Pad1.15x1.40mm_HandSolder; Manufacturer Part Number (none) -> 17-21SYGC/S530-E2/TR8
Changed lines of the file:
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@@
       (effects (font (size 1.27 1.27)) (justify right))
     )
-    (property "Footprint" "" (id 2) (at 135.89 160.02 0)
-      (effects (font (size 1.27 1.27)) hide)
-    )
-    (property "Datasheet" "~" (id 3) (at 135.89 160.02 0)
+    (property "Footprint" "LED_SMD:LED_0805_2012Metric_Pad1.15x1.40mm_HandSolder" (id 2) (at 135.89 160.02 0)
+      (effects (font (size 1.27 1.27)) hide)
+    )
+    (property "Datasheet" "https://datasheet.lcsc.com/lcsc/1811011222_Everlight-Elec-17-21SYGC-S530-E2-TR8_C73548.pdf" (id 3) (at 135.89 160.02 0)
+      (effects (font (size 1.27 1.27)) hide)
+    )
+    (property "Manufacturer Part Number" "17-21SYGC/S530-E2/TR8" (id 4) (at 135.89 160.02 0)
       (effects (font (size 1.27 1.27)) hide)
     )
@@
     )
     (path "/661ca651-e916-4763-a813-1266fdc56ef5"
-      (reference "D1") (unit 1) (value "LED") (footprint "")
+      (reference "D1") (unit 1) (value "LED") (footprint "LED_SMD:LED_0805_2012Metric_Pad1.15x1.40mm_HandSolder")
     )
     (path "/3c559a96-2c80-4f4c-b299-ee6165d1ac21"

Commit message: Progressed ECAD
Parts:
- Q1: Manufacturer Part Number (none) -> BC846,215
Connections:
- net VBUS: now also R3.1; no longer D1.2 (A)
- net at Q1.3 (C): now also D1.1 (K); no longer R3.2
- new net: D1.2 (A), R3.2
Other:
- moved on the sheet: D1, R3
Changed lines of the file:
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@@
       (effects (font (size 1.27 1.27) italic) (justify left) hide)
     )
-    (property "Datasheet" "https://assets.nexperia.com/documents/data-sheet/BC846_SER.pdf" (id 3) (at 133.35 176.53 0)
+    (property "Datasheet" "https://datasheet.lcsc.com/lcsc/1811141222_Nexperia-BC846-215_C179342.pdf" (id 3) (at 133.35 176.53 0)
       (effects (font (size 1.27 1.27)) (justify left) hide)
+    )
+    (property "Manufacturer Part Number" "BC846,215" (id 4) (at 133.35 176.53 0)
+      (effects (font (size 1.27 1.27)) hide)
     )
     (pin "1")
@@
     (pin "1")
   )
-  (symbol (lib_id "Device:LED") (at 135.89 160.02 90) (unit 1)
-    (in_bom yes) (on_board yes) (fields_autoplaced)
-    (property "Reference" "D1" (id 0) (at 139.7 160.3374 90)
-      (effects (font (size 1.27 1.27)) (justify right))
-    )
-    (property "Value" "LED" (id 1) (at 139.7 162.8774 90)
-      (effects (font (size 1.27 1.27)) (justify right))
-    )
-    (property "Footprint" "LED_SMD:LED_0805_2012Metric_Pad1.15x1.40mm_HandSolder" (id 2) (at 135.89 160.02 0)
-      (effects (font (size 1.27 1.27)) hide)
-    )
-    (property "Datasheet" "https://datasheet.lcsc.com/lcsc/1811011222_Everlight-Elec-17-21SYGC-S530-E2-TR8_C73548.pdf" (id 3) (at 135.89 160.02 0)
-      (effects (font (size 1.27 1.27)) hide)
-    )
-    (property "Manufacturer Part Number" "17-21SYGC/S530-E2/TR8" (id 4) (at 135.89 160.02 0)
+  (symbol (lib_id "Device:LED") (at 135.89 167.64 90) (unit 1)
+    (in_bom yes) (on_board yes) (fields_autoplaced)
+    (property "Reference" "D1" (id 0) (at 139.7 167.9574 90)
+      (effects (font (size 1.27 1.27)) (justify right))
+    )
+    (property "Value" "LED" (id 1) (at 139.7 170.4974 90)
+      (effects (font (size 1.27 1.27)) (justify right))
+    )
+    (property "Footprint" "LED_SMD:LED_0805_2012Metric_Pad1.15x1.40mm_HandSolder" (id 2) (at 135.89 167.64 0)
+      (effects (font (size 1.27 1.27)) hide)
+    )
+    (property "Datasheet" "https://datasheet.lcsc.com/lcsc/1811011222_Everlight-Elec-17-21SYGC-S530-E2-TR8_C73548.pdf" (id 3) (at 135.89 167.64 0)
+      (effects (font (size 1.27 1.27)) hide)
+    )
+    (property "Manufacturer Part Number" "17-21SYGC/S530-E2/TR8" (id 4) (at 135.89 167.64 0)
       (effects (font (size 1.27 1.27)) hide)
     )
@@
     (pin "2")
   )
-  (symbol (lib_id "Device:R") (at 135.89 167.64 0) (unit 1)
-    (in_bom yes) (on_board yes) (fields_autoplaced)
-    (property "Reference" "R3" (id 0) (at 138.43 166.3699 0)
-      (effects (font (size 1.27 1.27)) (justify left))
-    )
-    (property "Value" "R" (id 1) (at 138.43 168.9099 0)
-      (effects (font (size 1.27 1.27)) (justify left))
-    )
-    (property "Footprint" "" (id 2) (at 134.112 167.64 90)
-      (effects (font (size 1.27 1.27)) hide)
-    )
-    (property "Datasheet" "~" (id 3) (at 135.89 167.64 0)
-      (effects (font (size 1.27 1.27)) hide)
-    )
+  (symbol (lib_id "Device:R") (at 135.89 160.02 0) (unit 1)
+    (in_bom yes) (on_board yes) (fields_autoplaced)
+    (property "Reference" "R3" (id 0) (at 138.43 158.7499 0)
+      (effects (font (size 1.27 1.27)) (justify left))
+    )
+    (property "Value" "R" (id 1) (at 138.43 161.2899 0)
+      (effects (font (size 1.27 1.27)) (justify left))
+    )
+    (property "Footprint" "" (id 2) (at 134.112 160.02 90)
+      (effects (font (size 1.27 1.27)) hide)
+    )
+    (property "Datasheet" "~" (id 3) (at 135.89 160.02 0)
+      (effects (font (size 1.27 1.27)) hide)
+    )
