File: Tester/ECAD/_Deprecated/BrushedMotorDriver/BrushedMotorDriver.kicad_sch (KiCad schematic)
At the start: 41 parts, among them J1 SWIM connector, J2 Power connector, J3 RS485 connector, J4 Limit switch connector, J5 Limit switch connector, J6 Motor connector, Q1 BC846, U1 STM8S003F3P6, U2 SP485, U3 L78M05_TO252, U4 LM321, U5 74HCT2G17GV, Y1 Crystal_GND24

Commit message: Cleanup
Parts:
- removed R5: 1kR, Resistor_SMD:R_0805_2012Metric_Pad1.20x1.40mm_HandSolder, symbol Device:R
- J3: renamed from J1; footprint Connector_PinHeader_2.54mm:PinHeader_1x04_P2.54mm_Horizontal -> Connector_PinHeader_2.54mm:PinHeader_1x04_P2.54mm_Vertical; Manufacturer Part Number PZ254R-11-04P -> PZ254-1-04-Z-8.5
- R5: renamed from R6; value 1kR -> 2k1R; Manufacturer Part Number RC0805FR-071KL -> AC0805FR-072K1L
- renumbered J2 to J1, J3 to J2, R11 to R10, R12 to R11, R13 to R12, R7 to R6, R8 to R7, R9 to R8, R10 to R9
Connections:
- net ACT_LED: now also R5.1
Other:
- moved on the sheet: C1, C2, C3, C4, C5, C6, C8, D2, J3, Q1, R5, R6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
