File: Tester/ECAD/BDCMotorControlBoard/BDCMotorControlBoard.kicad_pcb (KiCad board)
At the start: 2 copper layers, 122 parts, among them J1 Limit switch connector, J2 Limit switch connector, J3 SWIM connector, J4 Power connector, J5 Motor connector, J6 RS485 connector, Q1 BC846, Q10 IRLR8726, Q11 IRLR8726, Q12 IRLR8726, Q2 BC846, Q3 BC846, Q4 BC846BPN, Q5 BC846, Q6 BC846, Q7 BC846, Q8 BC846, Q9 IRLR8726, U1 STM8S003F3P6, U2 74HCT2G17GV, U3 SP485, U4 L78M05_TO252, U5 INA180A2, U6 IR2103, U7 IR2103, Y1 Crystal_GND24

Commit message: Progressed CAD
Parts:
- moved R7 85.3 mm to (239.8, 149.2), turned to 180 degrees
- moved Q2 84.7 mm to (239.8, 152.2)
- moved D2 84.2 mm to (239.8, 155.2), turned to 180 degrees
- moved R8 83.8 mm to (239.8, 157.5), turned to 180 degrees
- moved R5 74.0 mm to (249.5, 149.5), turned to 180 degrees
- moved Q1 73.0 mm to (249.5, 152.5)
- moved D1 72.4 mm to (249.5, 155.5), turned to 180 degrees
- moved R6 72.0 mm to (249.5, 157.8), turned to 180 degrees
- moved C11 42.2 mm to (246.9, 96.8), turned to -90 degrees
- moved C12 42.0 mm to (237.1, 96.8), turned to -90 degrees
- moved U4 39.1 mm to (242.0, 98.8), turned to -90 degrees
- moved C13 24.5 mm to (207.7, 87.2)
- moved C14 24.5 mm to (217.0, 87.2)
- moved TP2 18.4 mm to (199.0, 83.0)
- moved C15 16.4 mm to (218.0, 119.4)
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Connections:
- C13 pad 1: +12V -> /H-bridge/Top_Rail
- C14 pad 1: +12V -> /H-bridge/Top_Rail
Other:
- board outline added: 96.5 x 67.5 mm

Commit message: Update BDCMotorControlBoard.kicad_pcb
Parts:
- moved H2 156.0 mm to (107.5, 127.5)
- moved J3 86.0 mm to (147.2, 151.3)
- moved H3 82.8 mm to (192.5, 127.5)
- moved U1 75.1 mm to (159.9, 154.9)
- moved C7 72.7 mm to (160.2, 171.2)
- moved C9 72.7 mm to (165.2, 166.3)
- moved Y1 72.7 mm to (160.8, 166.8)
- moved C1 72.5 mm to (162.2, 160.5)
- moved C4 71.7 mm to (157.2, 160.8)
- moved H4 71.4 mm to (192.5, 72.5)
- moved kibuzzard-6336230B 71.3 mm to (198.0, 116.5)
- moved kibuzzard-63362281 71.1 mm to (198.0, 94.5)
- moved J6 71.0 mm to (193.2, 119.0)
- moved R23 71.0 mm to (11.3, 55.5)
- moved R27 71.0 mm to (6.33, 55.5)
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Other:
- board size 96.5 x 67.5 mm -> 100 x 70 mm

Commit message: Update BDCMotorControlBoard.kicad_pcb
Parts:
- removed kibuzzard-633622A8: G***, kibuzzard-633622A8
- added D13: LED, LED_SMD:LED_0805_2012Metric_Pad1.15x1.40mm_HandSolder, F.Cu at (169.0, 130.0)
- added Q13: BC846, Package_TO_SOT_SMD:SOT-23, F.Cu at (164.0, 128.8)
- added R31: 2k1R, Resistor_SMD:R_0805_2012Metric_Pad1.20x1.40mm_HandSolder, F.Cu at (164.0, 125.2)
- added R32: 150R, Resistor_SMD:R_0805_2012Metric_Pad1.20x1.40mm_HandSolder, F.Cu at (169.0, 127.5)
- added kibuzzard-63375F99: G***, kibuzzard-63375F99, F.Cu at (183.0, 133.0)
- added kibuzzard-63376701: G***, kibuzzard-63376701, F.Cu at (176.0, 133.0)
- added kibuzzard-63376CDD: G***, kibuzzard-63376CDD, F.Cu at (169.0, 133.0)
- added kibuzzard-63376D3D: G***, kibuzzard-63376D3D, F.Cu at (102.0, 100.0)
- moved C7 69.3 mm to (153.1, 102.3), turned to -135 degrees
- moved C16 67.6 mm to (128.5, 91.8)
- moved C17 67.6 mm to (131.5, 91.8)
- moved D6 67.6 mm to (123.5, 91.8)
- moved Q3 67.6 mm to (128.5, 105.7)
- moved Q4 67.6 mm to (128.5, 101.8)
- moved R14 67.6 mm to (127.5, 111.8)
- moved R15 67.6 mm to (128.5, 108.8)
- moved R16 67.6 mm to (125.5, 101.8)
- moved TP1 67.6 mm to (122.5, 112.8)
- moved TP3 67.6 mm to (133.5, 102.8)
- moved TP4 67.6 mm to (129.5, 87.8)
- moved Y1 62.3 mm to (155.7, 104.8), turned to -135 degrees
- moved C9 60.1 mm to (152.8, 107.5), turned to 135 degrees
- moved C19 55.6 mm to (78.2, 75.5)
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Connections:
- U1 pad 10: unconnected-(U1-Pad10) -> /LSW_ACT_LED
- U1 pad 11: /LIM_POS_- -> /LIM_POS_+
- U1 pad 12: /LIM_POS_+ -> /LIM_POS_-

Commit message: Update BDCMotorControlBoard.kicad_pcb
Parts:
- removed kibuzzard-63362281: G***, kibuzzard-63362281
- removed kibuzzard-6336228B: G***, kibuzzard-6336228B
- removed kibuzzard-63362299: G***, kibuzzard-63362299
- removed kibuzzard-6336230B: G***, kibuzzard-6336230B
- added kibuzzard-63377EA3: G***, kibuzzard-63377EA3, F.Cu at (198.0, 85.0)
- added kibuzzard-63377EB6: G***, kibuzzard-63377EB6, F.Cu at (198.0, 95.0)
- added kibuzzard-63377EC7: G***, kibuzzard-63377EC7, F.Cu at (198.0, 105.0)
- added kibuzzard-63377ED3: G***, kibuzzard-63377ED3, F.Cu at (198.0, 115.0)
- moved Q1 29.4 mm to (183.0, 124.0)
- moved Q2 17.7 mm to (176.0, 124.0)
- moved R5 11.1 mm to (163.0, 118.8)
- moved Q13 6.90 mm to (169.0, 124.0)
- moved R7 5.84 mm to (163.0, 121.0)
- moved R31 2.24 mm to (163.0, 123.2)
- moved C10 1.50 mm to (180.0, 111.0)
- moved D5 1.50 mm to (185.5, 115.0)
- moved J4 1.50 mm to (193.2, 87.5)
- moved J6 1.50 mm to (193.2, 117.5)
- moved R10 1.50 mm to (171.5, 116.2)
- moved R11 1.50 mm to (185.5, 112.0)
- moved R12 1.50 mm to (185.5, 118.0)
- moved R9 1.50 mm to (171.5, 114.0)
- moved U3 1.50 mm to (178.5, 115.0)
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
Commit message: Update BDCMotorControlBoard.kicad_pcb
Parts:
- moved Q11 74.3 mm to (118.0, 92.5)
- moved Q12 72.4 mm to (118.1, 77.0)
- moved C16 65.2 mm to (166.0, 145.1)
- moved C17 65.2 mm to (169.0, 145.1)
- moved D6 65.2 mm to (161.0, 145.1)
- moved Q3 65.2 mm to (166.0, 159.0)
- moved Q4 65.2 mm to (166.0, 155.1)
- moved R14 65.2 mm to (165.0, 165.1)
- moved R15 65.2 mm to (166.0, 162.1)
- moved R16 65.2 mm to (163.0, 155.1)
- moved TP1 65.2 mm to (160.0, 166.1)
- moved TP3 65.2 mm to (171.0, 156.1)
- moved TP4 65.2 mm to (167.0, 141.1)
- moved R30 56.4 mm to (118.5, 112.0), turned to 0 degrees
- moved C35 56.3 mm to (122.5, 112.0), turned to 0 degrees
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
Commit message: Update BDCMotorControlBoard.kicad_pcb
Parts:
- removed kibuzzard-63376D3D: G***, kibuzzard-63376D3D
- added kibuzzard-633802D7: G***, kibuzzard-633802D7, F.Cu at (102.0, 100.0)
- moved R23 73.2 mm to (134.3, 90.6)
- moved R24 73.2 mm to (132.3, 80.6)
- moved R27 73.2 mm to (129.3, 90.6)
- moved R28 73.2 mm to (129.3, 80.6)
- moved U7 73.2 mm to (142.3, 85.6)
- moved R21 64.1 mm to (132.0, 120.0)
- moved R22 64.1 mm to (132.0, 111.0)
- moved R25 64.1 mm to (130.0, 120.0)
- moved R26 64.1 mm to (130.0, 111.0)
- moved U6 64.1 mm to (141.0, 116.0)
- moved C33 58.6 mm to (104.0, 91.0), turned to 180 degrees
- moved C31 54.2 mm to (104.0, 87.0), turned to 180 degrees
- moved C29 49.9 mm to (104.0, 83.0), turned to 180 degrees
- moved C32 49.3 mm to (104.0, 121.0), turned to 180 degrees
- moved C30 47.5 mm to (104.0, 117.0), turned to 180 degrees
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
Commit message: Update BDCMotorControlBoard.kicad_pcb
Parts:
- moved TP5 22.1 mm to (72.0, 148.0), turned to 180 degrees
- moved TP8 22.0 mm to (73.2, 82.5), turned to 180 degrees
- moved TP10 20.6 mm to (74.8, 60.5), turned to 180 degrees
- moved TP7 20.0 mm to (74.0, 127.0), turned to 180 degrees
- moved D3 17.5 mm to (179.0, 70.0), turned to -90 degrees
- moved C25 17.1 mm to (73.8, 65.5), turned to -90 degrees
- moved C22 16.8 mm to (73.0, 143.0), turned to 90 degrees
- moved C23 16.7 mm to (73.0, 132.0), turned to -90 degrees
- moved C24 16.5 mm to (74.2, 77.5), turned to 90 degrees
- moved TP6 16.3 mm to (72.0, 138.0), turned to 180 degrees
- moved TP9 15.7 mm to (73.2, 72.5), turned to 180 degrees
- moved D8 15.4 mm to (92.6, 78.5), turned to 0 degrees
- moved D7 15.2 mm to (92.0, 144.0), turned to 0 degrees
- moved R24 14.7 mm to (129.0, 95.0), turned to 0 degrees
- moved R28 13.8 mm to (126.0, 94.0), turned to -90 degrees
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
Commit message: Update BDCMotorControlBoard.kicad_pcb
Parts:
- moved D10 67.3 mm to (143.8, 113.8)
- moved Q6 67.3 mm to (140.8, 113.8)
- moved R18 67.3 mm to (146.8, 113.8)
- moved C18 65.3 mm to (148.6, 121.5)
- moved C20 65.3 mm to (145.6, 121.5)
- moved D7 65.3 mm to (153.6, 122.5)
- moved D9 65.3 mm to (138.6, 119.5)
- moved Q5 65.3 mm to (138.6, 122.5)
- moved R17 65.3 mm to (142.6, 121.5)
- moved D12 64.5 mm to (139.8, 89.2)
- moved Q8 64.5 mm to (136.8, 89.2)
- moved R20 63.8 mm to (142.0, 89.2)
- moved C25 62.4 mm to (132.0, 88.0), turned to 180 degrees
- moved C23 60.5 mm to (132.0, 118.5), turned to 180 degrees
- moved C22 59.1 mm to (125.0, 115.0)
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