File: Tester/ECAD/BDCMotorControlBoard/BDCMotorControlBoard.kicad_sch (KiCad schematic)
At the start: 52 parts, among them J1 Limit switch connector, J2 Limit switch connector, J3 SWIM connector, J4 Power connector, J5 Motor connector, J6 RS485 connector, Q1 2N7002, Q2 2N7002, Q7 2N7002, Q8 2N7002, SW1 SW_Push, U1 STM8S003F3P6, U3 SP485, U4 L78M05_TO252, Y1 Crystal_GND24

Commit message: Progressed CAD
Parts:
- removed C8: 0.1uC, Capacitor_SMD:C_0805_2012Metric_Pad1.18x1.45mm_HandSolder, symbol Device:C
- removed D7: LED, LED_SMD:LED_0805_2012Metric_Pad1.15x1.40mm_HandSolder, symbol Device:LED
- removed J1, J2: Limit switch connector, Connector_custom:JILN JL301-50002U01, symbol Connector:Screw_Terminal_01x02
- removed R1, R2: 4k7R, Resistor_SMD:R_0805_2012Metric_Pad1.20x1.40mm_HandSolder, symbol Device:R
- removed R22: 150R, Resistor_SMD:R_0805_2012Metric_Pad1.20x1.40mm_HandSolder, symbol Device:R
Connections:
- net LIM_SWITCH: no longer names the net of U1.11 (PB5)
- no-connect marks 0 -> 1
Other:
- note removed: "Limit Switch section"
- note removed: "Power LED"
- note removed: "V_ADC = 0V"
- note removed: "V_ADC = 2.5V"

Commit message: Progressed CAD
Parts:
- Y1: footprint Crystal:Crystal_SMD_3225-4Pin_3.2x2.5mm_HandSoldering -> Crystal:Crystal_SMD_3225-4Pin_3.2x2.5mm
Other:
- note added: "Power LED"
- note removed: "Limit Switch Activity LED"
- moved on the sheet: C2, C3, C4, U1

Commit message: Progressed CAD
Parts:
- removed U4: L78M05_TO252, Package_TO_SOT_SMD:TO-252-2, symbol Regulator_Linear:LM78M05_TO252
- added C22, C23, C25, C26, C8: C, symbol Device:C
- added L1: L, symbol Device:L
- added R1, R2: R, symbol Device:R
- added U4: TPS563201, Package_TO_SOT_SMD:SOT-23-6, symbol Regulator_Switching:TPS563200
- C11: value 1uC -> C; footprint Capacitor_SMD:C_0805_2012Metric_Pad1.18x1.45mm_HandSolder -> (none); Manufacturer Part Number GCM21BR71E105KA56L -> (none)
- H1, H2, H3, H4: Manufacturer Part Number (none) -> N/A
Connections:
- net +12V: now also C22.1, C8.1, U4.3 (VIN), U4.5 (EN)
- net +5V: now also C23.1, C25.2, C26.1, L1.2, R2.2; no longer C12.1
- net GND: now also C22.2, C23.2, C26.2, C8.2, R1.2, U4.1 (GND); no longer C12.2
- net C_ACT_LED renamed RS485_LED
- net LSW_ACT_LED renamed PWR_LED
- new net: C25.1, R1.1, R2.1, U4.4 (VFB)
- new net: C12.2, L1.1, U4.2 (SW)
- new net: C12.1, U4.6 (VBST)
Other:
- note added: "Power input and protection"
- moved on the sheet: C1, C10, C12, C2, C3, C4, C7, C9, D1, D13, D2, D3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

Commit message: Progressed CAD
Parts:
- removed C25: C, symbol Device:C
- C11, C8: value C -> 10uC; footprint (none) -> Capacitor_SMD:C_0805_2012Metric_Pad1.18x1.45mm_HandSolder
- C22: value C -> 0.1uC; footprint (none) -> Capacitor_SMD:C_0805_2012Metric_Pad1.18x1.45mm_HandSolder; Manufacturer Part Number (none) -> CC0805KRX7R8BB104
- C23, C26: value C -> 22uC; footprint (none) -> Capacitor_SMD:C_0805_2012Metric_Pad1.18x1.45mm_HandSolder
- L1: value L -> 3.3uL
- R1: value R -> 10kR; footprint (none) -> Resistor_SMD:R_0805_2012Metric_Pad1.20x1.40mm_HandSolder; Manufacturer Part Number (none) -> RC0805FR-0710KL
- R2: value R -> 54.9kR; footprint (none) -> Resistor_SMD:R_0805_2012Metric_Pad1.20x1.40mm_HandSolder
Other:
- note added: "1%"

Commit message: Progressed CAD
Parts:
- C11, C8: Manufacturer Part Number (none) -> C2012X5R1V106KT000E
- C23, C26: Manufacturer Part Number (none) -> C2012X5R1A226KT000N
- L1: footprint (none) -> Inductor_SMD:L_Bourns_SRN6045TA; Manufacturer Part Number (none) -> ABG06A45M3R3
Changed lines of the file:
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@@
       (effects (font (size 1.27 1.27)) hide)
     )
-    (property "Datasheet" "~" (id 3) (at 186.69 130.81 0)
+    (property "Datasheet" "https://datasheet.lcsc.com/lcsc/1912111437_TDK-C2012X5R1V106KT000E_C342722.pdf" (id 3) (at 186.69 130.81 0)
+      (effects (font (size 1.27 1.27)) hide)
+    )
+    (property "Manufacturer Part Number" "C2012X5R1V106KT000E" (id 4) (at 186.69 130.81 0)
       (effects (font (size 1.27 1.27)) hide)
     )
@@
     (property "Reference" "L1" (id 0) (at 243.84 119.38 90))
     (property "Value" "3.3uL" (id 1) (at 243.84 121.92 90))
-    (property "Footprint" "" (id 2) (at 243.84 125.73 0)
-      (effects (font (size 1.27 1.27)) hide)
-    )
-    (property "Datasheet" "~" (id 3) (at 243.84 125.73 0)
+    (property "Footprint" "Inductor_SMD:L_Bourns_SRN6045TA" (id 2) (at 243.84 125.73 0)
+      (effects (font (size 1.27 1.27)) hide)
+    )
+    (property "Datasheet" "https://datasheet.lcsc.com/lcsc/1809140622_COILANK-INTERNATIONAL-ABG06A45M3R3_C253598.pdf" (id 3) (at 243.84 125.73 0)
+      (effects (font (size 1.27 1.27)) hide)
+    )
+    (property "Manufacturer Part Number" "ABG06A45M3R3" (id 4) (at 243.84 125.73 0)
       (effects (font (size 1.27 1.27)) hide)
     )
@@
       (effects (font (size 1.27 1.27)) hide)
     )
-    (property "Datasheet" "~" (id 3) (at 251.46 130.81 0)
+    (property "Datasheet" "https://datasheet.lcsc.com/lcsc/1811151223_TDK-C2012X5R1A226KT000N_C76634.pdf" (id 3) (at 251.46 130.81 0)
+      (effects (font (size 1.27 1.27)) hide)
+    )
+    (property "Manufacturer Part Number" "C2012X5R1A226KT000N" (id 4) (at 251.46 130.81 0)
       (effects (font (size 1.27 1.27)) hide)
     )
@@
       (effects (font (size 1.27 1.27)) hide)
     )
-    (property "Datasheet" "~" (id 3) (at 175.26 130.81 0)
+    (property "Datasheet" "https://datasheet.lcsc.com/lcsc/1912111437_TDK-C2012X5R1V106KT000E_C342722.pdf" (id 3) (at 175.26 130.81 0)
+      (effects (font (size 1.27 1.27)) hide)
+    )
+    (property "Manufacturer Part Number" "C2012X5R1V106KT000E" (id 4) (at 175.26 130.81 0)
       (effects (font (size 1.27 1.27)) hide)
     )
@@
       (effects (font (size 1.27 1.27)) hide)
     )
-    (property "Datasheet" "~" (id 3) (at 264.16 130.81 0)
+    (property "Datasheet" "https://datasheet.lcsc.com/lcsc/1811151223_TDK-C2012X5R1A226KT000N_C76634.pdf" (id 3) (at 264.16 130.81 0)
+      (effects (font (size 1.27 1.27)) hide)
+    )
+    (property "Manufacturer Part Number" "C2012X5R1A226KT000N" (id 4) (at 264.16 130.81 0)
       (effects (font (size 1.27 1.27)) hide)
     )
@@
     )
     (path "/399b7709-217c-47bf-a504-7033f7138d54"
-      (reference "L1") (unit 1) (value "3.3uL") (footprint "")
+      (reference "L1") (unit 1) (value "3.3uL") (footprint "Inductor_SMD:L_Bourns_SRN6045TA")
     )
     (path "/bdb843bc-f6d0-4ca9-9dd4-e8379fadfb92"

Commit message: Progressed CAD
Parts:
- SW1: footprint Button_Switch_THT:SW_PUSH_6mm -> Button_Switch_SMD:SW_SPST_CK_RS282G05A3; Manufacturer Part Number TS-1002-04526 -> K2-1107ST-A4DW-06
Changed lines of the file:
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@@
       (effects (font (size 1.27 1.27)) (justify left))
     )
-    (property "Footprint" "Button_Switch_THT:SW_PUSH_6mm" (id 2) (at 107.95 50.8 0)
-      (effects (font (size 1.27 1.27)) hide)
-    )
-    (property "Datasheet" "https://datasheet.lcsc.com/lcsc/1912111437_XUNPU-TS-1002-04526_C455090.pdf" (id 3) (at 107.95 50.8 0)
-      (effects (font (size 1.27 1.27)) hide)
-    )
-    (property "Manufacturer Part Number" "TS-1002-04526" (id 4) (at 102.87 50.8 0)
+    (property "Footprint" "Button_Switch_SMD:SW_SPST_CK_RS282G05A3" (id 2) (at 107.95 50.8 0)
+      (effects (font (size 1.27 1.27)) hide)
+    )
+    (property "Datasheet" "https://datasheet.lcsc.com/lcsc/2108131530_Korean-Hroparts-Elec-K2-1107ST-A4DW-06_C118141.pdf" (id 3) (at 107.95 50.8 0)
+      (effects (font (size 1.27 1.27)) hide)
+    )
+    (property "Manufacturer Part Number" "K2-1107ST-A4DW-06" (id 4) (at 102.87 50.8 0)
       (effects (font (size 1.27 1.27)) hide)
     )
@@
     )
     (path "/77ce637e-066c-4c64-aa31-467dd0b75a01"
-      (reference "SW1") (unit 1) (value "SW_Push") (footprint "Button_Switch_THT:SW_PUSH_6mm")
+      (reference "SW1") (unit 1) (value "SW_Push") (footprint "Button_Switch_SMD:SW_SPST_CK_RS282G05A3")
     )
     (path "/a6597409-e020-48c5-b98f-177a095b88e4"

Commit message: Update BDCMotorControlBoard.kicad_sch
Parts:
- removed D3, D4: SMAJ13A, Diode_SMD:D_SMA, symbol Diode:SM6T68A
- removed D5: SM712_SOT23, Package_TO_SOT_SMD:SOT-23, symbol Diode:SM712_SOT23
- removed J4: Power connector, Connector_custom:JILN JL301-50002U01, symbol Connector:Screw_Terminal_01x02
- removed J5: Motor connector, Connector_custom:JILN JL301-50002U01, symbol Connector:Screw_Terminal_01x02
- removed J6: RS485 connector, Connector_custom:JILN JL301-50002U01, symbol Connector:Screw_Terminal_01x02
- removed R12: 10R, Resistor_SMD:R_0805_2012Metric_Pad1.20x1.40mm_HandSolder, symbol Device:R
- added J1: RS485, Connector_JST:JST_PH_S2B-PH-K_1x02_P2.00mm_Horizontal, symbol Connector_Generic:Conn_01x02
- added J2: 12V PWR, Connector_custom:HC-2510-2AW, symbol Connector_Generic:Conn_01x02
- R11: value 10R -> 120R; Manufacturer Part Number AC0805JR-0710RL -> RC0805JR-07120RL
- R2: Manufacturer Part Number (none) -> RC0805FR-0754K9L
Connections:
- net +12V: now also J2.1 (Pin_1)
- net GND: now also J2.2 (Pin_2)
- net at U3.6 (A): now also R11.2, J1.2 (Pin_2)
- net at U3.7 (B): now also R11.1, J1.1 (Pin_1); no longer R11.2

Commit message: Progressed ECAD
Parts:
- added J4: Motor, Connector_JST:JST_PH_S2B-PH-K_1x02_P2.00mm_Horizontal, symbol Connector_Generic:Conn_01x02
Connections:
- net H-bridge/Motor_L: now also J4.1 (Pin_1)
- net H-bridge/Motor_R: now also J4.2 (Pin_2)
