File: Tester/ECAD/USBGatewayBoard/RS232Interface.kicad_sch (KiCad schematic)
At the start: 9 parts, among them J3 RS232, U2 SP213E

Commit message: Progressed CAD
Parts:
- renumbered C3 to C1, C4 to C2, C5 to C3, C6 to C4, C7 to C5, C8 to C6, J3 to J2, R4 to R3, U2 to U1
Changed lines of the file:
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@@
   (symbol (lib_id "Connector:DB9_Male_MountingHoles") (at 218.44 88.9 0) (unit 1)
     (in_bom yes) (on_board yes) (fields_autoplaced)
-    (property "Reference" "J3" (id 0) (at 223.52 87.6299 0)
+    (property "Reference" "J2" (id 0) (at 223.52 87.6299 0)
       (effects (font (size 1.27 1.27)) (justify left))
     )
@@
   (symbol (lib_id "Interface_UART_custom:MAX213") (at 133.35 77.47 0) (unit 1)
     (in_bom yes) (on_board yes) (fields_autoplaced)
-    (property "Reference" "U2" (id 0) (at 135.3694 58.42 0)
+    (property "Reference" "U1" (id 0) (at 135.3694 58.42 0)
       (effects (font (size 1.27 1.27)) (justify left))
     )
@@
   (symbol (lib_id "power:GND") (at 133.35 109.22 0) (unit 1)
     (in_bom yes) (on_board yes) (fields_autoplaced)
-    (property "Reference" "#PWR011" (id 0) (at 133.35 115.57 0)
+    (property "Reference" "#PWR05" (id 0) (at 133.35 115.57 0)
       (effects (font (size 1.27 1.27)) hide)
     )
@@
   (symbol (lib_id "Device:C") (at 119.38 153.67 180) (unit 1)
     (in_bom yes) (on_board yes) (fields_autoplaced)
-    (property "Reference" "C3" (id 0) (at 123.19 152.3999 0)
+    (property "Reference" "C1" (id 0) (at 123.19 152.3999 0)
       (effects (font (size 1.27 1.27)) (justify right))
     )
@@
   (symbol (lib_id "Device:R") (at 224.79 118.11 0) (unit 1)
     (in_bom yes) (on_board yes) (fields_autoplaced)
-    (property "Reference" "R4" (id 0) (at 227.33 116.8399 0)
+    (property "Reference" "R3" (id 0) (at 227.33 116.8399 0)
       (effects (font (size 1.27 1.27)) (justify left))
     )
@@
   (symbol (lib_id "Device:C") (at 147.32 176.53 180) (unit 1)
     (in_bom yes) (on_board yes) (fields_autoplaced)
-    (property "Reference" "C7" (id 0) (at 151.13 175.2599 0)
+    (property "Reference" "C5" (id 0) (at 151.13 175.2599 0)
       (effects (font (size 1.27 1.27)) (justify right))
     )
@@
   (symbol (lib_id "Device:C") (at 212.09 118.11 0) (unit 1)
     (in_bom yes) (on_board yes) (fields_autoplaced)
-    (property "Reference" "C8" (id 0) (at 215.9 116.8399 0)
+    (property "Reference" "C6" (id 0) (at 215.9 116.8399 0)
       (effects (font (size 1.27 1.27)) (justify left))
     )
@@
   (symbol (lib_id "power:GND") (at 147.32 180.34 0) (unit 1)
     (in_bom yes) (on_board yes) (fields_autoplaced)
-    (property "Reference" "#PWR012" (id 0) (at 147.32 186.69 0)
+    (property "Reference" "#PWR06" (id 0) (at 147.32 186.69 0)
       (effects (font (size 1.27 1.27)) hide)
     )
@@
   (symbol (lib_id "power:GND") (at 119.38 180.34 0) (unit 1)
     (in_bom yes) (on_board yes) (fields_autoplaced)
-    (property "Reference" "#PWR010" (id 0) (at 119.38 186.69 0)
+    (property "Reference" "#PWR04" (id 0) (at 119.38 186.69 0)
       (effects (font (size 1.27 1.27)) hide)
     )
@@
   (symbol (lib_id "Device:C") (at 119.38 176.53 180) (unit 1)
     (in_bom yes) (on_board yes) (fields_autoplaced)
-    (property "Reference" "C4" (id 0) (at 123.19 175.2599 0)
+    (property "Reference" "C2" (id 0) (at 123.19 175.2599 0)
       (effects (font (size 1.27 1.27)) (justify right))
     )
@@
   (symbol (lib_id "power:GND") (at 218.44 123.19 0) (unit 1)
     (in_bom yes) (on_board yes) (fields_autoplaced)
-    (property "Reference" "#PWR014" (id 0) (at 218.44 129.54 0)
+    (property "Reference" "#PWR08" (id 0) (at 218.44 129.54 0)
       (effects (font (size 1.27 1.27)) hide)
     )
@@
   (symbol (lib_id "power:GND") (at 209.55 105.41 0) (unit 1)
     (in_bom yes) (on_board yes) (fields_autoplaced)
-    (property "Reference" "#PWR013" (id 0) (at 209.55 111.76 0)
+    (property "Reference" "#PWR07" (id 0) (at 209.55 111.76 0)
       (effects (font (size 1.27 1.27)) hide)
     )
@@
   (symbol (lib_id "Device:C") (at 133.35 176.53 180) (unit 1)
     (in_bom yes) (on_board yes) (fields_autoplaced)
-    (property "Reference" "C6" (id 0) (at 137.16 175.2599 0)
+    (property "Reference" "C4" (id 0) (at 137.16 175.2599 0)
       (effects (font (size 1.27 1.27)) (justify right))
     )
@@
   (symbol (lib_id "Device:C") (at 133.35 153.67 180) (unit 1)
     (in_bom yes) (on_board yes) (fields_autoplaced)
-    (property "Reference" "C5" (id 0) (at 137.16 152.3999 0)
-      (effects (font (size 1.27 1.27)) (justify right))
-    )
+    (property "Reference" "C3" (id 0) (at 137.16 152.3999 0)
+      (effects (font (size 1.27 1.27)) (justify right))
+    )

Commit message: Progressed CAD
Parts:
- added C? (x2): 1uC, symbol Device:C_Polarized
- added U?: MAX232, symbol Interface_UART:MAX232
- added U?: MAX3232, symbol Interface_UART:MAX3232
Connections:
- net 5V: now also U?.16 (VCC)
- net GND: now also U?.15 (GND)
- net RX: now also U?.12 (R1OUT), U?.13 (R1IN)
- net TX: now also U?.11 (T1IN), U?.14 (T1OUT)
- new net: C?.1, U?.1 (C1+)
- new net: C?.2, U?.3 (C1-)
- new net: C?.1, U?.4 (C2+)
- new net: C?.2, U?.5 (C2-)
Changed lines of the file:
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@@
+    (stroke (width 0) (type default) (color 0 0 0 0))
+  )
+  (wire (pts (xy 85.09 68.58) (xy 80.01 68.58))
     (stroke (width 0) (type default) (color 0 0 0 0))
   )
@@
     (stroke (width 0) (type default) (color 0 0 0 0))
   )
+  (wire (pts (xy 34.29 68.58) (xy 39.37 68.58))
+    (stroke (width 0) (type default) (color 0 0 0 0))
+  )
   (wire (pts (xy 144.78 100.33) (xy 149.86 100.33))
     (stroke (width 0) (type default) (color 0 0 0 0))
@@
     (stroke (width 0) (type default) (color 0 0 0 0))
   )
+  (wire (pts (xy 80.01 86.36) (xy 85.09 86.36))
+    (stroke (width 0) (type default) (color 0 0 0 0))
+  )
   (wire (pts (xy 144.78 78.74) (xy 149.86 78.74))
     (stroke (width 0) (type default) (color 0 0 0 0))
@@
     (stroke (width 0) (type default) (color 0 0 0 0))
   )
+  (wire (pts (xy 80.01 96.52) (xy 85.09 96.52))
+    (stroke (width 0) (type default) (color 0 0 0 0))
+  )
   (wire (pts (xy 144.78 97.79) (xy 149.86 97.79))
     (stroke (width 0) (type default) (color 0 0 0 0))
@@
     (stroke (width 0) (type default) (color 0 0 0 0))
   )
+  (wire (pts (xy 34.29 60.96) (xy 39.37 60.96))
+    (stroke (width 0) (type default) (color 0 0 0 0))
+  )
   (wire (pts (xy 133.35 144.78) (xy 133.35 149.86))
     (stroke (width 0) (type default) (color 0 0 0 0))
   )
+  (wire (pts (xy 85.09 60.96) (xy 80.01 60.96))
+    (stroke (width 0) (type default) (color 0 0 0 0))
+  )
   (text "RS232 Level Translator" (at 123.19 29.21 0)
     (effects (font (size 1.27 1.27)) (justify left bottom))
@@
     (effects (font (size 1.27 1.27)) (justify right bottom))
   )
+  (label "TX" (at 85.09 86.36 180)
+    (effects (font (size 1.27 1.27)) (justify right bottom))
+  )
   (label "TX" (at 149.86 78.74 180)
     (effects (font (size 1.27 1.27)) (justify right bottom))
@@
   )
   (label "V+" (at 149.86 66.04 180)
+    (effects (font (size 1.27 1.27)) (justify right bottom))
+  )
+  (label "RX" (at 85.09 96.52 180)
     (effects (font (size 1.27 1.27)) (justify right bottom))
   )
@@
     (effects (font (size 1.27 1.27)) (justify right))
   )
+  (hierarchical_label "RX" (shape output) (at 39.37 96.52 180)
+    (effects (font (size 1.27 1.27)) (justify right))
+  )
   (hierarchical_label "5V" (shape input) (at 147.32 172.72 90)
     (effects (font (size 1.27 1.27)) (justify left))
   )
+  (hierarchical_label "TX" (shape input) (at 39.37 86.36 180)
+    (effects (font (size 1.27 1.27)) (justify right))
+  )
   (hierarchical_label "CTS" (shape output) (at 123.19 92.71 180)
     (effects (font (size 1.27 1.27)) (justify right))
@@
   )
   (hierarchical_label "5V" (shape input) (at 133.35 172.72 90)
+    (effects (font (size 1.27 1.27)) (justify left))
+  )
+  (hierarchical_label "5V" (shape input) (at 59.69 53.34 90)
     (effects (font (size 1.27 1.27)) (justify left))
   )
@@
     (pin "1")
   )
+  (symbol (lib_id "Device:C_Polarized") (at 34.29 64.77 0) (unit 1)
+    (in_bom yes) (on_board yes) (fields_autoplaced)
+    (property "Reference" "C?" (id 0) (at 38.1 62.6109 0)
+      (effects (font (size 1.27 1.27)) (justify left))
+    )
+    (property "Value" "1uC" (id 1) (at 38.1 65.1509 0)
+      (effects (font (size 1.27 1.27)) (justify left))
+    )
+    (property "Footprint" "" (id 2) (at 35.2552 68.58 0)
+      (effects (font (size 1.27 1.27)) hide)
+    )
+    (property "Datasheet" "~" (id 3) (at 34.29 64.77 0)
+      (effects (font (size 1.27 1.27)) hide)
+    )
+    (pin "1")
+    (pin "2")
+  )
   (symbol (lib_id "power:GND") (at 119.38 180.34 0) (unit 1)
     (in_bom yes) (on_board yes) (fields_autoplaced)
@@
     (pin "1")
   )
+  (symbol (lib_id "Interface_UART:MAX232") (at 59.69 83.82 0) (unit 1)
+    (in_bom yes) (on_board yes) (fields_autoplaced)
+    (property "Reference" "U?" (id 0) (at 61.7094 53.34 0)
+      (effects (font (size 1.27 1.27)) (justify left))
+    )
+    (property "Value" "MAX232" (id 1) (at 61.7094 55.88 0)
+      (effects (font (size 1.27 1.27)) (justify left))
+    )
+    (property "Footprint" "" (id 2) (at 60.96 110.49 0)
+      (effects (font (size 1.27 1.27)) (justify left) hide)
+    )
+    (property "Datasheet" "http://www.ti.com/lit/ds/symlink/max232.pdf" (id 3) (at 59.69 81.28 0)
+      (effects (font (size 1.27 1.27)) hide)
+    )
+    (pin "1")
+    (pin "10")
+    (pin "11")
+    (pin "12")
+    (pin "13")
+    (pin "14")
+    (pin "15")
+    (pin "16")
+    (pin "2")
+    (pin "3")
+    (pin "4")
+    (pin "5")
+    (pin "6")
+    (pin "7")
+    (pin "8")
+    (pin "9")
+  )
+  (symbol (lib_id "power:GND") (at 59.69 114.3 0) (unit 1)
+    (in_bom yes) (on_board yes) (fields_autoplaced)
+    (property "Reference" "#PWR?" (id 0) (at 59.69 120.65 0)
+      (effects (font (size 1.27 1.27)) hide)
+    )
+    (property "Value" "GND" (id 1) (at 59.69 119.38 0))
+    (property "Footprint" "" (id 2) (at 59.69 114.3 0)
+      (effects (font (size 1.27 1.27)) hide)
+    )
+    (property "Datasheet" "" (id 3) (at 59.69 114.3 0)
+      (effects (font (size 1.27 1.27)) hide)
+    )
+    (pin "1")
+  )
+  (symbol (lib_id "Interface_UART:MAX3232") (at 59.69 154.94 0) (unit 1)
+    (in_bom yes) (on_board yes) (fields_autoplaced)
+    (property "Reference" "U?" (id 0) (at 61.7094 124.46 0)
+      (effects (font (size 1.27 1.27)) (justify left))
+    )
+    (property "Value" "MAX3232" (id 1) (at 61.7094 127 0)
+      (effects (font (size 1.27 1.27)) (justify left))
+    )
+    (property "Footprint" "" (id 2) (at 60.96 181.61 0)
+      (effects (font (size 1.27 1.27)) (justify left) hide)
+    )
+    (property "Datasheet" "https://datasheets.maximintegrated.com/en/ds/MAX3222-MAX3241.pdf" (id 3) (at 59.69 152.4 0)
+      (effects (font (size 1.27 1.27)) hide)
+    )
+    (pin "1")
+    (pin "10")
+    (pin "11")
+    (pin "12")
+    (pin "13")
+    (pin "14")
+    (pin "15")
+    (pin "16")
+    (pin "2")
+    (pin "3")
+    (pin "4")
+    (pin "5")
+    (pin "6")
+    (pin "7")
+    (pin "8")
+    (pin "9")
+  )
   (symbol (lib_id "Device:C") (at 133.35 176.53 180) (unit 1)
     (in_bom yes) (on_board yes) (fields_autoplaced)
@@
       (effects (font (size 1.27 1.27)) hide)
     )
+    (pin "1")
+    (pin "2")
+  )
+  (symbol (lib_id "Device:C_Polarized") (at 85.09 64.77 0) (unit 1)
+    (in_bom yes) (on_board yes) (fields_autoplaced)
+    (property "Reference" "C?" (id 0) (at 88.9 62.6109 0)
+      (effects (font (size 1.27 1.27)) (justify left))
+    )
+    (property "Value" "1uC" (id 1) (at 88.9 65.1509 0)
+      (effects (font (size 1.27 1.27)) (justify left))
+    )
+    (property "Footprint" "" (id 2) (at 86.0552 68.58 0)
+      (effects (font (size 1.27 1.27)) hide)
+    )
+    (property "Datasheet" "~" (id 3) (at 85.09 64.77 0)
+      (effects (font (size 1.27 1.27)) hide)
+    )

Commit message: Progressed CAD
Parts:
- removed C1, C2, C3, C4, C5: 0.1uC, Capacitor_SMD:C_0805_2012Metric_Pad1.18x1.45mm_HandSolder, symbol Device:C
- removed C? (x2): 1uC, symbol Device:C_Polarized
- removed U1: SP213E, Package_SO:SSOP-28_5.3x10.2mm_P0.65mm, symbol Interface_UART_custom:MAX213
- removed U?: MAX232, symbol Interface_UART:MAX232
- added C? (x5): 0.1uC, symbol Device:C_Polarized
- gave numbers to parts that had none: 1
- renumbered C6 to C8, J2 to J5
Connections:
- net GND: now also U2.15 (GND), C?.1, C?.2, C?.2
- net RX: now also U2.12 (R1OUT), U2.13 (R1IN)
- net TX: now also U2.11 (T1IN), U2.14 (T1OUT)
- net at U2.1 (C1+): now also C?.1
- net 3V3: now reaches U2.16 (VCC)
- net 3V3: now also C?.1
- net at U2.2 (VS+): now also C?.1
- net at U2.3 (C1-): now also C?.2
- net at U2.4 (C2+): now also C?.1
- net at U2.5 (C2-): now also C?.2
- net at U2.6 (VS-): now also C?.2
- no-connect marks 2 -> 0
Other:
- moved on the sheet: C8, J5, R3, U2

Commit message: Progressed ECAD
Parts:
- gave numbers to parts that had none: 5
Changed lines of the file:
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@@
   (symbol (lib_id "Device:C_Polarized") (at 71.12 148.59 0) (unit 1)
     (in_bom yes) (on_board yes) (fields_autoplaced)
-    (property "Reference" "C?" (id 0) (at 74.93 146.4309 0)
+    (property "Reference" "C2" (id 0) (at 74.93 146.4309 0)
       (effects (font (size 1.27 1.27)) (justify left))
     )
@@
   (symbol (lib_id "power:GND") (at 71.12 152.4 0) (unit 1)
     (in_bom yes) (on_board yes) (fields_autoplaced)
-    (property "Reference" "#PWR?" (id 0) (at 71.12 158.75 0)
+    (property "Reference" "#PWR0103" (id 0) (at 71.12 158.75 0)
       (effects (font (size 1.27 1.27)) hide)
     )
@@
   (symbol (lib_id "Device:C_Polarized") (at 118.11 91.44 0) (unit 1)
     (in_bom yes) (on_board yes) (fields_autoplaced)
-    (property "Reference" "C?" (id 0) (at 121.92 89.2809 0)
+    (property "Reference" "C5" (id 0) (at 121.92 89.2809 0)
       (effects (font (size 1.27 1.27)) (justify left))
     )
@@
   (symbol (lib_id "Device:C_Polarized") (at 111.76 99.06 0) (mirror x) (unit 1)
     (in_bom yes) (on_board yes)
-    (property "Reference" "C?" (id 0) (at 107.95 98.6789 0)
+    (property "Reference" "C4" (id 0) (at 107.95 98.6789 0)
       (effects (font (size 1.27 1.27)) (justify right))
     )
@@
   (symbol (lib_id "Device:C_Polarized") (at 45.72 77.47 0) (unit 1)
     (in_bom yes) (on_board yes)
-    (property "Reference" "C?" (id 0) (at 36.83 76.2 0)
+    (property "Reference" "C1" (id 0) (at 36.83 76.2 0)
       (effects (font (size 1.27 1.27)) (justify left))
     )
@@
   (symbol (lib_id "Device:C_Polarized") (at 96.52 77.47 0) (unit 1)
     (in_bom yes) (on_board yes) (fields_autoplaced)
-    (property "Reference" "C?" (id 0) (at 100.33 75.3109 0)
+    (property "Reference" "C3" (id 0) (at 100.33 75.3109 0)
       (effects (font (size 1.27 1.27)) (justify left))
     )
@@
   (symbol (lib_id "power:GND") (at 111.76 102.87 0) (unit 1)
     (in_bom yes) (on_board yes) (fields_autoplaced)
-    (property "Reference" "#PWR?" (id 0) (at 111.76 109.22 0)
+    (property "Reference" "#PWR0101" (id 0) (at 111.76 109.22 0)
       (effects (font (size 1.27 1.27)) hide)
     )
@@
   (symbol (lib_id "power:GND") (at 118.11 95.25 0) (unit 1)
     (in_bom yes) (on_board yes) (fields_autoplaced)
-    (property "Reference" "#PWR?" (id 0) (at 118.11 101.6 0)
-      (effects (font (size 1.27 1.27)) hide)
-    )
+    (property "Reference" "#PWR0102" (id 0) (at 118.11 101.6 0)
+      (effects (font (size 1.27 1.27)) hide)
+    )

Commit message: Progressed ECAD
Parts:
- removed C1, C2, C3, C4, C5: 0.1uC, symbol Device:C_Polarized
- removed U2: MAX3232, symbol Interface_UART:MAX3232
- added C1, C2, C3, C4, C5: 0.1uC, Capacitor_SMD:C_0805_2012Metric_Pad1.18x1.45mm_HandSolder, symbol Device:C
- added U1: SP213E, Package_SO:SSOP-28_5.3x10.2mm_P0.65mm, symbol Interface_UART_custom:MAX213
- renumbered C8 to C6, J5 to J4, R3 to R1
Connections:
- net CTS: now also U1.4 (RIN2), U1.5 (ROUT2)
- net DCD: now also U1.18 (RIN5), U1.19 (ROUT5)
- net DSR: now also U1.26 (ROUT3), U1.27 (RIN3)
- net DTR: now also U1.3 (DOUT2), U1.6 (DIN2)
- net GND: now also C2.1, C5.1, U1.10 (GND)
- net RI: now also U1.22 (ROUT4), U1.23 (RIN4)
- net RTS: now also U1.1 (DOUT3), U1.20 (DIN3)
- net RX: now also U1.8 (ROUT1), U1.9 (RIN1)
- net TX: now also U1.2 (DOUT1), U1.7 (DIN1)
- new net 5V: C4.2, C5.2, U1.11 (VCC), U1.24 (EN), U1.25 (~{SHDN})
- new net C1+: C1.2, U1.12 (C1+)
- new net C1-: C1.1, U1.14 (C1-)
- new net C2+: C3.2, U1.15 (C2+)
- new net C2-: C3.1, U1.16 (C2-)
- new net V+: C4.1, U1.13 (V+)
- new net V-: C2.2, U1.17 (V-)
- no-connect marks 0 -> 2
Other:
- moved on the sheet: C6, J4, R1
