File: Tester/ECAD/USBGatewayBoard/RS485Interface.kicad_sch (KiCad schematic)
At the start: 7 parts, among them J4 RS485 connector, U3 SP485

Commit message: Progressed CAD
Parts:
- renumbered C9 to C7, J4 to J3, R5 to R4, R6 to R5, R7 to R6, U3 to U2
Changed lines of the file:
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@@
   (symbol (lib_id "Device:C") (at 133.35 138.43 180) (unit 1)
     (in_bom yes) (on_board yes) (fields_autoplaced)
-    (property "Reference" "C9" (id 0) (at 137.16 137.1599 0)
+    (property "Reference" "C7" (id 0) (at 137.16 137.1599 0)
       (effects (font (size 1.27 1.27)) (justify right))
     )
@@
   (symbol (lib_id "Interface_UART:ST485EBDR") (at 133.35 101.6 0) (unit 1)
     (in_bom yes) (on_board yes) (fields_autoplaced)
-    (property "Reference" "U3" (id 0) (at 135.3694 88.9 0)
+    (property "Reference" "U2" (id 0) (at 135.3694 88.9 0)
       (effects (font (size 1.27 1.27)) (justify left))
     )
@@
   (symbol (lib_id "power:GND") (at 133.35 114.3 0) (unit 1)
     (in_bom yes) (on_board yes) (fields_autoplaced)
-    (property "Reference" "#PWR016" (id 0) (at 133.35 120.65 0)
+    (property "Reference" "#PWR010" (id 0) (at 133.35 120.65 0)
       (effects (font (size 1.27 1.27)) hide)
     )
@@
   (symbol (lib_id "Device:R") (at 116.84 111.76 0) (unit 1)
     (in_bom yes) (on_board yes) (fields_autoplaced)
-    (property "Reference" "R5" (id 0) (at 119.38 110.4899 0)
+    (property "Reference" "R4" (id 0) (at 119.38 110.4899 0)
       (effects (font (size 1.27 1.27)) (justify left))
     )
@@
   (symbol (lib_id "Connector:Screw_Terminal_01x02") (at 205.74 101.6 0) (unit 1)
     (in_bom yes) (on_board yes) (fields_autoplaced)
-    (property "Reference" "J4" (id 0) (at 208.28 101.5999 0)
+    (property "Reference" "J3" (id 0) (at 208.28 101.5999 0)
       (effects (font (size 1.27 1.27)) (justify left))
     )
@@
   (symbol (lib_id "Device:R") (at 172.72 111.76 90) (unit 1)
     (in_bom yes) (on_board yes) (fields_autoplaced)
-    (property "Reference" "R7" (id 0) (at 172.72 105.41 90))
+    (property "Reference" "R6" (id 0) (at 172.72 105.41 90))
     (property "Value" "10R" (id 1) (at 172.72 107.95 90))
     (property "Footprint" "Resistor_SMD:R_0805_2012Metric_Pad1.20x1.40mm_HandSolder" (id 2) (at 172.72 113.538 90)
@@
   (symbol (lib_id "power:GND") (at 149.86 114.3 0) (unit 1)
     (in_bom yes) (on_board yes) (fields_autoplaced)
-    (property "Reference" "#PWR018" (id 0) (at 149.86 120.65 0)
+    (property "Reference" "#PWR012" (id 0) (at 149.86 120.65 0)
       (effects (font (size 1.27 1.27)) hide)
     )
@@
   (symbol (lib_id "power:GND") (at 116.84 115.57 0) (unit 1)
     (in_bom yes) (on_board yes) (fields_autoplaced)
-    (property "Reference" "#PWR015" (id 0) (at 116.84 121.92 0)
+    (property "Reference" "#PWR09" (id 0) (at 116.84 121.92 0)
       (effects (font (size 1.27 1.27)) hide)
     )
@@
   (symbol (lib_id "Device:R") (at 172.72 93.98 90) (unit 1)
     (in_bom yes) (on_board yes) (fields_autoplaced)
-    (property "Reference" "R6" (id 0) (at 172.72 87.63 90))
+    (property "Reference" "R5" (id 0) (at 172.72 87.63 90))
     (property "Value" "10R" (id 1) (at 172.72 90.17 90))
     (property "Footprint" "Resistor_SMD:R_0805_2012Metric_Pad1.20x1.40mm_HandSolder" (id 2) (at 172.72 95.758 90)
@@
   (symbol (lib_id "power:GND") (at 133.35 142.24 0) (unit 1)
     (in_bom yes) (on_board yes) (fields_autoplaced)
-    (property "Reference" "#PWR017" (id 0) (at 133.35 148.59 0)
+    (property "Reference" "#PWR011" (id 0) (at 133.35 148.59 0)
       (effects (font (size 1.27 1.27)) hide)
     )

Commit message: Progressed CAD
Parts:
- renumbered C7 to C9, J3 to J6, U2 to U4
Changed lines of the file:
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@@
   (symbol (lib_id "Device:C") (at 133.35 138.43 180) (unit 1)
     (in_bom yes) (on_board yes) (fields_autoplaced)
-    (property "Reference" "C7" (id 0) (at 137.16 137.1599 0)
+    (property "Reference" "C9" (id 0) (at 137.16 137.1599 0)
       (effects (font (size 1.27 1.27)) (justify right))
     )
@@
   (symbol (lib_id "Interface_UART:ST485EBDR") (at 133.35 101.6 0) (unit 1)
     (in_bom yes) (on_board yes) (fields_autoplaced)
-    (property "Reference" "U2" (id 0) (at 135.3694 88.9 0)
+    (property "Reference" "U4" (id 0) (at 135.3694 88.9 0)
       (effects (font (size 1.27 1.27)) (justify left))
     )
@@
   (symbol (lib_id "power:GND") (at 133.35 114.3 0) (unit 1)
     (in_bom yes) (on_board yes) (fields_autoplaced)
-    (property "Reference" "#PWR010" (id 0) (at 133.35 120.65 0)
+    (property "Reference" "#PWR012" (id 0) (at 133.35 120.65 0)
       (effects (font (size 1.27 1.27)) hide)
     )
@@
   (symbol (lib_id "Connector:Screw_Terminal_01x02") (at 205.74 101.6 0) (unit 1)
     (in_bom yes) (on_board yes) (fields_autoplaced)
-    (property "Reference" "J3" (id 0) (at 208.28 101.5999 0)
+    (property "Reference" "J6" (id 0) (at 208.28 101.5999 0)
       (effects (font (size 1.27 1.27)) (justify left))
     )
@@
   (symbol (lib_id "power:GND") (at 149.86 114.3 0) (unit 1)
     (in_bom yes) (on_board yes) (fields_autoplaced)
-    (property "Reference" "#PWR012" (id 0) (at 149.86 120.65 0)
+    (property "Reference" "#PWR014" (id 0) (at 149.86 120.65 0)
       (effects (font (size 1.27 1.27)) hide)
     )
@@
   (symbol (lib_id "power:GND") (at 116.84 115.57 0) (unit 1)
     (in_bom yes) (on_board yes) (fields_autoplaced)
-    (property "Reference" "#PWR09" (id 0) (at 116.84 121.92 0)
+    (property "Reference" "#PWR011" (id 0) (at 116.84 121.92 0)
       (effects (font (size 1.27 1.27)) hide)
     )
@@
   (symbol (lib_id "power:GND") (at 133.35 142.24 0) (unit 1)
     (in_bom yes) (on_board yes) (fields_autoplaced)
-    (property "Reference" "#PWR011" (id 0) (at 133.35 148.59 0)
+    (property "Reference" "#PWR013" (id 0) (at 133.35 148.59 0)
       (effects (font (size 1.27 1.27)) hide)
     )

Commit message: Progressed ECAD
Parts:
- renumbered C9 to C7, D2 to D1, J6 to J5, R4 to R2, R5 to R3, R6 to R4, U4 to U2
Changed lines of the file:
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@@
     (stroke (width 0) (type default) (color 0 0 0 0))
   )
-  (text "RS485 Level Translator" (at 124.46 30.48 0)
+  (text "RS485 Level Translator" (at 123.19 81.28 0)
     (effects (font (size 1.27 1.27)) (justify left bottom))
   )
@@
   (symbol (lib_id "Device:C") (at 133.35 138.43 180) (unit 1)
     (in_bom yes) (on_board yes) (fields_autoplaced)
-    (property "Reference" "C9" (id 0) (at 137.16 137.1599 0)
+    (property "Reference" "C7" (id 0) (at 137.16 137.1599 0)
       (effects (font (size 1.27 1.27)) (justify right))
     )
@@
   (symbol (lib_id "Interface_UART:ST485EBDR") (at 133.35 101.6 0) (unit 1)
     (in_bom yes) (on_board yes) (fields_autoplaced)
-    (property "Reference" "U4" (id 0) (at 135.3694 88.9 0)
+    (property "Reference" "U2" (id 0) (at 135.3694 88.9 0)
       (effects (font (size 1.27 1.27)) (justify left))
     )
@@
   (symbol (lib_id "Diode:SM712_SOT23") (at 153.67 102.87 270) (mirror x) (unit 1)
     (in_bom yes) (on_board yes) (fields_autoplaced)
-    (property "Reference" "D2" (id 0) (at 156.21 101.5999 90)
+    (property "Reference" "D1" (id 0) (at 156.21 101.5999 90)
       (effects (font (size 1.27 1.27)) (justify left))
     )
@@
   (symbol (lib_id "power:GND") (at 133.35 114.3 0) (unit 1)
     (in_bom yes) (on_board yes) (fields_autoplaced)
-    (property "Reference" "#PWR012" (id 0) (at 133.35 120.65 0)
+    (property "Reference" "#PWR07" (id 0) (at 133.35 120.65 0)
       (effects (font (size 1.27 1.27)) hide)
     )
@@
   (symbol (lib_id "Device:R") (at 116.84 111.76 0) (unit 1)
     (in_bom yes) (on_board yes) (fields_autoplaced)
-    (property "Reference" "R4" (id 0) (at 119.38 110.4899 0)
+    (property "Reference" "R2" (id 0) (at 119.38 110.4899 0)
       (effects (font (size 1.27 1.27)) (justify left))
     )
@@
   (symbol (lib_id "Connector:Screw_Terminal_01x02") (at 205.74 101.6 0) (unit 1)
     (in_bom yes) (on_board yes) (fields_autoplaced)
-    (property "Reference" "J6" (id 0) (at 208.28 101.5999 0)
+    (property "Reference" "J5" (id 0) (at 208.28 101.5999 0)
       (effects (font (size 1.27 1.27)) (justify left))
     )
@@
   (symbol (lib_id "Device:R") (at 172.72 111.76 90) (unit 1)
     (in_bom yes) (on_board yes) (fields_autoplaced)
-    (property "Reference" "R6" (id 0) (at 172.72 105.41 90))
+    (property "Reference" "R4" (id 0) (at 172.72 105.41 90))
     (property "Value" "10R" (id 1) (at 172.72 107.95 90))
     (property "Footprint" "Resistor_SMD:R_0805_2012Metric_Pad1.20x1.40mm_HandSolder" (id 2) (at 172.72 113.538 90)
@@
   (symbol (lib_id "power:GND") (at 149.86 114.3 0) (unit 1)
     (in_bom yes) (on_board yes) (fields_autoplaced)
-    (property "Reference" "#PWR014" (id 0) (at 149.86 120.65 0)
+    (property "Reference" "#PWR09" (id 0) (at 149.86 120.65 0)
       (effects (font (size 1.27 1.27)) hide)
     )
@@
   (symbol (lib_id "power:GND") (at 116.84 115.57 0) (unit 1)
     (in_bom yes) (on_board yes) (fields_autoplaced)
-    (property "Reference" "#PWR011" (id 0) (at 116.84 121.92 0)
+    (property "Reference" "#PWR06" (id 0) (at 116.84 121.92 0)
       (effects (font (size 1.27 1.27)) hide)
     )
@@
   (symbol (lib_id "Device:R") (at 172.72 93.98 90) (unit 1)
     (in_bom yes) (on_board yes) (fields_autoplaced)
-    (property "Reference" "R5" (id 0) (at 172.72 87.63 90))
+    (property "Reference" "R3" (id 0) (at 172.72 87.63 90))
     (property "Value" "10R" (id 1) (at 172.72 90.17 90))
     (property "Footprint" "Resistor_SMD:R_0805_2012Metric_Pad1.20x1.40mm_HandSolder" (id 2) (at 172.72 95.758 90)
@@
   (symbol (lib_id "power:GND") (at 133.35 142.24 0) (unit 1)
     (in_bom yes) (on_board yes) (fields_autoplaced)
-    (property "Reference" "#PWR013" (id 0) (at 133.35 148.59 0)
-      (effects (font (size 1.27 1.27)) hide)
-    )
+    (property "Reference" "#PWR08" (id 0) (at 133.35 148.59 0)
+      (effects (font (size 1.27 1.27)) hide)
+    )
