File: Tester/ECAD/USBGatewayBoard/power_supply.kicad_sch (KiCad schematic)
At the start: 2 parts, among them J2 Barrel_Jack, J8 Barrel_Jack_MountingPin

Commit message: Progressed ECAD
Parts:
- removed J8: Barrel_Jack_MountingPin, Connector_BarrelJack:BarrelJack_CUI_PJ-063AH_Horizontal, symbol Connector:Barrel_Jack_MountingPin
- added C35, C36: 0.1nC, Capacitor_SMD:C_0805_2012Metric_Pad1.18x1.45mm_HandSolder, symbol Device:C
- added C37: 220uC, Capacitor_THT:CP_Radial_D8.0mm_P3.50mm, symbol Device:C_Polarized
- added D6: D_TVS, Diode_SMD:D_SMA, symbol Device:D_TVS
- added D7: D_Zener, symbol Device:D_Zener
- added F2: Fuse, symbol Device:Fuse
- added FB2: FerriteBead, Inductor_SMD:L_1806_4516Metric_Pad1.45x1.90mm_HandSolder, symbol Device:FerriteBead
- added Q5: IRF7404, Package_SO:SOIC-8_3.9x4.9mm_P1.27mm, symbol Transistor_FET:IRF7404
- added R28: R, Resistor_SMD:R_0805_2012Metric_Pad1.20x1.40mm_HandSolder, symbol Device:R
- J2: Manufacturer Part Number (none) -> DC-042C-W-2.5
Connections:
- net at J2.1: now also F2.1
- net GND: now reaches J2.2
- net GND: now also C35.2, C36.2, C37.2, D6.1 (A1), R28.2
- new net: C35.1, D7.1 (K), FB2.1, Q5.1 (S), Q5.2 (S), Q5.3 (S)
- new net: D6.2 (A2), F2.2, Q5.5 (D), Q5.6 (D), Q5.7 (D), Q5.8 (D)
- new net: D7.2 (A), Q5.4 (G), R28.1
- new net 12V: C36.1, C37.1, FB2.2
Other:
- moved on the sheet: J2

Commit message: Progressed ECAD
Parts:
- added J4: Power connector, Connector_custom:JILN JL301-50002U01, symbol Connector:Screw_Terminal_01x02
Connections:
- net 12V: now also J4.1 (Pin_1)
- net GND: now also J4.2 (Pin_2)
Changed lines of the file:
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@@
   (junction (at 198.12 85.09) (diameter 0) (color 0 0 0 0)
   )
+  (junction (at 215.9 85.09) (diameter 0) (color 0 0 0 0)
+  )
   (junction (at 181.61 85.09) (diameter 0) (color 0 0 0 0)
   )
@@
     (stroke (width 0) (type default) (color 0 0 0 0))
   )
+  (wire (pts (xy 215.9 96.52) (xy 215.9 105.41))
+    (stroke (width 0) (type default) (color 0 0 0 0))
+  )
   (wire (pts (xy 198.12 85.09) (xy 198.12 91.44))
     (stroke (width 0) (type default) (color 0 0 0 0))
   )
+  (wire (pts (xy 215.9 85.09) (xy 222.25 85.09))
+    (stroke (width 0) (type default) (color 0 0 0 0))
+  )
   (wire (pts (xy 140.97 85.09) (xy 160.02 85.09))
     (stroke (width 0) (type default) (color 0 0 0 0))
@@
     (stroke (width 0) (type default) (color 0 0 0 0))
   )
-  (wire (pts (xy 198.12 85.09) (xy 212.09 85.09))
+  (wire (pts (xy 198.12 85.09) (xy 215.9 85.09))
     (stroke (width 0) (type default) (color 0 0 0 0))
   )
@@
     (stroke (width 0) (type default) (color 0 0 0 0))
   )
+  (wire (pts (xy 218.44 93.98) (xy 215.9 93.98))
+    (stroke (width 0) (type default) (color 0 0 0 0))
+  )
   (wire (pts (xy 87.63 85.09) (xy 97.79 85.09))
     (stroke (width 0) (type default) (color 0 0 0 0))
@@
     (stroke (width 0) (type default) (color 0 0 0 0))
   )
+  (wire (pts (xy 218.44 96.52) (xy 215.9 96.52))
+    (stroke (width 0) (type default) (color 0 0 0 0))
+  )
   (wire (pts (xy 198.12 99.06) (xy 198.12 105.41))
     (stroke (width 0) (type default) (color 0 0 0 0))
@@
     (stroke (width 0) (type default) (color 0 0 0 0))
   )
+  (wire (pts (xy 215.9 93.98) (xy 215.9 85.09))
+    (stroke (width 0) (type default) (color 0 0 0 0))
+  )
   (wire (pts (xy 160.02 85.09) (xy 160.02 91.44))
     (stroke (width 0) (type default) (color 0 0 0 0))
@@
     (stroke (width 0) (type default) (color 0 0 0 0))
   )
-  (hierarchical_label "12V" (shape output) (at 212.09 85.09 0)
+  (hierarchical_label "12V" (shape output) (at 222.25 85.09 0)
     (effects (font (size 1.27 1.27)) (justify left))
   )
@@
       (effects (font (size 1.27 1.27)) hide)
     )
+    (pin "1")
+    (pin "2")
+  )
+  (symbol (lib_id "power:GND") (at 215.9 105.41 0) (unit 1)
+    (in_bom yes) (on_board yes) (fields_autoplaced)
+    (property "Reference" "#PWR01" (id 0) (at 215.9 111.76 0)
+      (effects (font (size 1.27 1.27)) hide)
+    )
+    (property "Value" "GND" (id 1) (at 215.9 110.49 0))
+    (property "Footprint" "" (id 2) (at 215.9 105.41 0)
+      (effects (font (size 1.27 1.27)) hide)
+    )
+    (property "Datasheet" "" (id 3) (at 215.9 105.41 0)
+      (effects (font (size 1.27 1.27)) hide)
+    )
+    (pin "1")
+  )
+  (symbol (lib_id "Connector:Screw_Terminal_01x02") (at 223.52 93.98 0) (unit 1)
+    (in_bom yes) (on_board yes) (fields_autoplaced)
+    (property "Reference" "J4" (id 0) (at 226.06 93.9799 0)
+      (effects (font (size 1.27 1.27)) (justify left))
+    )
+    (property "Value" "Power connector" (id 1) (at 226.06 96.5199 0)
+      (effects (font (size 1.27 1.27)) (justify left))
+    )
+    (property "Footprint" "Connector_custom:JILN JL301-50002U01" (id 2) (at 223.52 93.98 0)
+      (effects (font (size 1.27 1.27)) hide)
+    )
+    (property "Datasheet" "https://datasheet.lcsc.com/lcsc/1912111437_JILN-JL301-50002U02_C395214.pdf" (id 3) (at 223.52 93.98 0)
+      (effects (font (size 1.27 1.27)) hide)
+    )
+    (property "Manufacturer Part Number" "JL301-50002U02" (id 4) (at 223.52 93.98 0)
+      (effects (font (size 1.27 1.27)) hide)
+    )
