File: Tester/ECAD/USBGatewayBoard/USBGatewayBoard.kicad_pcb (KiCad board)
At the start: 2 copper layers, 120 x 45 mm, 30 parts, among them J2 Barrel_Jack_MountingPin, J4 Power connector, J5 RS232, J6 RS485 connector, J7 USB_B, J8 RS232, Q1 BC846, U4 SP485, U5 USBLC6-2SC6

Commit message: Progressed ECAD
Parts:
- removed J2: Barrel_Jack_MountingPin, Connector_BarrelJack:BarrelJack_CUI_PJ-063AH_Horizontal
- added C1: 0.1uC, Capacitor_SMD:C_0805_2012Metric_Pad1.18x1.45mm_HandSolder, F.Cu at (71.0, 94.5)
- added C12: 1uC, Capacitor_SMD:C_0805_2012Metric_Pad1.18x1.45mm_HandSolder, F.Cu at (74.7, 37.7)
- added C13: 1uC, Capacitor_SMD:C_0805_2012Metric_Pad1.18x1.45mm_HandSolder, F.Cu at (85.3, 33.1)
- added C14: 220uC, Capacitor_THT:CP_Radial_D8.0mm_P3.50mm, F.Cu at (58.0, 29.9)
- added C15: 1uC, Capacitor_SMD:C_0805_2012Metric_Pad1.18x1.45mm_HandSolder, F.Cu at (66.9, 33.1)
- added C16: 1uC, Capacitor_SMD:C_0805_2012Metric_Pad1.18x1.45mm_HandSolder, F.Cu at (80.5, 36.1)
- added C17: 0.1uC, Capacitor_SMD:C_0805_2012Metric_Pad1.18x1.45mm_HandSolder, F.Cu at (89.4, 29.6)
- added C18: 0.1uC, Capacitor_SMD:C_0805_2012Metric_Pad1.18x1.45mm_HandSolder, F.Cu at (74.7, 40.7)
- added C2: 0.1uC, Capacitor_SMD:C_0805_2012Metric_Pad1.18x1.45mm_HandSolder, F.Cu at (66.7, 103.0)
- added C20: 1uC, Capacitor_SMD:C_0805_2012Metric_Pad1.18x1.45mm_HandSolder, F.Cu at (114.5, 43.8)
- added C21: 0.1uC, Capacitor_SMD:C_0805_2012Metric_Pad1.18x1.45mm_HandSolder, F.Cu at (124.8, 33.1)
- added C22: 1uC, Capacitor_SMD:C_0805_2012Metric_Pad1.18x1.45mm_HandSolder, F.Cu at (119.0, 37.7)
- added C23: 1uC, Capacitor_SMD:C_0805_2012Metric_Pad1.18x1.45mm_HandSolder, F.Cu at (129.6, 33.1)
- added C24: 220uC, Capacitor_THT:CP_Radial_D8.0mm_P3.50mm, F.Cu at (102.3, 29.9)
- added C25: 1uC, Capacitor_SMD:C_0805_2012Metric_Pad1.18x1.45mm_HandSolder, F.Cu at (111.2, 33.1)
- added C26: 1uC, Capacitor_SMD:C_0805_2012Metric_Pad1.18x1.45mm_HandSolder, F.Cu at (124.8, 36.1)
- added C27: 0.1uC, Capacitor_SMD:C_0805_2012Metric_Pad1.18x1.45mm_HandSolder, F.Cu at (133.7, 29.6)
- added C28: 0.1uC, Capacitor_SMD:C_0805_2012Metric_Pad1.18x1.45mm_HandSolder, F.Cu at (119.0, 40.7)
- added C29: 1uC, Capacitor_SMD:C_0805_2012Metric_Pad1.18x1.45mm_HandSolder, F.Cu at (133.7, 26.6)
- added C3: 0.1uC, Capacitor_SMD:C_0805_2012Metric_Pad1.18x1.45mm_HandSolder, F.Cu at (66.2, 94.5)
- added C30: 0.1uC, Capacitor_SMD:C_0805_2012Metric_Pad1.18x1.45mm_HandSolder, F.Cu at (169.2, 43.5)
- added C31: 0.1uC, Capacitor_SMD:C_0805_2012Metric_Pad1.18x1.45mm_HandSolder, F.Cu at (193.9, 28.9)
- added C32: 0.1uC, Capacitor_SMD:C_0805_2012Metric_Pad1.18x1.45mm_HandSolder, F.Cu at (174.0, 43.5)
- added C33: 0.1uC, Capacitor_SMD:C_0805_2012Metric_Pad1.18x1.45mm_HandSolder, F.Cu at (178.8, 43.5)
- added C34: 1uC, Capacitor_SMD:C_0805_2012Metric_Pad1.18x1.45mm_HandSolder, F.Cu at (185.1, 35.5)
- added C4: 0.1uC, Capacitor_SMD:C_0805_2012Metric_Pad1.18x1.45mm_HandSolder, F.Cu at (71.5, 103.0)
- added C5: 0.1uC, Capacitor_SMD:C_0805_2012Metric_Pad1.18x1.45mm_HandSolder, F.Cu at (66.2, 97.5)
- added C6: 4.7nC, Capacitor_SMD:C_0805_2012Metric_Pad1.18x1.45mm_HandSolder, F.Cu at (66.7, 106.0)
- added C7: 0.1uC, Capacitor_SMD:C_0805_2012Metric_Pad1.18x1.45mm_HandSolder, F.Cu at (225.3, 34.4)
- added D3: PMEG6010ER, Diode_SMD:Nexperia_CFP3_SOD-123W, F.Cu at (84.2, 26.8)
- added D4: PMEG6010ER, Diode_SMD:Nexperia_CFP3_SOD-123W, F.Cu at (128.5, 30.0)
- added D5: PMEG6010ER, Diode_SMD:Nexperia_CFP3_SOD-123W, F.Cu at (128.5, 26.8)
- added J1: Motor connector, Connector_PinHeader_2.54mm:PinHeader_1x02_P2.54mm_Vertical, F.Cu at (109.8, 43.5)
- added J10: SW0 switch, Connector_JST:JST_PH_B2B-PH-K_1x02_P2.00mm_Vertical, F.Cu at (177.8, 38.2)
- added J11: SW1 switch, Connector_JST:JST_PH_B2B-PH-K_1x02_P2.00mm_Vertical, F.Cu at (186.5, 30.1)
- added J12: SW1 switch, Connector_JST:JST_PH_B2B-PH-K_1x02_P2.00mm_Vertical, F.Cu at (178.6, 30.1)
- added J9: SW0 switch, Connector_JST:JST_PH_B2B-PH-K_1x02_P2.00mm_Vertical, F.Cu at (169.8, 38.2)
- added Q2: AO4822A, Package_SO:SO-8_3.9x4.9mm_P1.27mm, F.Cu at (77.2, 28.4)
- added Q3: AO4822A, Package_SO:SO-8_3.9x4.9mm_P1.27mm, F.Cu at (113.0, 28.4)
- added Q4: AO4822A, Package_SO:SO-8_3.9x4.9mm_P1.27mm, F.Cu at (121.5, 28.4)
- added R10: 10R, Resistor_SMD:R_0805_2012Metric_Pad1.20x1.40mm_HandSolder, F.Cu at (75.0, 46.7)
- added R11: 10R, Resistor_SMD:R_0805_2012Metric_Pad1.20x1.40mm_HandSolder, F.Cu at (79.4, 39.1)
- added R12: 10R, Resistor_SMD:R_0805_2012Metric_Pad1.20x1.40mm_HandSolder, F.Cu at (84.2, 39.1)
- added R13: 10R, Resistor_SMD:R_0805_2012Metric_Pad1.20x1.40mm_HandSolder, F.Cu at (129.5, 36.1)
- added R14: 10R, Resistor_SMD:R_0805_2012Metric_Pad1.20x1.40mm_HandSolder, F.Cu at (119.3, 43.7)
- added R15: 10R, Resistor_SMD:R_0805_2012Metric_Pad1.20x1.40mm_HandSolder, F.Cu at (114.5, 46.7)
- added R16: 20mR, Resistor_SMD:R_2512_6332Metric_Pad1.40x3.35mm_HandSolder, F.Cu at (103.6, 37.1)
- added R17: 10R, Resistor_SMD:R_0805_2012Metric_Pad1.20x1.40mm_HandSolder, F.Cu at (119.3, 46.7)
- added R18: 10R, Resistor_SMD:R_0805_2012Metric_Pad1.20x1.40mm_HandSolder, F.Cu at (123.7, 39.1)
- added R19: 10R, Resistor_SMD:R_0805_2012Metric_Pad1.20x1.40mm_HandSolder, F.Cu at (128.5, 39.1)
- added R20: 10kR, Resistor_SMD:R_0805_2012Metric_Pad1.20x1.40mm_HandSolder, F.Cu at (198.7, 28.9)
- added R21: 10kR, Resistor_SMD:R_0805_2012Metric_Pad1.20x1.40mm_HandSolder, F.Cu at (189.8, 38.5)
- added R22: 10kR, Resistor_SMD:R_0805_2012Metric_Pad1.20x1.40mm_HandSolder, F.Cu at (185.1, 38.5)
- added R23: 10kR, Resistor_SMD:R_0805_2012Metric_Pad1.20x1.40mm_HandSolder, F.Cu at (183.6, 44.4)
- added R24: 10kR, Resistor_SMD:R_0805_2012Metric_Pad1.20x1.40mm_HandSolder, F.Cu at (185.1, 41.4)
- added R25: 10kR, Resistor_SMD:R_0805_2012Metric_Pad1.20x1.40mm_HandSolder, F.Cu at (193.8, 31.9)
- added R26: 10kR, Resistor_SMD:R_0805_2012Metric_Pad1.20x1.40mm_HandSolder, F.Cu at (194.7, 34.9)
- added R27: 10kR, Resistor_SMD:R_0805_2012Metric_Pad1.20x1.40mm_HandSolder, F.Cu at (189.9, 35.5)
- added R9: 20mR, Resistor_SMD:R_2512_6332Metric_Pad1.40x3.35mm_HandSolder, F.Cu at (59.3, 37.1)
- added U1: SP213E, Package_SO:SSOP-28_5.3x10.2mm_P0.65mm, F.Cu at (57.5, 101.0)
- added U10: 74HC7541, Package_SO:TSSOP-20_4.4x6.5mm_P0.65mm, F.Cu at (171.2, 31.4)
- added U2: SP485, Package_SO:SOIC-8_3.9x4.9mm_P1.27mm, F.Cu at (227.2, 29.6)
- added U3: USBLC6-2SC6, Package_TO_SOT_SMD:SOT-23-6, F.Cu at (117.0, 129.0)
- added U6: IR2103, Package_SO:SOIC-8_3.9x4.9mm_P1.27mm, F.Cu at (68.0, 37.9)
- added U7: IR2103, Package_SO:SOIC-8_3.9x4.9mm_P1.27mm, F.Cu at (103.3, 42.8)
- added U8: INA180A2, Package_TO_SOT_SMD:SOT-23-5_HandSoldering, F.Cu at (119.5, 33.9)
- added U9: IR2103, Package_SO:SOIC-8_3.9x4.9mm_P1.27mm, F.Cu at (112.3, 37.9)
- C10, C19: value 4.7nC -> 1uC
- D1: value LED -> SM712_SOT23; footprint LED_SMD:LED_0805_2012Metric_Pad1.15x1.40mm_HandSolder -> Package_TO_SOT_SMD:SOT-23
- D2: value SM712_SOT23 -> PMEG6010ER; footprint Package_TO_SOT_SMD:SOT-23 -> Diode_SMD:Nexperia_CFP3_SOD-123W
- J4: value Power connector -> RS232; footprint Connector_custom:JILN JL301-50002U01 -> Connector_Dsub:DSUB-9_Male_Vertical_P2.77x2.84mm_MountingHoles
- J5: value RS232 -> RS485 connector; footprint Connector_Dsub:DSUB-9_Male_Vertical_P2.77x2.84mm_MountingHoles -> Connector_custom:JILN JL301-50002U01
- J6: value RS485 connector -> USB_B; footprint Connector_custom:JILN JL301-50002U01 -> Connector_USB:USB_B_OST_USB-B1HSxx_Horizontal
- J7: value USB_B -> Motor connector; footprint Connector_USB:USB_B_OST_USB-B1HSxx_Horizontal -> Connector_PinHeader_2.54mm:PinHeader_1x02_P2.54mm_Vertical
- J8: value RS232 -> Barrel_Jack_MountingPin; footprint Connector_Dsub:DSUB-9_Male_Vertical_P2.77x2.84mm_MountingHoles -> Connector_BarrelJack:BarrelJack_CUI_PJ-063AH_Horizontal
- Q1: value BC846 -> AO4822A; footprint Package_TO_SOT_SMD:SOT-23 -> Package_SO:SO-8_3.9x4.9mm_P1.27mm
- R1: value 2k1R -> 1MR
- R2: value 150R -> 10kR
- R3, R7, R8: value 1MR -> 10R
- R4: value 10kR -> 10R
- R5: value 10R -> 1MR
- U4: value SP485 -> IR2103
- U5: value USBLC6-2SC6 -> INA180A2; footprint Package_TO_SOT_SMD:SOT-23-6 -> Package_TO_SOT_SMD:SOT-23-5_HandSoldering
- moved R4 208.9 mm to (233.8, 27.9)
- moved D1 205.8 mm to (213.7, 37.7)
- moved R3 200.0 mm to (223.3, 37.3)
- moved R2 197.5 mm to (218.5, 37.0)
- moved J8 178.0 mm to (192.5, 97.5)
- moved C19 173.5 mm to (89.4, 26.6)
- moved D2 131.0 mm to (84.2, 30.0)
- moved U5 129.5 mm to (75.2, 33.9)
- moved C11 129.4 mm to (80.5, 33.1)
- moved R8 126.5 mm to (70.2, 46.7)
- moved C10 125.8 mm to (70.2, 43.8)
- moved R7 125.8 mm to (75.0, 43.7)
- moved R6 113.8 mm to (85.2, 36.1)
- moved U4 110.9 mm to (59.0, 42.8)
- moved J7 105.0 mm to (65.5, 43.5), turned to 0 degrees
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Connections:
- C11 pad 1: GND -> Net-(C11-Pad1)
- C11 pad 2: VBUS -> /H-bridge #1/Motor_L
- C19 pad 1: Net-(C19-Pad1) -> Net-(C10-Pad1)
- C9 pad 2: /RS485 Interface - Port #1/5V -> VBUS
- D2 pad 1: Net-(D2-Pad1) -> Net-(C11-Pad1)
- J4 pad 1: unconnected-(J4-Pad1) -> /RS232 Interface - Port #1/DCD
- J4 pad 2: GND -> /RS232 Interface - Port #1/RX
- J5 pad 1: /RS232 Interface - Port #1/DCD -> Net-(J5-Pad1)
- J5 pad 2: /RS232 Interface - Port #1/RX -> Net-(J5-Pad2)
- J6 pad 1: Net-(J6-Pad1) -> Net-(F1-Pad1)
- J7 pad 1: Net-(F1-Pad1) -> /H-bridge #1/Motor_R
- J7 pad 2: Net-(J7-Pad2) -> /H-bridge #1/Motor_L
- J8 pad 1: /RS232 Interface - Port #2/DCD -> unconnected-(J8-Pad1)
- J8 pad 2: /RS232 Interface - Port #2/RX -> unconnected-(J8-Pad2)
- Q1 pad 1: Net-(Q1-Pad1) -> /H-bridge #1/Motor_L
- Q1 pad 2: GND -> Net-(R7-Pad2)
- Q1 pad 3: Net-(D1-Pad1) -> GND
- R1 pad 1: /TX_LED -> Net-(C6-Pad1)
- R1 pad 2: Net-(Q1-Pad1) -> GND
- R2 pad 1: VBUS -> /RS485 Interface - Port #1/DIR
- R2 pad 2: Net-(D1-Pad2) -> GND
- R3 pad 1: Net-(C8-Pad1) -> Net-(D1-Pad2)
- R3 pad 2: GND -> Net-(J5-Pad1)
- R4 pad 1: /RS485 Interface - Port #1/DIR -> Net-(D1-Pad1)
- R4 pad 2: GND -> Net-(J5-Pad2)
- R5 pad 1: Net-(D2-Pad2) -> Net-(C8-Pad1)
- R5 pad 2: Net-(J6-Pad1) -> GND
- R6 pad 1: Net-(D2-Pad1) -> Net-(C10-Pad1)
- R6 pad 2: Net-(J6-Pad2) -> Net-(D2-Pad2)
- R7 pad 1: Net-(C10-Pad1) -> Net-(R7-Pad1)
- R7 pad 2: GND -> Net-(R7-Pad2)
- R8 pad 1: Net-(C19-Pad1) -> Net-(R8-Pad1)
- R8 pad 2: GND -> Net-(R8-Pad2)
- U4 pad 1: /RS485 Interface - Port #1/RX -> Net-(C10-Pad1)
- U4 pad 2: /RS485 Interface - Port #1/DIR -> /H-bridge #1/PWM_L
- U4 pad 3: /RS485 Interface - Port #1/DIR -> /H-bridge #1/PWM_L
- U4 pad 4: /RS485 Interface - Port #1/TX -> GND
- U4 pad 5: GND -> Net-(R8-Pad1)
- U4 pad 6: Net-(D2-Pad1) -> /H-bridge #1/Motor_L
- U4 pad 7: Net-(D2-Pad2) -> Net-(R7-Pad1)
- U4 pad 8: /RS485 Interface - Port #1/5V -> Net-(C11-Pad1)
- U5 pad 1: Net-(J7-Pad2) -> /H-bridge #1/Motor_A_Sense
- U5 pad 3: Net-(J7-Pad3) -> /H-bridge #1/12V
- U5 pad 4: /USB Interface/USB_D+ -> Net-(C10-Pad1)
- U5 pad 5: VBUS -> /H-bridge #1/5V
Other:
- rule pad_to_mask_clearance: 0 -> 0.05

Commit message: Progressed ECAD
Parts:
- removed C1, C11, C17, C18, C2, C21, C27, C28, C3, C30, C31, C32, C33, C4, C5: 0.1uC, Capacitor_SMD:C_0805_2012Metric_Pad1.18x1.45mm_HandSolder
- removed C10, C12, C13, C15, C16, C19, C20, C22, C23, C25, C26, C29, C34: 1uC, Capacitor_SMD:C_0805_2012Metric_Pad1.18x1.45mm_HandSolder
- removed C14, C24: 220uC, Capacitor_THT:CP_Radial_D8.0mm_P3.50mm
- removed C6: 4.7nC, Capacitor_SMD:C_0805_2012Metric_Pad1.18x1.45mm_HandSolder
- removed D2, D3, D4, D5: PMEG6010ER, Diode_SMD:Nexperia_CFP3_SOD-123W
- removed J10, J9: SW0 switch, Connector_JST:JST_PH_B2B-PH-K_1x02_P2.00mm_Vertical
- removed J11, J12: SW1 switch, Connector_JST:JST_PH_B2B-PH-K_1x02_P2.00mm_Vertical
- removed J7: Motor connector, Connector_PinHeader_2.54mm:PinHeader_1x02_P2.54mm_Vertical
- removed J8: Barrel_Jack_MountingPin, Connector_BarrelJack:BarrelJack_CUI_PJ-063AH_Horizontal
- removed Q1, Q2, Q3, Q4: AO4822A, Package_SO:SO-8_3.9x4.9mm_P1.27mm
- removed R1: 1MR, Resistor_SMD:R_0805_2012Metric_Pad1.20x1.40mm_HandSolder
- removed R10, R11, R12, R13, R14, R15, R17, R18, R19, R6, R7, R8: 10R, Resistor_SMD:R_0805_2012Metric_Pad1.20x1.40mm_HandSolder
- removed R16, R9: 20mR, Resistor_SMD:R_2512_6332Metric_Pad1.40x3.35mm_HandSolder
- removed R20, R21, R22, R23, R24, R25, R26, R27: 10kR, Resistor_SMD:R_0805_2012Metric_Pad1.20x1.40mm_HandSolder
- removed U1: SP213E, Package_SO:SSOP-28_5.3x10.2mm_P0.65mm
- removed U10: 74HC7541, Package_SO:TSSOP-20_4.4x6.5mm_P0.65mm
- removed U4, U6, U7, U9: IR2103, Package_SO:SOIC-8_3.9x4.9mm_P1.27mm
- removed U5, U8: INA180A2, Package_TO_SOT_SMD:SOT-23-5_HandSoldering
- added C35: 0.1nC, Capacitor_SMD:C_0805_2012Metric_Pad1.18x1.45mm_HandSolder, F.Cu at (174.7, 83.7)
- added C36: 0.1nC, Capacitor_SMD:C_0805_2012Metric_Pad1.18x1.45mm_HandSolder, F.Cu at (164.6, 93.6)
- added C37: 220uC, Capacitor_THT:CP_Radial_D8.0mm_P3.50mm, F.Cu at (157.3, 87.0)
- added D6: D_TVS, Diode_SMD:D_SMA, F.Cu at (158.2, 94.0)
- added FB2: FerriteBead, Inductor_SMD:L_1806_4516Metric_Pad1.45x1.90mm_HandSolder, F.Cu at (167.6, 90.4)
- added Q5: IRF7404, Package_SO:SOIC-8_3.9x4.9mm_P1.27mm, F.Cu at (168.1, 85.5)
- added R28: R, Resistor_SMD:R_0805_2012Metric_Pad1.20x1.40mm_HandSolder, F.Cu at (173.7, 90.2)
- added kibuzzard-636D6560: G***, kibuzzard-636D6560, F.Cu at (91.5, 87.5)
- added kibuzzard-636D65C6: G***, kibuzzard-636D65C6, F.Cu at (188.5, 87.5)
- added kibuzzard-636D66E4: G***, kibuzzard-636D66E4, F.Cu at (91.5, 79.5)
- added kibuzzard-636D671C: G***, kibuzzard-636D671C, F.Cu at (188.5, 96.5)
- C7, C8, D1, R2, R3, R4, R5, U2: moved to B.Cu
- J1: value Motor connector -> Conn_02x20_Odd_Even; footprint Connector_PinHeader_2.54mm:PinHeader_1x02_P2.54mm_Vertical -> Connector_IDC:IDC-Header_2x20_P2.54mm_Vertical
- J4: value RS232 -> Power connector; footprint Connector_Dsub:DSUB-9_Male_Vertical_P2.77x2.84mm_MountingHoles -> Connector_custom:JILN JL301-50002U01
- moved R4 146.8 mm to (101.0, 90.5), turned to 180 degrees
- moved U2 132.0 mm to (108.5, 87.5), turned to 180 degrees
- moved R3 131.1 mm to (101.0, 84.5), turned to 180 degrees
- moved J5 129.5 mm to (96.8, 85.0), turned to -90 degrees
- moved C7 128.1 mm to (107.0, 83.5), turned to 180 degrees
- moved D1 121.8 mm to (102.5, 87.5)
- moved R2 115.6 mm to (114.5, 87.5)
- moved J4 95.3 mm to (183.2, 90.0), turned to 90 degrees
- moved C9 47.1 mm to (128.2, 81.6)
- moved FB1 47.1 mm to (123.0, 89.0)
- moved F1 47.1 mm to (133.0, 81.5)
- moved U3 47.1 mm to (123.2, 82.3)
- moved C8 35.3 mm to (114.0, 97.5), turned to 180 degrees
- moved R5 33.1 mm to (114.0, 100.5), turned to 180 degrees
- moved J1 28.9 mm to (115.9, 71.8), turned to 90 degrees
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Connections:
- J1 pad 1: /H-bridge #2/Motor_R -> unconnected-(J1-Pad1)
- J1 pad 2: /H-bridge #2/Motor_L -> unconnected-(J1-Pad2)
- J4 pad 1: /RS232 Interface - Port #1/DCD -> /Power Supply/12V
- J4 pad 2: /RS232 Interface - Port #1/RX -> GND
Other:
- board size 120 x 45 mm -> 100 x 45 mm

Commit message: Progressed ECAD
Parts:
- added U1: ATSAMD21G18A-A, Package_QFP:TQFP-48_7x7mm_P0.5mm, B.Cu at (132.0, 89.0)
- C35, C36, C9, D6, F1, FB1, FB2, Q5, R28, U3: moved to B.Cu
- moved FB2 8.72 mm to (169.0, 99.0), turned to 180 degrees
- moved J6 6.00 mm to (127.2, 100.4)
- moved C8 5.50 mm to (114.0, 103.0)
- moved R5 5.50 mm to (114.0, 106.0)
- moved D6 3.07 mm to (159.0, 97.0), turned to 180 degrees
- turned C35 to 180 degrees
- turned C36 to 180 degrees
- turned C9 to 180 degrees
- turned F1 to 180 degrees
- turned FB1 to 180 degrees
- turned Q5 to 180 degrees
- turned R28 to 180 degrees
- turned U3 to 180 degrees

Commit message: Progressed ECAD
Parts:
- moved U3 13.1 mm to (125.0, 95.2)
Changed lines of the file:
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@@
   )
   (footprint "Package_TO_SOT_SMD:SOT-23-6" (layer "B.Cu")
-    (at 123.2 82.29 180)
+    (at 125 95.25 180)
     (descr "SOT, 6 Pin (https://www.jedec.org/sites/default/files/docs/Mo-178c.PDF variant AB), generated with kicad-footprint-generator ipc_gullwing_generator.py")
     (tags "SOT TO_SOT_SMD")

Commit message: Progressed CAD
Parts:
- removed C35, C36: 0.1nC, Capacitor_SMD:C_0805_2012Metric_Pad1.18x1.45mm_HandSolder
- removed C37: 220uC, Capacitor_THT:CP_Radial_D8.0mm_P3.50mm
- removed C7, C9: 0.1uC, Capacitor_SMD:C_0805_2012Metric_Pad1.18x1.45mm_HandSolder
- removed C8: 4.7nC, Capacitor_SMD:C_0805_2012Metric_Pad1.18x1.45mm_HandSolder
- removed D6: D_TVS, Diode_SMD:D_SMA
- removed Q5: IRF7404, Package_SO:SOIC-8_3.9x4.9mm_P1.27mm
- removed R28: R, Resistor_SMD:R_0805_2012Metric_Pad1.20x1.40mm_HandSolder
- removed kibuzzard-636D6560: G***, kibuzzard-636D6560
- removed kibuzzard-636D65C6: G***, kibuzzard-636D65C6
- removed kibuzzard-636D66E4: G***, kibuzzard-636D66E4
- removed kibuzzard-636D671C: G***, kibuzzard-636D671C
- added C1: 0.1uC, Capacitor_SMD:C_0805_2012Metric_Pad1.18x1.45mm_HandSolder, F.Cu at (136.5, 152.0)
- added C2: 4.7nC, Capacitor_SMD:C_0805_2012Metric_Pad1.18x1.45mm_HandSolder, F.Cu at (131.7, 152.0)
- added C3: 0.1uC, Capacitor_SMD:C_0805_2012Metric_Pad1.18x1.45mm_HandSolder, F.Cu at (143.1, 144.1)
- added C4: 0.1nC, Capacitor_SMD:C_0805_2012Metric_Pad1.18x1.45mm_HandSolder, F.Cu at (165.2, 124.9)
- added C5: 0.1nC, Capacitor_SMD:C_0805_2012Metric_Pad1.18x1.45mm_HandSolder, F.Cu at (148.0, 143.0)
- added C6: 220uC, Capacitor_THT:CP_Radial_D8.0mm_P3.50mm, F.Cu at (134.2, 145.7)
- added D2: SM712_SOT23, Package_TO_SOT_SMD:SOT-23, F.Cu at (143.2, 140.4)
- added J3: USB_B, Connector_USB:USB_B_OST_USB-B1HSxx_Horizontal, F.Cu at (121.2, 94.4)
- added Q1: IRF7404, Package_SO:SOIC-8_3.9x4.9mm_P1.27mm, F.Cu at (158.5, 126.6)
- added R1: 1MR, Resistor_SMD:R_0805_2012Metric_Pad1.20x1.40mm_HandSolder, F.Cu at (154.2, 137.7)
- added kibuzzard-636F7E30: G***, kibuzzard-636F7E30, F.Cu at (92.0, 87.5)
- added kibuzzard-636F7E53: G***, kibuzzard-636F7E53, F.Cu at (188.0, 87.5)
- D1: value SM712_SOT23 -> D_TVS; footprint Package_TO_SOT_SMD:SOT-23 -> Diode_SMD:D_SMA; moved to F.Cu
- F1, FB1, FB2, R2, R4: moved to F.Cu
- J4: value Power connector -> Conn_01x02; footprint Connector_custom:JILN JL301-50002U01 -> Connector_JST:JST_PH_S2B-PH-K_1x02_P2.00mm_Horizontal
- J5: value RS485 connector -> Conn_ARM_JTAG_SWD_10; footprint Connector_custom:JILN JL301-50002U01 -> Connector_PinHeader_1.27mm:PinHeader_2x05_P1.27mm_Vertical
- J6: value USB_B -> Conn_01x02; footprint Connector_USB:USB_B_OST_USB-B1HSxx_Horizontal -> Connector_custom:HC-2510-2AW
- R3: value 10R -> R; moved to F.Cu
- R5: value 1MR -> 10R; moved to F.Cu
- U1: value ATSAMD21G18A-A -> SP485; footprint Package_QFP:TQFP-48_7x7mm_P0.5mm -> Package_SO:SOIC-8_3.9x4.9mm_P1.27mm; moved to F.Cu
- U2: value SP485 -> USBLC6-2SC6; footprint Package_SO:SOIC-8_3.9x4.9mm_P1.27mm -> Package_TO_SOT_SMD:SOT-23-6; moved to F.Cu
- U3: value USBLC6-2SC6 -> ATSAMD21G18A-A; footprint Package_TO_SOT_SMD:SOT-23-6 -> Package_QFP:TQFP-48_7x7mm_P0.5mm; moved to F.Cu
- moved J4 83.3 mm to (100.0, 86.5), turned to -90 degrees
- moved R3 75.4 mm to (143.1, 147.1), turned to 0 degrees
- moved R4 74.2 mm to (165.1, 127.8), turned to 0 degrees
- moved J5 71.7 mm to (148.5, 134.7), turned to 0 degrees
- moved R2 67.3 mm to (147.9, 145.9)
- moved U2 65.5 mm to (126.7, 150.4), turned to 0 degrees
- moved D1 65.3 mm to (120.1, 150.4)
- moved FB1 64.3 mm to (143.1, 150.0), turned to 0 degrees
- moved F1 62.8 mm to (154.2, 140.7), turned to 0 degrees
- moved R5 56.8 mm to (165.1, 130.8), turned to 0 degrees
- moved U1 51.4 mm to (158.5, 133.0), turned to 0 degrees
- moved J6 49.6 mm to (174.8, 86.2), turned to 0 degrees
- moved FB2 48.2 mm to (138.7, 136.4), turned to 0 degrees
- moved U3 37.2 mm to (140.7, 129.0), turned to 0 degrees
Connections:
- net /RS485 Interface - Port #1/TX renamed /USB_D+
- D1 pad 1: Net-(D1-Pad1) -> GND
- FB2 pad 2: /Power Supply/12V -> +12V
- J4 pad 1: /Power Supply/12V -> Net-(J4-Pad1)
- J4 pad 2: GND -> Net-(J4-Pad2)
- J5 pad 1: Net-(J5-Pad1) -> unconnected-(J5-Pad1)
- J5 pad 2: Net-(J5-Pad2) -> unconnected-(J5-Pad2)
- J6 pad 1: Net-(F1-Pad1) -> +12V
- J6 pad 2: Net-(J6-Pad2) -> GND
- R2 pad 1: /RS485 Interface - Port #1/DIR -> /RS485_DIR
- R3 pad 1: Net-(D1-Pad2) -> Net-(D3-Pad2)
- R3 pad 2: Net-(J5-Pad1) -> GND
- R4 pad 1: Net-(D1-Pad1) -> Net-(D2-Pad2)
- R4 pad 2: Net-(J5-Pad2) -> Net-(J4-Pad1)
- R5 pad 1: Net-(C8-Pad1) -> Net-(D2-Pad1)
- R5 pad 2: GND -> Net-(J4-Pad2)
- U1 pad 1: unconnected-(U1-Pad1) -> /RS485_RX
- U1 pad 2: unconnected-(U1-Pad2) -> /RS485_DIR
- U1 pad 3: unconnected-(U1-Pad3) -> /RS485_DIR
- U1 pad 4: unconnected-(U1-Pad4) -> /RS485_TX
- U1 pad 5: unconnected-(U1-Pad5) -> GND
- U1 pad 6: unconnected-(U1-Pad6) -> Net-(D2-Pad1)
- U1 pad 7: unconnected-(U1-Pad7) -> Net-(D2-Pad2)
- U2 pad 1: /RS485 Interface - Port #1/RX -> Net-(J3-Pad2)
- U2 pad 2: /RS485 Interface - Port #1/DIR -> GND
- U2 pad 3: /RS485 Interface - Port #1/DIR -> Net-(J3-Pad3)
- U2 pad 5: GND -> VBUS
- U2 pad 6: Net-(D1-Pad1) -> /USB_D-
- U3 pad 1: Net-(J6-Pad2) -> unconnected-(U3-Pad1)
- U3 pad 2: GND -> unconnected-(U3-Pad2)
- U3 pad 3: Net-(J6-Pad3) -> unconnected-(U3-Pad3)
- U3 pad 4: /USB Interface/USB_D+ -> unconnected-(U3-Pad4)
- U3 pad 5: VBUS -> unconnected-(U3-Pad5)
- U3 pad 6: /USB Interface/USB_D- -> unconnected-(U3-Pad6)

Commit message: Progressed ECAD
Parts:
- added H5: MountingHole, MountingHole:MountingHole_3.2mm_M3, F.Cu at (140.0, 105.0)
- added J2: Barrel_Jack_Switch, Connector_BarrelJack_custom:BarrelJack_DC-042C-W-2.5_Horizontal, F.Cu at (160.0, 106.5)
- added kibuzzard-636FAF85: G***, kibuzzard-636FAF85, F.Cu at (120.0, 108.0)
- added kibuzzard-636FAF98: G***, kibuzzard-636FAF98, F.Cu at (160.0, 108.0)
- moved J3 3.00 mm to (121.2, 91.4)

Commit message: Progressed ECAD
Parts:
- added D4: LED, LED_SMD:LED_0805_2012Metric, F.Cu at (94.2, 94.0)
- added D5: LED, LED_SMD:LED_0805_2012Metric, F.Cu at (149.1, 105.8)
- added D6: LED, LED_SMD:LED_0805_2012Metric, F.Cu at (94.2, 81.0)
- added kibuzzard-636FE537: G***, kibuzzard-636FE537, F.Cu at (149.0, 108.0)
- added kibuzzard-636FE58E: G***, kibuzzard-636FE58E, F.Cu at (92.0, 81.0)
- added kibuzzard-636FE59D: G***, kibuzzard-636FE59D, F.Cu at (92.0, 94.0)

Commit message: Progressed ECAD
Parts:
- removed kibuzzard-636FE537: G***, kibuzzard-636FE537
- added D3: MMSZ5240BT1G, Diode_SMD:D_SOD-123, F.Cu at (170.0, 119.0)
- added F2: Fuse, Fuse:Fuseholder_Littelfuse_100_series_5x20mm, F.Cu at (149.0, 99.2)
- added kibuzzard-63703123: G***, kibuzzard-63703123, F.Cu at (132.0, 108.0)
- added kibuzzard-6370312D: G***, kibuzzard-6370312D, F.Cu at (149.0, 108.0)
- C4, C5: value 0.1nC -> 0.1uC
- D1: value D_TVS -> SMAJ16CA
- FB2: footprint Inductor_SMD:L_1806_4516Metric_Pad1.45x1.90mm_HandSolder -> Inductor_SMD:L_1806_4516Metric
- Q1: value IRF7404 -> DMP3037LSS-13
- R3: value R -> 10kR
Connections:
- C4 pad 1: Net-(C4-Pad1) -> GND
- C4 pad 2: GND -> Net-(D3-Pad1)
- C5 pad 1: +12V -> GND
- C5 pad 2: GND -> +12V
- FB2 pad 1: Net-(C4-Pad1) -> Net-(D3-Pad1)
- Q1 pad 1: Net-(C4-Pad1) -> Net-(D3-Pad1)
- Q1 pad 2: Net-(C4-Pad1) -> Net-(D3-Pad1)
- Q1 pad 3: Net-(C4-Pad1) -> Net-(D3-Pad1)
