File: Tester/ECAD/USBGatewayBoard/USBGatewayBoard.kicad_sch (KiCad schematic)
At the start: 5 parts, among them J1 Conn_02x20_Odd_Even

Commit message: Progressed ECAD
Parts:
- J1: Manufacturer Part Number https://datasheet.lcsc.com/lcsc/1810311440_Nextron-Nextroni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 -> Z-231011020106
Changed lines of the file:
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@@
       (effects (font (size 1.27 1.27)) hide)
     )
-    (property "Datasheet" "Z-231011020106" (id 3) (at 227.33 96.52 0)
-      (effects (font (size 1.27 1.27)) hide)
-    )
-    (property "Manufacturer Part Number" "https://datasheet.lcsc.com/lcsc/1810311440_Nextron-Nextronics-Engineering-Z-231011020106_C221051.pdf" (id 4) (at 227.33 96.52 0)
+    (property "Datasheet" "https://datasheet.lcsc.com/lcsc/1810311440_Nextron-Nextronics-Engineering-Z-231011020106_C221051.pdf" (id 3) (at 227.33 96.52 0)
+      (effects (font (size 1.27 1.27)) hide)
+    )
+    (property "Manufacturer Part Number" "Z-231011020106" (id 4) (at 227.33 96.52 0)
       (effects (font (size 1.27 1.27)) hide)
     )
@@
       (reference "R28") (unit 1) (value "R") (footprint "Resistor_SMD:R_0805_2012Metric_Pad1.20x1.40mm_HandSolder")
     )
+    (path "/76be5f40-0efd-4be0-a528-34098d56af2b/50fcc21e-e085-4943-9a28-8f39c2cf0805"
+      (reference "U1") (unit 1) (value "ATSAMD21G18A-A") (footprint "Package_QFP:TQFP-48_7x7mm_P0.5mm")
+    )
     (path "/897e9868-1ae5-45cd-ab61-45d0dcbc33eb/22d82e24-0696-4dab-a97d-f101260ef0aa"

Commit message: Progressed ECAD
Parts:
- added C1, C3: 0.1uC, Capacitor_SMD:C_0805_2012Metric_Pad1.18x1.45mm_HandSolder, symbol Device:C
- added C2: 4.7nC, Capacitor_SMD:C_0805_2012Metric_Pad1.18x1.45mm_HandSolder, symbol Device:C
- added C4, C5: 0.1nC, Capacitor_SMD:C_0805_2012Metric_Pad1.18x1.45mm_HandSolder, symbol Device:C
- added C6: 220uC, Capacitor_THT:CP_Radial_D8.0mm_P3.50mm, symbol Device:C_Polarized
- added D1: D_TVS, Diode_SMD:D_SMA, symbol Device:D_TVS
- added D2: SM712_SOT23, Package_TO_SOT_SMD:SOT-23, symbol Diode:SM712_SOT23
- added D3: D_Zener, symbol Device:D_Zener
- added F1: Polyfuse, Fuse:Fuse_0805_2012Metric_Pad1.15x1.40mm_HandSolder, symbol Device:Polyfuse_Small
- added F2: Fuse, symbol Device:Fuse
- added FB1: FerriteBead, Inductor_SMD:L_0805_2012Metric_Pad1.15x1.40mm_HandSolder, symbol Device:FerriteBead_Small
- added FB2: FerriteBead, Inductor_SMD:L_1806_4516Metric_Pad1.45x1.90mm_HandSolder, symbol Device:FerriteBead
- added J2: Barrel_Jack, symbol Connector:Barrel_Jack
- added J3: USB_B, Connector_USB:USB_B_OST_USB-B1HSxx_Horizontal, symbol Connector:USB_B
- added J4, J6: Conn_01x02, symbol Connector_Generic:Conn_01x02
- added J5: Conn_ARM_JTAG_SWD_10, symbol Connector:Conn_ARM_JTAG_SWD_10
- added Q1: IRF7404, Package_SO:SOIC-8_3.9x4.9mm_P1.27mm, symbol Transistor_FET:IRF7404
- added R1: 1MR, Resistor_SMD:R_0805_2012Metric_Pad1.20x1.40mm_HandSolder, symbol Device:R
- added R2: 10kR, Resistor_SMD:R_0805_2012Metric_Pad1.20x1.40mm_HandSolder, symbol Device:R
- added R3: R, Resistor_SMD:R_0805_2012Metric_Pad1.20x1.40mm_HandSolder, symbol Device:R
- added R4, R5: 10R, Resistor_SMD:R_0805_2012Metric_Pad1.20x1.40mm_HandSolder, symbol Device:R
- added U1: SP485, Package_SO:SOIC-8_3.9x4.9mm_P1.27mm, symbol Interface_UART:ST485EBDR
- added U2: USBLC6-2SC6, Package_TO_SOT_SMD:SOT-23-6, symbol Power_Protection:USBLC6-2SC6
- added U3: ATSAMD21G18A-A, Package_QFP:TQFP-48_7x7mm_P0.5mm, symbol MCU_Microchip_SAMD:ATSAMD21G18A-A
Connections:
- new net: C4.1, D3.1 (K), FB2.1, Q1.1 (S), Q1.2 (S), Q1.3 (S)
- new net: D3.2 (A), Q1.4 (G), R3.1
- new net: D1.2 (A2), F2.2, Q1.5 (D), Q1.6 (D), Q1.7 (D), Q1.8 (D)
- new net: F2.1, J2.1
- new net: F1.1, J3.1 (VBUS)
- new net: J3.2 (D-), U2.1 (I/O1)
- new net: J3.3 (D+), U2.3 (I/O2)
- new net: C2.1, J3.5 (Shield), R1.1
- new net: D2.1 (A1), R5.1, U1.6 (A)
- new net: D2.2 (A2), R4.1, U1.7 (B)
- new net: J5.3 (GND), J5.5 (GND)
- new net: J4.1 (Pin_1), R4.2
- new net: J4.2 (Pin_2), R5.2
- new net: F1.2, FB1.2
- new net: U3.18 (GND), U3.35 (GND), U3.42 (GND)
- new net +12V: C5.1, C6.1, FB2.2, J6.1 (Pin_1)
- new net 5V: C1.2
- new net GND: C1.1, C2.2, C3.1, C4.2, C5.2, C6.2, D1.1 (A1), D2.3 (common), J2.2, J3.4 (GND), J6.2 (Pin_2), R1.2, R2.2, R3.2, U1.5 (GND), U2.2 (GND)
- new net RS485_DIR: R2.1, U1.2 (~{RE}), U1.3 (DE)
- new net RS485_RX: U1.1 (RO)
- new net RS485_TX: U1.4 (DI)
- new net USB_D+: U2.4 (I/O2)
- new net USB_D-: U2.6 (I/O1)
- new net VBUS: C3.2, FB1.1, U2.5 (VBUS)
Other:
- removed sheet MCU
- removed sheet Power Supply
- removed sheet RS485 Interface - Port #1
- removed sheet USB Interface
- note added: "Power input protection"
- note added: "RS485 Level Translator"
- note added: "USB interface"
- moved on the sheet: H1, H2, H3, H4, J1

Commit message: Progressed CAD
Parts:
- J4: footprint (none) -> Connector_JST:JST_PH_S2B-PH-K_1x02_P2.00mm_Horizontal; Manufacturer Part Number (none) -> S2B-PH-K-S(LF)(SN)
- J5: footprint (none) -> Connector_PinHeader_1.27mm:PinHeader_2x05_P1.27mm_Vertical
- J6: footprint (none) -> Connector_custom:HC-2510-2AW; Manufacturer Part Number (none) -> HC-2510-2AW
Other:
- note added: "Expansion port"
- moved on the sheet: J1
Changed lines of the file:
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@@
+    (effects (font (size 1.27 1.27)) (justify left bottom))
+  )
+  (text "Expansion port" (at 124.46 54.61 0)
     (effects (font (size 1.27 1.27)) (justify left bottom))
   )
@@
     (pin "1")
   )
-  (symbol (lib_id "Connector_Generic:Conn_02x20_Odd_Even") (at 165.1 101.6 0) (unit 1)
-    (in_bom yes) (on_board yes) (fields_autoplaced)
-    (property "Reference" "J1" (id 0) (at 166.37 72.39 0))
-    (property "Value" "Conn_02x20_Odd_Even" (id 1) (at 166.37 74.93 0))
-    (property "Footprint" "Connector_IDC:IDC-Header_2x20_P2.54mm_Vertical" (id 2) (at 165.1 101.6 0)
-      (effects (font (size 1.27 1.27)) hide)
-    )
-    (property "Datasheet" "https://datasheet.lcsc.com/lcsc/1810311440_Nextron-Nextronics-Engineering-Z-231011020106_C221051.pdf" (id 3) (at 165.1 101.6 0)
-      (effects (font (size 1.27 1.27)) hide)
-    )
-    (property "Manufacturer Part Number" "Z-231011020106" (id 4) (at 165.1 101.6 0)
+  (symbol (lib_id "Connector_Generic:Conn_02x20_Odd_Even") (at 129.54 86.36 0) (unit 1)
+    (in_bom yes) (on_board yes) (fields_autoplaced)
+    (property "Reference" "J1" (id 0) (at 130.81 57.15 0))
+    (property "Value" "Conn_02x20_Odd_Even" (id 1) (at 130.81 59.69 0))
+    (property "Footprint" "Connector_IDC:IDC-Header_2x20_P2.54mm_Vertical" (id 2) (at 129.54 86.36 0)
+      (effects (font (size 1.27 1.27)) hide)
+    )
+    (property "Datasheet" "https://datasheet.lcsc.com/lcsc/1810311440_Nextron-Nextronics-Engineering-Z-231011020106_C221051.pdf" (id 3) (at 129.54 86.36 0)
+      (effects (font (size 1.27 1.27)) hide)
+    )
+    (property "Manufacturer Part Number" "Z-231011020106" (id 4) (at 129.54 86.36 0)
       (effects (font (size 1.27 1.27)) hide)
     )
@@
       (effects (font (size 1.27 1.27)) (justify left))
     )
-    (property "Footprint" "" (id 2) (at 139.7 30.48 0)
-      (effects (font (size 1.27 1.27)) hide)
-    )
-    (property "Datasheet" "~" (id 3) (at 139.7 30.48 0)
+    (property "Footprint" "Connector_custom:HC-2510-2AW" (id 2) (at 139.7 30.48 0)
+      (effects (font (size 1.27 1.27)) hide)
+    )
+    (property "Datasheet" "https://datasheet.lcsc.com/lcsc/2203111830_HCTL-HC-2510-2AW_C2982041.pdf" (id 3) (at 139.7 30.48 0)
+      (effects (font (size 1.27 1.27)) hide)
+    )
+    (property "Manufacturer Part Number" "HC-2510-2AW" (id 4) (at 139.7 30.48 0)
       (effects (font (size 1.27 1.27)) hide)
     )
@@
       (effects (font (size 1.27 1.27)) (justify right))
     )
-    (property "Footprint" "" (id 2) (at 257.81 29.21 0)
+    (property "Footprint" "Connector_PinHeader_1.27mm:PinHeader_2x05_P1.27mm_Vertical" (id 2) (at 257.81 29.21 0)
       (effects (font (size 1.27 1.27)) hide)
     )
@@
       (effects (font (size 1.27 1.27)) (justify left))
     )
-    (property "Footprint" "" (id 2) (at 113.03 133.35 0)
-      (effects (font (size 1.27 1.27)) hide)
-    )
-    (property "Datasheet" "~" (id 3) (at 113.03 133.35 0)
+    (property "Footprint" "Connector_JST:JST_PH_S2B-PH-K_1x02_P2.00mm_Horizontal" (id 2) (at 113.03 133.35 0)
+      (effects (font (size 1.27 1.27)) hide)
+    )
+    (property "Datasheet" "https://datasheet.lcsc.com/lcsc/1810261107_JST-Sales-America-S2B-PH-K-S-LF-SN_C173752.pdf" (id 3) (at 113.03 133.35 0)
+      (effects (font (size 1.27 1.27)) hide)
+    )
+    (property "Manufacturer Part Number" "S2B-PH-K-S(LF)(SN)" (id 4) (at 113.03 133.35 0)
       (effects (font (size 1.27 1.27)) hide)
     )
@@
     )
     (path "/b33ad0cf-312d-4975-9ca2-4e031a0bd03c"
-      (reference "J4") (unit 1) (value "Conn_01x02") (footprint "")
+      (reference "J4") (unit 1) (value "Conn_01x02") (footprint "Connector_JST:JST_PH_S2B-PH-K_1x02_P2.00mm_Horizontal")
     )
     (path "/6c884b70-c320-4036-b417-0e6b6c78e111"
-      (reference "J5") (unit 1) (value "Conn_ARM_JTAG_SWD_10") (footprint "")
+      (reference "J5") (unit 1) (value "Conn_ARM_JTAG_SWD_10") (footprint "Connector_PinHeader_1.27mm:PinHeader_2x05_P1.27mm_Vertical")
     )
     (path "/6742674e-5f54-4fe9-8165-315021cf530e"
-      (reference "J6") (unit 1) (value "Conn_01x02") (footprint "")
+      (reference "J6") (unit 1) (value "Conn_01x02") (footprint "Connector_custom:HC-2510-2AW")
     )
     (path "/04105e0e-99e5-49fd-bf9b-54373ed0bfc7"

Commit message: Progressed ECAD
Parts:
- removed J2: Barrel_Jack, symbol Connector:Barrel_Jack
- added H5: MountingHole, MountingHole:MountingHole_3.2mm_M3, symbol Mechanical:MountingHole
- added J2: Barrel_Jack_Switch, Connector_BarrelJack_custom:BarrelJack_DC-042C-W-2.5_Horizontal, symbol Connector:Barrel_Jack_Switch
Connections:
- net GND: now also J2.2, J2.3
- net at F2.1: now also J2.1
Other:
- moved on the sheet: H1, H2, H3, H4, J5, U3

Commit message: Progressed ECAD
Parts:
- added D4, D5, D6: LED, LED_SMD:LED_0805_2012Metric, symbol Device:LED
- J5: Manufacturer Part Number 3220-10-0100-00 -> B-2101S10P-B110
Changed lines of the file:
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@@
     (pin "8")
+  )
+  (symbol (lib_id "Device:LED") (at 153.67 163.83 0) (unit 1)
+    (in_bom yes) (on_board yes) (fields_autoplaced)
+    (property "Reference" "D6" (id 0) (at 152.0825 157.48 0))
+    (property "Value" "LED" (id 1) (at 152.0825 160.02 0))
+    (property "Footprint" "LED_SMD:LED_0805_2012Metric" (id 2) (at 153.67 163.83 0)
+      (effects (font (size 1.27 1.27)) hide)
+    )
+    (property "Datasheet" "~" (id 3) (at 153.67 163.83 0)
+      (effects (font (size 1.27 1.27)) hide)
+    )
+    (pin "1")
+    (pin "2")
   )
   (symbol (lib_id "Device:Fuse") (at 35.56 26.67 90) (unit 1)
@@
     )
     (pin "1")
+  )
+  (symbol (lib_id "Device:LED") (at 153.67 140.97 0) (unit 1)
+    (in_bom yes) (on_board yes) (fields_autoplaced)
+    (property "Reference" "D4" (id 0) (at 152.0825 134.62 0))
+    (property "Value" "LED" (id 1) (at 152.0825 137.16 0))
+    (property "Footprint" "LED_SMD:LED_0805_2012Metric" (id 2) (at 153.67 140.97 0)
+      (effects (font (size 1.27 1.27)) hide)
+    )
+    (property "Datasheet" "~" (id 3) (at 153.67 140.97 0)
+      (effects (font (size 1.27 1.27)) hide)
+    )
+    (pin "1")
+    (pin "2")
+  )
+  (symbol (lib_id "Device:LED") (at 153.67 152.4 0) (unit 1)
+    (in_bom yes) (on_board yes) (fields_autoplaced)
+    (property "Reference" "D5" (id 0) (at 152.0825 146.05 0))
+    (property "Value" "LED" (id 1) (at 152.0825 148.59 0))
+    (property "Footprint" "LED_SMD:LED_0805_2012Metric" (id 2) (at 153.67 152.4 0)
+      (effects (font (size 1.27 1.27)) hide)
+    )
+    (property "Datasheet" "~" (id 3) (at 153.67 152.4 0)
+      (effects (font (size 1.27 1.27)) hide)
+    )
+    (pin "1")
+    (pin "2")
   )
   (symbol (lib_id "power:GND") (at 59.69 41.91 0) (unit 1)
@@
       (effects (font (size 1.27 1.27)) hide)
     )
-    (property "Datasheet" "http://infocenter.arm.com/help/topic/com.arm.doc.ddi0314h/DDI0314H_coresight_components_trm.pdf" (id 3) (at 186.69 134.62 90)
-      (effects (font (size 1.27 1.27)) hide)
-    )
-    (property "Manufacturer Part Number" "3220-10-0100-00" (id 4) (at 195.58 102.87 0)
+    (property "Datasheet" "https://datasheet.lcsc.com/lcsc/2109140930_Ckmtw-Shenzhen-Cankemeng-B-2101S10P-B110_C2895038.pdf" (id 3) (at 186.69 134.62 90)
+      (effects (font (size 1.27 1.27)) hide)
+    )
+    (property "Manufacturer Part Number" "B-2101S10P-B110" (id 4) (at 195.58 102.87 0)
       (effects (font (size 1.27 1.27)) hide)
     )
@@
       (reference "D3") (unit 1) (value "D_Zener") (footprint "")
     )
+    (path "/22092d1c-ba3e-42ba-b49a-f0365d5efbc1"
+      (reference "D4") (unit 1) (value "LED") (footprint "LED_SMD:LED_0805_2012Metric")
+    )
+    (path "/23c8d8fd-d134-4f24-99c7-5f28ac8f861e"
+      (reference "D5") (unit 1) (value "LED") (footprint "LED_SMD:LED_0805_2012Metric")
+    )
+    (path "/06325c7a-b85e-4eb8-9914-cc784f991912"
+      (reference "D6") (unit 1) (value "LED") (footprint "LED_SMD:LED_0805_2012Metric")
+    )
     (path "/fbbc567b-3a22-4738-b986-584ab49fcec0"

Commit message: Progressed ECAD
Parts:
- C1, C3: Manufacturer Part Number CC0805KRX7R8BB104 -> CL21B104KBCNNNC
- C4, C5: value 0.1nC -> 0.1uC; Manufacturer Part Number (none) -> CL21B104KBCNNNC
- D1: value D_TVS -> SMAJ16CA; Manufacturer Part Number SMAJ28CA -> SMAJ16CA-13-F
- D3: value D_Zener -> MMSZ5240BT1G; footprint (none) -> Diode_SMD:D_SOD-123; Manufacturer Part Number PDZ16BGWJ -> MMSZ5240BT1G
- F2: footprint (none) -> Fuse:Fuseholder_Littelfuse_100_series_5x20mm
- FB2: footprint Inductor_SMD:L_1806_4516Metric_Pad1.45x1.90mm_HandSolder -> Inductor_SMD:L_1806_4516Metric
- Q1: value IRF7404 -> DMP3037LSS-13
- R3: value R -> 10kR; Manufacturer Part Number RC0402FR-0747KL -> RC0805FR-0710KL
Connections:
- net +12V: now also C5.2; no longer C5.1
- net GND: now also C4.1, C5.1; no longer C4.2, C5.2
- net at D3.1 (K), FB2.1, Q1.1 (S)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: now also C4.2; no longer C4.1
Other:
- moved on the sheet: C6, FB2, J6

Commit message: Update USBGatewayBoard.kicad_sch
Parts:
- F1: Manufacturer Part Number SMD0805P020TF -> SMD250L-30V
- F2: footprint Fuse:Fuseholder_Littelfuse_100_series_5x20mm -> Fuse:Fuse_2920_7451Metric
Other:
- moved on the sheet: C4, C5, C6, D1

Commit message: Update USBGatewayBoard.kicad_sch
Parts:
- J1: footprint Connector_IDC:IDC-Header_2x20_P2.54mm_Vertical -> Connector_PinHeader_2.54mm:PinHeader_2x20_P2.54mm_Vertical; Manufacturer Part Number Z-231011020106 -> (none)
Changed lines of the file:
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@@
     (property "Reference" "J1" (id 0) (at 130.81 57.15 0))
     (property "Value" "Conn_02x20_Odd_Even" (id 1) (at 130.81 59.69 0))
-    (property "Footprint" "Connector_IDC:IDC-Header_2x20_P2.54mm_Vertical" (id 2) (at 129.54 86.36 0)
-      (effects (font (size 1.27 1.27)) hide)
-    )
-    (property "Datasheet" "https://datasheet.lcsc.com/lcsc/1810311440_Nextron-Nextronics-Engineering-Z-231011020106_C221051.pdf" (id 3) (at 129.54 86.36 0)
-      (effects (font (size 1.27 1.27)) hide)
-    )
-    (property "Manufacturer Part Number" "Z-231011020106" (id 4) (at 129.54 86.36 0)
+    (property "Footprint" "Connector_PinHeader_2.54mm:PinHeader_2x20_P2.54mm_Vertical" (id 2) (at 129.54 86.36 0)
+      (effects (font (size 1.27 1.27)) hide)
+    )
+    (property "Datasheet" "" (id 3) (at 129.54 86.36 0)
+      (effects (font (size 1.27 1.27)) hide)
+    )
+    (property "Manufacturer Part Number" "" (id 4) (at 129.54 86.36 0)
       (effects (font (size 1.27 1.27)) hide)
     )
@@
     )
     (path "/49ce806e-47b4-4d1f-a24e-4ff711543869"
-      (reference "J1") (unit 1) (value "Conn_02x20_Odd_Even") (footprint "Connector_IDC:IDC-Header_2x20_P2.54mm_Vertical")
+      (reference "J1") (unit 1) (value "Conn_02x20_Odd_Even") (footprint "Connector_PinHeader_2.54mm:PinHeader_2x20_P2.54mm_Vertical")
     )
     (path "/723bc676-a326-40fd-9720-acc4ea85ae42"
