File: Tester/ECAD/MotorControlDaughterBoard/MotorControlDaughterBoard.kicad_pcb (KiCad board)
At the start: 2 copper layers, 100 x 45 mm, 85 parts, among them J1 SW0 switch, J2 SW0 switch, J3 SW1 switch, J4 SW1 switch, J5 Conn_02x20_Odd_Even, J6 DB9_Male, J7 DB9_Male, J8 Motor connector, J9 Motor connector, Q1 Q_NMOS_GSD, Q2 Q_NMOS_GSD, Q3 Q_NMOS_GSD, Q4 Q_NMOS_GSD, Q5 Q_NMOS_GSD, Q6 Q_NMOS_GSD, Q7 Q_NMOS_GSD, Q8 Q_NMOS_GSD, U1 SP3243E, U2 SP3243E, U3 IR2103, U4 INA180A2, U5 IR2103, U6 IR2103, U7 INA180A2, U8 IR2103

Commit message: Progressed ECAD
Parts:
- C10, C11, C12, C13, C5, C6, C7, C8: value 0.1uC -> 0.22uC
- J1: value SW0 switch -> Conn_02x20_Odd_Even; footprint Connector_JST:JST_PH_B2B-PH-K_1x02_P2.00mm_Vertical -> Connector_PinSocket_2.54mm:PinSocket_2x20_P2.54mm_Vertical
- J3: value SW1 switch -> SW0 switch
- J5: value Conn_02x20_Odd_Even -> SW1 switch; footprint Connector_PinSocket_2.54mm:PinSocket_2x20_P2.54mm_Vertical -> Connector_JST:JST_PH_B2B-PH-K_1x02_P2.00mm_Vertical
- moved J4 53.7 mm to (97.7, -31.8)
- moved J7 53.4 mm to (145.5, -28.2)
- moved C10 53.3 mm to (150.6, -17.9)
- moved C11 53.3 mm to (145.7, -17.9)
- moved C12 53.3 mm to (145.7, -11.9)
- moved C13 53.3 mm to (150.6, -14.9)
- moved C14 53.3 mm to (145.7, -14.9)
- moved U2 53.3 mm to (139.0, -13.8)
- moved J1 37.7 mm to (92.5, -32.2)
- moved R6 35.6 mm to (101.9, -26.5)
- moved R1 30.8 mm to (97.1, -24.1)
- moved R4 26.1 mm to (116.1, -26.5)
- moved R3 21.5 mm to (101.9, -23.5)
- moved C25 20.9 mm to (179.3, -8.80)
- moved C26 20.9 mm to (193.0, -25.1)
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Connections:
- C13 pad 1: /RS232 port #2/V+ -> GND
- C13 pad 2: VBUS -> /RS232 port #2/V+
- C14 pad 2: VBUS -> +3V3
- C8 pad 1: /RS232 port #1/V+ -> GND
- C8 pad 2: VBUS -> /RS232 port #1/V+
- C9 pad 2: VBUS -> +3V3
- J1 pad 1: GND -> unconnected-(J1-Pad1)
- J1 pad 2: Net-(J1-Pad2) -> unconnected-(J1-Pad2)
- J5 pad 1: unconnected-(J5-Pad1) -> GND
- J5 pad 2: unconnected-(J5-Pad2) -> Net-(J5-Pad2)
- R1 pad 1: +5V -> Net-(J2-Pad2)
- R1 pad 2: Net-(J1-Pad2) -> /SW00
- R2 pad 1: +5V -> Net-(J3-Pad2)
- R2 pad 2: Net-(J2-Pad2) -> /SW01
- R3 pad 1: +5V -> Net-(J4-Pad2)
- R3 pad 2: Net-(J3-Pad2) -> /SW10
- R4 pad 1: +5V -> Net-(J5-Pad2)
- R4 pad 2: Net-(J4-Pad2) -> /SW11
- R5 pad 1: Net-(J1-Pad2) -> +3V3
- R5 pad 2: /SW00 -> Net-(J2-Pad2)
- R6 pad 1: Net-(J2-Pad2) -> +3V3
- R6 pad 2: /SW01 -> Net-(J3-Pad2)
- R7 pad 1: Net-(J3-Pad2) -> +3V3
- R7 pad 2: /SW10 -> Net-(J4-Pad2)
- R8 pad 1: Net-(J4-Pad2) -> +3V3
- R8 pad 2: /SW11 -> Net-(J5-Pad2)
- U1 pad 10: /RS232 port #1/DTR -> /RS232 port #1/RTS
- U1 pad 11: /RS232 port #1/RTS -> /RS232 port #1/DTR
- U1 pad 12: unconnected-(U1-Pad12) -> /RS232 port #1/DTR
- U1 pad 13: unconnected-(U1-Pad13) -> /RS232 port #1/RTS
- U1 pad 14: unconnected-(U1-Pad14) -> /RS232 port #1/TX
- U1 pad 15: unconnected-(U1-Pad15) -> /RS232 port #1/RI
- U1 pad 16: unconnected-(U1-Pad16) -> /RS232 port #1/DCD
- U1 pad 17: unconnected-(U1-Pad17) -> /RS232 port #1/DSR
- U1 pad 18: unconnected-(U1-Pad18) -> /RS232 port #1/CTS
- U1 pad 19: unconnected-(U1-Pad19) -> /RS232 port #1/RX
- U1 pad 22: unconnected-(U1-Pad22) -> +3V3
- U1 pad 23: unconnected-(U1-Pad23) -> +3V3
- U1 pad 7: /RS232 port #1/RI -> /RS232 port #1/DCD
- U1 pad 8: /RS232 port #1/DCD -> /RS232 port #1/RI
- U2 pad 10: /RS232 port #2/DTR -> /RS232 port #2/RTS
- U2 pad 11: /RS232 port #2/RTS -> /RS232 port #2/DTR
- U2 pad 12: unconnected-(U2-Pad12) -> /RS232 port #2/DTR
- U2 pad 13: unconnected-(U2-Pad13) -> /RS232 port #2/RTS
- U2 pad 14: unconnected-(U2-Pad14) -> /RS232 port #2/TX
- U2 pad 15: unconnected-(U2-Pad15) -> /RS232 port #2/RI
- U2 pad 16: unconnected-(U2-Pad16) -> /RS232 port #2/DCD
- U2 pad 17: unconnected-(U2-Pad17) -> /RS232 port #2/DSR
- U2 pad 18: unconnected-(U2-Pad18) -> /RS232 port #2/CTS
- U2 pad 19: unconnected-(U2-Pad19) -> /RS232 port #2/RX
- U2 pad 22: unconnected-(U2-Pad22) -> +3V3
- U2 pad 23: unconnected-(U2-Pad23) -> +3V3
- U2 pad 7: /RS232 port #2/RI -> /RS232 port #2/DCD
- U2 pad 8: /RS232 port #2/DCD -> /RS232 port #2/RI

Commit message: Progressed ECAD
Parts:
- J1: moved to B.Cu
- moved C25 169.4 mm to (158.7, 159.4)
- moved C26 169.4 mm to (172.4, 143.1)
- moved C33 169.4 mm to (177.6, 139.8)
- moved J9 169.4 mm to (162.8, 145.5)
- moved Q5 169.4 mm to (167.5, 143.8)
- moved C27 169.4 mm to (153.8, 163.7)
- moved C28 169.4 mm to (172.4, 146.1)
- moved C29 169.4 mm to (154.6, 138.4)
- moved C30 169.4 mm to (182.7, 135.2)
- moved C31 169.4 mm to (159.4, 156.3)
- moved C32 169.4 mm to (167.5, 150.5)
- moved C34 169.4 mm to (167.5, 147.5)
- moved D3 169.4 mm to (172.4, 139.9)
- moved D4 169.4 mm to (154.2, 156.2)
- moved Q6 169.4 mm to (162.3, 152.6)
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
Commit message: Progressed ECAD
Parts:
- removed C33: 0.1uC, Capacitor_SMD:C_0805_2012Metric_Pad1.18x1.45mm_HandSolder
- removed C34: 1uC, Capacitor_SMD:C_0805_2012Metric_Pad1.18x1.45mm_HandSolder
- added H1: MountingHole, MountingHole:MountingHole_3.2mm_M3, F.Cu at (107.6, 142.0)
- added J10: Motor connector, Connector_custom:HC-2510-2A, F.Cu at (172.6, 149.9)
- added R23: 10R, Resistor_SMD:R_0805_2012Metric_Pad1.20x1.40mm_HandSolder, F.Cu at (166.8, 166.7)
- added R24: 20mR, Resistor_SMD:R_2512_6332Metric_Pad1.40x3.35mm_HandSolder, F.Cu at (164.1, 150.0)
- added R25: 10R, Resistor_SMD:R_0805_2012Metric_Pad1.20x1.40mm_HandSolder, F.Cu at (161.9, 171.1)
- added R26: 10R, Resistor_SMD:R_0805_2012Metric_Pad1.20x1.40mm_HandSolder, F.Cu at (190.5, 144.0)
- added R27: 10R, Resistor_SMD:R_0805_2012Metric_Pad1.20x1.40mm_HandSolder, F.Cu at (183.3, 150.4)
- added U10: IR2103, Package_SO:SOIC-8_3.9x4.9mm_P1.27mm, F.Cu at (163.8, 155.7)
- added U9: INA180A2, Package_TO_SOT_SMD:SOT-23-5_HandSoldering, F.Cu at (180.7, 140.4)
- C1, C16, C2, C23, C26, C3, C32: value 0.1uC -> 1uC
- C10, C12, C13: value 0.22uC -> 1uC
- C11, C5, C6, C7, C8: value 0.22uC -> 0.1uC
- C14: value 0.1uC -> 220uC; footprint Capacitor_SMD:C_0805_2012Metric_Pad1.18x1.45mm_HandSolder -> Capacitor_THT:CP_Radial_D8.0mm_P3.50mm
- C17, C18, C24, C30, C31: value 1uC -> 0.1uC
- C19, C29: value 220uC -> 1uC; footprint Capacitor_THT:CP_Radial_D8.0mm_P3.50mm -> Capacitor_SMD:C_0805_2012Metric_Pad1.18x1.45mm_HandSolder
- C27: value 1uC -> 220uC; footprint Capacitor_SMD:C_0805_2012Metric_Pad1.18x1.45mm_HandSolder -> Capacitor_THT:CP_Radial_D8.0mm_P3.50mm
- J6, J7: value DB9_Male -> SW1 switch; footprint Connector_Dsub:DSUB-9_Male_Vertical_P2.77x2.84mm_MountingHoles -> Connector_JST:JST_PH_B2B-PH-K_1x02_P2.00mm_Vertical
- J8, J9: footprint Connector_PinHeader_2.54mm:PinHeader_1x02_P2.54mm_Vertical -> Connector_custom:HC-2510-2A
- R10, R11, R9: value 10R -> 10kR
- R12: value 20mR -> 10kR; footprint Resistor_SMD:R_2512_6332Metric_Pad1.40x3.35mm_HandSolder -> Resistor_SMD:R_0805_2012Metric_Pad1.20x1.40mm_HandSolder
- R16, R20: value 10R -> 20mR; footprint Resistor_SMD:R_0805_2012Metric_Pad1.20x1.40mm_HandSolder -> Resistor_SMD:R_2512_6332Metric_Pad1.40x3.35mm_HandSolder
- R19: value 20mR -> 10R; footprint Resistor_SMD:R_2512_6332Metric_Pad1.40x3.35mm_HandSolder -> Resistor_SMD:R_0805_2012Metric_Pad1.20x1.40mm_HandSolder
- U1: value SP3243E -> TLV70033DDCT; footprint Package_SO:TSSOP-28_4.4x9.7mm_P0.65mm -> Package_TO_SOT_SMD:SOT-23-5
- U2: value SP3243E -> 74HC14; footprint Package_SO:TSSOP-28_4.4x9.7mm_P0.65mm -> Package_SO:SO-14_3.9x8.65mm_P1.27mm
- U6: value IR2103 -> ZXBM5210-S
- moved R4 118.6 mm to (79.0, 156.3)
- moved R7 118.4 mm to (74.2, 159.4)
- moved J2 115.0 mm to (82.8, 151.0)
- moved J3 115.0 mm to (74.8, 151.0)
- moved J5 113.4 mm to (88.0, 163.0)
- moved R3 110.8 mm to (79.0, 159.2)
- moved R8 110.6 mm to (104.4, 156.4)
- moved C3 109.2 mm to (112.5, 153.0)
- moved C4 109.1 mm to (102.9, 150.5)
- moved R2 108.0 mm to (99.6, 153.5)
- moved J6 108.0 mm to (90.7, 147.3), turned to 0 degrees
- moved C2 106.4 mm to (107.7, 150.5)
- moved R5 104.8 mm to (94.9, 153.0)
- moved R6 103.4 mm to (94.9, 155.9)
- moved C1 98.4 mm to (114.0, 147.0)
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Connections:
- net /H-bridge #1/Motor_A_Sense renamed /HB_B1_A_SENSE
- net /H-bridge #1/PWM_L renamed /HB_B1_FWD
- net /H-bridge #1/PWM_R renamed /HB_B1_REV
- net /H-bridge #2/Motor_A_Sense renamed /HB_B3_A_SENSE
- net /H-bridge #2/PWM_R renamed /HB_B2_FWD
- C1 pad 1: /SW00 -> GND
- C1 pad 2: GND -> +5V
- C10 pad 1: /RS232 port #2/C1- -> Net-(C10-Pad1)
- C10 pad 2: /RS232 port #2/C1+ -> GND
- C11 pad 1: GND -> Net-(C11-Pad1)
- C11 pad 2: /RS232 port #2/V- -> /H-bridge #1/Motor_L
- C12 pad 1: /RS232 port #2/C2- -> Net-(C10-Pad1)
- C12 pad 2: /RS232 port #2/C2+ -> GND
- C13 pad 1: GND -> Net-(C10-Pad1)
- C13 pad 2: /RS232 port #2/V+ -> GND
- C14 pad 1: GND -> Net-(C10-Pad1)
- C14 pad 2: +3V3 -> GND
- C15 pad 1: Net-(C15-Pad1) -> Net-(C10-Pad1)
- C16 pad 1: Net-(C16-Pad1) -> Net-(C10-Pad1)
- C16 pad 2: /H-bridge #1/Motor_L -> GND
- C17 pad 1: Net-(C15-Pad1) -> Net-(C17-Pad1)
- C17 pad 2: GND -> /H-bridge #1/Motor_R
- C18 pad 1: Net-(C15-Pad1) -> +3V3
- C19 pad 1: Net-(C15-Pad1) -> Net-(C10-Pad1)
- C2 pad 1: /SW01 -> +3V3
- C20 pad 1: Net-(C15-Pad1) -> +5V
- C21 pad 1: Net-(C15-Pad1) -> Net-(U6-Pad2)
- C22 pad 1: Net-(C22-Pad1) -> +3V3
- C22 pad 2: /H-bridge #1/Motor_R -> GND
- C23 pad 1: +3V3 -> Net-(C23-Pad1)
- C24 pad 1: Net-(C15-Pad1) -> Net-(C24-Pad1)
- C24 pad 2: GND -> /H-bridge #2/Motor_L
- C25 pad 1: Net-(C25-Pad1) -> Net-(C23-Pad1)
- C26 pad 1: Net-(C26-Pad1) -> Net-(C23-Pad1)
- C26 pad 2: /H-bridge #2/Motor_L -> GND
- C27 pad 1: Net-(C25-Pad1) -> Net-(C23-Pad1)
- C28 pad 1: Net-(C25-Pad1) -> Net-(C23-Pad1)
- C29 pad 1: Net-(C25-Pad1) -> Net-(C23-Pad1)
- C3 pad 1: /SW10 -> GND
- C3 pad 2: GND -> +3.3V
- C30 pad 1: Net-(C25-Pad1) -> Net-(C30-Pad1)
- C30 pad 2: GND -> /H-bridge #2/Motor_R
- C31 pad 1: Net-(C25-Pad1) -> +3V3
- C32 pad 1: Net-(C32-Pad1) -> Net-(C23-Pad1)
- C32 pad 2: /H-bridge #2/Motor_R -> GND
- C4 pad 1: /SW11 -> Net-(C4-Pad1)
- C5 pad 1: /RS232 port #1/C1- -> Net-(C5-Pad1)
- C5 pad 2: /RS232 port #1/C1+ -> GND
- C6 pad 1: GND -> Net-(C6-Pad1)
- C6 pad 2: /RS232 port #1/V- -> GND
- C7 pad 1: /RS232 port #1/C2- -> Net-(C7-Pad1)
- C7 pad 2: /RS232 port #1/C2+ -> GND
- C8 pad 1: GND -> Net-(C8-Pad1)
- C8 pad 2: /RS232 port #1/V+ -> GND
- C9 pad 1: GND -> Net-(C9-Pad1)
- C9 pad 2: +3V3 -> GND
- D1 pad 1: Net-(C16-Pad1) -> Net-(C11-Pad1)
- D2 pad 1: Net-(C22-Pad1) -> Net-(C17-Pad1)
- D3 pad 1: Net-(C26-Pad1) -> Net-(C24-Pad1)
- D4 pad 1: Net-(C32-Pad1) -> Net-(C30-Pad1)
- J6 pad 1: /RS232 port #1/DCD -> GND
- J6 pad 2: /RS232 port #1/RX -> Net-(J6-Pad2)
- J7 pad 1: /RS232 port #2/DCD -> GND
- J7 pad 2: /RS232 port #2/RX -> Net-(J7-Pad2)
- J9 pad 1: /H-bridge #2/Motor_R -> Net-(U6-Pad1)
- J9 pad 2: /H-bridge #2/Motor_L -> Net-(U6-Pad7)
- Q1 pad 3: Net-(C15-Pad1) -> Net-(C10-Pad1)
- Q3 pad 3: Net-(C15-Pad1) -> Net-(C10-Pad1)
- Q5 pad 3: Net-(C25-Pad1) -> Net-(C23-Pad1)
- Q7 pad 3: Net-(C25-Pad1) -> Net-(C23-Pad1)
- R1 pad 2: /SW00 -> Net-(C4-Pad1)
- R10 pad 1: Net-(R10-Pad1) -> +3V3
- R10 pad 2: Net-(Q1-Pad1) -> Net-(J5-Pad2)
- R11 pad 1: Net-(R11-Pad1) -> +3V3
- R11 pad 2: Net-(Q2-Pad1) -> Net-(J6-Pad2)
- R12 pad 1: Net-(C15-Pad1) -> +3V3
- R12 pad 2: +12V -> Net-(J7-Pad2)
- R13 pad 1: Net-(Q3-Pad1) -> Net-(C10-Pad1)
- R13 pad 2: Net-(R13-Pad2) -> Net-(D1-Pad2)
- R14 pad 1: Net-(Q4-Pad1) -> Net-(R14-Pad1)
- R14 pad 2: Net-(R14-Pad2) -> Net-(Q1-Pad1)
- R15 pad 1: Net-(C15-Pad1) -> Net-(R15-Pad1)
- R15 pad 2: Net-(D2-Pad2) -> Net-(Q2-Pad1)
- R16 pad 1: Net-(C25-Pad1) -> Net-(C10-Pad1)
- R16 pad 2: Net-(D3-Pad2) -> +12V
- R17 pad 1: Net-(R17-Pad1) -> Net-(Q3-Pad1)
- R17 pad 2: Net-(Q5-Pad1) -> Net-(R17-Pad2)
- R18 pad 1: Net-(R18-Pad1) -> Net-(Q4-Pad1)
- R18 pad 2: Net-(Q6-Pad1) -> Net-(R18-Pad2)
- R19 pad 1: Net-(C25-Pad1) -> Net-(C10-Pad1)
- R19 pad 2: +12V -> Net-(D2-Pad2)
- R2 pad 2: /SW01 -> Net-(C5-Pad1)
- R20 pad 1: Net-(Q7-Pad1) -> Net-(U6-Pad2)
- R20 pad 2: Net-(R20-Pad2) -> +12V
- R21 pad 1: Net-(Q8-Pad1) -> Net-(C23-Pad1)
- R21 pad 2: Net-(R21-Pad2) -> Net-(D3-Pad2)
- R22 pad 1: Net-(C25-Pad1) -> Net-(R22-Pad1)
- R22 pad 2: Net-(D4-Pad2) -> Net-(Q5-Pad1)
- R3 pad 2: /SW10 -> Net-(C6-Pad1)
- R4 pad 2: /SW11 -> Net-(C7-Pad1)
- R5 pad 1: +3V3 -> Net-(J6-Pad2)
- R5 pad 2: Net-(J2-Pad2) -> Net-(C8-Pad1)
- R6 pad 1: +3V3 -> Net-(J7-Pad2)
- R6 pad 2: Net-(J3-Pad2) -> Net-(C9-Pad1)
- R7 pad 2: Net-(J4-Pad2) -> Net-(J2-Pad2)
- R8 pad 2: Net-(J5-Pad2) -> Net-(J3-Pad2)
- R9 pad 1: Net-(C15-Pad1) -> +3V3
- R9 pad 2: Net-(D1-Pad2) -> Net-(J4-Pad2)
- U1 pad 1: /RS232 port #1/C2+ -> +5V
- U1 pad 2: /RS232 port #1/C2- -> GND
- U1 pad 3: /RS232 port #1/V- -> +5V
- U1 pad 4: /RS232 port #1/RX -> unconnected-(U1-Pad4)
- U1 pad 5: /RS232 port #1/CTS -> +3.3V
- U2 pad 1: /RS232 port #2/C2+ -> Net-(C4-Pad1)
- U2 pad 10: /RS232 port #2/RTS -> /SW20
- U2 pad 11: /RS232 port #2/DTR -> Net-(C8-Pad1)
- U2 pad 12: /RS232 port #2/DTR -> /SW21
- U2 pad 13: /RS232 port #2/RTS -> Net-(C9-Pad1)
- U2 pad 14: /RS232 port #2/TX -> +3V3
- U2 pad 2: /RS232 port #2/C2- -> /SW00
- U2 pad 3: /RS232 port #2/V- -> Net-(C5-Pad1)
- U2 pad 4: /RS232 port #2/RX -> /SW01
- U2 pad 5: /RS232 port #2/CTS -> Net-(C6-Pad1)
- U2 pad 6: /RS232 port #2/DSR -> /SW10
- U2 pad 7: /RS232 port #2/DCD -> GND
- U2 pad 8: /RS232 port #2/RI -> /SW11
- U2 pad 9: /RS232 port #2/TX -> Net-(C7-Pad1)
- U3 pad 1: Net-(C15-Pad1) -> Net-(C10-Pad1)
- U3 pad 5: Net-(R11-Pad1) -> Net-(R15-Pad1)
- U3 pad 7: Net-(R10-Pad1) -> Net-(R14-Pad1)
- U3 pad 8: Net-(C16-Pad1) -> Net-(C11-Pad1)
- U4 pad 4: Net-(C15-Pad1) -> Net-(C10-Pad1)
- U5 pad 1: Net-(C15-Pad1) -> Net-(C10-Pad1)
- U5 pad 5: Net-(R14-Pad2) -> Net-(R18-Pad2)
- U5 pad 7: Net-(R13-Pad2) -> Net-(R17-Pad2)
- U5 pad 8: Net-(C22-Pad1) -> Net-(C17-Pad1)
- U6 pad 1: Net-(C25-Pad1) -> Net-(U6-Pad1)
- U6 pad 2: /H-bridge #2/PWM_L -> Net-(U6-Pad2)
- U6 pad 3: /H-bridge #2/PWM_L -> +5V
- U6 pad 4: GND -> /HB_B3_FWD
- U6 pad 5: Net-(R18-Pad1) -> /HB_B3_REV
- U6 pad 6: /H-bridge #2/Motor_L -> +5V
- U6 pad 7: Net-(R17-Pad1) -> Net-(U6-Pad7)
- U6 pad 8: Net-(C26-Pad1) -> GND
- U7 pad 4: Net-(C25-Pad1) -> Net-(U6-Pad2)
- U8 pad 1: Net-(C25-Pad1) -> Net-(C23-Pad1)
- U8 pad 5: Net-(R21-Pad2) -> Net-(R23-Pad1)
- U8 pad 6: /H-bridge #2/Motor_R -> /H-bridge #2/Motor_L
- U8 pad 7: Net-(R20-Pad2) -> Net-(R22-Pad1)
- U8 pad 8: Net-(C32-Pad1) -> Net-(C24-Pad1)
