File: Tester/ECAD/MotorControlDaughterBoard/lv_H_bridge.kicad_sch (KiCad schematic)
At the start: 7 parts, among them J9 Motor connector, U6 ZXBM5210-S, U7 INA180A2

Commit message: Update lv_H_bridge.kicad_sch
Parts:
- U6: Manufacturer Part Number (none) -> ZXBM5210-S-13
Changed lines of the file:
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@@
       (effects (font (size 1.27 1.27)) hide)
     )
-    (property "Datasheet" "https://www.diodes.com/assets/Datasheets/ZXBM5210.pdf" (id 3) (at 115.57 105.41 0)
+    (property "Datasheet" "https://datasheet.lcsc.com/lcsc/1912111437_Diodes-Incorporated-ZXBM5210-S-13_C460766.pdf" (id 3) (at 115.57 105.41 0)
       (effects (font (size 1.27 1.27)) hide)
     )
+    (property "Manufacturer Part Number" "ZXBM5210-S-13" (id 4) (at 115.57 105.41 0)
+      (effects (font (size 1.27 1.27)) hide)
+    )
