File: Tester/ECAD/BDCMotorControlShield/h_bridge.kicad_sch (KiCad schematic)
At the start: 25 parts, among them J5 Motor connector, Q1 Q_NMOS_GSD, Q2 Q_NMOS_GSD, Q3 Q_NMOS_GSD, Q4 Q_NMOS_GSD, U1 IR2103, U2 INA180A2, U3 IR2103

Commit message: Progressed ECAD
Parts:
- added R19, R20: 10R, Resistor_SMD:R_0805_2012Metric_Pad1.20x1.40mm_HandSolder, symbol Device:R
Connections:
- net +12V: no longer names the net of C1.1, R1.1, U1.1 (VCC)
- net +12V: now also C10.1, C11.1, C15.1, C4.1, C6.1, C7.1, Q1.3 (D), Q3.3 (D), U2.4 (-), U3.1 (VCC), R19.1, R20.1; no longer D1.2 (A), U2.3 (+)
- net +5V renamed 5V
- removed net A_Meas: C10.1, C11.1, C15.1, C4.1, C6.1, C7.1, D2.2 (A), Q1.3 (D), Q3.3 (D), R1.2, U2.4 (-), U3.1 (VCC)
- net Floating_Rail_L renamed Motor_L
- net Floating_Rail_R renamed Motor_R
- new net: D1.2 (A), R19.2
- new net: D2.2 (A), R20.2
- new net 12V: R1.2, U2.3 (+)
Other:
- moved on the sheet: C1, C13, C15, C2, C3, C4, D1, D2, J5, Q1, Q2, Q3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

Commit message: Progressed ECAD
Changed lines of the file:
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@@
     (stroke (width 0) (type default) (color 0 0 0 0))
   )
-  (wire (pts (xy 156.21 50.8) (xy 156.21 31.75))
+  (wire (pts (xy 156.21 50.8) (xy 156.21 48.26))
     (stroke (width 0) (type default) (color 0 0 0 0))
   )
@@
     (stroke (width 0) (type default) (color 0 0 0 0))
   )
-  (wire (pts (xy 156.21 31.75) (xy 148.59 31.75))
+  (wire (pts (xy 156.21 48.26) (xy 148.59 48.26))
     (stroke (width 0) (type default) (color 0 0 0 0))
   )
@@
     (stroke (width 0) (type default) (color 0 0 0 0))
   )
-  (wire (pts (xy 78.74 113.03) (xy 80.01 113.03))
+  (wire (pts (xy 74.93 113.03) (xy 80.01 113.03))
     (stroke (width 0) (type default) (color 0 0 0 0))
   )
@@
     (stroke (width 0) (type default) (color 0 0 0 0))
   )
-  (wire (pts (xy 231.14 113.03) (xy 232.41 113.03))
+  (wire (pts (xy 231.14 113.03) (xy 236.22 113.03))
     (stroke (width 0) (type default) (color 0 0 0 0))
   )
@@
     (effects (font (size 1.27 1.27)) (justify left))
   )
-  (hierarchical_label "12V" (shape input) (at 148.59 31.75 180)
+  (hierarchical_label "12V" (shape input) (at 148.59 48.26 180)
     (effects (font (size 1.27 1.27)) (justify right))
   )
@@
     (effects (font (size 1.27 1.27)) (justify left))
   )
-  (hierarchical_label "PWM_L" (shape input) (at 78.74 113.03 180)
+  (hierarchical_label "PWM_L" (shape input) (at 74.93 113.03 180)
     (effects (font (size 1.27 1.27)) (justify right))
   )
-  (hierarchical_label "PWM_R" (shape input) (at 232.41 113.03 0)
-    (effects (font (size 1.27 1.27)) (justify left))
-  )
+  (hierarchical_label "PWM_R" (shape input) (at 236.22 113.03 0)
+    (effects (font (size 1.27 1.27)) (justify left))
+  )

Commit message: Progressed ECAD
Parts:
- J5: footprint Connector_custom:HC-2510-2AW -> Connector_PinHeader_2.54mm:PinHeader_1x02_P2.54mm_Vertical
Changed lines of the file:
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@@
       (effects (font (size 1.27 1.27)) (justify left))
     )
-    (property "Footprint" "Connector_custom:HC-2510-2AW" (id 2) (at 157.48 133.35 0)
+    (property "Footprint" "Connector_PinHeader_2.54mm:PinHeader_1x02_P2.54mm_Vertical" (id 2) (at 157.48 133.35 0)
       (effects (font (size 1.27 1.27)) hide)
     )

Commit message: Progressed ECAD
Parts:
- removed C10, C11, C15, C6, C7: 1uC, Capacitor_SMD:C_0805_2012Metric_Pad1.18x1.45mm_HandSolder, symbol Device:C
- removed C13, C3: 0.1uC, Capacitor_SMD:C_0805_2012Metric_Pad1.18x1.45mm_HandSolder, symbol Device:C
- removed C4: 220uC, Capacitor_THT:CP_Radial_D8.0mm_P3.50mm, symbol Device:C_Polarized
- removed D1, D2: PMEG6010ER, Diode_SMD:Nexperia_CFP3_SOD-123W, symbol Diode:PMEG6010ER
- removed Q1, Q2, Q3, Q4: Q_NMOS_GSD, Package_TO_SOT_SMD:SOT-23, symbol Device:Q_NMOS_GSD
- removed R19, R2, R20, R3, R4, R5: 10R, Resistor_SMD:R_0805_2012Metric_Pad1.20x1.40mm_HandSolder, symbol Device:R
- removed U1, U3: IR2103, Package_SO:SOIC-8_3.9x4.9mm_P1.27mm, symbol Driver_FET:IR2103
- added C3: 220uC, Capacitor_THT:CP_Radial_D8.0mm_P3.50mm, symbol Device:C_Polarized
- added U1: DRV8870DDA, Package_SO:Texas_HTSOP-8-1EP_3.9x4.9mm_P1.27mm_EP2.95x4.9mm_Mask2.4x3.1mm_ThermalVias, symbol Driver_Motor:DRV8870DDA
- J5: footprint Connector_PinHeader_2.54mm:PinHeader_1x02_P2.54mm_Vertical -> Connector_custom:HC-2510-2A; Manufacturer Part Number HC-2510-2AW -> HC-2510-2A
Connections:
- net GND: now also C3.2
- net at R1.1, U2.4 (-): no longer C1.1
- net Motor_L: no longer names the net of J5.2 (Pin_2)
- net Motor_R: no longer names the net of J5.1 (Pin_1)
- new net: U1.1 (GND), U1.9 (GND)
Other:
- note removed: "H-bridge"
- moved on the sheet: J5

Commit message: Progressed ECAD
Parts:
- removed C1: 1uC, Capacitor_SMD:C_0805_2012Metric_Pad1.18x1.45mm_HandSolder, symbol Device:C
- added C?: 0.1uC, Capacitor_SMD:C_0805_2012Metric_Pad1.18x1.45mm_HandSolder, symbol Device:C
- U1: Manufacturer Part Number (none) -> DRV8870DDAR
Connections:
- net 12V: now also U1.5 (VM); no longer R1.2, U2.3 (+)
- net GND: now also R1.1, U1.1 (GND), U1.9 (GND), U2.4 (-), C?.2
- net PWM_L: now also U1.3 (IN1)
- net PWM_R: now also U1.2 (IN2)
- net at J5.1 (Pin_1): now also U1.6 (OUT1)
- net at J5.2 (Pin_2): now also U1.8 (OUT2)
- net at U1.7 (ISEN): now also R1.2, U2.3 (+)
Other:
- note added: "H-drive"
- moved on the sheet: C2, C3, J5, R1, U1, U2

Commit message: Progressed ECAD
Parts:
- added R2, R3: 10kR, Resistor_SMD:R_0805_2012Metric_Pad1.20x1.40mm_HandSolder, symbol Device:R
- C3: value 220uC -> 47uC; footprint Capacitor_THT:CP_Radial_D8.0mm_P3.50mm -> Capacitor_THT:CP_Radial_D5.0mm_P2.00mm; Manufacturer Part Number 25YXF220MEFC8X11.5 -> 35YXJ47M5X11
- R1: value 20mR -> 250mR; footprint Resistor_SMD:R_2512_6332Metric_Pad1.40x3.35mm_HandSolder -> Resistor_SMD:R_2010_5025Metric; Manufacturer Part Number RL2512FK-070R02L -> RL2010FK-070R25L
- U2: value INA180A2 -> INA180A1; footprint Package_TO_SOT_SMD:SOT-23-5_HandSoldering -> Package_TO_SOT_SMD:SOT-23-5; Manufacturer Part Number INA180A2IDBVR -> INA180A1IDBVR
- gave numbers to parts that had none: 1
Connections:
- net 12V: now also C1.1, C3.1
- net 5V: now also R2.1
- net GND: now also R3.2
- net at U1.4 (VREF): now also R2.2, R3.1
- net PWM_L renamed PWM1
- net PWM_R renamed PWM2
Other:
- note added: "2.5V"
- note added: "Current measurement 20 V/V Gain"
- note added: "I_trip = VREF/(10*RISEN) I_trip = 1 A"
- note removed: "Current measurement"
- moved on the sheet: C1, C2, C3, J5, R1, U1, U2

Commit message: Progessed ECAD
Parts:
- added C11: 10uC, Capacitor_SMD:C_1210_3225Metric_Pad1.33x2.70mm_HandSolder, symbol Device:C
Connections:
- net 12V: now also C11.1
- net GND: now also C11.2
Other:
- moved on the sheet: C1
Changed lines of the file:
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@@
+    (effects (font (size 1.27 1.27)) (justify left))
+  )
+  (hierarchical_label "12V" (shape input) (at 83.82 88.9 90)
     (effects (font (size 1.27 1.27)) (justify left))
   )
@@
     (effects (font (size 1.27 1.27)) (justify left))
   )
-  (hierarchical_label "12V" (shape input) (at 82.55 88.9 90)
+  (hierarchical_label "12V" (shape input) (at 69.85 88.9 90)
     (effects (font (size 1.27 1.27)) (justify left))
   )
@@
     (pin "1")
   )
-  (symbol (lib_id "power:GND") (at 82.55 96.52 0) (unit 1)
-    (in_bom yes) (on_board yes) (fields_autoplaced)
-    (property "Reference" "#PWR0103" (id 0) (at 82.55 102.87 0)
-      (effects (font (size 1.27 1.27)) hide)
-    )
-    (property "Value" "GND" (id 1) (at 82.55 101.6 0))
-    (property "Footprint" "" (id 2) (at 82.55 96.52 0)
-      (effects (font (size 1.27 1.27)) hide)
-    )
-    (property "Datasheet" "" (id 3) (at 82.55 96.52 0)
-      (effects (font (size 1.27 1.27)) hide)
-    )
-    (pin "1")
+  (symbol (lib_id "power:GND") (at 69.85 96.52 0) (unit 1)
+    (in_bom yes) (on_board yes) (fields_autoplaced)
+    (property "Reference" "#PWR0103" (id 0) (at 69.85 102.87 0)
+      (effects (font (size 1.27 1.27)) hide)
+    )
+    (property "Value" "GND" (id 1) (at 69.85 101.6 0))
+    (property "Footprint" "" (id 2) (at 69.85 96.52 0)
+      (effects (font (size 1.27 1.27)) hide)
+    )
+    (property "Datasheet" "" (id 3) (at 69.85 96.52 0)
+      (effects (font (size 1.27 1.27)) hide)
+    )
+    (pin "1")
+  )
+  (symbol (lib_id "Device:C") (at 83.82 92.71 0) (mirror y) (unit 1)
+    (in_bom yes) (on_board yes)
+    (property "Reference" "C11" (id 0) (at 91.44 91.44 0)
+      (effects (font (size 1.27 1.27)) (justify left))
+    )
+    (property "Value" "10uC" (id 1) (at 92.71 93.98 0)
+      (effects (font (size 1.27 1.27)) (justify left))
+    )
+    (property "Footprint" "Capacitor_SMD:C_1210_3225Metric_Pad1.33x2.70mm_HandSolder" (id 2) (at 82.8548 96.52 0)
+      (effects (font (size 1.27 1.27)) hide)
+    )
+    (property "Datasheet" "https://datasheet.lcsc.com/lcsc/1912111437_Taiyo-Yuden-UMK325AB7106KM-T_C386167.pdf" (id 3) (at 83.82 92.71 0)
+      (effects (font (size 1.27 1.27)) hide)
+    )
+    (property "Manufacturer Part Number" "UMK325AB7106KM-T" (id 4) (at 83.82 92.71 0)
+      (effects (font (size 1.27 1.27)) hide)
+    )
+    (pin "1")
+    (pin "2")
   )
   (symbol (lib_id "Driver_Motor:DRV8870DDA") (at 135.89 91.44 0) (unit 1)
@@
     (pin "2")
   )
-  (symbol (lib_id "Device:C") (at 82.55 92.71 0) (mirror y) (unit 1)
+  (symbol (lib_id "Device:C") (at 69.85 92.71 0) (mirror y) (unit 1)
     (in_bom yes) (on_board yes)
-    (property "Reference" "C1" (id 0) (at 88.9 91.44 0)
-      (effects (font (size 1.27 1.27)) (justify left))
-    )
-    (property "Value" "0.1uC" (id 1) (at 91.44 93.98 0)
-      (effects (font (size 1.27 1.27)) (justify left))
-    )
-    (property "Footprint" "Capacitor_SMD:C_0805_2012Metric_Pad1.18x1.45mm_HandSolder" (id 2) (at 81.5848 96.52 0)
-      (effects (font (size 1.27 1.27)) hide)
-    )
-    (property "Datasheet" "https://datasheet.lcsc.com/lcsc/2006111832_YAGEO-CC0805KRX7R8BB104_C519981.pdf" (id 3) (at 82.55 92.71 0)
-      (effects (font (size 1.27 1.27)) hide)
-    )
-    (property "Manufacturer Part Number" "CC0805KRX7R8BB104" (id 4) (at 82.55 92.71 0)
+    (property "Reference" "C1" (id 0) (at 76.2 91.44 0)
+      (effects (font (size 1.27 1.27)) (justify left))
+    )
+    (property "Value" "0.1uC" (id 1) (at 78.74 93.98 0)
+      (effects (font (size 1.27 1.27)) (justify left))
+    )
+    (property "Footprint" "Capacitor_SMD:C_0805_2012Metric_Pad1.18x1.45mm_HandSolder" (id 2) (at 68.8848 96.52 0)
+      (effects (font (size 1.27 1.27)) hide)
+    )
+    (property "Datasheet" "https://datasheet.lcsc.com/lcsc/2006111832_YAGEO-CC0805KRX7R8BB104_C519981.pdf" (id 3) (at 69.85 92.71 0)
+      (effects (font (size 1.27 1.27)) hide)
+    )
+    (property "Manufacturer Part Number" "CC0805KRX7R8BB104" (id 4) (at 69.85 92.71 0)
       (effects (font (size 1.27 1.27)) hide)
     )
@@
       (effects (font (size 1.27 1.27)) hide)
     )
+    (pin "1")
+  )
+  (symbol (lib_id "power:GND") (at 83.82 96.52 0) (unit 1)
+    (in_bom yes) (on_board yes) (fields_autoplaced)
+    (property "Reference" "#PWR021" (id 0) (at 83.82 102.87 0)
+      (effects (font (size 1.27 1.27)) hide)
+    )
+    (property "Value" "GND" (id 1) (at 83.82 101.6 0))
+    (property "Footprint" "" (id 2) (at 83.82 96.52 0)
+      (effects (font (size 1.27 1.27)) hide)
+    )
+    (property "Datasheet" "" (id 3) (at 83.82 96.52 0)
+      (effects (font (size 1.27 1.27)) hide)
+    )

Commit message: Progressed ECAD
Parts:
- added C15: 0.1uC, Capacitor_SMD:C_0805_2012Metric_Pad1.18x1.45mm_HandSolder, symbol Device:C
Connections:
- net GND: now also C15.2
- net at R2.2, R3.1, U1.4 (VREF): now also C15.1
Other:
- moved on the sheet: C1, C11, C3
