File: Tester/ECAD/BDCMotorControlShield/BDCMotorControlShield.kicad_sch (KiCad schematic)
At the start: 50 parts, among them J1 Power, J10 Limit switch, J11 Limit switch, J12 Limit switch, J13 Limit switch, J2 Digital/PWM, J3 Analog, J4 Digital/PWM, J6 Barrel_Jack_Switch, J7 Limit switch, J8 Limit switch, U10 74HC14, U11 PCA9535PW, U6 74HC2G08, U8 74HC2G08, U9 74HC2G08

Commit message: Progressed ECAD
Parts:
- added U?: TSOP531xx, OptoDevice:Vishay_MINIMOLD-3Pin, symbol Interface_Optical:TSOP531xx
Changed lines of the file:
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@@
     (pin "2")
+  )
+  (symbol (lib_id "Interface_Optical:TSOP531xx") (at -43.18 115.57 0) (unit 1)
+    (in_bom yes) (on_board yes) (fields_autoplaced)
+    (property "Reference" "U?" (id 0) (at -44.915 104.14 0))
+    (property "Value" "TSOP531xx" (id 1) (at -44.915 106.68 0))
+    (property "Footprint" "OptoDevice:Vishay_MINIMOLD-3Pin" (id 2) (at -44.45 125.095 0)
+      (effects (font (size 1.27 1.27)) hide)
+    )
+    (property "Datasheet" "https://datasheet.lcsc.com/lcsc/1912111437_Everlight-Elec-IRM-H638J7-TR2-CLW_C414640.pdf" (id 3) (at -26.67 107.95 0)
+      (effects (font (size 1.27 1.27)) hide)
+    )
+    (property "Manufacturer Part Number" "IRM-H638J7/TR2(CLW)" (id 4) (at -43.18 115.57 0)
+      (effects (font (size 1.27 1.27)) hide)
+    )
+    (pin "1")
+    (pin "2")
+    (pin "3")
   )
   (symbol (lib_id "Device:C") (at 189.23 140.97 0) (unit 1)
@@
       (reference "U11") (unit 1) (value "PCA9535PW") (footprint "Package_SO:TSSOP-24_4.4x7.8mm_P0.65mm")
     )
-  )
+    (path "/cab29b3a-e749-4d9a-a5d0-1de239719c00"
+      (reference "U?") (unit 1) (value "TSOP531xx") (footprint "OptoDevice:Vishay_MINIMOLD-3Pin")
+    )
+  )

Commit message: Progressed CAD
Parts:
- removed U?: TSOP531xx, OptoDevice:Vishay_MINIMOLD-3Pin, symbol Interface_Optical:TSOP531xx
- added C23: 4.7uC, Capacitor_SMD:C_0805_2012Metric_Pad1.18x1.45mm_HandSolder, symbol Device:C
- added R28: 10kR, Resistor_SMD:R_0805_2012Metric_Pad1.20x1.40mm_HandSolder, symbol Device:R
- added R29: 100R, Resistor_SMD:R_0805_2012Metric_Pad1.20x1.40mm_HandSolder, symbol Device:R
- added U12: IRM-H6XX, OptoDevice_custom:IRM-H6XX, symbol Inteface_Optical_custom:IRM-H6XX
- J1, J2, J3, J4: Manufacturer Part Number N/A -> (none)
Connections:
- net +5V: now also R28.1, R29.2
- net GND: now also C23.2, U12.1 (GND), U12.2 (GND)
- net at U6.2: now also U8.2, U9.2
- net at U9.6: now also U6.6, U8.6
- new net: C23.1, R29.1, U12.4 (Vs)
- new net: R28.2, U12.3 (OUT)
Other:
- note added: "I/O concentrator"
- note added: "IR receiver"
- note removed: "IR remote Limit switch Current limit Motor active"
- moved on the sheet: C22, D1, D2, D6, D8, J6, R10, R19, R20, R21, R22, R27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

Commit message: Progressed ECAD
Parts:
- J1, J3: Manufacturer Part Number (none) -> PZ254-1-06-Z-8.5
- J2, J4: Manufacturer Part Number (none) -> PZ254-1-08-Z-8.5
Connections:
- net *11: now also U6.2, U8.2, U9.2
- net *3: now also U6.6, U8.6, U9.6
- net +5V: no longer J1.8 (Pin_8)
- net 12: now also U9.1, U9.5
- net 13: now also R9.2, U11.1 (~{INT})
- net 2: now also U8.1, U8.5
- net 7: now also U6.1, U6.5
- net 8: now also R28.2, U12.3 (OUT)
- net SCL/A5: now also R19.2, U11.22 (SCL)
- net SDA/A4: now also R10.2, U11.23 (SDA)
- new net Vin: J1.8 (Pin_8)
- no-connect marks 7 -> 20

Commit message: Progressed ECAD
Parts:
- D1, D2, D6, D8: Manufacturer Part Number (none) -> 17-21SYGC/S530-E3/TR8
- R20, R21, R22, R27: value 2kR -> 160R; Manufacturer Part Number (none) -> AC0805FR-7W160RL
- R29: value 100R -> 160R; Manufacturer Part Number RC0805JR-07100RL -> AC0805FR-7W160RL
Changed lines of the file:
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@@
       (effects (font (size 1.27 1.27)) hide)
     )
-    (property "Datasheet" "" (id 3) (at 68.58 104.14 0)
-      (effects (font (size 1.27 1.27)) hide)
-    )
-    (property "Manufacturer Part Number" "" (id 4) (at 68.58 104.14 0)
+    (property "Datasheet" "https://datasheet.lcsc.com/lcsc/1810271707_Everlight-Elec-17-21SYGC-S530-E3-TR8_C142303.pdf" (id 3) (at 68.58 104.14 0)
+      (effects (font (size 1.27 1.27)) hide)
+    )
+    (property "Manufacturer Part Number" "17-21SYGC/S530-E3/TR8" (id 4) (at 68.58 104.14 0)
       (effects (font (size 1.27 1.27)) hide)
     )
@@
       (effects (font (size 1.27 1.27)) hide)
     )
-    (property "Datasheet" "" (id 3) (at 91.44 104.14 0)
-      (effects (font (size 1.27 1.27)) hide)
-    )
-    (property "Manufacturer Part Number" "" (id 4) (at 91.44 104.14 0)
+    (property "Datasheet" "https://datasheet.lcsc.com/lcsc/1810271707_Everlight-Elec-17-21SYGC-S530-E3-TR8_C142303.pdf" (id 3) (at 91.44 104.14 0)
+      (effects (font (size 1.27 1.27)) hide)
+    )
+    (property "Manufacturer Part Number" "17-21SYGC/S530-E3/TR8" (id 4) (at 91.44 104.14 0)
       (effects (font (size 1.27 1.27)) hide)
     )
@@
       (effects (font (size 1.27 1.27)) hide)
     )
-    (property "Datasheet" "" (id 3) (at 57.15 104.14 0)
-      (effects (font (size 1.27 1.27)) hide)
-    )
-    (property "Manufacturer Part Number" "" (id 4) (at 57.15 104.14 0)
+    (property "Datasheet" "https://datasheet.lcsc.com/lcsc/1810271707_Everlight-Elec-17-21SYGC-S530-E3-TR8_C142303.pdf" (id 3) (at 57.15 104.14 0)
+      (effects (font (size 1.27 1.27)) hide)
+    )
+    (property "Manufacturer Part Number" "17-21SYGC/S530-E3/TR8" (id 4) (at 57.15 104.14 0)
       (effects (font (size 1.27 1.27)) hide)
     )
@@
       (effects (font (size 1.27 1.27)) (justify left))
     )
-    (property "Value" "2kR" (id 1) (at 93.98 97.7899 0)
+    (property "Value" "160R" (id 1) (at 93.98 97.7899 0)
       (effects (font (size 1.27 1.27)) (justify left))
     )
@@
       (effects (font (size 1.27 1.27)) hide)
     )
-    (property "Datasheet" "" (id 3) (at 91.44 96.52 0)
-      (effects (font (size 1.27 1.27)) hide)
-    )
-    (property "Manufacturer Part Number" "" (id 4) (at 91.44 96.52 0)
+    (property "Datasheet" "https://datasheet.lcsc.com/lcsc/2012011712_YAGEO-AC0805FR-7W160RL_C727986.pdf" (id 3) (at 91.44 96.52 0)
+      (effects (font (size 1.27 1.27)) hide)
+    )
+    (property "Manufacturer Part Number" "AC0805FR-7W160RL" (id 4) (at 91.44 96.52 0)
       (effects (font (size 1.27 1.27)) hide)
     )
@@
       (effects (font (size 1.27 1.27)) hide)
     )
-    (property "Datasheet" "" (id 3) (at 80.01 104.14 0)
-      (effects (font (size 1.27 1.27)) hide)
-    )
-    (property "Manufacturer Part Number" "" (id 4) (at 80.01 104.14 0)
+    (property "Datasheet" "https://datasheet.lcsc.com/lcsc/1810271707_Everlight-Elec-17-21SYGC-S530-E3-TR8_C142303.pdf" (id 3) (at 80.01 104.14 0)
+      (effects (font (size 1.27 1.27)) hide)
+    )
+    (property "Manufacturer Part Number" "17-21SYGC/S530-E3/TR8" (id 4) (at 80.01 104.14 0)
       (effects (font (size 1.27 1.27)) hide)
     )
@@
       (effects (font (size 1.27 1.27)) (justify right))
     )
-    (property "Value" "100R" (id 1) (at 271.78 132.0799 0)
+    (property "Value" "160R" (id 1) (at 271.78 132.0799 0)
       (effects (font (size 1.27 1.27)) (justify right))
     )
@@
       (effects (font (size 1.27 1.27)) hide)
     )
-    (property "Datasheet" "https://datasheet.lcsc.com/lcsc/1811081022_YAGEO-RC0805JR-07100RL_C106949.pdf" (id 3) (at 269.24 130.81 0)
-      (effects (font (size 1.27 1.27)) hide)
-    )
-    (property "Manufacturer Part Number" "RC0805JR-07100RL" (id 4) (at 269.24 130.81 0)
+    (property "Datasheet" "https://datasheet.lcsc.com/lcsc/2012011712_YAGEO-AC0805FR-7W160RL_C727986.pdf" (id 3) (at 269.24 130.81 0)
+      (effects (font (size 1.27 1.27)) hide)
+    )
+    (property "Manufacturer Part Number" "AC0805FR-7W160RL" (id 4) (at 269.24 130.81 0)
       (effects (font (size 1.27 1.27)) hide)
     )
@@
       (effects (font (size 1.27 1.27)) (justify left))
     )
-    (property "Value" "2kR" (id 1) (at 71.12 97.7899 0)
+    (property "Value" "160R" (id 1) (at 71.12 97.7899 0)
       (effects (font (size 1.27 1.27)) (justify left))
     )
@@
       (effects (font (size 1.27 1.27)) hide)
     )
-    (property "Datasheet" "" (id 3) (at 68.58 96.52 0)
-      (effects (font (size 1.27 1.27)) hide)
-    )
-    (property "Manufacturer Part Number" "" (id 4) (at 68.58 96.52 0)
+    (property "Datasheet" "https://datasheet.lcsc.com/lcsc/2012011712_YAGEO-AC0805FR-7W160RL_C727986.pdf" (id 3) (at 68.58 96.52 0)
+      (effects (font (size 1.27 1.27)) hide)
+    )
+    (property "Manufacturer Part Number" "AC0805FR-7W160RL" (id 4) (at 68.58 96.52 0)
       (effects (font (size 1.27 1.27)) hide)
     )
@@
       (effects (font (size 1.27 1.27)) (justify left))
     )
-    (property "Value" "2kR" (id 1) (at 59.69 97.7899 0)
+    (property "Value" "160R" (id 1) (at 59.69 97.7899 0)
       (effects (font (size 1.27 1.27)) (justify left))
     )
@@
       (effects (font (size 1.27 1.27)) hide)
     )
-    (property "Datasheet" "" (id 3) (at 57.15 96.52 0)
-      (effects (font (size 1.27 1.27)) hide)
-    )
-    (property "Manufacturer Part Number" "" (id 4) (at 57.15 96.52 0)
+    (property "Datasheet" "https://datasheet.lcsc.com/lcsc/2012011712_YAGEO-AC0805FR-7W160RL_C727986.pdf" (id 3) (at 57.15 96.52 0)
+      (effects (font (size 1.27 1.27)) hide)
+    )
+    (property "Manufacturer Part Number" "AC0805FR-7W160RL" (id 4) (at 57.15 96.52 0)
       (effects (font (size 1.27 1.27)) hide)
     )
@@
       (effects (font (size 1.27 1.27)) (justify left))
     )
-    (property "Value" "2kR" (id 1) (at 82.55 97.7899 0)
+    (property "Value" "160R" (id 1) (at 82.55 97.7899 0)
       (effects (font (size 1.27 1.27)) (justify left))
     )
@@
       (effects (font (size 1.27 1.27)) hide)
     )
-    (property "Datasheet" "" (id 3) (at 80.01 96.52 0)
-      (effects (font (size 1.27 1.27)) hide)
-    )
-    (property "Manufacturer Part Number" "" (id 4) (at 80.01 96.52 0)
+    (property "Datasheet" "https://datasheet.lcsc.com/lcsc/2012011712_YAGEO-AC0805FR-7W160RL_C727986.pdf" (id 3) (at 80.01 96.52 0)
+      (effects (font (size 1.27 1.27)) hide)
+    )
+    (property "Manufacturer Part Number" "AC0805FR-7W160RL" (id 4) (at 80.01 96.52 0)
       (effects (font (size 1.27 1.27)) hide)
     )
@@
     )
     (path "/af030468-b35e-40dd-b52a-ff480b6a45e1"
-      (reference "R20") (unit 1) (value "2kR") (footprint "Resistor_SMD:R_0805_2012Metric_Pad1.20x1.40mm_HandSolder")
+      (reference "R20") (unit 1) (value "160R") (footprint "Resistor_SMD:R_0805_2012Metric_Pad1.20x1.40mm_HandSolder")
     )
     (path "/97a2d852-dc40-453f-a9e8-417149353da6"
-      (reference "R21") (unit 1) (value "2kR") (footprint "Resistor_SMD:R_0805_2012Metric_Pad1.20x1.40mm_HandSolder")
+      (reference "R21") (unit 1) (value "160R") (footprint "Resistor_SMD:R_0805_2012Metric_Pad1.20x1.40mm_HandSolder")
     )
     (path "/ca08b440-7798-4038-9a94-d92af3d9e7d6"
-      (reference "R22") (unit 1) (value "2kR") (footprint "Resistor_SMD:R_0805_2012Metric_Pad1.20x1.40mm_HandSolder")
+      (reference "R22") (unit 1) (value "160R") (footprint "Resistor_SMD:R_0805_2012Metric_Pad1.20x1.40mm_HandSolder")
     )
     (path "/74f0889c-0f1e-4158-a775-acfe9f971699"
@@
     )
     (path "/54506a66-042e-4641-ace6-26ddfe7f6e50"
-      (reference "R27") (unit 1) (value "2kR") (footprint "Resistor_SMD:R_0805_2012Metric_Pad1.20x1.40mm_HandSolder")
+      (reference "R27") (unit 1) (value "160R") (footprint "Resistor_SMD:R_0805_2012Metric_Pad1.20x1.40mm_HandSolder")
     )
     (path "/518edd02-a1ce-47ba-afbe-e8a8a6d6a4b3"
@@
     )
     (path "/76fc3f77-ecd1-48d7-9ddd-a687270c161a"
-      (reference "R29") (unit 1) (value "100R") (footprint "Resistor_SMD:R_0805_2012Metric_Pad1.20x1.40mm_HandSolder")
+      (reference "R29") (unit 1) (value "160R") (footprint "Resistor_SMD:R_0805_2012Metric_Pad1.20x1.40mm_HandSolder")
     )
     (path "/c73baced-111c-4c74-a3ea-6e5ed0fefcd0/69f20e10-ee91-4832-8671-180c2a7654ef"

Commit message: Progressed ECAD
Parts:
- C12, C19, C20, C21, C22, C29, C30, C37, C5, C8, C9: MPN (none) -> CC0805KRX7R8BB104; Manufacturer Part Number CC0805KRX7R8BB104 -> (none)
- C23: MPN (none) -> CC0805KKX7R8BB475; Manufacturer Part Number CC0805KKX7R8BB475 -> (none)
- D1, D2, D6, D8: MPN (none) -> 17-21SYGC/S530-E3/TR8; Manufacturer Part Number 17-21SYGC/S530-E3/TR8 -> (none)
- J1, J3: MPN (none) -> PZ254-1-06-Z-8.5; Manufacturer Part Number PZ254-1-06-Z-8.5 -> (none)
- J10, J11, J12, J13, J7, J8: MPN (none) -> B2B-PH-K-S(LF)(SN); Manufacturer Part Number B2B-PH-K-S(LF)(SN) -> (none)
- J2, J4: MPN (none) -> PZ254-1-08-Z-8.5; Manufacturer Part Number PZ254-1-08-Z-8.5 -> (none)
- J6: MPN (none) -> DC-005-20A; Manufacturer Part Number DC-005-20A -> (none)
- R10, R11, R12, R13, R14, R15, R16, R17, R18, R19, R23, R24, R25, R26, R28, R9: MPN (none) -> RC0805FR-0710KL; Manufacturer Part Number RC0805FR-0710KL -> (none)
- R20, R21, R22, R27, R29: MPN (none) -> AC0805FR-7W160RL; Manufacturer Part Number AC0805FR-7W160RL -> (none)
- U10: MPN (none) -> 74HC14S14-13; Manufacturer Part Number 74HC14S14-13 -> (none)
- U11: MPN (none) -> PCA9535PW,118; Manufacturer Part Number PCA9535PW,118 -> (none)
- U12: MPN (none) -> IRM-H638J7/TR2(CLW); Manufacturer Part Number IRM-H638J7/TR2(CLW) -> (none)
- U6, U8, U9: MPN (none) -> 74HC2G08DP,125; Manufacturer Part Number 74HC2G08DP,125 -> (none)

Commit message: Progressed ECAD
Parts:
- R20, R21, R22, R27: value 160R -> 1kR; MPN AC0805FR-7W160RL -> (none)
Changed lines of the file:
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@@
       (effects (font (size 1.27 1.27)) (justify left))
     )
-    (property "Value" "160R" (id 1) (at 93.98 97.7899 0)
+    (property "Value" "1kR" (id 1) (at 93.98 97.7899 0)
       (effects (font (size 1.27 1.27)) (justify left))
     )
@@
       (effects (font (size 1.27 1.27)) hide)
     )
-    (property "Datasheet" "https://datasheet.lcsc.com/lcsc/2012011712_YAGEO-AC0805FR-7W160RL_C727986.pdf" (id 3) (at 91.44 96.52 0)
-      (effects (font (size 1.27 1.27)) hide)
-    )
-    (property "MPN" "AC0805FR-7W160RL" (id 4) (at 91.44 96.52 0)
+    (property "Datasheet" "" (id 3) (at 91.44 96.52 0)
+      (effects (font (size 1.27 1.27)) hide)
+    )
+    (property "MPN" "" (id 4) (at 91.44 96.52 0)
       (effects (font (size 1.27 1.27)) hide)
     )
@@
       (effects (font (size 1.27 1.27)) (justify left))
     )
-    (property "Value" "160R" (id 1) (at 71.12 97.7899 0)
+    (property "Value" "1kR" (id 1) (at 71.12 97.7899 0)
       (effects (font (size 1.27 1.27)) (justify left))
     )
@@
       (effects (font (size 1.27 1.27)) hide)
     )
-    (property "Datasheet" "https://datasheet.lcsc.com/lcsc/2012011712_YAGEO-AC0805FR-7W160RL_C727986.pdf" (id 3) (at 68.58 96.52 0)
-      (effects (font (size 1.27 1.27)) hide)
-    )
-    (property "MPN" "AC0805FR-7W160RL" (id 4) (at 68.58 96.52 0)
+    (property "Datasheet" "" (id 3) (at 68.58 96.52 0)
+      (effects (font (size 1.27 1.27)) hide)
+    )
+    (property "MPN" "" (id 4) (at 68.58 96.52 0)
       (effects (font (size 1.27 1.27)) hide)
     )
@@
       (effects (font (size 1.27 1.27)) (justify left))
     )
-    (property "Value" "160R" (id 1) (at 59.69 97.7899 0)
+    (property "Value" "1kR" (id 1) (at 59.69 97.7899 0)
       (effects (font (size 1.27 1.27)) (justify left))
     )
@@
       (effects (font (size 1.27 1.27)) hide)
     )
-    (property "Datasheet" "https://datasheet.lcsc.com/lcsc/2012011712_YAGEO-AC0805FR-7W160RL_C727986.pdf" (id 3) (at 57.15 96.52 0)
-      (effects (font (size 1.27 1.27)) hide)
-    )
-    (property "MPN" "AC0805FR-7W160RL" (id 4) (at 57.15 96.52 0)
+    (property "Datasheet" "" (id 3) (at 57.15 96.52 0)
+      (effects (font (size 1.27 1.27)) hide)
+    )
+    (property "MPN" "" (id 4) (at 57.15 96.52 0)
       (effects (font (size 1.27 1.27)) hide)
     )
@@
       (effects (font (size 1.27 1.27)) (justify left))
     )
-    (property "Value" "160R" (id 1) (at 82.55 97.7899 0)
+    (property "Value" "1kR" (id 1) (at 82.55 97.7899 0)
       (effects (font (size 1.27 1.27)) (justify left))
     )
@@
       (effects (font (size 1.27 1.27)) hide)
     )
-    (property "Datasheet" "https://datasheet.lcsc.com/lcsc/2012011712_YAGEO-AC0805FR-7W160RL_C727986.pdf" (id 3) (at 80.01 96.52 0)
-      (effects (font (size 1.27 1.27)) hide)
-    )
-    (property "MPN" "AC0805FR-7W160RL" (id 4) (at 80.01 96.52 0)
+    (property "Datasheet" "" (id 3) (at 80.01 96.52 0)
+      (effects (font (size 1.27 1.27)) hide)
+    )
+    (property "MPN" "" (id 4) (at 80.01 96.52 0)
       (effects (font (size 1.27 1.27)) hide)
     )
@@
     )
     (path "/af030468-b35e-40dd-b52a-ff480b6a45e1"
-      (reference "R20") (unit 1) (value "160R") (footprint "Resistor_SMD:R_0805_2012Metric_Pad1.20x1.40mm_HandSolder")
+      (reference "R20") (unit 1) (value "1kR") (footprint "Resistor_SMD:R_0805_2012Metric_Pad1.20x1.40mm_HandSolder")
     )
     (path "/97a2d852-dc40-453f-a9e8-417149353da6"
-      (reference "R21") (unit 1) (value "160R") (footprint "Resistor_SMD:R_0805_2012Metric_Pad1.20x1.40mm_HandSolder")
+      (reference "R21") (unit 1) (value "1kR") (footprint "Resistor_SMD:R_0805_2012Metric_Pad1.20x1.40mm_HandSolder")
     )
     (path "/ca08b440-7798-4038-9a94-d92af3d9e7d6"
-      (reference "R22") (unit 1) (value "160R") (footprint "Resistor_SMD:R_0805_2012Metric_Pad1.20x1.40mm_HandSolder")
+      (reference "R22") (unit 1) (value "1kR") (footprint "Resistor_SMD:R_0805_2012Metric_Pad1.20x1.40mm_HandSolder")
     )
     (path "/74f0889c-0f1e-4158-a775-acfe9f971699"
@@
     )
     (path "/54506a66-042e-4641-ace6-26ddfe7f6e50"
-      (reference "R27") (unit 1) (value "160R") (footprint "Resistor_SMD:R_0805_2012Metric_Pad1.20x1.40mm_HandSolder")
+      (reference "R27") (unit 1) (value "1kR") (footprint "Resistor_SMD:R_0805_2012Metric_Pad1.20x1.40mm_HandSolder")
     )
     (path "/518edd02-a1ce-47ba-afbe-e8a8a6d6a4b3"

Commit message: Progressed ECAD
Parts:
- R20, R21, R22, R27: MPN (none) -> AC0805FR-7W1KL
Changed lines of the file:
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@@
       (effects (font (size 1.27 1.27)) hide)
     )
-    (property "Datasheet" "" (id 3) (at 91.44 96.52 0)
-      (effects (font (size 1.27 1.27)) hide)
-    )
-    (property "MPN" "" (id 4) (at 91.44 96.52 0)
+    (property "Datasheet" "https://datasheet.lcsc.com/lcsc/2010202005_YAGEO-AC0805FR-7W1KL_C727989.pdf" (id 3) (at 91.44 96.52 0)
+      (effects (font (size 1.27 1.27)) hide)
+    )
+    (property "MPN" "AC0805FR-7W1KL" (id 4) (at 91.44 96.52 0)
       (effects (font (size 1.27 1.27)) hide)
     )
@@
       (effects (font (size 1.27 1.27)) hide)
     )
-    (property "Datasheet" "" (id 3) (at 68.58 96.52 0)
-      (effects (font (size 1.27 1.27)) hide)
-    )
-    (property "MPN" "" (id 4) (at 68.58 96.52 0)
+    (property "Datasheet" "https://datasheet.lcsc.com/lcsc/2010202005_YAGEO-AC0805FR-7W1KL_C727989.pdf" (id 3) (at 68.58 96.52 0)
+      (effects (font (size 1.27 1.27)) hide)
+    )
+    (property "MPN" "AC0805FR-7W1KL" (id 4) (at 68.58 96.52 0)
       (effects (font (size 1.27 1.27)) hide)
     )
@@
       (effects (font (size 1.27 1.27)) hide)
     )
-    (property "Datasheet" "" (id 3) (at 57.15 96.52 0)
-      (effects (font (size 1.27 1.27)) hide)
-    )
-    (property "MPN" "" (id 4) (at 57.15 96.52 0)
+    (property "Datasheet" "https://datasheet.lcsc.com/lcsc/2010202005_YAGEO-AC0805FR-7W1KL_C727989.pdf" (id 3) (at 57.15 96.52 0)
+      (effects (font (size 1.27 1.27)) hide)
+    )
+    (property "MPN" "AC0805FR-7W1KL" (id 4) (at 57.15 96.52 0)
       (effects (font (size 1.27 1.27)) hide)
     )
@@
       (effects (font (size 1.27 1.27)) hide)
     )
-    (property "Datasheet" "" (id 3) (at 80.01 96.52 0)
-      (effects (font (size 1.27 1.27)) hide)
-    )
-    (property "MPN" "" (id 4) (at 80.01 96.52 0)
-      (effects (font (size 1.27 1.27)) hide)
-    )
+    (property "Datasheet" "https://datasheet.lcsc.com/lcsc/2010202005_YAGEO-AC0805FR-7W1KL_C727989.pdf" (id 3) (at 80.01 96.52 0)
+      (effects (font (size 1.27 1.27)) hide)
+    )
+    (property "MPN" "AC0805FR-7W1KL" (id 4) (at 80.01 96.52 0)
+      (effects (font (size 1.27 1.27)) hide)
+    )
