File: Tester/ECAD/BDCMotorControlShield/BDCMotorControlShield.kicad_pcb (KiCad board)
At the start: 4 copper layers, 68.6 x 53.3 mm, 98 parts, among them J1 Power, J10 Limit switch, J11 Limit switch, J12 Limit switch, J13 Limit switch, J14 Motor connector, J2 Digital/PWM, J3 Analog, J4 Digital/PWM, J5 Motor connector, J6 Barrel_Jack_Switch, J7 Limit switch, J8 Limit switch, J9 Motor connector, U1 DRV8870DDA, U10 74HC14, U11 PCA9535PW, U12 IRM-H6XX, U2 INA180A1, U3 DRV8870DDA, U4 DRV8870DDA, U5 INA180A1, U6 74HC2G08, U7 INA180A1, U8 74HC2G08, U9 74HC2G08

Commit message: Progressed ECAD
Parts:
- moved R28 0.25 mm to (111.5, 54.5)
Connections:
- U2 pad 1: /A0 -> /A1
- U5 pad 1: /A1 -> /A2
- U7 pad 1: /A2 -> /A0
Routing:
- net GND: track 0.00 -> 14.5 mm
- net /H-bridge #3/PWM2: track 0.00 -> 6.97 mm
- net /H-bridge #1/PWM2: track 0.00 -> 6.97 mm
- net /H-bridge #2/PWM2: track 0.00 -> 6.80 mm
- net +5V: track 0.00 -> 6.76 mm
- net Net-(C18-Pad1): track 0.00 -> 6.59 mm
- net Net-(C15-Pad1): track 0.00 -> 6.59 mm
- net Net-(C16-Pad1): track 0.00 -> 6.59 mm
- net Net-(C23-Pad1): track 0.00 -> 5.98 mm
- net Net-(R30-Pad2): track 0.00 -> 5.90 mm
- net Net-(R1-Pad2): track 0.00 -> 5.76 mm
- net Net-(R6-Pad2): track 0.00 -> 5.70 mm
- net /H-bridge #3/PWM1: track 0.00 -> 5.37 mm
- net /H-bridge #1/PWM1: track 0.00 -> 5.37 mm
- net /H-bridge #2/PWM1: track 0.00 -> 5.17 mm
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- added copper zone on F.Cu, net Net-(R1-Pad2)
- added copper zone on F.Cu, net Net-(R30-Pad2)
- added copper zone on F.Cu, net Net-(R6-Pad2)

Commit message: Progressed ECAD
Routing:
- net Net-(C30-Pad1): track 0.00 -> 2.02 mm
Changed lines of the file:
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@@
   (segment (start 151.75 90.0375) (end 151.7125 90) (width 0.25) (layer "B.Cu") (net 40))
   (segment (start 151.75 92) (end 151.75 90.0375) (width 0.25) (layer "B.Cu") (net 40))
+  (segment (start 131.25 86.9625) (end 133.2125 86.9625) (width 0.25) (layer "B.Cu") (net 41))
+  (segment (start 133.2125 86.9625) (end 133.25 86.925) (width 0.25) (layer "B.Cu") (net 41))
   (segment (start 121.75 92) (end 121.75 90.0375) (width 0.25) (layer "B.Cu") (net 42))
   (segment (start 121.75 90.0375) (end 121.7125 90) (width 0.25) (layer "B.Cu") (net 42))
@@
   (segment (start 127.6 55.525) (end 126.85 55.525) (width 0.25) (layer "F.Cu") (net 60))
   (zone (net 46) (net_name "Net-(R1-Pad2)") (layer "F.Cu") (hatch edge 0.508)
+    (priority 1)
     (connect_pads (clearance 0.508))
     (min_thickness 0.254) (filled_areas_thickness no)
@@
   )
   (zone (net 28) (net_name "+12V") (layer "F.Cu") (hatch edge 0.508)
+    (priority 1)
     (connect_pads yes (clearance 0.508))
     (min_thickness 0.254) (filled_areas_thickness no)
@@
   )
   (zone (net 28) (net_name "+12V") (layer "F.Cu") (hatch edge 0.508)
+    (priority 1)
     (connect_pads yes (clearance 0.508))
     (min_thickness 0.254) (filled_areas_thickness no)
@@
     )
   )
+  (zone (net 1) (net_name "GND") (layers F&B.Cu) (hatch edge 0.508)
+    (connect_pads (clearance 0.508))
+    (min_thickness 0.254) (filled_areas_thickness no)
+    (fill yes (thermal_gap 0.508) (thermal_bridge_width 0.508))
+    (polygon
+      (pts
+        (xy 169 101)
+        (xy 99 101)
+        (xy 99 46)
+        (xy 169 46)
+      )
+    )
+  )
   (zone (net 28) (net_name "+12V") (layer "F.Cu") (hatch edge 0.508)
+    (priority 1)
     (connect_pads yes (clearance 0.508))
     (min_thickness 0.254) (filled_areas_thickness no)
@@
   )
   (zone (net 49) (net_name "Net-(R6-Pad2)") (layer "F.Cu") (hatch edge 0.508)
+    (priority 1)
     (connect_pads (clearance 0.508))
     (min_thickness 0.254) (filled_areas_thickness no)
@@
   )
   (zone (net 53) (net_name "Net-(R30-Pad2)") (layer "F.Cu") (hatch edge 0.508)
+    (priority 1)
     (connect_pads (clearance 0.508))
     (min_thickness 0.254) (filled_areas_thickness no)
@@
       )
     )
-  )
-  (zone (net 1) (net_name "GND") (layer "B.Cu") (hatch edge 0.508)
-    (connect_pads (clearance 0.508))
-    (min_thickness 0.254) (filled_areas_thickness no)
-    (fill yes (thermal_gap 0.508) (thermal_bridge_width 0.508))
-    (polygon
-      (pts
-        (xy 169 101)
-        (xy 99 101)
-        (xy 99 46)
-        (xy 169 46)
-      )
-    )

Commit message: Progressed ECAD
Routing:
- net /A2: track 0.00 -> 32.3 mm
- net GND: track 14.5 -> 24.5 mm, vias 34 -> 52
- net /2: track 0.00 -> 5.11 mm
- net /7: track 0.00 -> 5.11 mm
- net /12: track 0.00 -> 5.11 mm
- net Net-(R6-Pad2): track 5.70 -> 10.3 mm
- net Net-(R1-Pad2): track 5.76 -> 10.3 mm
- net Net-(R30-Pad2): track 5.90 -> 10.3 mm
- net /H-bridge #3/PWM2: track 6.97 -> 9.32 mm
- net /H-bridge #2/PWM2: track 6.80 -> 9.02 mm
- net /H-bridge #1/PWM2: track 6.97 -> 9.13 mm

Commit message: Progressed ECAD
Parts:
- moved R20 2.25 mm to (110.0, 74.0)
- moved R21 2.25 mm to (110.0, 72.0)
- moved R22 2.25 mm to (110.0, 70.0)
- moved R27 2.25 mm to (110.0, 68.0)
- moved C29 0.50 mm to (152.8, 89.5)
- moved C37 0.50 mm to (122.8, 89.5)
- moved C8 0.50 mm to (137.8, 89.5)
- moved R11 0.50 mm to (137.8, 91.5)
- moved R14 0.50 mm to (152.8, 91.5)
- moved R16 0.50 mm to (122.8, 91.5)
- moved R17 0.50 mm to (137.8, 93.5)
- moved R24 0.50 mm to (152.8, 93.5)
- moved R26 0.50 mm to (122.8, 93.5)
- moved C12 0.25 mm to (163.0, 88.0)
- moved C30 0.25 mm to (133.0, 88.0)
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Connections:
- U10 pad 10: /LIM_SW04 -> /LIM_SW01
- U10 pad 11: Net-(C30-Pad1) -> Net-(C9-Pad1)
- U10 pad 12: /LIM_SW05 -> /LIM_SW04
- U10 pad 13: Net-(C37-Pad1) -> Net-(C30-Pad1)
- U10 pad 3: Net-(C9-Pad1) -> Net-(C37-Pad1)
- U10 pad 4: /LIM_SW01 -> /LIM_SW05
Routing:
- net Net-(C12-Pad1): track 2.02 -> 79.7 mm, vias 0 -> 1
- net Net-(C9-Pad1): track 2.02 -> 58.2 mm, vias 0 -> 1
- net Net-(C29-Pad1): track 2.02 -> 57.2 mm, vias 0 -> 1
- net Net-(C8-Pad1): track 2.02 -> 41.5 mm, vias 0 -> 1
- net Net-(C30-Pad1): track 2.02 -> 27.9 mm, vias 0 -> 1
- net Net-(C37-Pad1): track 2.02 -> 26.6 mm, vias 0 -> 1
- net +5V: track 6.76 -> 8.51 mm, vias 0 -> 1
- net /12: track 5.11 -> 5.91 mm
- net /7: track 5.11 -> 5.91 mm
- net /2: track 5.11 -> 5.91 mm
- net Net-(J12-Pad2): track 4.56 -> 5.30 mm
- net Net-(J8-Pad2): track 4.61 -> 5.22 mm
- net Net-(J10-Pad2): track 4.66 -> 5.27 mm
- net GND: vias 52 -> 63

Commit message: Update BDCMotorControlShield.kicad_pcb
Parts:
- moved R20 18.4 mm to (93.2, 81.4)
- moved R27 18.4 mm to (92.0, 71.6)
- moved R22 18.2 mm to (92.4, 74.6)
- moved R21 18.0 mm to (93.0, 77.8)
Routing:
- net /LIM_SW02: track 0.00 -> 25.8 mm, vias 0 -> 2
- net /LIM_SW03: track 0.00 -> 23.4 mm, vias 0 -> 1
- net /LIM_SW05: track 0.00 -> 18.6 mm, vias 0 -> 2
- net /LIM_SW01: track 0.00 -> 18.6 mm, vias 0 -> 1
- net /LIM_SW04: track 0.00 -> 18.4 mm, vias 0 -> 1
- net /LIM_SW00: track 0.00 -> 16.2 mm, vias 0 -> 2
Changed lines of the file:
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@@
   )
   (footprint "Resistor_SMD:R_0805_2012Metric_Pad1.20x1.40mm_HandSolder" (layer "B.Cu")
-    (at 110 72 180)
+    (at 93 77.8 180)
     (descr "Resistor SMD 0805 (2012 Metric), square (rectangular) end terminal, IPC_7351 nominal with elongated pad for handsoldering. (Body size source: IPC-SM-782 page 72, https://www.pcb-3d.com/wordpress/wp-content/uploads/ipc-sm-782a_amendment_1_and_2.pdf), generated with kicad-footprint-generator")
     (tags "resistor handsolder")
@@
   )
   (footprint "Resistor_SMD:R_0805_2012Metric_Pad1.20x1.40mm_HandSolder" (layer "B.Cu")
-    (at 110 74 180)
+    (at 93.2 81.4 180)
     (descr "Resistor SMD 0805 (2012 Metric), square (rectangular) end terminal, IPC_7351 nominal with elongated pad for handsoldering. (Body size source: IPC-SM-782 page 72, https://www.pcb-3d.com/wordpress/wp-content/uploads/ipc-sm-782a_amendment_1_and_2.pdf), generated with kicad-footprint-generator")
     (tags "resistor handsolder")
@@
   )
   (footprint "Resistor_SMD:R_0805_2012Metric_Pad1.20x1.40mm_HandSolder" (layer "B.Cu")
-    (at 110 68 180)
+    (at 92 71.6 180)
     (descr "Resistor SMD 0805 (2012 Metric), square (rectangular) end terminal, IPC_7351 nominal with elongated pad for handsoldering. (Body size source: IPC-SM-782 page 72, https://www.pcb-3d.com/wordpress/wp-content/uploads/ipc-sm-782a_amendment_1_and_2.pdf), generated with kicad-footprint-generator")
     (tags "resistor handsolder")
@@
   )
   (footprint "Resistor_SMD:R_0805_2012Metric_Pad1.20x1.40mm_HandSolder" (layer "B.Cu")
-    (at 110 70 180)
+    (at 92.4 74.6 180)
     (descr "Resistor SMD 0805 (2012 Metric), square (rectangular) end terminal, IPC_7351 nominal with elongated pad for handsoldering. (Body size source: IPC-SM-782 page 72, https://www.pcb-3d.com/wordpress/wp-content/uploads/ipc-sm-782a_amendment_1_and_2.pdf), generated with kicad-footprint-generator")
     (tags "resistor handsolder")
@@
   (segment (start 127.365 58.135) (end 127.75 57.75) (width 0.25) (layer "F.Cu") (net 60))
   (segment (start 127.6 55.525) (end 126.85 55.525) (width 0.25) (layer "F.Cu") (net 60))
+  (segment (start 109.1 72.2) (end 107.6 73.7) (width 0.25) (layer "F.Cu") (net 69))
+  (segment (start 107.6 73.7) (end 107.6 76.4) (width 0.25) (layer "F.Cu") (net 69))
+  (segment (start 117.775134 65.4985) (end 117.3145 65.4985) (width 0.25) (layer "F.Cu") (net 69))
+  (segment (start 107.6 76.4) (end 108.16 76.96) (width 0.25) (layer "F.Cu") (net 69))
+  (segment (start 117.3145 65.4985) (end 116.941 65.125) (width 0.25) (layer "F.Cu") (net 69))
+  (segment (start 108.16 76.96) (end 110.525 76.96) (width 0.25) (layer "F.Cu") (net 69))
+  (segment (start 112.2 72.2) (end 109.1 72.2) (width 0.25) (layer "F.Cu") (net 69))
+  (segment (start 116.941 65.125) (end 115.8625 65.125) (width 0.25) (layer "F.Cu") (net 69))
+  (via (at 117.775134 65.4985) (size 0.8) (drill 0.4) (layers "F.Cu" "B.Cu") (net 69))
+  (via (at 112.2 72.2) (size 0.8) (drill 0.4) (layers "F.Cu" "B.Cu") (net 69))
+  (segment (start 117.775134 65.4985) (end 117.775134 68.575134) (width 0.25) (layer "B.Cu") (net 69))
+  (segment (start 119 79.6) (end 119 75.8) (width 0.25) (layer "F.Cu") (net 70))
+  (segment (start 118.415 64.694) (end 117.399 64.694) (width 0.25) (layer "F.Cu") (net 70))
+  (segment (start 117.8 74.6) (end 117.8 72.2) (width 0.25) (layer "F.Cu") (net 70))
+  (segment (start 117.83 80.77) (end 119 79.6) (width 0.25) (layer "F.Cu") (net 70))
+  (segment (start 117.399 64.694) (end 117.18 64.475) (width 0.25) (layer "F.Cu") (net 70))
+  (segment (start 117.18 64.475) (end 115.8625 64.475) (width 0.25) (layer "F.Cu") (net 70))
+  (segment (start 119 75.8) (end 117.8 74.6) (width 0.25) (layer "F.Cu") (net 70))
+  (segment (start 115.475 80.77) (end 117.83 80.77) (width 0.25) (layer "F.Cu") (net 70))
+  (via (at 118.415 64.694) (size 0.8) (drill 0.4) (layers "F.Cu" "B.Cu") (net 70))
+  (segment (start 118.6 65.4) (end 118.6 66) (width 0.25) (layer "B.Cu") (net 70))
+  (segment (start 118.6 64.879) (end 118.6 65.4) (width 0.25) (layer "B.Cu") (net 70))
+  (segment (start 118.415 64.694) (end 118.6 64.879) (width 0.25) (layer "B.Cu") (net 70))
+  (segment (start 118.4 66.2) (end 118.4 68.6) (width 0.25) (layer "B.Cu") (net 70))
+  (segment (start 118.6 66) (end 118.4 66.2) (width 0.25) (layer "B.Cu") (net 70))
+  (segment (start 108.24 82.04) (end 106.4 80.2) (width 0.25) (layer "F.Cu") (net 71))
+  (segment (start 117.7055 63.825) (end 115.8625 63.825) (width 0.25) (layer "F.Cu") (net 71))
+  (segment (start 110.525 82.04) (end 108.24 82.04) (width 0.25) (layer "F.Cu") (net 71))
+  (segment (start 108.9 70.6) (end 112.2 70.6) (width 0.25) (layer "F.Cu") (net 71))
+  (segment (start 106.4 73.1) (end 108.9 70.6) (width 0.25) (layer "F.Cu") (net 71))
+  (segment (start 117.78 63.8995) (end 117.7055 63.825) (width 0.25) (layer "F.Cu") (net 71))
+  (segment (start 106.4 80.2) (end 106.4 73.1) (width 0.25) (layer "F.Cu") (net 71))
+  (via (at 117.78 63.8995) (size 0.8) (drill 0.4) (layers "F.Cu" "B.Cu") (net 71))
+  (via (at 112.2 70.6) (size 0.8) (drill 0.4) (layers "F.Cu" "B.Cu") (net 71))
+  (segment (start 117.78 63.8995) (end 117 64.6795) (width 0.25) (layer "B.Cu") (net 71))
+  (segment (start 117 66.2) (end 117 68.6) (width 0.25) (layer "B.Cu") (net 71))
+  (segment (start 117 64.6795) (end 117 66.2) (width 0.25) (layer "B.Cu") (net 71))
+  (segment (start 118.415 63.043) (end 118.283 63.175) (width 0.25) (layer "F.Cu") (net 72))
+  (segment (start 119.6 81.6) (end 119.6 74.8) (width 0.25) (layer "F.Cu") (net 72))
+  (segment (start 118.283 63.175) (end 115.8625 63.175) (width 0.25) (layer "F.Cu") (net 72))
+  (segment (start 117.89 83.31) (end 119.6 81.6) (width 0.25) (layer "F.Cu") (net 72))
+  (segment (start 115.475 83.31) (end 117.89 83.31) (width 0.25) (layer "F.Cu") (net 72))
+  (segment (start 119.6 74.8) (end 118.6 73.8) (width 0.25) (layer "F.Cu") (net 72))
+  (segment (start 118.6 73.8) (end 118.6 72) (width 0.25) (layer "F.Cu") (net 72))
+  (via (at 118.415 63.043) (size 0.8) (drill 0.4) (layers "F.Cu" "B.Cu") (net 72))
+  (segment (start 119.2 63.828) (end 119.2 66.4) (width 0.25) (layer "B.Cu") (net 72))
+  (segment (start 119.2 66.4) (end 119 66.6) (width 0.25) (layer "B.Cu") (net 72))
+  (segment (start 119 66.6) (end 119 68.6) (width 0.25) (layer "B.Cu") (net 72))
+  (segment (start 118.415 63.043) (end 119.2 63.828) (width 0.25) (layer "B.Cu") (net 72))
+  (segment (start 117 75) (end 117 72) (width 0.25) (layer "F.Cu") (net 73))
+  (segment (start 115.475 78.23) (end 117.77 78.23) (width 0.25) (layer "F.Cu") (net 73))
+  (segment (start 117.379602 62.525) (end 115.8625 62.525) (width 0.25) (layer "F.Cu") (net 73))
+  (segment (start 118.4 77.6) (end 118.4 76.4) (width 0.25) (layer "F.Cu") (net 73))
+  (segment (start 117.758733 62.145869) (end 117.379602 62.525) (width 0.25) (layer "F.Cu") (net 73))
+  (segment (start 117.77 78.23) (end 118.4 77.6) (width 0.25) (layer "F.Cu") (net 73))
+  (segment (start 118.4 76.4) (end 117 75) (width 0.25) (layer "F.Cu") (net 73))
+  (via (at 117.758733 62.145869) (size 0.8) (drill 0.4) (layers "F.Cu" "B.Cu") (net 73))
+  (segment (start 116.4 63.504602) (end 116.4 68.6) (width 0.25) (layer "B.Cu") (net 73))
+  (segment (start 117.758733 62.145869) (end 116.4 63.504602) (width 0.25) (layer "B.Cu") (net 73))
+  (segment (start 108.3 79.5) (end 107 78.2) (width 0.25) (layer "F.Cu") (net 74))
+  (segment (start 118.415 61.392) (end 117.399 61.392) (width 0.25) (layer "F.Cu") (net 74))
+  (segment (start 107 78.2) (end 107 73.4) (width 0.25) (layer "F.Cu") (net 74))
+  (segment (start 117.399 61.392) (end 116.916 61.875) (width 0.25) (layer "F.Cu") (net 74))
+  (segment (start 116.916 61.875) (end 115.8625 61.875) (width 0.25) (layer "F.Cu") (net 74))
+  (segment (start 110.525 79.5) (end 108.3 79.5) (width 0.25) (layer "F.Cu") (net 74))
+  (segment (start 107 73.4) (end 109 71.4) (width 0.25) (layer "F.Cu") (net 74))
+  (segment (start 109 71.4) (end 113.2 71.4) (width 0.25) (layer "F.Cu") (net 74))
+  (via (at 118.415 61.392) (size 0.8) (drill 0.4) (layers "F.Cu" "B.Cu") (net 74))
+  (via (at 113.2 71.4) (size 0.8) (drill 0.4) (layers "F.Cu" "B.Cu") (net 74))
   (zone (net 46) (net_name "Net-(R1-Pad2)") (layer "F.Cu") (hatch edge 0.508)
     (priority 1)

Commit message: Update BDCMotorControlShield.kicad_pcb
Routing:
- net /LIM_SW05: track 18.6 -> 32.7 mm
- net /LIM_SW00: track 16.2 -> 23.5 mm
- net /LIM_SW04: track 18.4 -> 24.9 mm, vias 1 -> 2
- net /LIM_SW02: track 25.8 -> 31.4 mm
- net /LIM_SW01: track 18.6 -> 23.1 mm, vias 1 -> 2
- net /LIM_SW03: track 23.4 -> 27.7 mm, vias 1 -> 2

Commit message: Update BDCMotorControlShield.kicad_pcb
Parts:
- moved R27 12.5 mm to (104.5, 70.5), turned to 90 degrees
- moved R22 12.1 mm to (104.5, 74.5), turned to 90 degrees
- moved R21 11.5 mm to (104.5, 78.5), turned to 90 degrees
- moved R20 11.4 mm to (104.5, 82.5), turned to 90 degrees
- moved R10 2.00 mm to (113.0, 65.5)
- moved R19 2.00 mm to (113.0, 63.5)
Routing:
- net GND: track 24.5 -> 43.5 mm
- net /13: track 0.00 -> 8.34 mm, vias 0 -> 1
- net /SCL/A5: track 0.00 -> 6.28 mm, vias 0 -> 1
- net /SDA/A4: track 0.00 -> 5.87 mm, vias 0 -> 1
- net +5V: track 8.51 -> 11.8 mm

Commit message: Update BDCMotorControlShield.kicad_pcb
Parts:
- moved R20 2.30 mm to (106.8, 83.0)
- moved R21 2.30 mm to (106.8, 79.0)
- moved R22 2.30 mm to (106.8, 75.0)
- moved R27 2.30 mm to (106.8, 71.0)
Changed lines of the file:
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@@
   )
   (footprint "Resistor_SMD:R_0805_2012Metric_Pad1.20x1.40mm_HandSolder" (layer "B.Cu")
-    (at 104.5 78.5 90)
+    (at 106.75 79 90)
     (descr "Resistor SMD 0805 (2012 Metric), square (rectangular) end terminal, IPC_7351 nominal with elongated pad for handsoldering. (Body size source: IPC-SM-782 page 72, https://www.pcb-3d.com/wordpress/wp-content/uploads/ipc-sm-782a_amendment_1_and_2.pdf), generated with kicad-footprint-generator")
     (tags "resistor handsolder")
@@
   )
   (footprint "Resistor_SMD:R_0805_2012Metric_Pad1.20x1.40mm_HandSolder" (layer "B.Cu")
-    (at 104.5 82.5 90)
+    (at 106.75 83 90)
     (descr "Resistor SMD 0805 (2012 Metric), square (rectangular) end terminal, IPC_7351 nominal with elongated pad for handsoldering. (Body size source: IPC-SM-782 page 72, https://www.pcb-3d.com/wordpress/wp-content/uploads/ipc-sm-782a_amendment_1_and_2.pdf), generated with kicad-footprint-generator")
     (tags "resistor handsolder")
@@
   )
   (footprint "Resistor_SMD:R_0805_2012Metric_Pad1.20x1.40mm_HandSolder" (layer "B.Cu")
-    (at 104.5 70.5 90)
+    (at 106.75 71 90)
     (descr "Resistor SMD 0805 (2012 Metric), square (rectangular) end terminal, IPC_7351 nominal with elongated pad for handsoldering. (Body size source: IPC-SM-782 page 72, https://www.pcb-3d.com/wordpress/wp-content/uploads/ipc-sm-782a_amendment_1_and_2.pdf), generated with kicad-footprint-generator")
     (tags "resistor handsolder")
@@
   )
   (footprint "Resistor_SMD:R_0805_2012Metric_Pad1.20x1.40mm_HandSolder" (layer "B.Cu")
-    (at 104.5 74.5 90)
-    (descr "Resistor SMD 0805 (2012 Metric), square (rectangular) end terminal, IPC_7351 nominal with elongated pad for handsoldering. (Body size source: IPC-SM-782 page 72, https://www.pcb-3d.com/wordpress/wp-content/uploads/ipc-sm-782a_amendment_1_and_2.pdf), generated with kicad-footprint-generator")
-    (tags "resistor handsolder")
+    (at 106.75 75 90)
+    (descr "Resistor SMD 0805 (2012 Metric), square (rectangular) end terminal, IPC_7351 nominal with elongated pad for handsoldering. (Body size source: IPC-SM-782 page 72, https://www.pcb-3d.com/wordpress/wp-content/uploads/ipc-sm-782a_amendment_1_and_2.pdf), generated with kicad-footprint-generator")
+    (tags "resistor handsolder")
