File: Tester/ECAD/LimitSwitchBoard/LimitSwitchBoard.kicad_pcb (KiCad board)
At the start: 2 copper layers, 18.5 x 23 mm, 3 parts, among them J1 Conn_01x03, SW1 SW_SPDT

Commit message: Final version for production
Parts:
- J1: footprint Connector_PinHeader_2.54mm:PinHeader_1x03_P2.54mm_Vertical -> Connector_PinSocket_2.00mm:PinSocket_1x03_P2.00mm_Vertical
- moved J1 2.55 mm to (136.0, 72.0)
Routing:
- net Net-(J1-Pad3): track 16.6 -> 18.1 mm
- net Net-(J1-Pad1): track 4.35 -> 5.03 mm
- added copper zone on B.Cu, net (none)
- added copper zone on F.Cu, net (none)
Changed lines of the file:
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@@
   (net 2 "Net-(J1-Pad1)")
   (net 3 "Net-(J1-Pad2)")
-  (footprint "Connector_PinHeader_2.54mm:PinHeader_1x03_P2.54mm_Vertical" (layer "F.Cu")
-    (at 136.5 69.5)
-    (descr "Through hole straight pin header, 1x03, 2.54mm pitch, single row")
-    (tags "Through hole pin header THT 1x03 2.54mm single row")
-    (property "Sheetfile" "Limit_Switch_Board_Simple.kicad_sch")
+  (footprint "Connector_PinSocket_2.00mm:PinSocket_1x03_P2.00mm_Vertical" (layer "F.Cu")
+    (at 136 72)
+    (descr "Through hole straight socket strip, 1x03, 2.00mm pitch, single row (from Kicad 4.0.7), script generated")
+    (tags "Through hole socket strip THT 1x03 2.00mm single row")
+    (property "Sheetfile" "LimitSwitchBoard.kicad_sch")
     (property "Sheetname" "")
     (attr through_hole)
-    (fp_text reference "J1" (at 0 -2.33) (layer "F.SilkS")
+    (fp_text reference "J1" (at 0 -2.5) (layer "F.SilkS")
       (effects (font (size 1 1) (thickness 0.15)))
     )
-    (fp_text value "Conn_01x03" (at 0 7.41) (layer "F.Fab")
+    (fp_text value "Conn_01x03" (at 0 6.5) (layer "F.Fab")
       (effects (font (size 1 1) (thickness 0.15)))
     )
-    (fp_text user "${REFERENCE}" (at 0 2.54 90) (layer "F.Fab")
+    (fp_text user "${REFERENCE}" (at 0 2 90) (layer "F.Fab")
       (effects (font (size 1 1) (thickness 0.15)))
     )
-    (fp_line (start 1.33 1.27) (end 1.33 6.41) (layer "F.SilkS") (width 0.12))
-    (fp_line (start -1.33 0) (end -1.33 -1.33) (layer "F.SilkS") (width 0.12))
-    (fp_line (start -1.33 1.27) (end -1.33 6.41) (layer "F.SilkS") (width 0.12))
-    (fp_line (start -1.33 -1.33) (end 0 -1.33) (layer "F.SilkS") (width 0.12))
-    (fp_line (start -1.33 1.27) (end 1.33 1.27) (layer "F.SilkS") (width 0.12))
-    (fp_line (start -1.33 6.41) (end 1.33 6.41) (layer "F.SilkS") (width 0.12))
-    (fp_line (start -1.8 -1.8) (end -1.8 6.85) (layer "F.CrtYd") (width 0.05))
-    (fp_line (start 1.8 6.85) (end 1.8 -1.8) (layer "F.CrtYd") (width 0.05))
-    (fp_line (start -1.8 6.85) (end 1.8 6.85) (layer "F.CrtYd") (width 0.05))
-    (fp_line (start 1.8 -1.8) (end -1.8 -1.8) (layer "F.CrtYd") (width 0.05))
-    (fp_line (start -0.635 -1.27) (end 1.27 -1.27) (layer "F.Fab") (width 0.1))
-    (fp_line (start -1.27 -0.635) (end -0.635 -1.27) (layer "F.Fab") (width 0.1))
-    (fp_line (start -1.27 6.35) (end -1.27 -0.635) (layer "F.Fab") (width 0.1))
-    (fp_line (start 1.27 -1.27) (end 1.27 6.35) (layer "F.Fab") (width 0.1))
-    (fp_line (start 1.27 6.35) (end -1.27 6.35) (layer "F.Fab") (width 0.1))
-    (pad "1" thru_hole rect (at 0 0) (size 1.7 1.7) (drill 1) (layers *.Cu *.Mask)
+    (fp_line (start 1.06 -1.06) (end 1.06 0) (layer "F.SilkS") (width 0.12))
+    (fp_line (start 0 -1.06) (end 1.06 -1.06) (layer "F.SilkS") (width 0.12))
+    (fp_line (start 1.06 1) (end 1.06 5.06) (layer "F.SilkS") (width 0.12))
+    (fp_line (start -1.06 5.06) (end 1.06 5.06) (layer "F.SilkS") (width 0.12))
+    (fp_line (start -1.06 1) (end 1.06 1) (layer "F.SilkS") (width 0.12))
+    (fp_line (start -1.06 1) (end -1.06 5.06) (layer "F.SilkS") (width 0.12))
+    (fp_line (start 1.5 -1.5) (end 1.5 5.5) (layer "F.CrtYd") (width 0.05))
+    (fp_line (start -1.5 -1.5) (end 1.5 -1.5) (layer "F.CrtYd") (width 0.05))
+    (fp_line (start -1.5 5.5) (end -1.5 -1.5) (layer "F.CrtYd") (width 0.05))
+    (fp_line (start 1.5 5.5) (end -1.5 5.5) (layer "F.CrtYd") (width 0.05))
+    (fp_line (start 0.5 -1) (end 1 -0.5) (layer "F.Fab") (width 0.1))
+    (fp_line (start 1 5) (end -1 5) (layer "F.Fab") (width 0.1))
+    (fp_line (start -1 5) (end -1 -1) (layer "F.Fab") (width 0.1))
+    (fp_line (start -1 -1) (end 0.5 -1) (layer "F.Fab") (width 0.1))
+    (fp_line (start 1 -0.5) (end 1 5) (layer "F.Fab") (width 0.1))
+    (pad "1" thru_hole rect (at 0 0) (size 1.35 1.35) (drill 0.8) (layers *.Cu *.Mask)
       (net 2 "Net-(J1-Pad1)") (pinfunction "Pin_1") (pintype "passive"))
-    (pad "2" thru_hole oval (at 0 2.54) (size 1.7 1.7) (drill 1) (layers *.Cu *.Mask)
+    (pad "2" thru_hole oval (at 0 2) (size 1.35 1.35) (drill 0.8) (layers *.Cu *.Mask)
       (net 3 "Net-(J1-Pad2)") (pinfunction "Pin_2") (pintype "passive"))
-    (pad "3" thru_hole oval (at 0 5.08) (size 1.7 1.7) (drill 1) (layers *.Cu *.Mask)
+    (pad "3" thru_hole oval (at 0 4) (size 1.35 1.35) (drill 0.8) (layers *.Cu *.Mask)
       (net 1 "Net-(J1-Pad3)") (pinfunction "Pin_3") (pintype "passive"))
-    (model "${KICAD6_3DMODEL_DIR}/Connector_PinHeader_2.54mm.3dshapes/PinHeader_1x03_P2.54mm_Vertical.wrl"
+    (model "${KICAD6_3DMODEL_DIR}/Connector_PinSocket_2.00mm.3dshapes/PinSocket_1x03_P2.00mm_Vertical.wrl"
       (offset (xyz 0 0 0))
       (scale (xyz 1 1 1))
@@
     (descr "Mounting Hole 5.3mm, no annular, M5")
     (tags "mounting hole 5.3mm no annular m5")
-    (property "Sheetfile" "Limit_Switch_Board_Simple.kicad_sch")
+    (property "Sheetfile" "LimitSwitchBoard.kicad_sch")
     (property "Sheetname" "")
     (attr exclude_from_pos_files)
@@
   (footprint "Limit_Switch_custom:SS075Q102F035V2A" (layer "F.Cu")
     (at 127.5 68.455)
-    (property "Sheetfile" "Limit_Switch_Board_Simple.kicad_sch")
+    (property "Sheetfile" "LimitSwitchBoard.kicad_sch")
     (property "Sheetname" "")
     (attr through_hole)
@@
   )
   (gr_rect (start 120 60) (end 138.5 83) (layer "Edge.Cuts") (width 0.1) (fill none))
-  (segment (start 136.5 74.58) (end 133.58 74.58) (width 1) (layer "B.Cu") (net 1))
-  (segment (start 133.58 74.58) (end 130.5 71.5) (width 1) (layer "B.Cu") (net 1))
-  (segment (start 125.465 71.5) (end 122.42 68.455) (width 1) (layer "B.Cu") (net 1))
-  (segment (start 130.5 71.5) (end 125.465 71.5) (width 1) (layer "B.Cu") (net 1))
-  (segment (start 136.5 69.5) (end 135.5 68.5) (width 1) (layer "F.Cu") (net 2))
-  (segment (start 135.5 68.5) (end 132.625 68.5) (width 1) (layer "F.Cu") (net 2))
+  (segment (start 122.42 70.92) (end 122.42 68.455) (width 0.4) (layer "F.Cu") (net 1))
+  (segment (start 124 72.5) (end 122.42 70.92) (width 0.4) (layer "F.Cu") (net 1))
+  (segment (start 132.5 72.5) (end 124 72.5) (width 0.4) (layer "F.Cu") (net 1))
+  (segment (start 136 76) (end 132.5 72.5) (width 0.4) (layer "F.Cu") (net 1))
+  (segment (start 132.58 68.455) (end 136 71.875) (width 0.4) (layer "F.Cu") (net 2))
   (segment (start 132.625 68.5) (end 132.58 68.455) (width 1) (layer "F.Cu") (net 2))
-  (segment (start 131.145 72.1) (end 127.5 68.455) (width 1) (layer "F.Cu") (net 3))
-  (segment (start 136.5 72.04) (end 136.44 72.1) (width 1) (layer "F.Cu") (net 3))
-  (segment (start 136.44 72.1) (end 131.145 72.1) (width 1) (layer "F.Cu") (net 3))
+  (segment (start 136 71.875) (end 136 72) (width 0.4) (layer "F.Cu") (net 2))
+  (segment (start 133 71) (end 130.045 71) (width 0.4) (layer "F.Cu") (net 3))
+  (segment (start 136 74) (end 133 71) (width 0.4) (layer "F.Cu") (net 3))
+  (segment (start 130.045 71) (end 127.5 68.455) (width 0.4) (layer "F.Cu") (net 3))
+  (zone (net 0) (net_name "") (layers F&B.Cu) (hatch edge 0.508)
+    (connect_pads (clearance 0.508))
+    (min_thickness 0.254) (filled_areas_thickness no)
+    (fill yes (thermal_gap 0.508) (thermal_bridge_width 0.508))
+    (polygon
+      (pts
+        (xy 139 83.5)
+        (xy 119.5 83.5)
+        (xy 119.5 59.5)
+        (xy 139 59.5)
+      )
+    )
+  )
 )
