File: ECAD/DataDisplay/DataDisplay.kicad_pcb (KiCad board)
At the start: 2 copper layers, 38.1 x 69.3 mm, 10 parts, among them J1 Conn_01x04, J2 LCD, U1 ATmega328PB-A, U2 ST485EBDR, U3 IRM-H6XX

Commit message: Progressed ECAD.
Parts:
- removed C2: 4.7uC, Capacitor_SMD:C_0805_2012Metric
- removed J1: Conn_01x04, Connector_JST:JST_EH_B4B-EH-A_1x04_P2.50mm_Vertical
- removed R1: R, Resistor_SMD:R_1206_3216Metric
- removed R2: 10kR, Resistor_SMD:R_0805_2012Metric_Pad1.20x1.40mm_HandSolder
- removed R3: 160R, Resistor_SMD:R_0805_2012Metric_Pad1.20x1.40mm_HandSolder
- removed U3: IRM-H6XX, OptoDevice_custom:IRM-H6XX
- C1: value 0.1uC -> 100nC
- U1: value ATmega328PB-A -> PCA9615DP; footprint Package_QFP:TQFP-32_7x7mm_P0.8mm -> Package_SO:TSSOP-10_3x3mm_P0.5mm
- U2: value ST485EBDR -> PCA9555P; footprint Package_SO:SOIC-8_3.9x4.9mm_P1.27mm -> Package_SO:TSSOP-24_4.4x7.8mm_P0.65mm
Connections:
- U1 pad 1: unconnected-(U1-PD3-Pad1) -> +5V
- U1 pad 10: unconnected-(U1-PD6-Pad10) -> +5V
- U1 pad 4: +5V -> unconnected-(U1-SCL-Pad4)
- U2 pad 1: /RX -> unconnected-(U2-~{INT}-Pad1)
- U2 pad 2: /~{RE} -> unconnected-(U2-A1-Pad2)
- U2 pad 3: /DE -> unconnected-(U2-A2-Pad3)
- U2 pad 4: /TX -> /DB0
- U2 pad 5: GND -> /DB1
- U2 pad 6: Net-(J1-Pin_3) -> /DB2
- U2 pad 7: Net-(J1-Pin_2) -> /DB3
- U2 pad 8: +5V -> /DB4

Commit message: Progressed ECAD.
Parts:
- added C2: 0.1uC, Capacitor_SMD:C_0805_2012Metric, F.Cu at (138.9, 106.9)
- added C3: 4n7C, Capacitor_SMD:C_0805_2012Metric, F.Cu at (138.9, 109.9)
- added C4: 100nC, Capacitor_SMD:C_0805_2012Metric, F.Cu at (138.9, 113.0)
- added C5: 10uC, Capacitor_SMD:CP_Elec_4x5.4, F.Cu at (149.4, 120.8)
- added C6: 13pC, Capacitor_SMD:C_0805_2012Metric, F.Cu at (138.9, 116.0)
- added C7: 100nC, Capacitor_SMD:C_0805_2012Metric, F.Cu at (138.9, 119.0)
- added C8: 100nC, Capacitor_SMD:C_0805_2012Metric, F.Cu at (138.9, 122.0)
- added D1: LED, LED_SMD:LED_0805_2012Metric, F.Cu at (138.9, 125.0)
- added D2: 4148, Diode_SMD:D_SOD-123, F.Cu at (148.4, 125.5)
- added J1: Conn_01x04, Connector_JST:JST_EH_B4B-EH-A_1x04_P2.50mm_Vertical, F.Cu at (144.6, 108.0)
- added L1: 10uL, Inductor_SMD:L_0805_2012Metric, F.Cu at (155.6, 119.3)
- added L2: 10uL, Inductor_SMD:L_0805_2012Metric, F.Cu at (155.6, 122.0)
- added Q1: BC847, Package_TO_SOT_SMD:SOT-23, F.Cu at (156.5, 113.7)
- added R2: 10kR, Resistor_SMD:R_0805_2012Metric, F.Cu at (143.3, 112.8)
- added R3: 1kR, Resistor_SMD:R_0805_2012Metric, F.Cu at (143.3, 115.7)
- added R4: 100kR, Resistor_SMD:R_0805_2012Metric, F.Cu at (143.3, 118.7)
- added R5: 10kR, Resistor_SMD:R_0805_2012Metric, F.Cu at (143.3, 121.6)
- added SW1: SW_Push, Button_Switch_SMD:SW_Push_1P1T_XKB_TS-1187A, F.Cu at (149.8, 114.6)
- added Y1: 16MHz, Crystal:Crystal_SMD_3225-4Pin_3.2x2.5mm, F.Cu at (155.9, 125.7)
- C1: value 100nC -> 13pC
- U1: value PCA9615DP -> ST485E; footprint Package_SO:TSSOP-10_3x3mm_P0.5mm -> Package_SO:SOIC-8_3.9x4.9mm_P1.27mm
- U2: value PCA9555P -> ATmega328PB-A; footprint Package_SO:TSSOP-24_4.4x7.8mm_P0.65mm -> Package_QFP:TQFP-32_7x7mm_P0.8mm
- moved U1 14.1 mm to (144.0, 72.0)
- moved C1 13.0 mm to (152.1, 85.5)
- moved J2 10.9 mm to (129.0, 65.4)
- moved U2 10.7 mm to (140.4, 84.2)
Connections:
- C1 pad 1: +5V -> /XTAL2
- U1 pad 1: +5V -> /RX
- U1 pad 2: unconnected-(U1-SDA-Pad2) -> /~{RE}
- U1 pad 3: unconnected-(U1-EN-Pad3) -> /DE
- U1 pad 4: unconnected-(U1-SCL-Pad4) -> /TX
- U1 pad 6: unconnected-(U1-DSCLM-Pad6) -> Net-(J1-Pin_2)
- U1 pad 7: unconnected-(U1-DSCLP-Pad7) -> Net-(J1-Pin_3)
- U1 pad 8: unconnected-(U1-DSDAP-Pad8) -> +5V
- U2 pad 1: unconnected-(U2-~{INT}-Pad1) -> /DB3
- U2 pad 12: GND -> /~{RE}
- U2 pad 13: /RS -> /DE
- U2 pad 14: /R/~{W} -> unconnected-(U2-PB2-Pad14)
- U2 pad 15: /E -> /TX
- U2 pad 16: unconnected-(U2-IO1_3-Pad16) -> /RX
- U2 pad 18: unconnected-(U2-IO1_5-Pad18) -> +5VA
- U2 pad 2: unconnected-(U2-A1-Pad2) -> /DB4
- U2 pad 20: unconnected-(U2-IO1_7-Pad20) -> /AREF
- U2 pad 21: unconnected-(U2-A0-Pad21) -> GND
- U2 pad 24: +5V -> unconnected-(U2-PC1-Pad24)
- U2 pad 3: unconnected-(U2-A2-Pad3) -> /LED_IND
- U2 pad 4: /DB0 -> +5VD
- U2 pad 5: /DB1 -> GND
- U2 pad 6: /DB2 -> unconnected-(U2-PE1-Pad6)
- U2 pad 7: /DB3 -> /XTAL1
- U2 pad 8: /DB4 -> /XTAL2

Commit message: Progressed ECAD.
Parts:
- added C9: 4.7uC, Capacitor_SMD:C_0805_2012Metric_Pad1.18x1.45mm_HandSolder, F.Cu at (173.5, 80.0)
- added Q2: BC847, Package_TO_SOT_SMD:SOT-23, F.Cu at (168.7, 80.9)
- added R6: 10kR, Resistor_SMD:R_0805_2012Metric, F.Cu at (164.0, 73.4)
- added R7: 10kR, Resistor_SMD:R_0805_2012Metric, F.Cu at (164.0, 76.3)
- added R8: 10kR, Resistor_SMD:R_0805_2012Metric, F.Cu at (164.0, 79.3)
- added R9: 160R, Resistor_SMD:R_0805_2012Metric_Pad1.20x1.40mm_HandSolder, F.Cu at (173.5, 83.0)
- added U3: IRM-H6XX, OptoDevice_custom:IRM-H6XX, F.Cu at (171.0, 75.2)
Connections:
- J2 pad 15: /A -> +5V
- J2 pad 16: GND -> /K
- U2 pad 13: /DE -> /BL_PWM
- U2 pad 14: unconnected-(U2-PB2-Pad14) -> /DE
- U2 pad 19: unconnected-(U2-PE2-Pad19) -> /IR
- U2 pad 22: unconnected-(U2-PE3-Pad22) -> /PHOTO
- U2 pad 23: unconnected-(U2-PC0-Pad23) -> /RS
- U2 pad 24: unconnected-(U2-PC1-Pad24) -> /R/~{W}
- U2 pad 25: unconnected-(U2-PC2-Pad25) -> /E
