File: ECAD/DataDisplay/DataDisplay.kicad_sch (KiCad schematic)
At the start: 13 parts, among them J1 Conn_01x04, J2 LCD, Q1 Q_Photo_NPN, U1 ATmega328PB-A, U2 ST485EBDR, U3 IRM-H6XX

Commit message: Progressed ECAD.
Parts:
- added J3: SD_Card, symbol Connector:SD_Card
Changed lines of the file:
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@@
+	)
+	(symbol
+		(lib_id "Connector:SD_Card")
+		(at 142.24 165.1 0)
+		(unit 1)
+		(exclude_from_sim no)
+		(in_bom yes)
+		(on_board yes)
+		(dnp no)
+		(fields_autoplaced yes)
+		(property "Reference" "J3"
+			(at 142.24 147.32 0)
+			(effects
+				(font
+					(size 1.27 1.27)
+				)
+			)
+		)
+		(property "Value" "SD_Card"
+			(at 142.24 149.86 0)
+			(effects
+				(font
+					(size 1.27 1.27)
+				)
+			)
+		)
+		(property "Footprint" ""
+			(at 142.24 165.1 0)
+			(effects
+				(font
+					(size 1.27 1.27)
+				)
+				(hide yes)
+			)
+		)
+		(property "Datasheet" "http://portal.fciconnect.com/Comergent//fci/drawing/10067847.pdf"
+			(at 142.24 165.1 0)
+			(effects
+				(font
+					(size 1.27 1.27)
+				)
+				(hide yes)
+			)
+		)
+		(property "Description" "SD Card Reader"
+			(at 142.24 165.1 0)
+			(effects
+				(font
+					(size 1.27 1.27)
+				)
+				(hide yes)
+			)
+		)
+		(pin "2"
+		)
+		(pin "12"
+		)
+		(pin "11"
+		)
+		(pin "13"
+		)
+		(pin "5"
+		)
+		(pin "8"
+		)
+		(pin "6"
+		)
+		(pin "7"
+		)
+		(pin "9"
+		)
+		(pin "4"
+		)
+		(pin "3"
+		)
+		(pin "1"
+		)
+		(pin "10"
+		)
+		(instances
+			(project "DataDisplay"
+				(path "/418d3b0b-b1a8-4336-b4b3-60f2ac533fa0"
+					(reference "J3")
+					(unit 1)
+				)
+			)
+		)
 	)
 	(symbol

Commit message: Progressed ECAD.
Parts:
- removed C2: 4.7uC, Capacitor_SMD:C_0805_2012Metric, symbol Device:C
- removed J1: Conn_01x04, Connector_JST:JST_EH_B4B-EH-A_1x04_P2.50mm_Vertical, symbol Connector_Generic:Conn_01x04
- removed J3: SD_Card, symbol Connector:SD_Card
- removed Q1: Q_Photo_NPN, symbol Device:Q_Photo_NPN
- removed R1: R, Resistor_SMD:R_1206_3216Metric, symbol Device:R
- removed R2, R4: 10kR, Resistor_SMD:R_0805_2012Metric_Pad1.20x1.40mm_HandSolder, symbol Device:R
- removed R3: 160R, Resistor_SMD:R_0805_2012Metric_Pad1.20x1.40mm_HandSolder, symbol Device:R
- removed U1: ATmega328PB-A, Package_QFP:TQFP-32_7x7mm_P0.8mm, symbol MCU_Microchip_ATmega:ATmega328PB-A
- removed U2: ST485EBDR, Package_SO:SOIC-8_3.9x4.9mm_P1.27mm, symbol Interface_UART:ST485EBDR
- removed U3: IRM-H6XX, OptoDevice_custom:IRM-H6XX, symbol Inteface_Optical_custom:IRM-H6XX
- added U1: PCA9615DP, Package_SO:TSSOP-10_3x3mm_P0.5mm, symbol Interface:PCA9615DP
- added U2: PCA9555P, Package_SO:TSSOP-24_4.4x7.8mm_P0.65mm, symbol Interface_Expansion:PCA9555PW
- C1: value 0.1uC -> 100nC
Connections:
- net +5V: now also U1.1 (V_{DD(A)}), U1.10 (V_{DD(B)}), U2.24 (VDD)
- net DB0: now also U2.4 (IO0_0)
- net DB1: now also U2.5 (IO0_1)
- net DB2: now also U2.6 (IO0_2)
- net DB3: now also U2.7 (IO0_3)
- net DB4: now also U2.8 (IO0_4)
- net DB5: now also U2.9 (IO0_5)
- net DB6: now also U2.10 (IO0_6)
- net DB7: now also U2.11 (IO0_7)
- net E: now also U2.15 (IO1_2)
- net GND: now also U1.5 (V_{SS}), U2.12 (VSS)
- net RS: now also U2.13 (IO1_0)
- net R/~{W}: now also U2.14 (IO1_1)

Commit message: Progressed ECAD.
Parts:
- removed U1: PCA9615DP, Package_SO:TSSOP-10_3x3mm_P0.5mm, symbol Interface:PCA9615DP
- removed U2: PCA9555P, Package_SO:TSSOP-24_4.4x7.8mm_P0.65mm, symbol Interface_Expansion:PCA9555PW
- added C2: 0.1uC, Capacitor_SMD:C_0805_2012Metric, symbol Device:C
- added C3: 4n7C, Capacitor_SMD:C_0805_2012Metric, symbol Device:C
- added C4, C7, C8: 100nC, Capacitor_SMD:C_0805_2012Metric, symbol Device:C
- added C5: 10uC, Capacitor_SMD:CP_Elec_4x5.4, symbol Device:C_Polarized
- added C6: 13pC, Capacitor_SMD:C_0805_2012Metric, symbol Device:C
- added D1: LED, LED_SMD:LED_0805_2012Metric, symbol Device:LED
- added D2: 4148, Diode_SMD:D_SOD-123, symbol Device:D
- added J1: Conn_01x04, Connector_JST:JST_EH_B4B-EH-A_1x04_P2.50mm_Vertical, symbol Connector_Generic:Conn_01x04
- added L1, L2: 10uL, Inductor_SMD:L_0805_2012Metric, symbol Device:L
- added Q1: BC847, Package_TO_SOT_SMD:SOT-23, symbol Transistor_BJT:BC847
- added R1: R, symbol Device:R
- added R2, R5: 10kR, Resistor_SMD:R_0805_2012Metric, symbol Device:R
- added R3: 1kR, Resistor_SMD:R_0805_2012Metric, symbol Device:R
- added R4: 100kR, Resistor_SMD:R_0805_2012Metric, symbol Device:R
- added SW1: SW_Push, Button_Switch_SMD:SW_Push_1P1T_XKB_TS-1187A, symbol Switch:SW_Push
- added U1: ST485E, Package_SO:SOIC-8_3.9x4.9mm_P1.27mm, symbol Interface_UART:ST485E
- added U2: ATmega328PB-A, Package_QFP:TQFP-32_7x7mm_P0.8mm, symbol MCU_Microchip_ATmega:ATmega328PB-A
- added Y1: 16MHz, Crystal:Crystal_SMD_3225-4Pin_3.2x2.5mm, symbol Device:Crystal_GND24
- C1: value 100nC -> 13pC
Connections:
- net +5V: now also C2.1, C5.1, D2.1 (K), J1.1 (Pin_1), L1.1, L2.1, R2.1, R3.2, U1.8 (VCC); no longer C1.1
- net DB0: now also U2.30 (PD0)
- net DB1: now also U2.31 (PD1)
- net DB2: now also U2.32 (PD2)
- net DB3: now also U2.1 (PD3)
- net DB4: now also U2.2 (PD4)
- net DB5: now also U2.9 (PD5)
- net DB6: now also U2.10 (PD6)
- net DB7: now also U2.11 (PD7)
- net GND: now also C2.2, C3.2, C4.2, C5.2, C6.2, C7.2, C8.2, J1.4 (Pin_4), Q1.2 (E), SW1.1, U1.5 (GND), U2.21 (GND), U2.5 (GND), Y1.2, Y1.4
- new net: Q1.1 (B), R5.1
- new net: D1.1 (K), Q1.3 (C)
- new net: J1.2 (Pin_2), R1.1, U1.6 (A)
- new net: J1.3 (Pin_3), R1.2, U1.7 (B)
- new net: D1.2 (A), R3.1
- new net +5VA: C8.1, L2.2, U2.18 (AVCC)
- new net +5VD: C7.1, L1.2, U2.4 (VCC)
- new net AREF: C4.1, U2.20 (AREF)
- new net DE: U1.3 (DE), U2.13 (PB1)
- new net LED_IND: R5.2, U2.3 (PE0)
- new net RX: U1.1 (RO), U2.16 (PB4)
- new net TX: U1.4 (DI), U2.15 (PB3)
- new net XTAL1: C6.1, R4.2, U2.7 (XTAL1/PB6), Y1.3
- new net XTAL2: C1.1, R4.1, U2.8 (XTAL2/PB7), Y1.1
- new net ~{RESET}: C3.1, D2.2 (A), R2.2, SW1.2, U2.29 (~{RESET}/PC6)
- new net ~{RE}: U1.2 (~{RE}), U2.12 (PB0)
- no-connect marks 0 -> 6
Other:
- note added: "Guideline: C6 = C9 = 2*(CL - Cstray) Cstray assumed to be 5pF"
- moved on the sheet: J2, RV1

Commit message: Progressed ECAD.
Parts:
- added C9: 4.7uC, Capacitor_SMD:C_0805_2012Metric_Pad1.18x1.45mm_HandSolder, symbol Device:C
- added Q2: BC847, Package_TO_SOT_SMD:SOT-23, symbol Transistor_BJT:BC847
- added Q3: TEMT6000, symbol Device:Q_Photo_NPN
- added R6, R7, R8: 10kR, Resistor_SMD:R_0805_2012Metric, symbol Device:R
- added R9: 160R, Resistor_SMD:R_0805_2012Metric_Pad1.20x1.40mm_HandSolder, symbol Device:R
- added U3: IRM-H6XX, OptoDevice_custom:IRM-H6XX, symbol Inteface_Optical_custom:IRM-H6XX
Connections:
- net A is gone; now on net +5V: J2.15 (Pin_15)
- net +5V: now also Q3.1 (C), R8.1, R9.2
- net DE: now also U2.14 (PB2); no longer U2.13 (PB1)
- net E: now also U2.25 (PC2)
- net GND: now also C9.2, Q2.2 (E), R6.2, U3.1 (GND), U3.2 (GND); no longer J2.16 (Pin_16)
- net RS: now also U2.23 (PC0)
- net R/~{W}: now also U2.24 (PC1)
- net IR: now reaches U2.19 (PE2)
- net IR: now also R8.2, U3.3 (OUT)
- net PHOTO: now reaches U2.22 (PE3)
- net PHOTO: now also Q3.2 (E), R6.1
- new net: Q2.1 (B), R7.1
- new net: C9.1, R9.1, U3.4 (Vs)
- new net BL_PWM: R7.2, U2.13 (PB1)
- new net K: J2.16 (Pin_16), Q2.3 (C)
- no-connect marks 6 -> 5
Other:
- note added: "A"
- note added: "ADC7 (ADC)"
- note added: "Guideline: C1 = C6 = 2*(CL - Cstray) Cstray assumed to be 5pF"
- note added: "ICP3 (Timer/Counter3)"
- note added: "IR receiver"
- note added: "OC1A (Timer/Counter1)"
- note added: "RXD1 (USART1)"
- note added: "TXD1 (USART1)"
- note added: "VDD"
- note added: "VSS"
- note removed: "Guideline: C6 = C9 = 2*(CL - Cstray) Cstray assumed to be 5pF"
- moved on the sheet: C2, J1, J2, R1, RV1, U1, U2
