File: ECAD/RS485Board/RS485Board.kicad_pcb (KiCad board)
At the start: 2 copper layers, 45 x 45 mm, 10 parts, among them J1 Conn_02x03_Odd_Even, J2 Conn_02x03_Odd_Even, J3 Barrel_Jack_Switch

Commit message: Progressed ECAD.
Parts:
- moved R2 0.50 mm to (112.5, 131.0)
- moved R1 0.50 mm to (112.5, 94.0)
Routing:
- net Net-(J2-Pin_2): track 0.00 -> 3.08 mm
- net Net-(J2-Pin_1): track 0.00 -> 3.08 mm
- net Net-(J1-Pin_2): track 0.00 -> 3.08 mm
- net Net-(J1-Pin_1): track 0.00 -> 3.08 mm
Other:
- board text added: "1 - B 2 - A 3, 4 - GND 5, 6 - 12 V"
- board text added: "2 4 6 1 3 5"
Changed lines of the file:
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@@
 			(at 0 -6.3 0)
 			(layer "F.SilkS")
+			(hide yes)
 			(effects
 				(font
@@
 			(at 0 6.3 0)
 			(layer "F.Fab")
+			(hide yes)
 			(effects
 				(font
@@
 			(at 0 -6.3 0)
 			(layer "F.SilkS")
+			(hide yes)
 			(effects
 				(font
@@
 			(at 0 6.3 0)
 			(layer "F.Fab")
+			(hide yes)
 			(effects
 				(font
@@
 			(at 0 -6.3 0)
 			(layer "F.SilkS")
+			(hide yes)
 			(effects
 				(font
@@
 			(at 0 6.3 0)
 			(layer "F.Fab")
+			(hide yes)
 			(effects
 				(font
@@
 			(at 0 -6.3 0)
 			(layer "F.SilkS")
+			(hide yes)
 			(effects
 				(font
@@
 			(at 0 6.3 0)
 			(layer "F.Fab")
+			(hide yes)
 			(effects
 				(font
@@
 			(at 1.27 11.18 0)
 			(layer "F.Fab")
+			(hide yes)
 			(effects
 				(font
@@
 				(font
 					(size 0.001 0.001)
+					(thickness 0.15)
 				)
 			)
@@
 				(font
 					(size 0.001 0.001)
+					(thickness 0.15)
 				)
 			)
@@
 			(at -6.2 -5.5 0)
 			(layer "F.Fab")
+			(hide yes)
 			(effects
 				(font
@@
 			(at 1.27 11.18 0)
 			(layer "F.Fab")
+			(hide yes)
 			(effects
 				(font
@@
 	(footprint "Resistor_SMD:R_1206_3216Metric"
 		(layer "B.Cu")
-		(at 112.5 93.5 180)
+		(at 112.5 94 180)
 		(descr "Resistor SMD 1206 (3216 Metric), square (rectangular) end terminal, IPC_7351 nominal, (Body size source: IPC-SM-782 page 72, https://www.pcb-3d.com/wordpress/wp-content/uploads/ipc-sm-782a_amendment_1_and_2.pdf), generated with kicad-footprint-generator")
 		(tags "resistor")
@@
 	(footprint "Resistor_SMD:R_1206_3216Metric"
 		(layer "B.Cu")
-		(at 112.5375 131.5)
+		(at 112.5 131)
 		(descr "Resistor SMD 1206 (3216 Metric), square (rectangular) end terminal, IPC_7351 nominal, (Body size source: IPC-SM-782 page 72, https://www.pcb-3d.com/wordpress/wp-content/uploads/ipc-sm-782a_amendment_1_and_2.pdf), generated with kicad-footprint-generator")
 		(tags "resistor")
 		(property "Reference" "R2"
-			(at 0 1.82 360)
+			(at 0 1.82 0)
 			(layer "B.SilkS")
 			(effects
@@
 		)
 		(property "Value" "120R"
-			(at 0 -1.82 360)
+			(at 0 -1.82 0)
 			(layer "B.Fab")
 			(effects
@@
 		)
 		(fp_text user "${REFERENCE}"
-			(at 0 0 360)
+			(at 0 0 0)
 			(layer "B.Fab")
 			(effects
@@
 		)
 	)
+	(gr_line
+		(start 109.25 114.5)
+		(end 109.25 110.5)
+		(stroke
+			(width 0.1)
+			(type default)
+		)
+		(layer "F.SilkS")
+	)
+	(gr_line
+		(start 111.25 114.5)
+		(end 109.25 114.5)
+		(stroke
+			(width 0.1)
+			(type default)
+		)
+		(layer "F.SilkS")
+	)
+	(gr_line
+		(start 114.75 110.5)
+		(end 114.75 114.5)
+		(stroke
+			(width 0.1)
+			(type default)
+		)
+		(layer "F.SilkS")
+	)
+	(gr_line
+		(start 114.75 114.5)
+		(end 112.75 114.5)
+		(stroke
+			(width 0.1)
+			(type default)
+		)
+		(layer "F.SilkS")
+	)
+	(gr_line
+		(start 109.25 110.5)
+		(end 114.75 110.5)
+		(stroke
+			(width 0.1)
+			(type default)
+		)
+		(layer "F.SilkS")
+	)
 	(gr_arc
 		(start 92 135)
@@
 		(layer "Edge.Cuts")
 	)
+	(gr_text "2 4 6\n1 3 5"
+		(at 109.75 114 0)
+		(layer "F.SilkS")
+		(effects
+			(font
+				(size 1 1)
+				(thickness 0.1)
+			)
+			(justify left bottom)
+		)
+	)
+	(gr_text "1 - B\n2 - A\n3, 4 - GND\n5, 6 - 12 V"
+		(at 120 115.5 0)
+		(layer "F.SilkS")
+		(effects
+			(font
+				(size 1 1)
+				(thickness 0.1)
+			)
+			(justify left bottom)
+		)
+	)
+	(segment
+		(start 113.9625 94)
+		(end 113.9625 96.8075)
+		(width 1)
+		(layer "B.Cu")
+		(net 2)
+	)
+	(segment
+		(start 113.9625 96.8075)
+		(end 113.77 97)
+		(width 1)
+		(layer "B.Cu")
+		(net 2)
+	)
+	(segment
+		(start 111.0375 94)
+		(end 111.0375 96.8075)
+		(width 1)
+		(layer "B.Cu")
+		(net 3)
+	)
+	(segment
+		(start 111.0375 96.8075)
+		(end 111.23 97)
+		(width 1)
+		(layer "B.Cu")
+		(net 3)
+	)
+	(segment
+		(start 113.9625 128.1925)
+		(end 113.77 128)
+		(width 1)
+		(layer "B.Cu")
+		(net 5)
+	)
+	(segment
+		(start 113.9625 131)
+		(end 113.9625 128.1925)
+		(width 1)
+		(layer "B.Cu")
+		(net 5)
+	)
+	(segment
+		(start 111.0375 128.1925)
+		(end 111.23 128)
+		(width 1)
+		(layer "B.Cu")
+		(net 6)
+	)
+	(segment
+		(start 111.0375 131)
+		(end 111.0375 128.1925)
+		(width 1)
+		(layer "B.Cu")
+		(net 6)
+	)
 	(zone

Commit message: Progressed ECAD.
Parts:
- removed kibuzzard-66804287: G***, kibuzzard-66804287
- added REF**: Symbol_Barrel_Polarity, Symbol:Symbol_Barrel_Polarity, F.Cu at (92.0, 122.0)
- J1, J2: value Conn_02x03_Odd_Even -> RS485
Other:
- board text added: "DC IN (8V - 15V)"
- board text added: "RS485 termination and power board Pinout: 1 - RS485 B 2 - RS485 A 3, 4 - GND 5, 6 - 12 V"
- board text removed: "1 - B 2 - A 3, 4 - GND 5, 6 - 12 V"

Commit message: Progressed ECAD.
Other:
- board text added: "RS485 termination and power board Pinout: 1 - RS485 A 2 - RS485 B 3, 4 - GND 5, 6 - 12 V"
- board text removed: "RS485 termination and power board Pinout: 1 - RS485 B 2 - RS485 A 3, 4 - GND 5, 6 - 12 V"
Changed lines of the file:
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@@
 		)
 	)
-	(gr_text "RS485 termination\nand power board\nPinout:\n1 - RS485 B\n2 - RS485 A\n3, 4 - GND\n5, 6 - 12 V"
+	(gr_text "RS485 termination\nand power board\nPinout:\n1 - RS485 A\n2 - RS485 B\n3, 4 - GND\n5, 6 - 12 V"
 		(at 119 118 0)
 		(layer "F.SilkS")
