File: ECAD/RotationEncoder/RotationEncoder.kicad_pcb (KiCad board)
At the start: 2 copper layers, 37.5 x 31.6 mm, 31 parts, among them J1 Conn_01x04, Q1 BC847, SW1 SW_Push, U1 ST485E, U2 AS5600, U3 ATmega328PB-A, Y1 16MHz

Commit message: Progressed ECAD.
Parts:
- added R1: 120R, Resistor_SMD:R_1206_3216Metric, F.Cu at (122.0, 112.0)
- J1: value Conn_01x04 -> Conn_02x03_Odd_Even; footprint Connector_JST:JST_EH_B4B-EH-A_1x04_P2.50mm_Vertical -> Connector_IDC:IDC-Header_2x03_P2.54mm_Vertical
- moved J1 10.2 mm to (116.5, 77.5)
Connections:
- J1 pad 1: +5V -> Net-(J1-Pin_1)
- J1 pad 3: Net-(J1-Pin_3) -> GND
- U1 pad 7: Net-(J1-Pin_3) -> Net-(J1-Pin_1)

Commit message: Progressed ECAD.
Parts:
- added C10: 10uC, Capacitor_SMD:C_1206_3216Metric, F.Cu at (148.5, 64.8)
- added C11: 10uC, Capacitor_SMD:C_1206_3216Metric, F.Cu at (151.5, 73.2)
- added C13: 100nC, Capacitor_SMD:C_0805_2012Metric, F.Cu at (138.4, 73.4)
- added C14: 100nC, Capacitor_SMD:C_0805_2012Metric, F.Cu at (138.4, 76.4)
- added C15: 68pC, Capacitor_SMD:C_0805_2012Metric, F.Cu at (138.4, 79.4)
- added C16: 10uC, Capacitor_SMD:C_1206_3216Metric, F.Cu at (151.5, 76.5)
- added C17: 47uC, Capacitor_SMD:C_1210_3225Metric, F.Cu at (148.5, 69.0)
- added D3: CMS30I30A, Diode_SMD:D_SOD-128, F.Cu at (145.0, 73.5)
- added J2: ICSP, Connector_PinHeader_2.54mm:PinHeader_2x03_P2.54mm_Vertical, F.Cu at (104.0, 74.4)
- added L3: 4u7L, Inductor_SMD:L_1008_2520Metric, F.Cu at (128.4, 77.5)
- added R10: 10kR, Resistor_SMD:R_0805_2012Metric, F.Cu at (143.5, 70.0)
- added R8: 12k1R, Resistor_SMD:R_0805_2012Metric, F.Cu at (143.5, 64.1)
- added R9: 61k9R, Resistor_SMD:R_0805_2012Metric, F.Cu at (143.5, 67.0)
- added U4: TPS561208DDCR, Package_TO_SOT_SMD:SOT-23-6, F.Cu at (138.7, 65.0)
- added U5: TLV75801PDBVR, Package_TO_SOT_SMD:SOT-23-5, F.Cu at (138.7, 69.7)
- J1: value Conn_02x03_Odd_Even -> RS485
- R1: value 120R -> 97k6R; footprint Resistor_SMD:R_1206_3216Metric -> Resistor_SMD:R_0805_2012Metric
Connections:
- J1 pad 5: unconnected-(J1-Pin_5-Pad5) -> +12V
- J1 pad 6: unconnected-(J1-Pin_6-Pad6) -> +12V
- R1 pad 1: Net-(J1-Pin_2) -> +5V
- R1 pad 2: Net-(J1-Pin_1) -> Net-(U5-FB)
Other:
- board size 37.5 x 31.6 mm -> 70.3 x 53.5 mm

Commit message: Progressed ECAD.
Parts:
- added J3: Wire RS485, Connector_IDC:IDC-Header_2x03_P2.54mm_Vertical, F.Cu at (161.5, 68.4)
- C10, C16: footprint Capacitor_SMD:C_1206_3216Metric -> Capacitor_SMD:C_0805_2012Metric
- C11: value 10uC -> 100nC; footprint Capacitor_SMD:C_1206_3216Metric -> Capacitor_SMD:C_0805_2012Metric
- C12: footprint Capacitor_SMD:CP_Elec_4x5.4 -> Capacitor_SMD:C_0805_2012Metric
- C15: value 68pC -> 13pC
- R1: value 97k6R -> 80k6R
- R8: value 12k1R -> 10kR
- moved J2 1.80 mm to (105.5, 75.4)
Connections:
- C11 pad 1: /5V5 -> GND
- C11 pad 2: GND -> +12V
- C12 pad 1: +5V -> +12V
- J2 pad 2: unconnected-(J2-Pin_2-Pad2) -> +5V
- J2 pad 5: unconnected-(J2-Pin_5-Pad5) -> /~{RESET}
- J2 pad 6: unconnected-(J2-Pin_6-Pad6) -> GND
- U3 pad 15: unconnected-(U3-PB3-Pad15) -> /ICSP_MOSI
- U3 pad 16: unconnected-(U3-PB4-Pad16) -> /ICSP_MISO
- U3 pad 17: unconnected-(U3-PB5-Pad17) -> /ICSP_SCK

Commit message: Progressed ECAD.
Parts:
- removed J3: Wire RS485, Connector_IDC:IDC-Header_2x03_P2.54mm_Vertical
- moved L1 77.3 mm to (231.3, 50.3)
- moved R2 77.3 mm to (236.9, 66.0)
- moved R3 77.3 mm to (236.9, 69.0)
- moved U2 77.3 mm to (219.4, 66.0)
- moved C2 77.3 mm to (232.5, 66.1)
- moved C3 77.3 mm to (232.5, 69.1)
- moved D2 71.6 mm to (198.7, 74.8)
- moved C1 71.6 mm to (177.5, 68.8)
- moved C4 71.6 mm to (177.5, 71.8)
- moved C5 71.6 mm to (177.5, 74.8)
- moved C6 71.6 mm to (177.5, 77.9)
- moved C7 71.6 mm to (177.5, 80.9)
- moved C8 71.6 mm to (177.5, 83.9)
- moved C9 71.6 mm to (177.5, 86.9)
- moved D1 71.6 mm to (177.6, 89.9)
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Other:
- board size 70.3 x 53.5 mm -> 50 x 50 mm
- copper layers 2 -> 6
- board text added: "1 - B 2 - A 3, 4 - GND 5, 6 - 12 V"
- board text added: "2 4 6 1 3 5"

Commit message: Progressed ECAD.
Parts:
- removed H3, H4: MountingHole, MountingHole:MountingHole_3.2mm_M3
- added C18: 100nC, Capacitor_SMD:C_0805_2012Metric, F.Cu at (105.5, 73.5)
- added R11: 10kR, Resistor_SMD:R_0805_2012Metric, B.Cu at (157.6, 100.2)
- C1, C15, C7, D2, Q1, R10, R4, R5, R7, R9, U2: moved to B.Cu
- moved C2 132.0 mm to (104.7, 99.0)
- moved C3 132.0 mm to (104.7, 102.0)
- moved R2 132.0 mm to (109.1, 99.0)
- moved R3 132.0 mm to (109.1, 102.0)
- moved L1 117.5 mm to (116.9, 77.2)
- moved L2 86.8 mm to (111.7, 89.6)
- moved C4 79.1 mm to (98.5, 76.0)
- moved C5 79.1 mm to (98.5, 79.1)
- moved C8 79.1 mm to (98.5, 88.1)
- moved U2 78.2 mm to (145.0, 90.0), turned to 180 degrees
- moved D2 75.6 mm to (123.5, 83.0), turned to 90 degrees
- moved J2 67.0 mm to (124.8, 102.5), turned to 180 degrees
- moved U1 66.1 mm to (132.0, 100.5)
- moved SW1 64.4 mm to (124.2, 83.2)
- moved Y1 63.0 mm to (136.5, 90.0)
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Connections:
- D1 pad 2: Net-(D1-A) -> +5V
- J2 pad 1: unconnected-(J2-Pin_1-Pad1) -> /ICSP_MISO
- J2 pad 3: unconnected-(J2-Pin_3-Pad3) -> /ICSP_SCK
- J2 pad 4: unconnected-(J2-Pin_4-Pad4) -> /ICSP_MOSI
- Q1 pad 3: Net-(D1-K) -> Net-(Q1-C)
- R5 pad 1: Net-(D1-A) -> Net-(Q1-C)
- R5 pad 2: +5V -> Net-(D1-K)
- U1 pad 6: Net-(J1-Pin_2) -> Net-(J1-Pin_1)
- U1 pad 7: Net-(J1-Pin_1) -> Net-(J1-Pin_2)
- U3 pad 1: /DE -> unconnected-(U3-PD3-Pad1)
- U3 pad 10: unconnected-(U3-PD6-Pad10) -> /DIR
- U3 pad 13: unconnected-(U3-PB1-Pad13) -> /~{RE}
- U3 pad 14: unconnected-(U3-PB2-Pad14) -> /DE
- U3 pad 19: unconnected-(U3-PE2-Pad19) -> /OUT
- U3 pad 22: unconnected-(U3-PE3-Pad22) -> /LED_IND
- U3 pad 23: /OUT -> unconnected-(U3-PC0-Pad23)
- U3 pad 25: /PGO -> unconnected-(U3-PC2-Pad25)
- U3 pad 26: /DIR -> unconnected-(U3-PC3-Pad26)
- U3 pad 3: /LED_IND -> unconnected-(U3-PE0-Pad3)
- U3 pad 32: /~{RE} -> unconnected-(U3-PD2-Pad32)
- U3 pad 9: unconnected-(U3-PD5-Pad9) -> /PGO
- U4 pad 5: +12V -> Net-(U4-EN)
Routing:
- net GND: vias 0 -> 2
Other:
- board size 50 x 50 mm -> 50 x 25 mm
- copper layers 6 -> 4
- board text added: "1 - RS485 A 2 - RS485 B 3, 4 - GND 5, 6 - 12 V"
- board text added: "RS485"
- board text removed: "1 - B 2 - A 3, 4 - GND 5, 6 - 12 V"

Commit message: Update RotationEncoder.kicad_pcb
Parts:
- C2, C3, C4, C5, L1, L2, R2, R3: moved to B.Cu
- moved C5 54.1 mm to (151.5, 90.0), turned to 180 degrees
- moved C8 54.0 mm to (152.5, 87.5)
- moved C3 43.1 mm to (144.0, 84.5), turned to 180 degrees
- moved C2 43.0 mm to (147.5, 95.0), turned to 180 degrees
- moved R3 42.9 mm to (148.5, 85.0), turned to 180 degrees
- moved C4 41.7 mm to (139.5, 84.0), turned to 180 degrees
- moved L2 39.9 mm to (151.5, 92.0)
- moved R2 33.3 mm to (142.1, 94.5), turned to 180 degrees
- moved C18 26.7 mm to (131.0, 81.5)
- moved L1 24.3 mm to (139.5, 86.0)
- moved C1 2.67 mm to (132.5, 98.0)
- moved U1 2.55 mm to (132.5, 98.0), turned to -90 degrees
- moved R1 1.92 mm to (166.5, 83.5)
- moved C16 1.62 mm to (155.0, 85.0)
- moved D3 1.61 mm to (160.5, 83.0)
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
Commit message: Progressed ECAD.
Parts:
- added L4: 10uL, Inductor_SMD:L_0805_2012Metric, B.Cu at (132.6, 100.0)
- added L5: 10uL, Inductor_SMD:L_0805_2012Metric, B.Cu at (142.1, 81.5)
Connections:
- C1 pad 1: +5V -> +5VD
- C3 pad 1: +5V -> +5VD
- U1 pad 8: +5V -> +5VD
- U2 pad 1: +5V -> +5VD

Commit message: Progressed ECAD.
Parts:
- moved R11 11.7 mm to (168.5, 96.0)
- moved C15 6.65 mm to (164.5, 96.0)
- moved R10 4.99 mm to (156.0, 96.0)
- moved L3 1.12 mm to (161.5, 95.5)
- moved C13 1.00 mm to (165.6, 97.5)
- moved C17 0.50 mm to (157.5, 96.5)
Routing:
- net +12V: track 0.00 -> 20.7 mm
- net Net-(U4-SW): track 0.00 -> 6.68 mm, vias 0 -> 5
- net Net-(U4-BOOT): track 0.00 -> 3.69 mm
- net GND: vias 2 -> 9
- added copper zone on In2.Cu, net +5V
- added copper zone on F.Cu, net /5V5
- added copper zone on F.Cu, net GND
- added copper zone on In1.Cu, net GND
- added copper zone on In2.Cu, net GND
- added copper zone on B.Cu, net Net-(U4-SW)
