File: ECAD/RS232Board/RS232Board.kicad_pcb (KiCad board)
At the start: 2 copper layers, 101.6 x 53.3 mm, 9 parts, among them J1 Conn_01x20, J8 RS232, J9 RS232

Commit message: Progressed ECAD.
Parts:
- moved J1 59.9 mm to (197.4, 78.4), turned to 90 degrees
- moved J9 1.69 mm to (176.4, 54.7)
- moved J8 1.09 mm to (140.5, 54.7)
Connections:
- J1 pad 1: unconnected-(J1-Pin_1-Pad1) -> /RI_0
- J1 pad 10: unconnected-(J1-Pin_10-Pad10) -> GND
- J1 pad 11: unconnected-(J1-Pin_11-Pad11) -> /RI_1
- J1 pad 12: unconnected-(J1-Pin_12-Pad12) -> /DTR_1
- J1 pad 13: unconnected-(J1-Pin_13-Pad13) -> /CTS_1
- J1 pad 14: unconnected-(J1-Pin_14-Pad14) -> /TX_1
- J1 pad 15: unconnected-(J1-Pin_15-Pad15) -> /RTS_1
- J1 pad 16: unconnected-(J1-Pin_16-Pad16) -> /RX_1
- J1 pad 17: unconnected-(J1-Pin_17-Pad17) -> /DSR_1
- J1 pad 18: unconnected-(J1-Pin_18-Pad18) -> /DCD_1
- J1 pad 19: unconnected-(J1-Pin_19-Pad19) -> GND
- J1 pad 2: unconnected-(J1-Pin_2-Pad2) -> /DTR_0
- J1 pad 20: unconnected-(J1-Pin_20-Pad20) -> GND
- J1 pad 3: unconnected-(J1-Pin_3-Pad3) -> /CTS_0
- J1 pad 4: unconnected-(J1-Pin_4-Pad4) -> /TX_0
- J1 pad 5: unconnected-(J1-Pin_5-Pad5) -> /RTS_0
- J1 pad 6: unconnected-(J1-Pin_6-Pad6) -> /RX_0
- J1 pad 7: unconnected-(J1-Pin_7-Pad7) -> /DSR_0
- J1 pad 8: unconnected-(J1-Pin_8-Pad8) -> /DCD_0
- J1 pad 9: unconnected-(J1-Pin_9-Pad9) -> GND
- J8 pad 1: /DCD -> /DCD_0
- J8 pad 2: /RX -> /RX_0
- J8 pad 3: /TX -> /TX_0
- J8 pad 4: /DTR -> /DTR_0
- J8 pad 6: /DSR -> /DSR_0
- J8 pad 7: /RTS -> /RTS_0
- J8 pad 8: /CTS -> /CTS_0
- J8 pad 9: /RI -> /RI_0
- J9 pad 1: /DCD -> /DCD_1
- J9 pad 2: /RX -> /RX_1
- J9 pad 3: /TX -> /TX_1
- J9 pad 4: /DTR -> /DTR_1
- J9 pad 6: /DSR -> /DSR_1
- J9 pad 7: /RTS -> /RTS_1
- J9 pad 8: /CTS -> /CTS_1
- J9 pad 9: /RI -> /RI_1
Routing:
- added copper zone on B.Cu, net GND
- added copper zone on F.Cu, net GND

Commit message: Progressed ECAD.
Parts:
- J1: footprint Connector_FFC-FPC:Molex_200528-0200_1x20-1MP_P1.00mm_Horizontal -> Connector_FFC-FPC:TE_2-84952-0_1x20-1MP_P1.0mm_Horizontal
- moved J1 3.28 mm to (194.2, 78.4)

Commit message: Progressed ECAD.
Parts:
- moved J1 3.37 mm to (195.9, 75.5)
Connections:
- J1 pad 1: /RI_0 -> /DCD_0
- J1 pad 11: /RI_1 -> /DCD_1
- J1 pad 12: /DTR_1 -> /DSR_1
- J1 pad 13: /CTS_1 -> /RX_1
- J1 pad 14: /TX_1 -> /CTS_1
- J1 pad 15: /RTS_1 -> /RI_1
- J1 pad 16: /RX_1 -> /TX_1
- J1 pad 17: /DSR_1 -> /DTR_1
- J1 pad 18: /DCD_1 -> /RTS_1
- J1 pad 2: /DTR_0 -> /DSR_0
- J1 pad 3: /CTS_0 -> /RX_0
- J1 pad 4: /TX_0 -> /CTS_0
- J1 pad 5: /RTS_0 -> /RI_0
- J1 pad 6: /RX_0 -> /TX_0
- J1 pad 7: /DSR_0 -> /DTR_0
- J1 pad 8: /DCD_0 -> /RTS_0
Routing:
- net /RI_0: track 0.00 -> 92.5 mm, vias 0 -> 1
- net /CTS_0: track 0.00 -> 90.7 mm, vias 0 -> 1
- net /DSR_0: track 0.00 -> 87.2 mm, vias 0 -> 1
- net /DTR_0: track 0.00 -> 86.2 mm, vias 0 -> 1
- net /RX_0: track 0.00 -> 84.7 mm, vias 0 -> 1
- net /TX_0: track 0.00 -> 84.5 mm, vias 0 -> 1
- net /DCD_0: track 0.00 -> 83.9 mm, vias 0 -> 1
- net /RTS_0: track 0.00 -> 83.9 mm, vias 0 -> 1
- net /RI_1: track 0.00 -> 55.6 mm, vias 0 -> 1
- net /DTR_1: track 0.00 -> 49.7 mm, vias 0 -> 1
- net /CTS_1: track 0.00 -> 44.8 mm, vias 0 -> 1
- net /DSR_1: track 0.00 -> 41.3 mm, vias 0 -> 1
- net /RX_1: track 0.00 -> 38.8 mm, vias 0 -> 1
- net /TX_1: track 0.00 -> 38.5 mm, vias 0 -> 1
- net /DCD_1: track 0.00 -> 38.0 mm, vias 0 -> 1
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
Commit message: Added Gerbers.
Parts:
- added kibuzzard-66E5B9FC: G***, kibuzzard-66E5B9FC, F.Cu at (125.0, 60.0)
- added kibuzzard-66E5BA0D: G***, kibuzzard-66E5BA0D, F.Cu at (161.2, 60.0)
Connections:
- J1 pad 1: /DCD_0 -> GND
- J1 pad 10: GND -> /DCD_1
- J1 pad 11: /DCD_1 -> GND
- J1 pad 12: /DSR_1 -> GND
- J1 pad 13: /RX_1 -> /RTS_0
- J1 pad 14: /CTS_1 -> /DTR_0
- J1 pad 15: /RI_1 -> /TX_0
- J1 pad 16: /TX_1 -> /RI_0
- J1 pad 17: /DTR_1 -> /CTS_0
- J1 pad 18: /RTS_1 -> /RX_0
- J1 pad 19: GND -> /DSR_0
- J1 pad 2: /DSR_0 -> GND
- J1 pad 20: GND -> /DCD_0
- J1 pad 3: /RX_0 -> /RTS_1
- J1 pad 4: /CTS_0 -> /DTR_1
- J1 pad 5: /RI_0 -> /TX_1
- J1 pad 6: /TX_0 -> /RI_1
- J1 pad 7: /DTR_0 -> /CTS_1
- J1 pad 8: /RTS_0 -> /RX_1
- J1 pad 9: GND -> /DSR_1
Routing:
- net /DSR_0: track 87.2 -> 70.2 mm
- net /DCD_0: track 83.9 -> 68.7 mm
- net /RX_0: track 84.7 -> 69.7 mm
- net /RTS_1: track 38.0 -> 53.0 mm
- net /CTS_0: track 90.7 -> 77.7 mm
- net /DTR_1: track 49.7 -> 62.2 mm
- net /TX_1: track 38.5 -> 49.6 mm
- net /RI_0: track 92.5 -> 81.5 mm
- net /TX_0: track 84.5 -> 75.5 mm
- net /RI_1: track 55.6 -> 64.6 mm
- net /DTR_0: track 86.2 -> 79.2 mm
- net /CTS_1: track 44.8 -> 51.8 mm
- net /RX_1: track 38.8 -> 43.8 mm
- net /RTS_0: track 83.9 -> 78.9 mm
- net /DSR_1: track 41.3 -> 44.3 mm
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