File: ECAD/BDCMotorControlBoard/h_bridge.kicad_sch (KiCad schematic)
At the start: 2 parts, among them U2 DRV8870DDA, U3 INA180A1

Commit message: Progressed ECAD.
Parts:
- U2: MPN (none) -> DRV8870DDAR; Status (none) -> OK
Changed lines of the file:
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@@
+			)
+		)
+		(property "Status" "OK"
+			(at 125.73 74.93 0)
+			(effects
+				(font
+					(size 1.27 1.27)
+				)
+				(hide yes)
+			)
+		)
+		(property "MPN" "DRV8870DDAR"
+			(at 125.73 74.93 0)
+			(effects
+				(font
+					(size 1.27 1.27)
+				)
+				(hide yes)
 			)
 		)
@@
 			(at 151.13 93.98 0)
 			(effects
+				(font
+					(size 1.27 1.27)
+				)
+				(hide yes)
+			)
+		)
+		(property "Status" ""
+			(at 151.13 93.98 0)
+			(effects
