File: ECAD/BDCMotorControlBoard/BDCMotorControlBoard.kicad_pcb (KiCad board)
At the start: 4 copper layers, 105.5 x 38 mm, 67 parts, among them J1 Motor Connector, J2 RS485 PCB, J4 Limit switch, J5 Limit switch, J6 Conn_ARM_JTAG_SWD_10, J9 USB_C_Receptacle_USB2.0_16P, U1 RP2040, U2 DRV8870DDA, U3 INA180A1, U5 SP3485EN, U6 TLV75533PDBV, U7 TPS54202DDC, U8 W25Q16JVUXIQ, U9 TLV75533PDBV, Y1 ABM8-272-T3

Commit message: Progressed ECAD.
Parts:
- added C34: 100nC, Capacitor_SMD:C_0805_2012Metric, F.Cu at (148.6, 127.5)
- added Q1: BC847, Package_TO_SOT_SMD:SOT-23, F.Cu at (148.8, 121.8)
- added Q2: BC847, Package_TO_SOT_SMD:SOT-23, F.Cu at (140.1, 120.2)
- added Q3: BC847, Package_TO_SOT_SMD:SOT-23, F.Cu at (140.1, 124.9)
- added Q4: BC847, Package_TO_SOT_SMD:SOT-23, F.Cu at (140.1, 129.5)
- added R18: 5k1R, Resistor_SMD:R_0402_1005Metric, F.Cu at (134.5, 121.5)
- added R19: 5k1R, Resistor_SMD:R_0402_1005Metric, F.Cu at (134.5, 123.5)
- added R20: 5k1R, Resistor_SMD:R_0402_1005Metric, F.Cu at (134.5, 125.5)
- added R21: 5k1R, Resistor_SMD:R_0402_1005Metric, F.Cu at (134.5, 127.5)
Connections:
- D1 pad 1: GND -> Net-(D1-K)
- D2 pad 1: GND -> Net-(D2-K)
- D4 pad 1: GND -> Net-(D4-K)
- D5 pad 1: GND -> Net-(D5-K)

Commit message: Progressed ECAD.
Parts:
- added C35: 100nC, Capacitor_SMD:C_0805_2012Metric, F.Cu at (171.1, 119.5)
- added C36: 100nC, Capacitor_SMD:C_0805_2012Metric, F.Cu at (171.1, 122.5)
- added C37: 10uC, Capacitor_SMD:C_0805_2012Metric, F.Cu at (177.6, 119.5)
- added U10: PGA112, Package_SO:VSSOP-10_3x3mm_P0.5mm, F.Cu at (172.6, 113.7)
Connections:
- C34 pad 1: +3.3VA -> +3.3V
- R18 pad 2: unconnected-(R18-Pad2) -> /MCU/ON_LED
- R19 pad 2: unconnected-(R19-Pad2) -> /MCU/MOTOR_LIM_LED
- R20 pad 2: unconnected-(R20-Pad2) -> /MCU/RS485_LED
- R21 pad 2: unconnected-(R21-Pad2) -> /MCU/MOTOR_LED

Commit message: Progressed ECAD.
Parts:
- added C38: 100nC, Capacitor_SMD:C_0805_2012Metric, F.Cu at (173.3, 98.2)
- added R22: 1R, Resistor_SMD:R_0402_1005Metric, F.Cu at (176.5, 93.2)
- added R23: 200R, Resistor_SMD:R_0603_1608Metric, F.Cu at (173.1, 93.5)
- added U11: LM4040DBZ-3, Package_TO_SOT_SMD:SOT-23, F.Cu at (173.5, 90.0)
Connections:
- C27 pad 1: +3.3VA -> Net-(U1-ADC_AVDD)
- U1 pad 43: +3.3VA -> Net-(U1-ADC_AVDD)
- U10 pad 1: unconnected-(U10-AV_{DD}-Pad1) -> +3V0
- U10 pad 10: unconnected-(U10-DV_{DD}-Pad10) -> +3.3VA
- U10 pad 2: unconnected-(U10-CH1-Pad2) -> /Motor Control/A_SENSE_BASE
- U10 pad 3: unconnected-(U10-CH0/V_{CAL}-Pad3) -> +3V0
- U10 pad 4: unconnected-(U10-V_{REF}-Pad4) -> GND
- U10 pad 5: unconnected-(U10-V_{OUT}-Pad5) -> /Motor Control/A_SENSE
- U10 pad 6: unconnected-(U10-GND-Pad6) -> GND
- U3 pad 1: /Motor Control/A_SENSE -> /Motor Control/A_SENSE_BASE
- U3 pad 5: +3.3VA -> +3V0

Commit message: Progressed ECAD.
Parts:
- moved J4 33.6 mm to (198.6, 111.2), turned to 90 degrees
- moved J5 29.8 mm to (198.8, 85.5), turned to 90 degrees
- moved J1 4.55 mm to (199.1, 102.5)
Other:
- outline, holes or cut-outs redrawn

Commit message: Progressed ECAD.
Parts:
- added C40: 2u2C, Capacitor_SMD:C_0402_1005Metric, F.Cu at (168.8, 83.3)
- added C41: 2u2C, Capacitor_SMD:C_0402_1005Metric, F.Cu at (168.8, 85.2)
- added C42: 100nC, Capacitor_SMD:C_0805_2012Metric, F.Cu at (165.1, 83.8)
- added C43: 100nC, Capacitor_SMD:C_0805_2012Metric, F.Cu at (165.1, 86.8)
Connections:
- C27 pad 1: Net-(U1-ADC_AVDD) -> +3.3VA
- C38 pad 1: +3V0 -> +3.3VA
- R22 pad 2: Net-(U1-ADC_AVDD) -> unconnected-(R22-Pad2)
- R23 pad 1: +3.3VA -> unconnected-(R23-Pad1)
- U1 pad 43: Net-(U1-ADC_AVDD) -> +3.3VA
- U10 pad 1: +3V0 -> +3.3VA
- U3 pad 5: +3V0 -> +3.3VA

Commit message: Progressed ECAD.
Parts:
- added C44: 100nC, Capacitor_SMD:C_0201_0603Metric, F.Cu at (178.2, 88.0)
- added C45: 100nC, Capacitor_SMD:C_0201_0603Metric, F.Cu at (178.2, 89.8)
- added D3: 1N4148WT, Diode_SMD:D_SOD-523, F.Cu at (178.8, 81.5)
- added D6: 1N4148WT, Diode_SMD:D_SOD-523, F.Cu at (178.8, 83.9)
- C43: value 100nC -> 2u2C; footprint Capacitor_SMD:C_0805_2012Metric -> Capacitor_SMD:C_0402_1005Metric
- moved C43 17.8 mm to (182.0, 81.2)
Connections:
- net Net-(C4-Pad1) renamed /Motor Control/LIM1
- net Net-(C5-Pad1) renamed /Motor Control/LIM2
- U10 pad 3: +3V0 -> +3.3VA
- U10 pad 7: unconnected-(U10-SCLK-Pad7) -> /Motor Control/PGA_SCLK
- U10 pad 8: unconnected-(U10-DIO-Pad8) -> /Motor Control/PGA_DIO
- U10 pad 9: unconnected-(U10-~{CS}-Pad9) -> /Motor Control/~{PGA_CS}
Other:
- board size 105.5 x 38 mm -> 110 x 38 mm

Commit message: Progressed ECAD.
Parts:
- removed C29: 10uC, Capacitor_SMD:C_0805_2012Metric
- removed C36: 100nC, Capacitor_SMD:C_0805_2012Metric
- removed D3, D6: 1N4148WT, Diode_SMD:D_SOD-523
- removed R22: 1R, Resistor_SMD:R_0402_1005Metric
- removed R23: 200R, Resistor_SMD:R_0603_1608Metric
- removed U11: LM4040DBZ-3, Package_TO_SOT_SMD:SOT-23
- removed U9: TLV75533PDBV, Package_TO_SOT_SMD:SOT-23-5
- added C46: 100nC, Capacitor_SMD:C_0201_0603Metric, F.Cu at (170.7, 94.0)
- added R24: 27R, Resistor_SMD:R_0201_0603Metric, F.Cu at (166.2, 87.4)
- added R28: 27R, Resistor_SMD:R_0201_0603Metric, F.Cu at (166.2, 89.1)
- added R30: 27R, Resistor_SMD:R_0201_0603Metric, F.Cu at (166.2, 90.9)
- added U12: REF3033, Package_TO_SOT_SMD:SOT-23, F.Cu at (171.9, 88.9)
- C41: value 2u2C -> 15pC; footprint Capacitor_SMD:C_0402_1005Metric -> Capacitor_SMD:C_0201_0603Metric
- C44: value 100nC -> 15pC
Connections:
- C41 pad 1: +3.3VA -> GND
- C41 pad 2: GND -> /Motor Control/ENCODER_A
- C44 pad 1: +3.3VA -> GND
- C44 pad 2: GND -> /Motor Control/ENCODER_B
- J1 pad 3: /Motor Control/ENCODER- -> +3.3V
- J1 pad 4: /Motor Control/ENCODER+ -> GND
- U10 pad 5: /Motor Control/A_SENSE -> Net-(U10-V_{OUT})

Commit message: Progressed ECAD.
Parts:
- R24: value 27R -> 250R
- moved Q4 62.2 mm to (99.9, 82.0)
- moved D5 53.4 mm to (99.0, 87.0)
- moved R20 50.8 mm to (102.5, 86.0)
Other:
- board size 110 x 38 mm -> 110 x 37 mm
Changed lines of the file:
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@@
 	(footprint "Resistor_SMD:R_0402_1005Metric"
 		(layer "F.Cu")
-		(at 134.49 125.51)
+		(at 102.49 86)
 		(descr "Resistor SMD 0402 (1005 Metric), square (rectangular) end terminal, IPC-7351 nominal, (Body size source: IPC-SM-782 page 72, https://www.pcb-3d.com/wordpress/wp-content/uploads/ipc-sm-782a_amendment_1_and_2.pdf), generated with kicad-footprint-generator")
 		(tags "resistor")
@@
 	(footprint "Package_TO_SOT_SMD:SOT-23"
 		(layer "F.Cu")
-		(at 140.0625 129.5)
+		(at 99.9375 81.95)
 		(descr "SOT, 3 Pin (JEDEC TO-236 Var AB https://www.jedec.org/document_search?search_api_views_fulltext=TO-236), generated with kicad-footprint-generator ipc_gullwing_generator.py")
 		(tags "SOT TO_SOT_SMD")
@@
 			)
 		)
-		(property "Value" "27R"
+		(property "Value" "250R"
 			(at 0 1.05 0)
 			(layer "F.Fab")
@@
 			)
 		)
-		(property "MPN" "RC0201FR-0727RL"
+		(property "MPN" ""
 			(at 0 0 0)
 			(unlocked yes)
@@
 	(footprint "LED_SMD:LED_0805_2012Metric"
 		(layer "F.Cu")
-		(at 144.5 115)
+		(at 99 87)
 		(descr "LED SMD 0805 (2012 Metric), square (rectangular) end terminal, IPC-7351 nominal, (Body size source: https://docs.google.com/spreadsheets/d/1BsfQQcO9C6DZCsRaXUlFlo91Tg2WpOkGARC1WS5S8t0/edit?usp=sharing), generated with kicad-footprint-generator")
 		(tags "LED")
@@
 		)
 	)
-	(gr_arc
-		(start 97 106)
-		(mid 96.292893 105.707107)
-		(end 96 105)
-		(stroke
-			(width 0.05)
-			(type default)
-		)
-		(layer "Edge.Cuts")
-	)
-	(gr_arc
-		(start 103.5 88)
-		(mid 103.207107 88.707107)
-		(end 102.5 89)
-		(stroke
-			(width 0.05)
-			(type default)
-		)
-		(layer "Edge.Cuts")
-	)
-	(gr_line
-		(start 103.5 110)
-		(end 103.5 107)
-		(stroke
-			(width 0.05)
-			(type default)
-		)
-		(layer "Edge.Cuts")
-	)
-	(gr_arc
-		(start 96 90)
-		(mid 96.292893 89.292893)
-		(end 97 89)
-		(stroke
-			(width 0.05)
-			(type default)
-		)
-		(layer "Edge.Cuts")
-	)
-	(gr_line
-		(start 110 78.5)
-		(end 206 78.5)
-		(stroke
-			(width 0.05)
-			(type default)
-		)
-		(layer "Edge.Cuts")
-	)
 	(gr_line
-		(start 206 78.5)
-		(end 206 116.5)
+		(start 96 79)
+		(end 206 79)
 		(stroke
 			(width 0.05)
@@
 	)
 	(gr_line
-		(start 96 105)
-		(end 96 90)
+		(start 206 79)
+		(end 206 116)
 		(stroke
 			(width 0.05)
@@
 	)
 	(gr_line
-		(start 103.5 88)
-		(end 103.5 85)
-		(stroke
-			(width 0.05)
-			(type default)
-		)
-		(layer "Edge.Cuts")
-	)
-	(gr_line
-		(start 102.5 106)
-		(end 97 106)
-		(stroke
-			(width 0.05)
-			(type default)
-		)
-		(layer "Edge.Cuts")
-	)
-	(gr_line
-		(start 110 116.5)
-		(end 206 116.5)
-		(stroke
-			(width 0.05)
-			(type default)
-		)
-		(layer "Edge.Cuts")
-	)
-	(gr_arc
-		(start 103.5 85)
-		(mid 105.403806 80.403806)
-		(end 110 78.5)
-		(stroke
-			(width 0.05)
-			(type default)
-		)
-		(layer "Edge.Cuts")
-	)
-	(gr_arc
-		(start 102.5 106)
-		(mid 103.207107 106.292893)
-		(end 103.5 107)
-		(stroke
-			(width 0.05)
-			(type default)
-		)
-		(layer "Edge.Cuts")
-	)
-	(gr_arc
-		(start 110 116.5)
-		(mid 105.403806 114.596194)
-		(end 103.5 110)
+		(start 96 116)
+		(end 96 79)
 		(stroke
 			(width 0.05)
@@
 	)
 	(gr_line
-		(start 102.5 89)
-		(end 97 89)
+		(start 96 116)
+		(end 206 116)
 		(stroke
 			(width 0.05)
