File: ECAD/BDCMotorControlBoard/BDCMotorControlBoard.kicad_sch (KiCad schematic)
At the start: 1 part, among them J1 Conn_01x06

Commit message: Progressed ECAD.
Other:
- added sheet RS485 (rs485.kicad_sch)
Changed lines of the file:
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@@
+		)
+	)
+	(sheet
+		(at 106.68 111.76)
+		(size 30.48 26.67)
+		(exclude_from_sim no)
+		(in_bom yes)
+		(on_board yes)
+		(dnp no)
+		(fields_autoplaced yes)
+		(stroke
+			(width 0.1524)
+			(type solid)
+		)
+		(fill
+			(color 0 0 0 0.0000)
+		)
+		(property "Sheetname" "RS485"
+			(at 106.68 111.0484 0)
+			(effects
+				(font
+					(size 1.27 1.27)
+				)
+				(justify left bottom)
+			)
+		)
+		(property "Sheetfile" "rs485.kicad_sch"
+			(at 106.68 139.0146 0)
+			(effects
+				(font
+					(size 1.27 1.27)
+				)
+				(justify left top)
+			)
+		)
+		(instances
+			(project "BDCMotorControlBoard"
+				(path "/249dd5db-06ad-47dc-a5d6-b66af80e4bef"
+					(page "5")
+				)
+			)
 		)
 	)

Commit message: Progressed ECAD.
Parts:
- J1: footprint (none) -> Connector_JST:JST_PH_S6B-PH-K_1x06_P2.00mm_Horizontal
Changed lines of the file:
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@@
 			)
 		)
-		(property "Footprint" ""
+		(property "Footprint" "Connector_JST:JST_PH_S6B-PH-K_1x06_P2.00mm_Horizontal"
 			(at 254 62.23 0)
 			(effects

Commit message: Progressed ECAD.
Parts:
- removed J1: Conn_01x06, Connector_JST:JST_PH_S6B-PH-K_1x06_P2.00mm_Horizontal, symbol Connector_Generic:Conn_01x06
Other:
- removed sheet H-Bridge
- added sheet Motor Control (motor_control.kicad_sch)
Changed lines of the file:
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@@
 	(generator_version "9.0")
 	(paper "A4")
-	(symbol
-		(lib_id "Connector_Generic:Conn_01x06")
-		(at 254 62.23 0)
-		(unit 1)
-		(exclude_from_sim no)
-		(in_bom yes)
-		(on_board yes)
-		(dnp no)
-		(fields_autoplaced yes)
-		(property "Reference" "J1"
-			(at 256.54 62.2299 0)
-			(effects
-				(font
-					(size 1.27 1.27)
-				)
-				(justify left)
-			)
-		)
-		(property "Value" "Conn_01x06"
-			(at 256.54 64.7699 0)
-			(effects
-				(font
-					(size 1.27 1.27)
-				)
-				(justify left)
-			)
-		)
-		(property "Footprint" "Connector_JST:JST_PH_S6B-PH-K_1x06_P2.00mm_Horizontal"
-			(at 254 62.23 0)
-			(effects
-				(font
-					(size 1.27 1.27)
-				)
-				(hide yes)
-			)
-		)
-		(property "Datasheet" "~"
-			(at 254 62.23 0)
-			(effects
-				(font
-					(size 1.27 1.27)
-				)
-				(hide yes)
-			)
-		)
-		(property "Description" "Generic connector, single row, 01x06, script generated (kicad-library-utils/schlib/autogen/connector/)"
-			(at 254 62.23 0)
-			(effects
-				(font
-					(size 1.27 1.27)
-				)
-				(hide yes)
-			)
-		)
-		(property "Status" ""
-			(at 254 62.23 0)
-			(effects
-				(font
-					(size 1.27 1.27)
-				)
-				(hide yes)
-			)
-		)
-		(pin "2"
-		)
-		(pin "4"
-		)
-		(pin "1"
-		)
-		(pin "5"
-		)
-		(pin "3"
-		)
-		(pin "6"
-		)
-		(instances
-			(project ""
-				(path "/249dd5db-06ad-47dc-a5d6-b66af80e4bef"
-					(reference "J1")
-					(unit 1)
-				)
-			)
-		)
-	)
 	(sheet
-		(at 124.46 53.34)
+		(at 198.12 111.76)
 		(size 35.56 38.1)
 		(exclude_from_sim no)
@@
 		)
 		(property "Sheetname" "Power Supply"
-			(at 124.46 52.6284 0)
+			(at 198.12 111.0484 0)
 			(effects
 				(font
@@
 		)
 		(property "Sheetfile" "power_supply.kicad_sch"
-			(at 124.46 92.0246 0)
+			(at 198.12 150.4446 0)
 			(effects
 				(font
@@
 	)
 	(sheet
-		(at 187.96 40.64)
+		(at 107.95 68.58)
 		(size 25.4 22.86)
 		(exclude_from_sim no)
@@
 		)
 		(property "Sheetname" "MCU"
-			(at 187.96 39.9284 0)
+			(at 107.95 67.8684 0)
 			(effects
 				(font
@@
 		)
 		(property "Sheetfile" "mcu.kicad_sch"
-			(at 187.96 64.0846 0)
+			(at 107.95 92.0246 0)
 			(effects
 				(font
@@
 	)
 	(sheet
-		(at 185.42 85.09)
-		(size 34.29 30.48)
+		(at 194.31 54.61)
+		(size 30.48 19.05)
 		(exclude_from_sim no)
 		(in_bom yes)
@@
 			(color 0 0 0 0.0000)
 		)
-		(property "Sheetname" "H-Bridge"
-			(at 185.42 84.3784 0)
+		(property "Sheetname" "Motor Control"
+			(at 194.31 53.8984 0)
 			(effects
 				(font
@@
 			)
 		)
-		(property "Sheetfile" "h_bridge.kicad_sch"
-			(at 185.42 116.1546 0)
+		(property "Sheetfile" "motor_control.kicad_sch"
+			(at 194.31 74.2446 0)
 			(effects
 				(font
@@
 			(project "BDCMotorControlBoard"
 				(path "/249dd5db-06ad-47dc-a5d6-b66af80e4bef"
-					(page "3")
+					(page "7")
 				)
 			)

Commit message: Progressed ECAD.
Other:
- sheet MCU ports: added MOTOR_A_SENSE, MOTOR_LIM1, MOTOR_LIM2, MOTOR_PWM1, MOTOR_PWM2, RS485_DE, RS485_RX, RS485_TX, RS485_~{RE}; removed none
- sheet Motor Control ports: added A_SENSE, LIM1, LIM2, PWM1, PWM2; removed none
- sheet RS485 ports: added DE, RX, TX, ~{RE}; removed none
Changed lines of the file:
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@@
 	(paper "A4")
 	(sheet
-		(at 198.12 111.76)
+		(at 214.63 114.3)
 		(size 35.56 38.1)
 		(exclude_from_sim no)
@@
 		)
 		(property "Sheetname" "Power Supply"
-			(at 198.12 111.0484 0)
+			(at 214.63 113.5884 0)
 			(effects
 				(font
@@
 		)
 		(property "Sheetfile" "power_supply.kicad_sch"
-			(at 198.12 150.4446 0)
+			(at 214.63 152.9846 0)
 			(effects
 				(font
@@
 	(sheet
 		(at 107.95 68.58)
-		(size 25.4 22.86)
+		(size 41.91 35.56)
 		(exclude_from_sim no)
 		(in_bom yes)
@@
 		)
 		(property "Sheetfile" "mcu.kicad_sch"
-			(at 107.95 92.0246 0)
+			(at 107.95 104.7246 0)
 			(effects
 				(font
@@
 				)
 				(justify left top)
+			)
+		)
+		(pin "RS485_DE" output
+			(at 107.95 76.2 180)
+			(effects
+				(font
+					(size 1.27 1.27)
+				)
+				(justify left)
+			)
+		)
+		(pin "RS485_RX" input
+			(at 107.95 85.09 180)
+			(effects
+				(font
+					(size 1.27 1.27)
+				)
+				(justify left)
+			)
+		)
+		(pin "RS485_TX" output
+			(at 107.95 78.74 180)
+			(effects
+				(font
+					(size 1.27 1.27)
+				)
+				(justify left)
+			)
+		)
+		(pin "RS485_~{RE}" output
+			(at 107.95 82.55 180)
+			(effects
+				(font
+					(size 1.27 1.27)
+				)
+				(justify left)
+			)
+		)
+		(pin "MOTOR_A_SENSE" input
+			(at 149.86 82.55 0)
+			(effects
+				(font
+					(size 1.27 1.27)
+				)
+				(justify right)
+			)
+		)
+		(pin "MOTOR_PWM1" output
+			(at 149.86 76.2 0)
+			(effects
+				(font
+					(size 1.27 1.27)
+				)
+				(justify right)
+			)
+		)
+		(pin "MOTOR_PWM2" output
+			(at 149.86 78.74 0)
+			(effects
+				(font
+					(size 1.27 1.27)
+				)
+				(justify right)
+			)
+		)
+		(pin "MOTOR_LIM1" input
+			(at 149.86 85.09 0)
+			(effects
+				(font
+					(size 1.27 1.27)
+				)
+				(justify right)
+			)
+		)
+		(pin "MOTOR_LIM2" input
+			(at 149.86 87.63 0)
+			(effects
+				(font
+					(size 1.27 1.27)
+				)
+				(justify right)
 			)
 		)
@@
 	)
 	(sheet
-		(at 194.31 54.61)
+		(at 167.64 69.85)
 		(size 30.48 19.05)
 		(exclude_from_sim no)
@@
 		)
 		(property "Sheetname" "Motor Control"
-			(at 194.31 53.8984 0)
+			(at 167.64 69.1384 0)
 			(effects
 				(font
@@
 		)
 		(property "Sheetfile" "motor_control.kicad_sch"
-			(at 194.31 74.2446 0)
+			(at 167.64 89.4846 0)
 			(effects
 				(font
@@
 				)
 				(justify left top)
+			)
+		)
+		(pin "A_SENSE" output
+			(at 167.64 82.55 180)
+			(effects
+				(font
+					(size 1.27 1.27)
+				)
+				(justify left)
+			)
+		)
+		(pin "PWM1" input
+			(at 167.64 73.66 180)
+			(effects
+				(font
+					(size 1.27 1.27)
+				)
+				(justify left)
+			)
+		)
+		(pin "PWM2" input
+			(at 167.64 76.2 180)
+			(effects
+				(font
+					(size 1.27 1.27)
+				)
+				(justify left)
+			)
+		)
+		(pin "LIM1" output
+			(at 167.64 85.09 180)
+			(effects
+				(font
+					(size 1.27 1.27)
+				)
+				(justify left)
+			)
+		)
+		(pin "LIM2" output
+			(at 167.64 87.63 180)
+			(effects
+				(font
+					(size 1.27 1.27)
+				)
+				(justify left)
 			)
 		)
@@
 	)
 	(sheet
-		(at 106.68 111.76)
-		(size 30.48 26.67)
+		(at 45.72 73.66)
+		(size 30.48 13.97)
 		(exclude_from_sim no)
 		(in_bom yes)
@@
 		)
 		(property "Sheetname" "RS485"
-			(at 106.68 111.0484 0)
+			(at 45.72 72.9484 0)
 			(effects
 				(font
@@
 		)
 		(property "Sheetfile" "rs485.kicad_sch"
-			(at 106.68 139.0146 0)
+			(at 45.72 88.2146 0)
 			(effects
 				(font
@@
 			)
 		)
+		(pin "DE" input
+			(at 76.2 76.2 0)
+			(effects
+				(font
+					(size 1.27 1.27)
+				)
+				(justify right)
+			)
+		)
+		(pin "RX" output
+			(at 76.2 85.09 0)
+			(effects
+				(font
+					(size 1.27 1.27)
+				)
+				(justify right)
+			)
+		)
+		(pin "TX" input
+			(at 76.2 78.74 0)
+			(effects
+				(font
+					(size 1.27 1.27)
+				)
+				(justify right)
+			)
+		)
+		(pin "~{RE}" input
+			(at 76.2 82.55 0)
+			(effects
+				(font
+					(size 1.27 1.27)
+				)
+				(justify right)
+			)
+		)

Commit message: Progressed ECAD.
Other:
- sheet Motor Control ports: added A_SENSE_LP; removed none
Changed lines of the file:
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@@
 	(sheet
 		(at 167.64 69.85)
-		(size 30.48 19.05)
+		(size 30.48 20.32)
 		(exclude_from_sim no)
 		(in_bom yes)
@@
 		)
 		(property "Sheetfile" "motor_control.kicad_sch"
-			(at 167.64 89.4846 0)
+			(at 167.64 90.7546 0)
 			(effects
 				(font
@@
 		)
 		(pin "A_SENSE" output
-			(at 167.64 82.55 180)
+			(at 167.64 80.01 180)
 			(effects
 				(font
@@
 		)
 		(pin "PWM1" input
-			(at 167.64 73.66 180)
+			(at 167.64 72.39 180)
 			(effects
 				(font
@@
 		)
 		(pin "PWM2" input
-			(at 167.64 76.2 180)
+			(at 167.64 74.93 180)
 			(effects
 				(font
@@
 			(effects
 				(font
+					(size 1.27 1.27)
+				)
+				(justify left)
+			)
+		)
+		(pin "A_SENSE_LP" output
+			(at 167.64 82.55 180)
+			(effects
+				(font

Commit message: Progressed ECAD.
Other:
- sheet MCU ports: added MOTOR_ENCODER_A, MOTOR_ENCODER_B, MOTOR_PGA_DIO, MOTOR_PGA_SCLK, ~{MOTOR_PGA_CS}; removed none
- sheet Motor Control ports: added ENCODER_A, ENCODER_B, PGA_DIO, PGA_SCLK, ~{PGA_CS}; removed A_SENSE_LP
