File: ECAD/BDCMotorControlShieldMega/motor_control.kicad_sch (KiCad schematic)
At the start: 5 parts, among them U15 MCP6S26

Commit message: Progressed ECAD.
Parts:
- U15: MPN (none) -> MCP6S26-I/SL
Connections:
- net A_SENSE_BASE renamed A_SENSE
Other:
- moved on the sheet: C24, R30
Changed lines of the file:
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@@
 	)
 	(junction
-		(at 59.69 119.38)
+		(at 68.58 119.38)
 		(diameter 0)
 		(color 0 0 0 0)
@@
 	(wire
 		(pts
-			(xy 50.8 119.38) (xy 35.56 119.38)
+			(xy 59.69 119.38) (xy 58.42 119.38)
 		)
 		(stroke
@@
 	(wire
 		(pts
-			(xy 59.69 119.38) (xy 91.44 119.38)
+			(xy 68.58 119.38) (xy 91.44 119.38)
 		)
 		(stroke
@@
 	(wire
 		(pts
-			(xy 58.42 119.38) (xy 59.69 119.38)
+			(xy 67.31 119.38) (xy 68.58 119.38)
 		)
 		(stroke
@@
 	(wire
 		(pts
-			(xy 59.69 119.38) (xy 59.69 120.65)
+			(xy 68.58 119.38) (xy 68.58 120.65)
 		)
 		(stroke
@@
 			)
 			(justify right bottom)
-		)
-	)
-	(label "A_SENSE_BASE"
-		(at 35.56 119.38 0)
-		(effects
-			(font
-				(size 1.27 1.27)
-			)
-			(justify left bottom)
 		)
 	)
@@
 		(shape input)
 		(at 210.82 46.99 180)
+		(effects
+			(font
+				(size 1.27 1.27)
+			)
+			(justify right)
+		)
+	)
+	(hierarchical_label "A_SENSE"
+		(shape output)
+		(at 58.42 119.38 180)
 		(effects
 			(font
@@
 	(symbol
 		(lib_id "Device:R")
-		(at 54.61 119.38 270)
+		(at 63.5 119.38 270)
 		(mirror x)
 		(unit 1)
@@
 		(fields_autoplaced yes)
 		(property "Reference" "R30"
-			(at 54.61 113.03 90)
+			(at 63.5 113.03 90)
 			(effects
 				(font
@@
 		)
 		(property "Value" "1kR"
-			(at 54.61 115.57 90)
+			(at 63.5 115.57 90)
 			(effects
 				(font
@@
 		)
 		(property "Footprint" "Resistor_SMD:R_0402_1005Metric"
-			(at 54.61 121.158 90)
+			(at 63.5 121.158 90)
 			(effects
 				(font
@@
 		)
 		(property "Datasheet" "~"
-			(at 54.61 119.38 0)
+			(at 63.5 119.38 0)
 			(effects
 				(font
@@
 		)
 		(property "Description" "Resistor"
-			(at 54.61 119.38 0)
+			(at 63.5 119.38 0)
 			(effects
 				(font
@@
 		)
 		(property "MPN" "RC0402FR-071KL"
-			(at 54.61 119.38 90)
+			(at 63.5 119.38 90)
 			(effects
 				(font
@@
 	(symbol
 		(lib_id "power:GND")
-		(at 59.69 128.27 0)
+		(at 68.58 128.27 0)
 		(unit 1)
 		(exclude_from_sim no)
@@
 		(fields_autoplaced yes)
 		(property "Reference" "#PWR0119"
-			(at 59.69 134.62 0)
+			(at 68.58 134.62 0)
 			(effects
 				(font
@@
 		)
 		(property "Value" "GND"
-			(at 59.69 133.35 0)
+			(at 68.58 133.35 0)
 			(effects
 				(font
@@
 		)
 		(property "Footprint" ""
-			(at 59.69 128.27 0)
+			(at 68.58 128.27 0)
 			(effects
 				(font
@@
 		)
 		(property "Datasheet" ""
-			(at 59.69 128.27 0)
+			(at 68.58 128.27 0)
 			(effects
 				(font
@@
 		)
 		(property "Description" "Power symbol creates a global label with name \"GND\" , ground"
-			(at 59.69 128.27 0)
+			(at 68.58 128.27 0)
 			(effects
 				(font
@@
 			)
 		)
+		(property "MPN" "MCP6S26-I/SL"
+			(at 102.87 111.76 0)
+			(effects
+				(font
+					(size 1.27 1.27)
+				)
+				(hide yes)
+			)
+		)
 		(pin "5"
 		)
@@
 	(symbol
 		(lib_id "Device:C")
-		(at 59.69 124.46 0)
+		(at 68.58 124.46 0)
 		(unit 1)
 		(exclude_from_sim no)
@@
 		(fields_autoplaced yes)
 		(property "Reference" "C24"
-			(at 63.5 123.1899 0)
+			(at 72.39 123.1899 0)
 			(effects
 				(font
@@
 		)
 		(property "Value" "100pC"
-			(at 63.5 125.7299 0)
+			(at 72.39 125.7299 0)
 			(effects
 				(font
@@
 		)
 		(property "Footprint" "Capacitor_SMD:C_0402_1005Metric"
-			(at 60.6552 128.27 0)
+			(at 69.5452 128.27 0)
 			(effects
 				(font
@@
 		)
 		(property "Datasheet" "~"
-			(at 59.69 124.46 0)
+			(at 68.58 124.46 0)
 			(effects
 				(font
@@
 		)
 		(property "Description" "Unpolarized capacitor"
-			(at 59.69 124.46 0)
-			(effects
-				(font
+			(at 68.58 124.46 0)
+			(effects
+				(font

Commit message: Progressed ECAD.
Parts:
- C53: renamed from C24; footprint Capacitor_SMD:C_0402_1005Metric -> Capacitor_SMD:C_0805_2012Metric
- C54: renamed from C23; MPN (none) -> C0805F104K5RACAUTO
- C55: renamed from C22; MPN (none) -> C0805F104K5RACAUTO
- R39: renamed from R30; footprint Resistor_SMD:R_0402_1005Metric -> Resistor_SMD:R_0805_2012Metric; MPN RC0402FR-071KL -> AC0805FR-7W1KL
- renumbered U15 to U23

Commit message: Progressed ECAD.
Parts:
- added L4: 10uL, Inductor_SMD:L_0805_2012Metric, symbol Device:L
- renumbered C53 to C57, C54 to C58, C55 to C59, R39 to R37
Connections:
- net +5V: now also L4.1; no longer C59.1
- net GND: now also U23.8 (V_{REF})
- net ~{PG_CS}: now reaches U23.10 (~{CS})
- net PGA_SI: now reaches U23.11 (SI)
- net PGA_SO: now reaches U23.12 (SO)
- net PGA_SCK: now reaches U23.13 (SCK)
- net at U23.14 (V_{DD}): now also C59.1, L4.2
Other:
- sheet H-bridge #1 ports: added ~{ENABLE_ENCODER}; removed none
- sheet H-bridge #2 ports: added ~{ENABLE_ENCODER}; removed none
- sheet H-bridge #3 ports: added ~{ENABLE_ENCODER}; removed none
- moved on the sheet: C58, C59

Commit message: Progressed ECAD.
Parts:
- added C60: 100nC, Capacitor_SMD:C_0805_2012Metric, symbol Device:C
- added U24: 74AHC1G79, Package_TO_SOT_SMD:SOT-353_SC-70-5, symbol 74xGxx:74AUC1G79
Connections:
- net +5V: now also C60.1, U24.5 (VCC)
- net ENCODER_A: now also U24.1 (D)
- net ENCODER_B: now also U24.2 (C)
- net GND: now also C60.2, U24.3 (GND)

Commit message: Progressed ECAD.
Parts:
- removed C57: 100pC, Capacitor_SMD:C_0805_2012Metric, symbol Device:C
- removed C60: 100nC, Capacitor_SMD:C_0805_2012Metric, symbol Device:C
- removed R37: 1kR, Resistor_SMD:R_0805_2012Metric, symbol Device:R
- removed U24: 74AHC1G79, Package_TO_SOT_SMD:SOT-353_SC-70-5, symbol 74xGxx:74AUC1G79
- C58, C59: Status (none) -> OK
Connections:
- net A_SENSE: now also U23.1 (V_{OUT})
Other:
- note removed: "SAR ADC Charge bucket filter Low pass filter -3dB Cutoff Frequency: 1,6 MHz"
- moved on the sheet: C58, C59, L4, U23

Commit message: Progressed ECAD.
Parts:
- U23: Status (none) -> OK
Changed lines of the file:
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@@
+			)
+		)
+		(property "Status" "OK"
+			(at 116.84 95.25 0)
+			(effects
+				(font
+					(size 1.27 1.27)
+				)
+				(hide yes)
 			)
 		)

Commit message: Progressed ECAD.
Parts:
- added C15, C16, C17, C26, C41, C42, C52: 100nC, Capacitor_SMD:C_0805_2012Metric, symbol Device:C
- added J10, J11, J13, J14, J16, J17: Limit switch, Connector_JST:JST_PH_B2B-PH-K_1x02_P2.00mm_Vertical, symbol Connector_Generic:Conn_01x02
- added R14, R15, R16, R17, R23, R24, R25, R26, R32, R33, R34, R35: 10kR, Resistor_SMD:R_0805_2012Metric, symbol Device:R
- added U5: 74AHC14, Package_SO:TSSOP-14_4.4x5mm_P0.65mm, symbol 74xx:74HC14
Connections:
- net +5V: now also C15.1, R16.2, R17.2, R24.2, R33.2, R34.2, R35.2, U5.14 (VCC)
- net GND: now also C15.2, C16.2, C17.2, C26.2, C41.2, C42.2, C52.2, J10.2 (Pin_2), J11.2 (Pin_2), J13.2 (Pin_2), J14.2 (Pin_2), J16.2 (Pin_2), J17.2 (Pin_2), U5.7 (GND)
- net CURRENT1: no longer names the net of U23.2 (CH0)
- net CURRENT2: no longer names the net of U23.3 (CH1)
- net CURRENT3: no longer names the net of U23.4 (CH2)
- new net: J16.1 (Pin_1), R26.2, R34.1
- new net: J17.1 (Pin_1), R32.2, R35.1
- new net: C16.1, R14.1, U5.5
- new net: J13.1 (Pin_1), R23.2, R24.1
- new net: J14.1 (Pin_1), R25.2, R33.1
- new net: C41.1, R25.1, U5.13
- new net: C17.1, R15.1, U5.9
- new net: J11.1 (Pin_1), R15.2, R17.1
- new net: C26.1, R23.1, U5.11
- new net: J10.1 (Pin_1), R14.2, R16.1
- new net: C52.1, R32.1, U5.1
- new net: C42.1, R26.1, U5.3
- new net LIM_SW_1: U5.6
- new net LIM_SW_2: U5.8
- new net LIM_SW_3: U5.10
- new net LIM_SW_4: U5.12
- new net LIM_SW_5: U5.4
- new net LIM_SW_6: U5.2
Other:
- added sheet H-bridge #4 (h_bridge.kicad_sch)
- added sheet H-bridge #5 (h_bridge.kicad_sch)
- added sheet H-bridge #6 (h_bridge.kicad_sch)
- sheet H-bridge #1 ports: added ENABLE_MOTOR, FORWARD/~{REVERSE}, PWM; removed ENABLE_PWM, LIM1, LIM2, PWM1, PWM2, ~{ENABLE_ENCODER}
- sheet H-bridge #2 ports: added ENABLE_MOTOR, FORWARD/~{REVERSE}, PWM; removed ENABLE_PWM, LIM1, LIM2, PWM1, PWM2, ~{ENABLE_ENCODER}
- sheet H-bridge #3 ports: added ENABLE_MOTOR, FORWARD/~{REVERSE}, PWM; removed ENABLE_PWM, LIM1, LIM2, PWM1, PWM2, ~{ENABLE_ENCODER}
- note added: "Limit switches debouncing"
- moved on the sheet: C58, C59, L4, U23

Commit message: Progressed ECAD.
Parts:
- added C65, C66: 100nC, Capacitor_SMD:C_0805_2012Metric, symbol Device:C
- added L8: 10uL, Inductor_SMD:L_0805_2012Metric, symbol Device:L
- added U12: MCP6S26, Package_SO:SOIC-14_3.9x8.7mm_P1.27mm, symbol Analog_custom:MCP6S26
Connections:
- net +5V: now also C66.1, L8.1
- net CURRENT_M1A: now also U23.2 (CH0), U12.2 (CH0)
- net CURRENT_M1B: now also U23.3 (CH1), U12.3 (CH1)
- net CURRENT_M2A: now also U23.4 (CH2), U12.4 (CH2)
- net CURRENT_M2B: now also U23.5 (CH3), U12.5 (CH3)
- net CURRENT_M3A: now also U23.6 (CH4), U12.6 (CH4)
- net CURRENT_M3B: now also U23.7 (CH5), U12.7 (CH5)
- net GND: now also C65.2, C66.2, U12.8 (V_{REF}), U12.9 (GND); no longer U23.5 (CH3), U23.6 (CH4), U23.7 (CH5)
- net PGA_SCK: now also U12.13 (SCK)
- net PGA_SI: now also U12.11 (SI)
- net PGA_SO: now also U12.12 (SO)
- net A_SENSE renamed A_SENSE_0
- net ~{PG_CS} renamed ~{PG_CS}_0
- new net: C65.1, L8.2, U12.14 (V_{DD})
- new net A_SENSE_1: U12.1 (V_{OUT})
- new net ~{PG_CS}_1: U12.10 (~{CS})
Other:
- moved on the sheet: C15, C58, C59, L4, U23, U5G
