File: ECAD/BDCMotorControlShieldMega/BDCMotorControlShieldMega.kicad_pcb (KiCad board)
At the start: 2 copper layers, 101.6 x 53.3 mm, 104 parts, among them J1 Power, J10 Limit switch, J11 Motor Connector, J12 Limit switch, J13 Limit switch, J14 Motor Connector, J15 Barrel_Jack_Switch, J18 Motor Connector, J19 Limit switch, J2 PWM, J3 Analog, J4 PWM, J5 Analog, J6 Communication, J7 Digital, J8 Limit switch, J9 Limit switch, U1 DRV8870DDA, U14 INA180A1, U2 INA180A1, U3 DRV8870DDA, U4 INA180A1, U5 PCA9535PW, U6 LM4040DBZ-4.1, U7 DRV8870DDA, U8 CY62148ELL-45ZSXIT, U9 PGA112

Commit message: Progressed ECAD.
Parts:
- removed J19: Limit switch, Connector_JST:JST_PH_B2B-PH-K_1x02_P2.00mm_Vertical
- removed R40: 10kR, Capacitor_SMD:C_0805_2012Metric
- removed R42, R43: 10kR, Resistor_SMD:R_0805_2012Metric_Pad1.20x1.40mm_HandSolder
- removed R47: 250mR, Resistor_SMD:R_2010_5025Metric
- added C25: 0.1uC, Capacitor_SMD:C_0805_2012Metric_Pad1.18x1.45mm_HandSolder, F.Cu at (235.9, 97.2)
- added C26: 0.1uC, Capacitor_SMD:C_0805_2012Metric_Pad1.18x1.45mm_HandSolder, F.Cu at (235.9, 100.2)
- added C28: 10uC, Capacitor_SMD:C_1210_3225Metric_Pad1.33x2.70mm_HandSolder, F.Cu at (240.1, 84.7)
- added C29: 47uC, Capacitor_THT:CP_Radial_D5.0mm_P2.00mm, F.Cu at (240.7, 99.0)
- added C30: 0.1uC, Capacitor_SMD:C_0805_2012Metric_Pad1.18x1.45mm_HandSolder, F.Cu at (235.9, 106.3)
- added C32: 100nC, Capacitor_SMD:C_0805_2012Metric, F.Cu at (231.3, 90.6)
- added C35: 0.1uC, Capacitor_SMD:C_0805_2012Metric_Pad1.18x1.45mm_HandSolder, F.Cu at (283.7, 49.7)
- added C37: 0.1uC, Capacitor_SMD:C_0805_2012Metric_Pad1.18x1.45mm_HandSolder, F.Cu at (283.7, 55.8)
- added C39: 47uC, Capacitor_THT:CP_Radial_D5.0mm_P2.00mm, F.Cu at (288.4, 51.5)
- added C40: 0.1uC, Capacitor_SMD:C_0805_2012Metric_Pad1.18x1.45mm_HandSolder, F.Cu at (283.7, 58.8)
- added C42: 100nC, Capacitor_SMD:C_0805_2012Metric, F.Cu at (279.1, 43.1)
- added C43: 100nC, Capacitor_SMD:C_0805_2012Metric, F.Cu at (279.1, 46.1)
- added C44: 100pC, Capacitor_SMD:C_0402_1005Metric, F.Cu at (294.1, 51.2)
- added C45: 10uC, Capacitor_SMD:C_1206_3216Metric, F.Cu at (264.1, 48.1)
- added C46: 100nC, Capacitor_SMD:C_0805_2012Metric, F.Cu at (260.8, 68.6)
- added C47: 100nC, Capacitor_SMD:C_0805_2012Metric, F.Cu at (260.8, 71.6)
- added C48: 100nC, Capacitor_SMD:C_0805_2012Metric, F.Cu at (260.8, 74.6)
- added J16: Limit switch, Connector_JST:JST_PH_B2B-PH-K_1x02_P2.00mm_Vertical, F.Cu at (271.9, 44.3)
- added J17: Limit switch, Connector_JST:JST_PH_B2B-PH-K_1x02_P2.00mm_Vertical, F.Cu at (271.9, 50.9)
- added L1: 10uL, Inductor_SMD:L_0805_2012Metric, F.Cu at (275.6, 102.9)
- added L2: 10uL, Inductor_SMD:L_0805_2012Metric, F.Cu at (256.9, 96.0)
- added L3: 10uL, Inductor_SMD:L_0805_2012Metric, F.Cu at (260.8, 57.0)
- added L4: 10uL, Inductor_SMD:L_0805_2012Metric, F.Cu at (260.8, 59.7)
- added R32: 10kR, Capacitor_SMD:C_0805_2012Metric, F.Cu at (279.1, 49.1)
- added R33: 10kR, Capacitor_SMD:C_0805_2012Metric, F.Cu at (279.1, 52.1)
- added R34: 10kR, Capacitor_SMD:C_0805_2012Metric, F.Cu at (279.1, 55.1)
- added R35: 10kR, Capacitor_SMD:C_0805_2012Metric, F.Cu at (279.1, 58.1)
- added R36: 1kR, Resistor_SMD:R_0402_1005Metric, F.Cu at (294.5, 57.8)
- added R37: 10kR, Resistor_SMD:R_0805_2012Metric, F.Cu at (227.8, 69.8)
- added R38: 10kR, Resistor_SMD:R_0805_2012Metric, F.Cu at (227.8, 72.8)
- added U10: 74HC2G08, Package_SO:TSSOP-8_3x3mm_P0.65mm, F.Cu at (241.8, 104.6)
- added U11: DRV8870DDA, Package_SO:Texas_HTSOP-8-1EP_3.9x4.9mm_P1.27mm_EP2.95x4.9mm_Mask2.4x3.1mm_ThermalVias, F.Cu at (238.2, 92.5)
- added U12: INA180A1, Package_TO_SOT_SMD:SOT-23-5, F.Cu at (245.7, 84.9)
- added U13: 74HC2G08, Package_SO:TSSOP-8_3x3mm_P0.65mm, F.Cu at (289.6, 57.1)
- added U15: INA180A1, Package_TO_SOT_SMD:SOT-23-5, F.Cu at (293.4, 37.4)
- added U16: PCA9555PW, Package_SO:TSSOP-24_4.4x7.8mm_P0.65mm, F.Cu at (235.0, 51.1)
- added U17: 74AHC373, Package_SO:TSSOP-20_4.4x6.5mm_P0.65mm, F.Cu at (244.1, 72.5)
- C1, C2, C27: value 100pC -> 0.1uC; footprint Capacitor_SMD:C_0402_1005Metric -> Capacitor_SMD:C_0805_2012Metric_Pad1.18x1.45mm_HandSolder
- C10: value 100nC -> 100pC; footprint Capacitor_SMD:C_0805_2012Metric -> Capacitor_SMD:C_0402_1005Metric
- C11, C18, C8: value 100pC -> 100nC; footprint Capacitor_SMD:C_0402_1005Metric -> Capacitor_SMD:C_0805_2012Metric
- C13, C17, C19, C9: value 0.1uC -> 100nC; footprint Capacitor_SMD:C_0805_2012Metric_Pad1.18x1.45mm_HandSolder -> Capacitor_SMD:C_0805_2012Metric
- C14: value 10uC -> 100nC; footprint Capacitor_SMD:C_1210_3225Metric_Pad1.33x2.70mm_HandSolder -> Capacitor_SMD:C_0805_2012Metric
- C16: value 47uC -> 100nC; footprint Capacitor_THT:CP_Radial_D5.0mm_P2.00mm -> Capacitor_SMD:C_0805_2012Metric
- C3: value 100nC -> 0.1uC; footprint Capacitor_SMD:C_0805_2012Metric -> Capacitor_SMD:C_0805_2012Metric_Pad1.18x1.45mm_HandSolder
- C31, C41, C7: value 0.1uC -> 100pC; footprint Capacitor_SMD:C_0805_2012Metric_Pad1.18x1.45mm_HandSolder -> Capacitor_SMD:C_0402_1005Metric
- C34: value 10uC -> 100pC; footprint Capacitor_SMD:C_1210_3225Metric_Pad1.33x2.70mm_HandSolder -> Capacitor_SMD:C_0402_1005Metric
- C36, C6: value 47uC -> 0.1uC; footprint Capacitor_THT:CP_Radial_D5.0mm_P2.00mm -> Capacitor_SMD:C_0805_2012Metric_Pad1.18x1.45mm_HandSolder
- C38, C4: value 0.1uC -> 10uC; footprint Capacitor_SMD:C_0805_2012Metric_Pad1.18x1.45mm_HandSolder -> Capacitor_SMD:C_1210_3225Metric_Pad1.33x2.70mm_HandSolder
- C5: value 10uC -> 47uC; footprint Capacitor_SMD:C_1210_3225Metric_Pad1.33x2.70mm_HandSolder -> Capacitor_THT:CP_Radial_D5.0mm_P2.00mm
- J10: value Limit switch -> Motor Connector; footprint Connector_JST:JST_PH_B2B-PH-K_1x02_P2.00mm_Vertical -> Connector_JST:JST_PH_B6B-PH-K_1x06_P2.00mm_Vertical
- J11: value Motor Connector -> Conn_01x20; footprint Connector_JST:JST_PH_B6B-PH-K_1x06_P2.00mm_Vertical -> Connector_FFC-FPC:TE_2-84952-0_1x20-1MP_P1.0mm_Horizontal
- R1, R2: value 1kR -> 10kR; footprint Resistor_SMD:R_0402_1005Metric -> Resistor_SMD:R_0805_2012Metric_Pad1.20x1.40mm_HandSolder
- R10, R19: value 250mR -> 10kR; footprint Resistor_SMD:R_2010_5025Metric -> Resistor_SMD:R_0805_2012Metric_Pad1.20x1.40mm_HandSolder
- R11, R20: footprint Capacitor_SMD:C_0805_2012Metric -> Resistor_SMD:R_0805_2012Metric_Pad1.20x1.40mm_HandSolder
- R12, R21, R3: value 10kR -> 250mR; footprint Capacitor_SMD:C_0805_2012Metric -> Resistor_SMD:R_2010_5025Metric
- R16, R7: value 1kR -> 10kR; footprint Resistor_SMD:R_0402_1005Metric -> Capacitor_SMD:C_0805_2012Metric
- R17, R8: footprint Resistor_SMD:R_0805_2012Metric_Pad1.20x1.40mm_HandSolder -> Capacitor_SMD:C_0805_2012Metric
- R18, R9: value 10kR -> 1kR; footprint Resistor_SMD:R_0805_2012Metric_Pad1.20x1.40mm_HandSolder -> Resistor_SMD:R_0402_1005Metric
- R31: value 10kR -> 1kR; footprint Capacitor_SMD:C_0805_2012Metric -> Resistor_SMD:R_0402_1005Metric
- R39: footprint Capacitor_SMD:C_0805_2012Metric -> Resistor_SMD:R_0805_2012Metric
- U1: value DRV8870DDA -> 74HC2G08; footprint Package_SO:Texas_HTSOP-8-1EP_3.9x4.9mm_P1.27mm_EP2.95x4.9mm_Mask2.4x3.1mm_ThermalVias -> Package_SO:TSSOP-8_3x3mm_P0.65mm
- U14, U2: value INA180A1 -> DRV8870DDA; footprint Package_TO_SOT_SMD:SOT-23-5 -> Package_SO:Texas_HTSOP-8-1EP_3.9x4.9mm_P1.27mm_EP2.95x4.9mm_Mask2.4x3.1mm_ThermalVias
- U3: value DRV8870DDA -> INA180A1; footprint Package_SO:Texas_HTSOP-8-1EP_3.9x4.9mm_P1.27mm_EP2.95x4.9mm_Mask2.4x3.1mm_ThermalVias -> Package_TO_SOT_SMD:SOT-23-5
- U4: value INA180A1 -> SP213; footprint Package_TO_SOT_SMD:SOT-23-5 -> Package_SO:SSOP-28_5.3x10.2mm_P0.65mm
- U7: value DRV8870DDA -> SP213; footprint Package_SO:Texas_HTSOP-8-1EP_3.9x4.9mm_P1.27mm_EP2.95x4.9mm_Mask2.4x3.1mm_ThermalVias -> Package_SO:SSOP-28_5.3x10.2mm_P0.65mm
- moved J18 147.4 mm to (271.9, 37.8)
- moved J11 127.8 mm to (236.1, 38.9)
- moved U1 80.4 mm to (289.6, 84.4)
- moved R9 78.3 mm to (294.5, 85.0)
- moved J14 75.2 mm to (224.1, 85.3)
- moved C10 71.3 mm to (294.1, 78.4)
- moved R16 67.3 mm to (231.3, 102.6)
- moved C7 67.1 mm to (294.1, 76.5)
- moved U8 66.8 mm to (246.6, 57.4)
- moved R13 64.6 mm to (246.7, 103.3)
- moved R4 64.2 mm to (294.5, 83.0)
- moved J9 63.9 mm to (271.9, 78.1)
- moved C5 63.9 mm to (288.4, 78.7)
- moved C4 63.6 mm to (287.8, 64.4)
- moved R8 62.5 mm to (279.1, 85.4)
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Connections:
- net /H-bridge1/PWM2 renamed /H-bridge #1/PWM1
- C1 pad 1: /H-bridge/ENCODER_A -> +5V
- C10 pad 1: /H-bridge1/LIM1 -> /H-bridge #1/ENCODER_B
- C11 pad 1: /H-bridge2/ENCODER_A -> /RS232 Interface #2/C1+
- C11 pad 2: GND -> /RS232 Interface #2/C1-
- C12 pad 1: /H-bridge2/LIM2 -> /RS232 Interface #2/V-
- C13 pad 1: +12V -> /RS232 Interface #2/C2+
- C13 pad 2: GND -> /RS232 Interface #2/C2-
- C14 pad 1: +12V -> +5V
- C14 pad 2: GND -> /RS232 Interface #2/V+
- C15 pad 1: /H-bridge/LIM2 -> +5VD
- C16 pad 1: +12V -> /RS232 Interface #1/C1+
- C16 pad 2: GND -> /RS232 Interface #1/C1-
- C17 pad 1: Net-(U3-VREF) -> /RS232 Interface #1/V-
- C18 pad 1: /H-bridge2/ENCODER_B -> /RS232 Interface #1/C2+
- C18 pad 2: GND -> /RS232 Interface #1/C2-
- C19 pad 2: GND -> /RS232 Interface #1/V+
- C2 pad 1: /H-bridge1/ENCODER_A -> Net-(U2-VREF)
- C20 pad 1: /H-bridge2/LIM1 -> +5VD
- C27 pad 1: /H-bridge/ENCODER_B -> +12V
- C3 pad 1: /H-bridge1/LIM2 -> +12V
- C31 pad 1: +12V -> /H-bridge #2/ENCODER_A
- C33 pad 1: /H-bridge/LIM1 -> /H-bridge #2/LIM2
- C34 pad 1: +12V -> /H-bridge #2/ENCODER_B
- C36 pad 1: +12V -> Net-(U14-VREF)
- C38 pad 1: Net-(U7-VREF) -> +12V
- C41 pad 1: +5V -> /H-bridge #3/ENCODER_A
- C6 pad 1: +12V -> +5V
- C7 pad 1: Net-(U1-VREF) -> /H-bridge #1/ENCODER_A
- C8 pad 1: /H-bridge1/ENCODER_B -> /H-bridge #1/LIM1
- C9 pad 1: +5V -> /H-bridge #1/LIM2
- J1 pad 8: VCC -> +5V
- J10 pad 1: Net-(J10-Pin_1) -> /H-bridge #1/MOTOR+
- J10 pad 2: GND -> /H-bridge #1/MOTOR-
- J11 pad 1: /H-bridge1/MOTOR+ -> GND
- J11 pad 2: /H-bridge1/MOTOR- -> GND
- J11 pad 3: +5V -> /RTS_LINE1
- J11 pad 4: GND -> /DTR_LINE1
- J11 pad 5: /H-bridge1/ENCODER_A -> /TX_LINE1
- J11 pad 6: /H-bridge1/ENCODER_B -> /RI_LINE1
- J14 pad 1: /H-bridge2/MOTOR+ -> /H-bridge #2/MOTOR+
- J14 pad 2: /H-bridge2/MOTOR- -> /H-bridge #2/MOTOR-
- J14 pad 5: /H-bridge2/ENCODER_A -> /H-bridge #2/ENCODER_A
- J14 pad 6: /H-bridge2/ENCODER_B -> /H-bridge #2/ENCODER_B
- J18 pad 1: /H-bridge/MOTOR+ -> /H-bridge #3/MOTOR+
- J18 pad 2: /H-bridge/MOTOR- -> /H-bridge #3/MOTOR-
- J18 pad 5: /H-bridge/ENCODER_A -> /H-bridge #3/ENCODER_A
- J18 pad 6: /H-bridge/ENCODER_B -> /H-bridge #3/ENCODER_B
- R1 pad 1: /H-bridge/ENCODER_A -> +5V
- R1 pad 2: /H-bridge/ENCODER_A -> Net-(U2-VREF)
- R10 pad 1: GND -> +5V
- R10 pad 2: Net-(U1-ISEN) -> Net-(U11-VREF)
- R11 pad 1: /H-bridge1/LIM1 -> Net-(U11-VREF)
- R11 pad 2: Net-(J10-Pin_1) -> GND
- R12 pad 1: Net-(J10-Pin_1) -> GND
- R12 pad 2: +5V -> Net-(U11-ISEN)
- R13 pad 1: /H-bridge2/ENCODER_A -> /H-bridge #2/ENCODER_A
- R13 pad 2: /H-bridge2/ENCODER_A -> /H-bridge #2/ENCODER_A
- R14 pad 1: /H-bridge2/LIM2 -> /H-bridge #2/LIM1
- R15 pad 1: Net-(J12-Pin_1) -> /H-bridge #2/LIM2
- R15 pad 2: +5V -> Net-(J13-Pin_1)
- R16 pad 1: /H-bridge2/ENCODER_B -> Net-(J12-Pin_1)
- R16 pad 2: /H-bridge2/ENCODER_B -> +5V
- R17 pad 1: +5V -> Net-(J13-Pin_1)
- R17 pad 2: Net-(U3-VREF) -> +5V
- R18 pad 1: Net-(U3-VREF) -> /H-bridge #2/ENCODER_B
- R18 pad 2: GND -> /H-bridge #2/ENCODER_B
- R19 pad 1: GND -> +5V
- R19 pad 2: Net-(U3-ISEN) -> Net-(U14-VREF)
- R2 pad 1: /H-bridge/ENCODER_B -> Net-(U2-VREF)
- R2 pad 2: /H-bridge/ENCODER_B -> GND
- R20 pad 1: /H-bridge2/LIM1 -> Net-(U14-VREF)
- R20 pad 2: Net-(J13-Pin_1) -> GND
- R21 pad 1: Net-(J13-Pin_1) -> GND
- R21 pad 2: +5V -> Net-(U14-ISEN)
- R3 pad 1: /H-bridge/LIM2 -> GND
- R3 pad 2: Net-(J8-Pin_1) -> Net-(U2-ISEN)
- R31 pad 1: Net-(J8-Pin_1) -> /H-bridge #3/ENCODER_A
- R31 pad 2: +5V -> /H-bridge #3/ENCODER_A
- R39 pad 1: /H-bridge/LIM1 -> /SCL/21
- R39 pad 2: Net-(J19-Pin_1) -> +5V
- R4 pad 1: /H-bridge1/ENCODER_A -> /H-bridge #1/ENCODER_A
- R4 pad 2: /H-bridge1/ENCODER_A -> /H-bridge #1/ENCODER_A
- R5 pad 1: /H-bridge1/LIM2 -> /H-bridge #1/LIM1
- R5 pad 2: Net-(J9-Pin_1) -> Net-(J8-Pin_1)
- R6 pad 1: Net-(J9-Pin_1) -> /H-bridge #1/LIM2
- R6 pad 2: +5V -> Net-(J9-Pin_1)
- R7 pad 1: /H-bridge1/ENCODER_B -> Net-(J8-Pin_1)
- R7 pad 2: /H-bridge1/ENCODER_B -> +5V
- R8 pad 1: +5V -> Net-(J9-Pin_1)
- R8 pad 2: Net-(U1-VREF) -> +5V
- R9 pad 1: Net-(U1-VREF) -> /H-bridge #1/ENCODER_B
- R9 pad 2: GND -> /H-bridge #1/ENCODER_B
- U1 pad 1: GND -> /H-bridge #1/ENABLE_PWM
- U1 pad 3: /H-bridge1/PWM1 -> Net-(U2-IN2)
- U1 pad 4: Net-(U1-VREF) -> GND
- U1 pad 5: +12V -> /H-bridge #1/ENABLE_PWM
- U1 pad 6: /H-bridge1/MOTOR+ -> /H-bridge #1/PWM2
- U1 pad 7: Net-(U1-ISEN) -> Net-(U2-IN1)
- U1 pad 8: /H-bridge1/MOTOR- -> +5V
- U14 pad 1: /H-bridge/A_SENSE -> GND
- U14 pad 2: GND -> Net-(U14-IN2)
- U14 pad 3: Net-(U14-+) -> Net-(U14-IN1)
- U14 pad 4: GND -> Net-(U14-VREF)
- U14 pad 5: +5V -> +12V
- U2 pad 1: /H-bridge1/A_SENSE -> GND
- U2 pad 2: GND -> Net-(U2-IN2)
- U2 pad 3: Net-(U1-ISEN) -> Net-(U2-IN1)
- U2 pad 4: GND -> Net-(U2-VREF)
- U2 pad 5: +5V -> +12V
- U3 pad 1: GND -> /H-bridge #1/A_SENSE
- U3 pad 2: /H-bridge2/PWM2 -> GND
- U3 pad 3: /H-bridge2/PWM1 -> Net-(U2-ISEN)
- U3 pad 4: Net-(U3-VREF) -> GND
- U3 pad 5: +12V -> +5V
- U4 pad 1: /H-bridge2/A_SENSE -> /RTS_LINE2
- U4 pad 2: GND -> /DTR_LINE2
- U4 pad 3: Net-(U3-ISEN) -> /TX_LINE2
- U4 pad 4: GND -> /RI_LINE2
- U4 pad 5: +5V -> /RI_IN2
- U7 pad 1: GND -> /RTS_LINE1
- U7 pad 2: /H-bridge/PWM2 -> /DTR_LINE1
- U7 pad 3: /H-bridge/PWM1 -> /TX_LINE1
- U7 pad 4: Net-(U7-VREF) -> /RI_LINE1
- U7 pad 5: +12V -> /RI_IN1
- U7 pad 6: /H-bridge/MOTOR+ -> /TX3/14
- U7 pad 7: Net-(U14-+) -> /DTR_IN1
- U7 pad 8: /H-bridge/MOTOR- -> /CTS_IN1
- U7 pad 9: GND -> /CTS_LINE1
- U8 pad 16: unconnected-(U8-GND-Pad16) -> GND
- U8 pad 32: unconnected-(U8-VDD-Pad32) -> +5VD

Commit message: Progressed ECAD.
Parts:
- removed U17: 74AHC373, Package_SO:TSSOP-20_4.4x6.5mm_P0.65mm
- added C51: 100nC, Capacitor_SMD:C_0805_2012Metric, F.Cu at (227.0, 101.5)
- added L5: 10uL, Inductor_SMD:L_0805_2012Metric, F.Cu at (231.5, 101.2)
- added U18: 74AHC573, Package_SO:TSSOP-20_4.4x6.5mm_P0.65mm, F.Cu at (229.5, 93.0)
- moved J10 58.6 mm to (213.3, 64.5)
- moved J8 58.6 mm to (213.3, 71.0)
- moved J9 58.6 mm to (213.3, 77.6)
- moved R1 58.6 mm to (234.5, 69.8)
- moved R2 58.6 mm to (234.5, 72.7)
- moved U3 58.6 mm to (234.8, 64.2)
- moved C1 58.6 mm to (225.1, 76.4)
- moved C2 58.6 mm to (225.1, 79.5)
- moved C3 58.6 mm to (225.1, 82.5)
- moved C5 58.6 mm to (229.9, 78.2)
- moved C6 58.6 mm to (225.1, 85.5)
- moved C8 58.6 mm to (220.5, 69.8)
- moved C9 58.6 mm to (220.5, 72.8)
- moved R4 58.6 mm to (235.9, 82.5)
- moved R5 58.6 mm to (220.5, 75.8)
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Connections:
- net /RS232 Interface #1/C1+ renamed /Serial ports/RS232 Interface #2/C1+
- net /RS232 Interface #1/C1- renamed /Serial ports/RS232 Interface #2/C1-
- net /RS232 Interface #1/C2+ renamed /Serial ports/RS232 Interface #2/C2+
- net /RS232 Interface #1/C2- renamed /Serial ports/RS232 Interface #2/C2-
- net /RS232 Interface #1/V+ renamed /Serial ports/RS232 Interface #2/V+
- net /RS232 Interface #1/V- renamed /Serial ports/RS232 Interface #2/V-
- net /RS232 Interface #2/C1+ renamed /Serial ports/RS232 Interface #1/C1+
- net /RS232 Interface #2/C1- renamed /Serial ports/RS232 Interface #1/C1-
- net /RS232 Interface #2/C2+ renamed /Serial ports/RS232 Interface #1/C2+
- net /RS232 Interface #2/C2- renamed /Serial ports/RS232 Interface #1/C2-
- net /RS232 Interface #2/V+ renamed /Serial ports/RS232 Interface #1/V+
- net /RS232 Interface #2/V- renamed /Serial ports/RS232 Interface #1/V-
- J11 pad 10: /DCD_LINE1 -> /Serial ports/DCD_LINE1
- J11 pad 13: /RTS_LINE2 -> /Serial ports/RTS_LINE2
- J11 pad 14: /DTR_LINE2 -> /Serial ports/DTR_LINE2
- J11 pad 15: /TX_LINE2 -> /Serial ports/TX_LINE2
- J11 pad 16: /RI_LINE2 -> /Serial ports/RI_LINE2
- J11 pad 17: /CTS_LINE2 -> /Serial ports/CTS_LINE2
- J11 pad 18: /RX_LINE2 -> /Serial ports/RX_LINE2
- J11 pad 19: /DSR_LINE2 -> /Serial ports/DSR_LINE2
- J11 pad 20: /DCD_LINE2 -> /Serial ports/DCD_LINE2
- J11 pad 3: /RTS_LINE1 -> /Serial ports/RTS_LINE1
- J11 pad 4: /DTR_LINE1 -> /Serial ports/DTR_LINE1
- J11 pad 5: /TX_LINE1 -> /Serial ports/TX_LINE1
- J11 pad 6: /RI_LINE1 -> /Serial ports/RI_LINE1
- J11 pad 7: /CTS_LINE1 -> /Serial ports/CTS_LINE1
- J11 pad 8: /RX_LINE1 -> /Serial ports/RX_LINE1
- J11 pad 9: /DSR_LINE1 -> /Serial ports/DSR_LINE1
- R37 pad 1: /A8 -> /Serial ports/A8
- R38 pad 1: /SDA/20 -> /Serial ports/SDA/20
- R39 pad 1: /SCL/21 -> /Serial ports/SCL/21
- U16 pad 1: /A8 -> /Serial ports/A8
- U16 pad 10: /~{SHDN_IN1} -> /Serial ports/~{SHDN_IN1}
- U16 pad 11: /DCD_IN1 -> /Serial ports/DCD_IN1
- U16 pad 13: /RI_IN2 -> /Serial ports/RI_IN2
- U16 pad 14: /~{SHDN_IN2} -> /Serial ports/~{SHDN_IN2}
- U16 pad 15: /DCD_IN2 -> /Serial ports/DCD_IN2
- U16 pad 16: /DTR_IN2 -> /Serial ports/DTR_IN2
- U16 pad 17: /CTS_IN2 -> /Serial ports/CTS_IN2
- U16 pad 18: /DSR_IN2 -> /Serial ports/DSR_IN2
- U16 pad 19: /EN_IN2 -> /Serial ports/EN_IN2
- U16 pad 20: /RTS_IN2 -> /Serial ports/RTS_IN2
- U16 pad 22: /SCL/21 -> /Serial ports/SCL/21
- U16 pad 23: /SDA/20 -> /Serial ports/SDA/20
- U16 pad 4: /EN_IN1 -> /Serial ports/EN_IN1
- U16 pad 5: /RTS_IN1 -> /Serial ports/RTS_IN1
- U16 pad 6: /DSR_IN1 -> /Serial ports/DSR_IN1
- U16 pad 7: /CTS_IN1 -> /Serial ports/CTS_IN1
- U16 pad 8: /DTR_IN1 -> /Serial ports/DTR_IN1
- U16 pad 9: /RI_IN1 -> /Serial ports/RI_IN1
- U4 pad 1: /RTS_LINE2 -> /Serial ports/RTS_LINE1
- U4 pad 18: /RX_LINE2 -> /Serial ports/RX_LINE1
- U4 pad 19: /RX2/17 -> /Serial ports/RX3/15
- U4 pad 2: /DTR_LINE2 -> /Serial ports/DTR_LINE1
- U4 pad 20: /RTS_IN2 -> /Serial ports/RTS_IN1
- U4 pad 22: /DSR_IN2 -> /Serial ports/DSR_IN1
- U4 pad 23: /DSR_LINE2 -> /Serial ports/DSR_LINE1
- U4 pad 24: /EN_IN2 -> /Serial ports/EN_IN1
- U4 pad 25: /~{SHDN_IN2} -> /Serial ports/~{SHDN_IN1}
- U4 pad 26: /DCD_IN2 -> /Serial ports/DCD_IN1
- U4 pad 27: /DCD_LINE2 -> /Serial ports/DCD_LINE1
- U4 pad 3: /TX_LINE2 -> /Serial ports/TX_LINE1
- U4 pad 4: /RI_LINE2 -> /Serial ports/RI_LINE1
- U4 pad 5: /RI_IN2 -> /Serial ports/RI_IN1
- U4 pad 6: /TX2/16 -> /Serial ports/TX3/14
- U4 pad 7: /DTR_IN2 -> /Serial ports/DTR_IN1
- U4 pad 8: /CTS_IN2 -> /Serial ports/CTS_IN1
- U4 pad 9: /CTS_LINE2 -> /Serial ports/CTS_LINE1
- U7 pad 1: /RTS_LINE1 -> /Serial ports/RTS_LINE2
- U7 pad 18: /RX_LINE1 -> /Serial ports/RX_LINE2
- U7 pad 19: /RX3/15 -> /Serial ports/RX2/17
- U7 pad 2: /DTR_LINE1 -> /Serial ports/DTR_LINE2
- U7 pad 20: /RTS_IN1 -> /Serial ports/RTS_IN2
- U7 pad 22: /DSR_IN1 -> /Serial ports/DSR_IN2
- U7 pad 23: /DSR_LINE1 -> /Serial ports/DSR_LINE2
- U7 pad 24: /EN_IN1 -> /Serial ports/EN_IN2
- U7 pad 25: /~{SHDN_IN1} -> /Serial ports/~{SHDN_IN2}
- U7 pad 26: /DCD_IN1 -> /Serial ports/DCD_IN2
- U7 pad 27: /DCD_LINE1 -> /Serial ports/DCD_LINE2
- U7 pad 3: /TX_LINE1 -> /Serial ports/TX_LINE2
- U7 pad 4: /RI_LINE1 -> /Serial ports/RI_LINE2
- U7 pad 5: /RI_IN1 -> /Serial ports/RI_IN2
- U7 pad 6: /TX3/14 -> /Serial ports/TX2/16
- U7 pad 7: /DTR_IN1 -> /Serial ports/DTR_IN2
- U7 pad 8: /CTS_IN1 -> /Serial ports/CTS_IN2
- U7 pad 9: /CTS_LINE1 -> /Serial ports/CTS_LINE2
- U8 pad 1: unconnected-(U8-A17-Pad1) -> /External RAM/A17
- U8 pad 10: unconnected-(U8-A2-Pad10) -> Net-(U18-Q2)
- U8 pad 11: unconnected-(U8-A1-Pad11) -> Net-(U18-Q1)
- U8 pad 12: unconnected-(U8-A0-Pad12) -> Net-(U18-Q0)
- U8 pad 13: unconnected-(U8-I/O0-Pad13) -> /External RAM/AD0
- U8 pad 14: unconnected-(U8-I/O1-Pad14) -> /External RAM/AD1
- U8 pad 15: unconnected-(U8-I/O2-Pad15) -> /External RAM/AD2
- U8 pad 17: unconnected-(U8-I/O3-Pad17) -> /External RAM/AD3
- U8 pad 18: unconnected-(U8-I/O4-Pad18) -> /External RAM/AD4
- U8 pad 19: unconnected-(U8-I/O5-Pad19) -> /External RAM/AD5
- U8 pad 2: unconnected-(U8-A16-Pad2) -> /External RAM/A16
- U8 pad 20: unconnected-(U8-I/O6-Pad20) -> /External RAM/AD6
- U8 pad 21: unconnected-(U8-I/O7-Pad21) -> /External RAM/AD7
- U8 pad 22: unconnected-(U8-~{CE}-Pad22) -> GND
- U8 pad 23: unconnected-(U8-A10-Pad23) -> /External RAM/A10
- U8 pad 24: unconnected-(U8-~{OE}-Pad24) -> /External RAM/~{RD}
- U8 pad 25: unconnected-(U8-A11-Pad25) -> /External RAM/A11
- U8 pad 26: unconnected-(U8-A9-Pad26) -> /External RAM/A09
- U8 pad 27: unconnected-(U8-A8-Pad27) -> /External RAM/A08
- U8 pad 28: unconnected-(U8-A13-Pad28) -> /External RAM/A13
- U8 pad 29: unconnected-(U8-~{WE}-Pad29) -> /External RAM/~{WR}
- U8 pad 3: unconnected-(U8-A14-Pad3) -> /External RAM/A14
- U8 pad 30: unconnected-(U8-A18-Pad30) -> /External RAM/A18
- U8 pad 31: unconnected-(U8-A15-Pad31) -> /External RAM/A15
- U8 pad 4: unconnected-(U8-A12-Pad4) -> /External RAM/A12
- U8 pad 5: unconnected-(U8-A7-Pad5) -> Net-(U18-Q7)
- U8 pad 6: unconnected-(U8-A6-Pad6) -> Net-(U18-Q6)
- U8 pad 7: unconnected-(U8-A5-Pad7) -> Net-(U18-Q5)
- U8 pad 8: unconnected-(U8-A4-Pad8) -> Net-(U18-Q4)
- U8 pad 9: unconnected-(U8-A3-Pad9) -> Net-(U18-Q3)

Commit message: Progressed ECAD.
Parts:
- added C49: 100nC, Capacitor_SMD:C_0805_2012Metric, F.Cu at (223.6, 83.2)
- added C50: 100nC, Capacitor_SMD:C_0805_2012Metric, F.Cu at (283.4, 104.4)
- added C52: 100nC, Capacitor_SMD:C_0805_2012Metric, F.Cu at (256.5, 87.7)
- added C53: 100pC, Capacitor_SMD:C_0402_1005Metric, F.Cu at (282.8, 67.1)
- added C54: 100nC, Capacitor_SMD:C_0805_2012Metric, F.Cu at (283.6, 59.6)
- added C55: 100nC, Capacitor_SMD:C_0805_2012Metric, F.Cu at (283.6, 62.6)
- added U17: 74AHC14, Package_SO:TSSOP-14_4.4x5mm_P0.65mm, F.Cu at (230.2, 97.9)
- added U19: INA180A1, Package_TO_SOT_SMD:SOT-23-5, F.Cu at (235.4, 85.3)
- added U20: 74AHC573, Package_SO:TSSOP-20_4.4x6.5mm_P0.65mm, F.Cu at (286.0, 98.8)
- added U21: CY62148ELL-45ZSXIT, Package_SO:TSOP-II-32_21.0x10.2mm_P1.27mm, F.Cu at (274.0, 105.8)
- added U22: PCA9555PW, Package_SO:TSSOP-24_4.4x7.8mm_P0.65mm, F.Cu at (245.5, 88.2)
- added U23: MCP6S26, Package_SO:SOIC-14_3.9x8.7mm_P1.27mm, F.Cu at (277.2, 63.3)
- C10, C44: value 100pC -> 10uC; footprint Capacitor_SMD:C_0402_1005Metric -> Capacitor_SMD:C_1210_3225Metric_Pad1.33x2.70mm_HandSolder
- C11, C23: value 100nC -> 47uC; footprint Capacitor_SMD:C_0805_2012Metric -> Capacitor_THT:CP_Radial_D5.0mm_P2.00mm
- C12, C13, C16, C17, C18, C19, C46, C47: value 100nC -> 0.1uC; footprint Capacitor_SMD:C_0805_2012Metric -> Capacitor_SMD:C_0805_2012Metric_Pad1.18x1.45mm_HandSolder
- C2: value 0.1uC -> 10uC; footprint Capacitor_SMD:C_0805_2012Metric_Pad1.18x1.45mm_HandSolder -> Capacitor_SMD:C_1206_3216Metric
- C20, C42, C43, C8, C9: value 100nC -> 100pC; footprint Capacitor_SMD:C_0805_2012Metric -> Capacitor_SMD:C_0402_1005Metric
- C21: value 0.1uC -> 100pC; footprint Capacitor_SMD:C_0805_2012Metric_Pad1.18x1.45mm_HandSolder -> Capacitor_SMD:C_0402_1005Metric
- C22: value 100nC -> 10uC; footprint Capacitor_SMD:C_0805_2012Metric -> Capacitor_SMD:C_1210_3225Metric_Pad1.33x2.70mm_HandSolder
- C24, C41, C7: value 100pC -> 0.1uC; footprint Capacitor_SMD:C_0402_1005Metric -> Capacitor_SMD:C_0805_2012Metric_Pad1.18x1.45mm_HandSolder
- C26, C27, C3, C30, C35, C36, C37: value 0.1uC -> 100nC; footprint Capacitor_SMD:C_0805_2012Metric_Pad1.18x1.45mm_HandSolder -> Capacitor_SMD:C_0805_2012Metric
- C28: value 10uC -> 100nC; footprint Capacitor_SMD:C_1210_3225Metric_Pad1.33x2.70mm_HandSolder -> Capacitor_SMD:C_0805_2012Metric
- C29: value 47uC -> 100nC; footprint Capacitor_THT:CP_Radial_D5.0mm_P2.00mm -> Capacitor_SMD:C_0805_2012Metric
- C31, C34: value 100pC -> 100nC; footprint Capacitor_SMD:C_0402_1005Metric -> Capacitor_SMD:C_0805_2012Metric
- C38, C4: value 10uC -> 0.1uC; footprint Capacitor_SMD:C_1210_3225Metric_Pad1.33x2.70mm_HandSolder -> Capacitor_SMD:C_0805_2012Metric_Pad1.18x1.45mm_HandSolder
- C39, C5: value 47uC -> 0.1uC; footprint Capacitor_THT:CP_Radial_D5.0mm_P2.00mm -> Capacitor_SMD:C_0805_2012Metric_Pad1.18x1.45mm_HandSolder
- C45: value 10uC -> 47uC; footprint Capacitor_SMD:C_1206_3216Metric -> Capacitor_THT:CP_Radial_D5.0mm_P2.00mm
- J10, J14: value Motor Connector -> Limit switch; footprint Connector_JST:JST_PH_B6B-PH-K_1x06_P2.00mm_Vertical -> Connector_JST:JST_PH_B2B-PH-K_1x02_P2.00mm_Vertical
- J11: value Conn_01x20 -> Limit switch; footprint Connector_FFC-FPC:TE_2-84952-0_1x20-1MP_P1.0mm_Horizontal -> Connector_JST:JST_PH_B2B-PH-K_1x02_P2.00mm_Vertical
- J12, J9: value Limit switch -> Motor Connector; footprint Connector_JST:JST_PH_B2B-PH-K_1x02_P2.00mm_Vertical -> Connector_JST:JST_PH_B6B-PH-K_1x06_P2.00mm_Vertical
- J15: value Barrel_Jack_Switch -> Motor Connector; footprint Connector_BarrelJack:BarrelJack_Horizontal -> Connector_JST:JST_PH_B6B-PH-K_1x06_P2.00mm_Vertical
- J18: value Motor Connector -> Conn_01x20; footprint Connector_JST:JST_PH_B6B-PH-K_1x06_P2.00mm_Vertical -> Connector_FFC-FPC:TE_2-84952-0_1x20-1MP_P1.0mm_Horizontal
- J8: value Limit switch -> Barrel_Jack_Switch; footprint Connector_JST:JST_PH_B2B-PH-K_1x02_P2.00mm_Vertical -> Connector_BarrelJack:BarrelJack_Horizontal
- R1, R2: value 10kR -> 1kR
- R11, R20: value 10kR -> 1kR; footprint Resistor_SMD:R_0805_2012Metric_Pad1.20x1.40mm_HandSolder -> Resistor_SMD:R_0402_1005Metric
- R12, R21: value 250mR -> 1kR; footprint Resistor_SMD:R_2010_5025Metric -> Resistor_SMD:R_0402_1005Metric
- R13, R31: value 1kR -> 250mR; footprint Resistor_SMD:R_0402_1005Metric -> Resistor_SMD:R_2010_5025Metric
- R18, R9: value 1kR -> 10kR; footprint Resistor_SMD:R_0402_1005Metric -> Resistor_SMD:R_0805_2012Metric_Pad1.20x1.40mm_HandSolder
- R22: value 10kR -> 250mR; footprint Resistor_SMD:R_0805_2012Metric_Pad1.20x1.40mm_HandSolder -> Resistor_SMD:R_2010_5025Metric
- R23, R25: footprint Resistor_SMD:R_0805_2012Metric_Pad1.20x1.40mm_HandSolder -> Capacitor_SMD:C_0805_2012Metric
- R24, R26: value 1kR -> 10kR; footprint Resistor_SMD:R_0805_2012Metric_Pad1.20x1.40mm_HandSolder -> Capacitor_SMD:C_0805_2012Metric
- R27, R28: value 1kR -> 10kR
- R29: footprint Resistor_SMD:R_0805_2012Metric_Pad1.20x1.40mm_HandSolder -> Resistor_SMD:R_0402_1005Metric
- R3: value 250mR -> 1kR; footprint Resistor_SMD:R_2010_5025Metric -> Resistor_SMD:R_0805_2012Metric_Pad1.20x1.40mm_HandSolder
- R36: value 1kR -> 10kR; footprint Resistor_SMD:R_0402_1005Metric -> Resistor_SMD:R_0805_2012Metric
- R39: value 10kR -> 1kR; footprint Resistor_SMD:R_0805_2012Metric -> Resistor_SMD:R_0402_1005Metric
- R4: footprint Resistor_SMD:R_0402_1005Metric -> Resistor_SMD:R_0805_2012Metric_Pad1.20x1.40mm_HandSolder
- R5: value 10kR -> 1kR; footprint Capacitor_SMD:C_0805_2012Metric -> Resistor_SMD:R_0805_2012Metric_Pad1.20x1.40mm_HandSolder
- R6, R7, R8: footprint Capacitor_SMD:C_0805_2012Metric -> Resistor_SMD:R_0805_2012Metric_Pad1.20x1.40mm_HandSolder
- U1: value 74HC2G08 -> LM4040DBZ-4.1; footprint Package_SO:TSSOP-8_3x3mm_P0.65mm -> Package_TO_SOT_SMD:SOT-23
- U10: value 74HC2G08 -> 74AHC14; footprint Package_SO:TSSOP-8_3x3mm_P0.65mm -> Package_SO:TSSOP-14_4.4x5mm_P0.65mm
- U13: value 74HC2G08 -> SP213; footprint Package_SO:TSSOP-8_3x3mm_P0.65mm -> Package_SO:SSOP-28_5.3x10.2mm_P0.65mm
- U14: value DRV8870DDA -> SP213; footprint Package_SO:Texas_HTSOP-8-1EP_3.9x4.9mm_P1.27mm_EP2.95x4.9mm_Mask2.4x3.1mm_ThermalVias -> Package_SO:SSOP-28_5.3x10.2mm_P0.65mm
- U15, U3: value INA180A1 -> 74AHC2G125; footprint Package_TO_SOT_SMD:SOT-23-5 -> Package_SO:TSSOP-8_3x3mm_P0.65mm
- U16: value PCA9555PW -> 74AHC2G08; footprint Package_SO:TSSOP-24_4.4x7.8mm_P0.65mm -> Package_SO:TSSOP-8_3x3mm_P0.65mm
- U18: value 74AHC573 -> DRV8870DDA; footprint Package_SO:TSSOP-20_4.4x6.5mm_P0.65mm -> Package_SO:Texas_HTSOP-8-1EP_3.9x4.9mm_P1.27mm_EP2.95x4.9mm_Mask2.4x3.1mm_ThermalVias
- U2: value DRV8870DDA -> PCA9555PW; footprint Package_SO:Texas_HTSOP-8-1EP_3.9x4.9mm_P1.27mm_EP2.95x4.9mm_Mask2.4x3.1mm_ThermalVias -> Package_SO:TSSOP-24_4.4x7.8mm_P0.65mm
- U4: value SP213 -> 74AHC2G08; footprint Package_SO:SSOP-28_5.3x10.2mm_P0.65mm -> Package_SO:TSSOP-8_3x3mm_P0.65mm
- U5: value PCA9535PW -> 74AHC14; footprint Package_SO:TSSOP-24_4.4x7.8mm_P0.65mm -> Package_SO:TSSOP-14_4.4x5mm_P0.65mm
- U6: value LM4040DBZ-4.1 -> DRV8870DDA; footprint Package_TO_SOT_SMD:SOT-23 -> Package_SO:Texas_HTSOP-8-1EP_3.9x4.9mm_P1.27mm_EP2.95x4.9mm_Mask2.4x3.1mm_ThermalVias
- U7: value SP213 -> INA180A1; footprint Package_SO:SSOP-28_5.3x10.2mm_P0.65mm -> Package_TO_SOT_SMD:SOT-23-5
- U8: value CY62148ELL-45ZSXIT -> 74AHC2G125; footprint Package_SO:TSOP-II-32_21.0x10.2mm_P1.27mm -> Package_SO:TSSOP-8_3x3mm_P0.65mm
- U9: value PGA112 -> 74AHC2G08; footprint Package_SO:VSSOP-10_3x3mm_P0.5mm -> Package_SO:TSSOP-8_3x3mm_P0.65mm
- moved C32 69.5 mm to (275.0, 85.7)
- moved U8 68.4 mm to (261.5, 49.9)
- moved C41 61.1 mm to (219.0, 89.2)
- moved C11 58.9 mm to (211.0, 64.0)
- moved C28 58.8 mm to (275.0, 73.6)
- moved C38 58.7 mm to (219.0, 80.2)
- moved L4 57.1 mm to (287.9, 107.0)
- moved C51 56.7 mm to (283.4, 107.4)
- moved U15 56.1 mm to (229.3, 81.0)
- moved J11 55.9 mm to (211.6, 56.9)
- moved J8 55.1 mm to (260.1, 100.2)
- moved C33 54.8 mm to (275.2, 42.5)
- moved C1 54.4 mm to (261.5, 116.9)
- moved C30 54.3 mm to (275.0, 79.7)
- moved R39 53.3 mm to (282.9, 65.1)
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Connections:
- net /H-bridge #2/PWM2 renamed /Motor Control/H-bridge #2/LIM1
- net /H-bridge #3/PWM2 renamed /Serial ports/TX1
- C10 pad 1: /H-bridge #1/ENCODER_B -> +12V
- C11 pad 1: /Serial ports/RS232 Interface #1/C1+ -> +12V
- C11 pad 2: /Serial ports/RS232 Interface #1/C1- -> GND
- C12 pad 1: /Serial ports/RS232 Interface #1/V- -> +5V
- C13 pad 1: /Serial ports/RS232 Interface #1/C2+ -> +5V
- C13 pad 2: /Serial ports/RS232 Interface #1/C2- -> GND
- C14 pad 1: +5V -> Net-(C14-Pad1)
- C14 pad 2: /Serial ports/RS232 Interface #1/V+ -> GND
- C15 pad 1: +5VD -> Net-(C15-Pad1)
- C16 pad 1: /Serial ports/RS232 Interface #2/C1+ -> +5V
- C16 pad 2: /Serial ports/RS232 Interface #2/C1- -> GND
- C17 pad 1: /Serial ports/RS232 Interface #2/V- -> +5V
- C18 pad 1: /Serial ports/RS232 Interface #2/C2+ -> Net-(U11-VREF)
- C18 pad 2: /Serial ports/RS232 Interface #2/C2- -> GND
- C19 pad 1: +5V -> +12V
- C19 pad 2: /Serial ports/RS232 Interface #2/V+ -> GND
- C2 pad 1: Net-(U2-VREF) -> +5V
- C20 pad 1: +5VD -> Net-(C20-Pad1)
- C21 pad 1: +5V -> Net-(C21-Pad1)
- C22 pad 1: +5V -> +12V
- C23 pad 1: +5V -> +12V
- C24 pad 1: Net-(U9-V_{OUT}) -> +5V
- C26 pad 1: Net-(U11-VREF) -> Net-(C26-Pad1)
- C27 pad 1: +12V -> Net-(C27-Pad1)
- C28 pad 1: +12V -> /Serial ports/RS232 Interface #1/C1+
- C28 pad 2: GND -> /Serial ports/RS232 Interface #1/C1-
- C29 pad 1: +12V -> /Serial ports/RS232 Interface #1/V-
- C3 pad 1: +12V -> +5V
- C30 pad 1: +5V -> /Serial ports/RS232 Interface #1/C2+
- C30 pad 2: GND -> /Serial ports/RS232 Interface #1/C2-
- C31 pad 1: /H-bridge #2/ENCODER_A -> +5V
- C31 pad 2: GND -> /Serial ports/RS232 Interface #1/V+
- C32 pad 1: /H-bridge #2/LIM1 -> +5VD
- C33 pad 1: /H-bridge #2/LIM2 -> /Serial ports/RS232 Interface #2/C1+
- C33 pad 2: GND -> /Serial ports/RS232 Interface #2/C1-
- C34 pad 1: /H-bridge #2/ENCODER_B -> /Serial ports/RS232 Interface #2/V-
- C35 pad 1: +5V -> /Serial ports/RS232 Interface #2/C2+
- C35 pad 2: GND -> /Serial ports/RS232 Interface #2/C2-
- C36 pad 1: Net-(U14-VREF) -> +5V
- C36 pad 2: GND -> /Serial ports/RS232 Interface #2/V+
- C37 pad 1: +12V -> +5VD
- C38 pad 1: +12V -> +5V
- C39 pad 1: +12V -> +5V
- C4 pad 1: +12V -> +5V
- C40 pad 1: +5V -> Net-(U18-VREF)
- C41 pad 1: /H-bridge #3/ENCODER_A -> +12V
- C42 pad 1: /H-bridge #3/LIM1 -> Net-(C42-Pad1)
- C43 pad 1: /H-bridge #3/LIM2 -> Net-(C43-Pad1)
- C44 pad 1: /H-bridge #3/ENCODER_B -> +12V
- C45 pad 1: +5V -> +12V
- C47 pad 1: +5VD -> +5V
- C48 pad 1: +5VD -> Net-(C48-Pad1)
- C5 pad 1: +12V -> +5V
- C6 pad 1: +5V -> Net-(U6-VREF)
- C7 pad 1: /H-bridge #1/ENCODER_A -> +12V
- C8 pad 1: /H-bridge #1/LIM1 -> Net-(C8-Pad1)
- C9 pad 1: /H-bridge #1/LIM2 -> Net-(C9-Pad1)
- J1 pad 8: +5V -> VCC
- J10 pad 1: /H-bridge #1/MOTOR+ -> Net-(J10-Pin_1)
- J10 pad 2: /H-bridge #1/MOTOR- -> GND
- J11 pad 1: GND -> Net-(J11-Pin_1)
- J12 pad 1: Net-(J12-Pin_1) -> /Motor Control/H-bridge #2/MOTOR+
- J12 pad 2: GND -> /Motor Control/H-bridge #2/MOTOR-
- J14 pad 1: /H-bridge #2/MOTOR+ -> Net-(J14-Pin_1)
- J14 pad 2: /H-bridge #2/MOTOR- -> GND
- J15 pad 1: +12V -> /Motor Control/H-bridge #3/MOTOR+
- J15 pad 2: GND -> /Motor Control/H-bridge #3/MOTOR-
- J15 pad 3: GND -> +5V
- J18 pad 1: /H-bridge #3/MOTOR+ -> GND
- J18 pad 2: /H-bridge #3/MOTOR- -> GND
- J18 pad 3: +5V -> /Serial ports/RTS_LINE1
- J18 pad 4: GND -> /Serial ports/DTR_LINE1
- J18 pad 5: /H-bridge #3/ENCODER_A -> /Serial ports/TX_LINE1
- J18 pad 6: /H-bridge #3/ENCODER_B -> /Serial ports/RI_LINE1
- J8 pad 1: Net-(J8-Pin_1) -> +12V
- J9 pad 1: Net-(J9-Pin_1) -> /Motor Control/H-bridge #1/MOTOR+
- J9 pad 2: GND -> /Motor Control/H-bridge #1/MOTOR-
- R1 pad 2: Net-(U2-VREF) -> Net-(D1-A)
- R10 pad 1: +5V -> Net-(U6-VREF)
- R10 pad 2: Net-(U11-VREF) -> GND
- R11 pad 1: Net-(U11-VREF) -> Net-(C8-Pad1)
- R11 pad 2: GND -> /Motor Control/H-bridge #1/ENCODER_A
- R12 pad 1: GND -> Net-(C9-Pad1)
- R12 pad 2: Net-(U11-ISEN) -> /Motor Control/H-bridge #1/ENCODER_B
- R13 pad 1: /H-bridge #2/ENCODER_A -> GND
- R13 pad 2: /H-bridge #2/ENCODER_A -> Net-(U6-ISEN)
- R14 pad 1: /H-bridge #2/LIM1 -> Net-(C14-Pad1)
- R14 pad 2: Net-(J12-Pin_1) -> Net-(J10-Pin_1)
- R15 pad 1: /H-bridge #2/LIM2 -> Net-(C15-Pad1)
- R15 pad 2: Net-(J13-Pin_1) -> Net-(J11-Pin_1)
- R16 pad 1: Net-(J12-Pin_1) -> Net-(J10-Pin_1)
- R17 pad 1: Net-(J13-Pin_1) -> Net-(J11-Pin_1)
- R18 pad 1: /H-bridge #2/ENCODER_B -> +5V
- R18 pad 2: /H-bridge #2/ENCODER_B -> Net-(U11-VREF)
- R19 pad 1: +5V -> Net-(U11-VREF)
- R19 pad 2: Net-(U14-VREF) -> GND
- R2 pad 1: Net-(U2-VREF) -> +5V
- R2 pad 2: GND -> Net-(D2-A)
- R20 pad 1: Net-(U14-VREF) -> Net-(C20-Pad1)
- R20 pad 2: GND -> /Motor Control/H-bridge #1/ENCODER_A
- R21 pad 1: GND -> Net-(C21-Pad1)
- R21 pad 2: Net-(U14-ISEN) -> /Motor Control/H-bridge #1/ENCODER_B
- R22 pad 1: +5V -> GND
- R22 pad 2: /13 -> Net-(U11-ISEN)
- R23 pad 1: +5V -> Net-(C26-Pad1)
- R23 pad 2: /SDA/A4 -> Net-(J13-Pin_1)
- R24 pad 1: +5V -> Net-(C27-Pad1)
- R24 pad 2: Net-(D1-A) -> Net-(J14-Pin_1)
- R25 pad 1: +5V -> Net-(J13-Pin_1)
- R25 pad 2: /SCL/A5 -> +5V
- R26 pad 1: +5V -> Net-(J14-Pin_1)
- R26 pad 2: Net-(D2-A) -> +5V
- R27 pad 2: Net-(D3-A) -> Net-(U18-VREF)
- R28 pad 1: +5V -> Net-(U18-VREF)
- R28 pad 2: Net-(D4-A) -> GND
- R29 pad 1: +5V -> Net-(C42-Pad1)
- R29 pad 2: /AREF -> /Motor Control/H-bridge #1/ENCODER_A
- R3 pad 1: GND -> +5V
- R3 pad 2: Net-(U2-ISEN) -> Net-(D3-A)
- R30 pad 1: Net-(U9-V_{OUT}) -> Net-(C43-Pad1)
- R30 pad 2: /A_SENSE_BASE -> /Motor Control/H-bridge #1/ENCODER_B
- R31 pad 1: /H-bridge #3/ENCODER_A -> GND
- R31 pad 2: /H-bridge #3/ENCODER_A -> Net-(U18-ISEN)
- R32 pad 1: /H-bridge #3/LIM1 -> Net-(C48-Pad1)
- R33 pad 1: /H-bridge #3/LIM2 -> Net-(C49-Pad1)
- R36 pad 1: /H-bridge #3/ENCODER_B -> /Serial ports/~{INT}
- R36 pad 2: /H-bridge #3/ENCODER_B -> +5V
- R37 pad 1: /Serial ports/A8 -> /SDA/A4
- R38 pad 1: /Serial ports/SDA/20 -> /SCL/A5
- R39 pad 1: /Serial ports/SCL/21 -> Net-(U23-V_{OUT})
- R39 pad 2: +5V -> /Motor Control/A_SENSE
- R4 pad 1: /H-bridge #1/ENCODER_A -> +5V
- R4 pad 2: /H-bridge #1/ENCODER_A -> Net-(D4-A)
- R5 pad 1: /H-bridge #1/LIM1 -> +5V
- R5 pad 2: Net-(J8-Pin_1) -> /AREF
- R6 pad 1: /H-bridge #1/LIM2 -> +5V
- R6 pad 2: Net-(J9-Pin_1) -> /13
- R7 pad 1: Net-(J8-Pin_1) -> +5V
- R7 pad 2: +5V -> /SDA/A4
- R8 pad 1: Net-(J9-Pin_1) -> +5V
- R8 pad 2: +5V -> /SCL/A5
- R9 pad 1: /H-bridge #1/ENCODER_B -> +5V
- R9 pad 2: /H-bridge #1/ENCODER_B -> Net-(U6-VREF)
- U1 pad 1: /H-bridge #1/ENABLE_PWM -> /AREF
- U1 pad 2: /H-bridge #1/PWM1 -> GND
- U1 pad 3: Net-(U2-IN2) -> unconnected-(U1-NC-Pad3)
- U10 pad 1: /H-bridge #2/ENABLE_PWM -> Net-(C21-Pad1)
- U10 pad 2: /H-bridge #2/PWM1 -> Net-(U10-Pad2)
- U10 pad 3: Net-(U11-IN2) -> Net-(U10-Pad2)
- U10 pad 4: GND -> Net-(U10-Pad4)
- U10 pad 5: /H-bridge #2/ENABLE_PWM -> Net-(C26-Pad1)
- U10 pad 7: Net-(U11-IN1) -> GND
- U10 pad 8: +5V -> /Motor Control/H-bridge #2/LIM2
- U11 pad 6: /H-bridge #2/MOTOR+ -> /Motor Control/H-bridge #2/MOTOR+
- U11 pad 8: /H-bridge #2/MOTOR- -> /Motor Control/H-bridge #2/MOTOR-
- U12 pad 1: /H-bridge #2/A_SENSE -> /Motor Control/CURRENT2
- U13 pad 1: /H-bridge #3/ENABLE_PWM -> /Serial ports/RTS_LINE1
- U13 pad 2: /H-bridge #3/PWM1 -> /Serial ports/DTR_LINE1
- U13 pad 3: Net-(U14-IN2) -> /Serial ports/TX_LINE1
- U13 pad 4: GND -> /Serial ports/RI_LINE1
- U13 pad 5: /H-bridge #3/ENABLE_PWM -> /Serial ports/RI_IN1
- U13 pad 7: Net-(U14-IN1) -> /Serial ports/DTR_IN1
- U13 pad 8: +5V -> /Serial ports/CTS_IN1
- U14 pad 1: GND -> /Serial ports/RTS_LINE2
- U14 pad 2: Net-(U14-IN2) -> /Serial ports/DTR_LINE2
- U14 pad 3: Net-(U14-IN1) -> /Serial ports/TX_LINE2
- U14 pad 4: Net-(U14-VREF) -> /Serial ports/RI_LINE2
- U14 pad 5: +12V -> /Serial ports/RI_IN2
- U14 pad 6: /H-bridge #3/MOTOR+ -> /Serial ports/TX2
- U14 pad 7: Net-(U14-ISEN) -> /Serial ports/DTR_IN2
- U14 pad 8: /H-bridge #3/MOTOR- -> /Serial ports/CTS_IN2
- U14 pad 9: GND -> /Serial ports/CTS_LINE2
- U15 pad 1: /H-bridge #3/A_SENSE -> /Motor Control/EN_MOTOR3
- U15 pad 2: GND -> Net-(U15-Pad2)
- U15 pad 3: Net-(U14-ISEN) -> /Motor Control/H-bridge #1/ENCODER_A
- U15 pad 5: +5V -> Net-(U15-Pad5)
- U16 pad 1: /Serial ports/A8 -> /Motor Control/EN_MOTOR3
- U16 pad 2: +5VD -> /Motor Control/PWM1
- U16 pad 3: +5VD -> Net-(U18-IN2)
- U16 pad 4: /Serial ports/EN_IN1 -> GND
- U16 pad 5: /Serial ports/RTS_IN1 -> /Motor Control/EN_MOTOR3
- U16 pad 6: /Serial ports/DSR_IN1 -> /Motor Control/PWM2
- U16 pad 7: /Serial ports/CTS_IN1 -> Net-(U18-IN1)
- U16 pad 8: /Serial ports/DTR_IN1 -> +5V
- U18 pad 2: /External RAM/AD0 -> Net-(U18-IN2)
- U18 pad 3: /External RAM/AD1 -> Net-(U18-IN1)
- U18 pad 4: /External RAM/AD2 -> Net-(U18-VREF)
- U18 pad 5: /External RAM/AD3 -> +12V
- U18 pad 6: /External RAM/AD4 -> /Motor Control/H-bridge #3/MOTOR+
- U18 pad 7: /External RAM/AD5 -> Net-(U18-ISEN)
- U18 pad 8: /External RAM/AD6 -> /Motor Control/H-bridge #3/MOTOR-
- U18 pad 9: /External RAM/AD7 -> GND
- U2 pad 1: GND -> /13
- U2 pad 2: Net-(U2-IN2) -> GND
- U2 pad 3: Net-(U2-IN1) -> GND
- U2 pad 4: Net-(U2-VREF) -> /LIM_SW00
- U2 pad 5: +12V -> /LIM_SW01
- U2 pad 6: /H-bridge #1/MOTOR+ -> /LIM_SW02
- U2 pad 7: Net-(U2-ISEN) -> /LIM_SW03
- U2 pad 8: /H-bridge #1/MOTOR- -> /LIM_SW04
- U2 pad 9: GND -> /LIM_SW05
- U3 pad 1: /H-bridge #1/A_SENSE -> /Motor Control/EN_MOTOR1
- U3 pad 2: GND -> Net-(U3-Pad2)
- U3 pad 3: Net-(U2-ISEN) -> /Motor Control/H-bridge #1/ENCODER_A
- U3 pad 5: +5V -> Net-(U3-Pad5)
- U4 pad 1: /Serial ports/RTS_LINE1 -> /Motor Control/EN_MOTOR1
- U4 pad 2: /Serial ports/DTR_LINE1 -> /Motor Control/PWM1
- U4 pad 3: /Serial ports/TX_LINE1 -> Net-(U6-IN2)
- U4 pad 4: /Serial ports/RI_LINE1 -> GND
- U4 pad 5: /Serial ports/RI_IN1 -> /Motor Control/EN_MOTOR1
- U4 pad 6: /Serial ports/TX3/14 -> /Motor Control/PWM2
- U4 pad 7: /Serial ports/DTR_IN1 -> Net-(U6-IN1)
- U4 pad 8: /Serial ports/CTS_IN1 -> +5V
- U5 pad 1: /13 -> Net-(C9-Pad1)
- U5 pad 10: unconnected-(U5-IO0_6-Pad10) -> Net-(U5-Pad10)
- U5 pad 11: unconnected-(U5-IO0_7-Pad11) -> Net-(C8-Pad1)
- U5 pad 12: GND -> Net-(U3-Pad5)
- U5 pad 13: /LED00 -> Net-(U5-Pad10)
- U5 pad 14: /LED01 -> +5V
- U5 pad 2: GND -> Net-(U5-Pad2)
- U5 pad 3: GND -> Net-(U5-Pad2)
- U5 pad 4: /LIM_SW00 -> Net-(U3-Pad2)
- U5 pad 5: /LIM_SW01 -> Net-(C14-Pad1)
- U5 pad 6: /LIM_SW02 -> /Motor Control/H-bridge #1/LIM1
- U5 pad 7: /LIM_SW03 -> GND
- U5 pad 8: /LIM_SW04 -> /Motor Control/H-bridge #1/LIM2
- U5 pad 9: /LIM_SW05 -> Net-(C15-Pad1)
- U6 pad 1: /AREF -> GND
- U6 pad 2: GND -> Net-(U6-IN2)
- U6 pad 3: unconnected-(U6-NC-Pad3) -> Net-(U6-IN1)
- U7 pad 1: /Serial ports/RTS_LINE2 -> /Motor Control/CURRENT1
- U7 pad 2: /Serial ports/DTR_LINE2 -> GND
- U7 pad 3: /Serial ports/TX_LINE2 -> Net-(U6-ISEN)
- U7 pad 4: /Serial ports/RI_LINE2 -> GND
- U7 pad 5: /Serial ports/RI_IN2 -> +5V
- U8 pad 1: /External RAM/A17 -> /Motor Control/EN_MOTOR2
- U8 pad 2: /External RAM/A16 -> Net-(U10-Pad4)
- U8 pad 3: /External RAM/A14 -> /Motor Control/H-bridge #1/ENCODER_A
- U8 pad 4: /External RAM/A12 -> GND
- U8 pad 5: Net-(U18-Q7) -> Net-(U10-Pad12)
- U8 pad 6: Net-(U18-Q6) -> /Motor Control/H-bridge #1/ENCODER_B
- U8 pad 7: Net-(U18-Q5) -> /Motor Control/EN_MOTOR2
- U8 pad 8: Net-(U18-Q4) -> +5V
- U9 pad 1: +5V -> /Motor Control/EN_MOTOR2
- U9 pad 2: unconnected-(U9-CH1-Pad2) -> /Motor Control/PWM1
- U9 pad 3: unconnected-(U9-CH0/V_{CAL}-Pad3) -> Net-(U11-IN2)
- U9 pad 5: Net-(U9-V_{OUT}) -> /Motor Control/EN_MOTOR2
- U9 pad 6: GND -> /Motor Control/PWM2
- U9 pad 7: unconnected-(U9-SCLK-Pad7) -> Net-(U11-IN1)
- U9 pad 8: unconnected-(U9-DIO-Pad8) -> +5V
