File: ECAD/BDCMotorControlShieldMega/BDCMotorControlShieldMega.kicad_pcb (KiCad board)
At the start: 2 copper layers, 101.6 x 53.3 mm, 150 parts, among them J1 Power, J10 Limit switch, J11 Limit switch, J12 Motor Connector, J13 Limit switch, J14 Limit switch, J15 Motor Connector, J16 Limit switch, J17 Limit switch, J18 Conn_01x20, J2 PWM, J3 Analog, J4 PWM, J5 Analog, J6 Communication, J7 Digital, J8 Barrel_Jack_Switch, J9 Motor Connector, U1 LM4040DBZ-4.1, U10 74AHC14, U11 DRV8870DDA, U12 INA180A1, U13 SP213, U14 SP213, U15 74AHC2G125, U16 74AHC2G08, U17 74AHC14, U18 DRV8870DDA, U19 INA180A1, U2 PCA9555PW, U20 74AHC573, U21 CY62148ELL-45ZSXIT, U22 PCA9555PW, U23 MCP6S26, U3 74AHC2G125, U4 74AHC2G08, U5 74AHC14, U6 DRV8870DDA, U7 INA180A1, U8 74AHC2G125, U9 74AHC2G08

Commit message: Progressed ECAD.
Parts:
- removed L5: 10uL, Inductor_SMD:L_0805_2012Metric
- removed R38: 10kR, Resistor_SMD:R_0805_2012Metric
- removed R39: 1kR, Resistor_SMD:R_0402_1005Metric
- added C56: 100nC, Capacitor_SMD:C_0805_2012Metric, F.Cu at (255.4, 88.2)
- added C57: 100pC, Capacitor_SMD:C_0805_2012Metric, F.Cu at (286.1, 61.0)
- added C58: 100nC, Capacitor_SMD:C_0805_2012Metric, F.Cu at (286.1, 64.0)
- added C59: 100nC, Capacitor_SMD:C_0805_2012Metric, F.Cu at (286.1, 67.0)
- added C60: 100nC, Capacitor_SMD:C_0805_2012Metric, F.Cu at (210.2, 113.8)
- added U24: 74AHC1G79, Package_TO_SOT_SMD:SOT-353_SC-70-5, F.Cu at (210.1, 117.3)
- C1, C13, C16, C17, C18, C19, C38, C39, C4, C40, C41, C5, C6, C7: value 0.1uC -> 100nC; footprint Capacitor_SMD:C_0805_2012Metric_Pad1.18x1.45mm_HandSolder -> Capacitor_SMD:C_0805_2012Metric
- C10: value 10uC -> 100pC; footprint Capacitor_SMD:C_1210_3225Metric_Pad1.33x2.70mm_HandSolder -> Capacitor_SMD:C_0805_2012Metric
- C11, C23: value 47uC -> 100pC; footprint Capacitor_THT:CP_Radial_D5.0mm_P2.00mm -> Capacitor_SMD:C_0805_2012Metric
- C12, C25: value 0.1uC -> 47uC; footprint Capacitor_SMD:C_0805_2012Metric_Pad1.18x1.45mm_HandSolder -> Capacitor_THT:CP_Radial_D5.0mm_P2.00mm
- C2: value 10uC -> 100nC; footprint Capacitor_SMD:C_1206_3216Metric -> Capacitor_SMD:C_0805_2012Metric
- C20, C21, C42, C43, C53, C8: value 100pC -> 100nC; footprint Capacitor_SMD:C_0402_1005Metric -> Capacitor_SMD:C_0805_2012Metric
- C22: footprint Capacitor_SMD:C_1210_3225Metric_Pad1.33x2.70mm_HandSolder -> Capacitor_SMD:C_1210_3225Metric
- C24, C46, C47: value 0.1uC -> 100pC; footprint Capacitor_SMD:C_0805_2012Metric_Pad1.18x1.45mm_HandSolder -> Capacitor_SMD:C_0805_2012Metric
- C3: value 100nC -> 10uC; footprint Capacitor_SMD:C_0805_2012Metric -> Capacitor_SMD:C_1206_3216Metric
- C44: value 10uC -> 100nC; footprint Capacitor_SMD:C_1210_3225Metric_Pad1.33x2.70mm_HandSolder -> Capacitor_SMD:C_0805_2012Metric
- C45: value 47uC -> 10uC; footprint Capacitor_THT:CP_Radial_D5.0mm_P2.00mm -> Capacitor_SMD:C_1210_3225Metric
- C48: value 100nC -> 47uC; footprint Capacitor_SMD:C_0805_2012Metric -> Capacitor_THT:CP_Radial_D5.0mm_P2.00mm
- C9: value 100pC -> 10uC; footprint Capacitor_SMD:C_0402_1005Metric -> Capacitor_SMD:C_1210_3225Metric
- R1, R10, R18, R19, R2, R27, R28, R3, R4, R6, R8, R9: footprint Resistor_SMD:R_0805_2012Metric_Pad1.20x1.40mm_HandSolder -> Resistor_SMD:R_0805_2012Metric
- R11, R12, R20, R21, R29, R30: footprint Resistor_SMD:R_0402_1005Metric -> Resistor_SMD:R_0805_2012Metric
- R14, R15, R16, R17, R23, R24, R25, R26, R32, R33, R34, R35: footprint Capacitor_SMD:C_0805_2012Metric -> Resistor_SMD:R_0805_2012Metric
- R37: value 10kR -> 1kR
- R5: value 1kR -> 10kR; footprint Resistor_SMD:R_0805_2012Metric_Pad1.20x1.40mm_HandSolder -> Resistor_SMD:R_0805_2012Metric
- R7: value 10kR -> 1kR; footprint Resistor_SMD:R_0805_2012Metric_Pad1.20x1.40mm_HandSolder -> Resistor_SMD:R_0805_2012Metric
- moved C50 82.8 mm to (223.7, 47.0)
- moved C51 82.8 mm to (223.7, 50.0)
- moved C4 80.3 mm to (259.8, 118.2)
- moved L3 68.3 mm to (236.2, 59.7)
- moved C38 66.0 mm to (277.6, 50.0)
- moved C39 66.0 mm to (277.6, 53.0)
- moved C40 66.0 mm to (277.6, 56.0)
- moved C53 60.2 mm to (223.7, 56.0)
- moved R13 59.4 mm to (220.8, 102.1)
- moved R29 50.5 mm to (214.8, 49.8)
- moved U7 50.3 mm to (228.5, 104.0)
- moved R30 49.6 mm to (214.8, 52.8)
- moved C54 48.3 mm to (288.6, 107.6)
- moved C55 48.3 mm to (288.6, 110.6)
- moved C52 47.8 mm to (223.7, 53.0)
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Connections:
- C10 pad 1: +12V -> Net-(C10-Pad1)
- C11 pad 1: +12V -> Net-(C11-Pad1)
- C12 pad 1: +5V -> +12V
- C14 pad 1: Net-(C14-Pad1) -> Net-(U7-V+)
- C15 pad 1: Net-(C15-Pad1) -> +5V
- C16 pad 1: +5V -> Net-(C16-Pad1)
- C17 pad 1: +5V -> Net-(C17-Pad1)
- C18 pad 1: Net-(U11-VREF) -> +5V
- C19 pad 1: +12V -> +5V
- C2 pad 1: +5V -> /AREF
- C20 pad 1: Net-(C20-Pad1) -> Net-(U11-VREF)
- C21 pad 1: Net-(C21-Pad1) -> +12V
- C23 pad 1: +12V -> Net-(C23-Pad1)
- C24 pad 1: +5V -> Net-(C24-Pad1)
- C25 pad 1: +5V -> +12V
- C26 pad 1: Net-(C26-Pad1) -> +5V
- C27 pad 1: Net-(C27-Pad1) -> Net-(U12-V+)
- C28 pad 1: /Serial ports/RS232 Interface #1/C1+ -> +5V
- C28 pad 2: /Serial ports/RS232 Interface #1/C1- -> GND
- C29 pad 1: /Serial ports/RS232 Interface #1/V- -> Net-(C29-Pad1)
- C30 pad 1: /Serial ports/RS232 Interface #1/C2+ -> Net-(C30-Pad1)
- C30 pad 2: /Serial ports/RS232 Interface #1/C2- -> GND
- C31 pad 1: +5V -> /Serial ports/RS232 Interface #1/C1+
- C31 pad 2: /Serial ports/RS232 Interface #1/V+ -> /Serial ports/RS232 Interface #1/C1-
- C32 pad 1: +5VD -> /Serial ports/RS232 Interface #1/V-
- C33 pad 1: /Serial ports/RS232 Interface #2/C1+ -> /Serial ports/RS232 Interface #1/C2+
- C33 pad 2: /Serial ports/RS232 Interface #2/C1- -> /Serial ports/RS232 Interface #1/C2-
- C34 pad 1: /Serial ports/RS232 Interface #2/V- -> +5V
- C34 pad 2: GND -> /Serial ports/RS232 Interface #1/V+
- C35 pad 1: /Serial ports/RS232 Interface #2/C2+ -> +5V
- C35 pad 2: /Serial ports/RS232 Interface #2/C2- -> GND
- C36 pad 1: +5V -> /Serial ports/RS232 Interface #2/C1+
- C36 pad 2: /Serial ports/RS232 Interface #2/V+ -> /Serial ports/RS232 Interface #2/C1-
- C37 pad 1: +5VD -> /Serial ports/RS232 Interface #2/V-
- C38 pad 1: +5V -> /Serial ports/RS232 Interface #2/C2+
- C38 pad 2: GND -> /Serial ports/RS232 Interface #2/C2-
- C39 pad 2: GND -> /Serial ports/RS232 Interface #2/V+
- C40 pad 1: Net-(U18-VREF) -> +5V
- C41 pad 1: +12V -> +5V
- C42 pad 1: Net-(C42-Pad1) -> +5V
- C43 pad 1: Net-(C43-Pad1) -> Net-(U18-VREF)
- C46 pad 1: +5V -> Net-(C46-Pad1)
- C47 pad 1: +5V -> Net-(C47-Pad1)
- C48 pad 1: Net-(C48-Pad1) -> +12V
- C49 pad 1: Net-(C49-Pad1) -> +5V
- C50 pad 1: +5VD -> Net-(U19-V+)
- C51 pad 1: +5VD -> +5V
- C52 pad 1: +5VD -> Net-(C52-Pad1)
- C53 pad 1: Net-(U23-V_{OUT}) -> Net-(C53-Pad1)
- C6 pad 1: Net-(U6-VREF) -> +5V
- C7 pad 1: +12V -> Net-(U6-VREF)
- C8 pad 1: Net-(C8-Pad1) -> +12V
- C9 pad 1: Net-(C9-Pad1) -> +12V
- J1 pad 2: /IOREF -> unconnected-(J1-Pin_2-Pad2)
- J1 pad 3: /~{RESET} -> unconnected-(J1-Pin_3-Pad3)
- J1 pad 4: +3V3 -> unconnected-(J1-Pin_4-Pad4)
- J1 pad 8: VCC -> unconnected-(J1-Pin_8-Pad8)
- L1 pad 2: +5VD -> Net-(U7-V+)
- L2 pad 2: +5VD -> Net-(U12-V+)
- L3 pad 2: +5VD -> Net-(U19-V+)
- L4 pad 2: +5VD -> Net-(U23-V_{DD})
- R11 pad 1: Net-(C8-Pad1) -> Net-(C10-Pad1)
- R12 pad 1: Net-(C9-Pad1) -> Net-(C11-Pad1)
- R14 pad 1: Net-(C14-Pad1) -> Net-(C16-Pad1)
- R15 pad 1: Net-(C15-Pad1) -> Net-(C17-Pad1)
- R20 pad 1: Net-(C20-Pad1) -> Net-(C23-Pad1)
- R21 pad 1: Net-(C21-Pad1) -> Net-(C24-Pad1)
- R23 pad 1: Net-(C26-Pad1) -> Net-(C29-Pad1)
- R24 pad 1: Net-(C27-Pad1) -> Net-(C30-Pad1)
- R29 pad 1: Net-(C42-Pad1) -> Net-(C46-Pad1)
- R30 pad 1: Net-(C43-Pad1) -> Net-(C47-Pad1)
- R32 pad 1: Net-(C48-Pad1) -> Net-(C52-Pad1)
- R33 pad 1: Net-(C49-Pad1) -> Net-(C53-Pad1)
- R36 pad 1: /Serial ports/~{INT} -> /RX3/15
- R37 pad 1: /SDA/A4 -> Net-(U23-V_{OUT})
- R37 pad 2: +5V -> /A0
- R5 pad 2: /AREF -> /SCL/21
- R6 pad 2: /13 -> /SDA/20
- R7 pad 2: /SDA/A4 -> /AREF
- R8 pad 2: /SCL/A5 -> /13
- U10 pad 1: Net-(C21-Pad1) -> Net-(C24-Pad1)
- U10 pad 11: Net-(C20-Pad1) -> Net-(C23-Pad1)
- U10 pad 5: Net-(C26-Pad1) -> Net-(C29-Pad1)
- U10 pad 6: /Motor Control/H-bridge #2/LIM1 -> /LIM_SW02
- U10 pad 8: /Motor Control/H-bridge #2/LIM2 -> /LIM_SW03
- U10 pad 9: Net-(C27-Pad1) -> Net-(C30-Pad1)
- U12 pad 5: +5V -> Net-(U12-V+)
- U13 pad 11: +5VD -> +5V
- U13 pad 19: /Serial ports/RX1 -> /RX1/19
- U13 pad 6: /Serial ports/TX1 -> /TX1/18
- U14 pad 11: +5VD -> +5V
- U14 pad 19: /Serial ports/RX2 -> /RX2/17
- U14 pad 6: /Serial ports/TX2 -> /TX2/16
- U15 pad 1: /Motor Control/EN_MOTOR3 -> /Motor Control/EN_ENC_MOTOR3
- U15 pad 7: /Motor Control/EN_MOTOR3 -> /Motor Control/EN_ENC_MOTOR3
- U17 pad 1: Net-(C43-Pad1) -> Net-(C47-Pad1)
- U17 pad 11: Net-(C42-Pad1) -> Net-(C46-Pad1)
- U17 pad 5: Net-(C48-Pad1) -> Net-(C52-Pad1)
- U17 pad 6: /Motor Control/H-bridge #3/LIM1 -> /LIM_SW04
- U17 pad 8: /Motor Control/H-bridge #3/LIM2 -> /LIM_SW05
- U17 pad 9: Net-(C49-Pad1) -> Net-(C53-Pad1)
- U19 pad 5: +5V -> Net-(U19-V+)
- U20 pad 11: /External RAM/ALE -> /39
- U20 pad 2: /External RAM/AD0 -> /22
- U20 pad 20: +5VD -> +5V
- U20 pad 3: /External RAM/AD1 -> /23
- U20 pad 4: /External RAM/AD2 -> /24
- U20 pad 5: /External RAM/AD3 -> /25
- U20 pad 6: /External RAM/AD4 -> /26
- U20 pad 7: /External RAM/AD5 -> /27
- U20 pad 8: /External RAM/AD6 -> /28
- U20 pad 9: /External RAM/AD7 -> /29
- U21 pad 1: /External RAM/A17 -> /43
- U21 pad 13: /External RAM/AD0 -> /22
- U21 pad 14: /External RAM/AD1 -> /23
- U21 pad 15: /External RAM/AD2 -> /24
- U21 pad 17: /External RAM/AD3 -> /25
- U21 pad 18: /External RAM/AD4 -> /26
- U21 pad 19: /External RAM/AD5 -> /27
- U21 pad 2: /External RAM/A16 -> /42
- U21 pad 20: /External RAM/AD6 -> /28
- U21 pad 21: /External RAM/AD7 -> /29
- U21 pad 23: /External RAM/A10 -> /35
- U21 pad 24: /External RAM/~{RD} -> /40
- U21 pad 25: /External RAM/A11 -> /34
- U21 pad 26: /External RAM/A09 -> /36
- U21 pad 27: /External RAM/A08 -> /37
- U21 pad 28: /External RAM/A13 -> /32
- U21 pad 29: /External RAM/~{WR} -> /41
- U21 pad 3: /External RAM/A14 -> /31
- U21 pad 30: /External RAM/A18 -> /*44
- U21 pad 31: /External RAM/A15 -> /30
- U21 pad 32: +5VD -> +5V
- U21 pad 4: /External RAM/A12 -> /33
- U22 pad 1: /Serial ports/~{INT} -> /RX3/15
- U22 pad 2: +5VD -> +5V
- U22 pad 21: +5VD -> +5V
- U22 pad 22: /SCL/A5 -> /SCL/21
- U22 pad 23: /SDA/A4 -> /SDA/20
- U22 pad 24: +5VD -> +5V
- U22 pad 3: +5VD -> +5V
- U23 pad 10: unconnected-(U23-~{CS}-Pad10) -> /53
- U23 pad 11: unconnected-(U23-SI-Pad11) -> /51
- U23 pad 12: unconnected-(U23-SO-Pad12) -> /50
- U23 pad 13: unconnected-(U23-SCK-Pad13) -> /*52
- U23 pad 14: unconnected-(U23-V_{DD}-Pad14) -> Net-(U23-V_{DD})
- U23 pad 8: unconnected-(U23-V_{REF}-Pad8) -> GND
- U3 pad 1: /Motor Control/EN_MOTOR1 -> /Motor Control/EN_ENC_MOTOR1
- U3 pad 7: /Motor Control/EN_MOTOR1 -> /Motor Control/EN_ENC_MOTOR1
- U5 pad 1: Net-(C9-Pad1) -> Net-(C11-Pad1)
- U5 pad 11: Net-(C8-Pad1) -> Net-(C10-Pad1)
- U5 pad 5: Net-(C14-Pad1) -> Net-(C16-Pad1)
- U5 pad 6: /Motor Control/H-bridge #1/LIM1 -> /LIM_SW00
- U5 pad 8: /Motor Control/H-bridge #1/LIM2 -> /LIM_SW01
- U5 pad 9: Net-(C15-Pad1) -> Net-(C17-Pad1)
- U7 pad 5: +5V -> Net-(U7-V+)
- U8 pad 1: /Motor Control/EN_MOTOR2 -> /Motor Control/EN_ENC_MOTOR2
- U8 pad 7: /Motor Control/EN_MOTOR2 -> /Motor Control/EN_ENC_MOTOR2

Commit message: Progressed ECAD.
Parts:
- added R38: 160R, Resistor_SMD:R_0805_2012Metric, F.Cu at (224.1, 114.0)
- C3: footprint Capacitor_SMD:C_1206_3216Metric -> Capacitor_SMD:C_1210_3225Metric
- C57: value 100pC -> 4.7uC
- R13, R22, R31: value 250mR -> 150mR; footprint Resistor_SMD:R_2010_5025Metric -> Resistor_SMD:R_1206_3216Metric
- R37: value 1kR -> 10kR
- U24: value 74AHC1G79 -> IRM-H6XX; footprint Package_TO_SOT_SMD:SOT-353_SC-70-5 -> OptoDevice_custom:IRM-H6XX
- moved U24 5.22 mm to (215.0, 119.0)
Connections:
- C57 pad 1: Net-(U23-V_{OUT}) -> Net-(U24-Vs)
- R37 pad 1: Net-(U23-V_{OUT}) -> +5V
- R37 pad 2: /A0 -> /*8
- U23 pad 1: Net-(U23-V_{OUT}) -> /A0
- U24 pad 1: /Motor Control/H-bridge #1/ENCODER_A -> GND
- U24 pad 2: /Motor Control/H-bridge #1/ENCODER_B -> GND
- U24 pad 3: GND -> /*8
- U24 pad 4: unconnected-(U24-Q-Pad4) -> Net-(U24-Vs)

Commit message: Progressed ECAD.
Parts:
- removed C54, C55, C60: 100nC, Capacitor_SMD:C_0805_2012Metric
- removed U20: 74AHC573, Package_SO:TSSOP-20_4.4x6.5mm_P0.65mm
- removed U21: CY62148ELL-45ZSXIT, Package_SO:TSOP-II-32_21.0x10.2mm_P1.27mm

Commit message: Progressed ECAD.
Parts:
- removed D1, D2, D3, D4: LED, LED_SMD:LED_0805_2012Metric
- removed R1, R2, R3, R4: 1kR, Resistor_SMD:R_0805_2012Metric
- removed U10: 74AHC14, Package_SO:TSSOP-14_4.4x5mm_P0.65mm
- removed U11, U18: DRV8870DDA, Package_SO:Texas_HTSOP-8-1EP_3.9x4.9mm_P1.27mm_EP2.95x4.9mm_Mask2.4x3.1mm_ThermalVias
- removed U4: 74AHC2G08, Package_SO:TSSOP-8_3x3mm_P0.65mm
- removed U8: 74AHC2G125, Package_SO:TSSOP-8_3x3mm_P0.65mm
- added C100: 100nC, Capacitor_SMD:C_0805_2012Metric, F.Cu at (264.9, 76.0)
- added C101: 100nC, Capacitor_SMD:C_0805_2012Metric, F.Cu at (287.9, 36.3)
- added C102: 100nC, Capacitor_SMD:C_0805_2012Metric, F.Cu at (287.9, 39.3)
- added C103: 100nC, Capacitor_SMD:C_0805_2012Metric, F.Cu at (287.9, 42.3)
- added C104: 100nC, Capacitor_SMD:C_0805_2012Metric, F.Cu at (287.9, 45.3)
- added C105: 100pC, Capacitor_SMD:C_0805_2012Metric, F.Cu at (287.9, 48.4)
- added C106: 100pC, Capacitor_SMD:C_0805_2012Metric, F.Cu at (287.9, 51.4)
- added C107: 100nC, Capacitor_SMD:C_0805_2012Metric, F.Cu at (292.4, 36.3)
- added C109: 100nC, Capacitor_SMD:C_0805_2012Metric, F.Cu at (292.4, 39.3)
- added C110: 100nC, Capacitor_SMD:C_0805_2012Metric, F.Cu at (292.4, 42.3)
- added C111: 10uC, Capacitor_SMD:C_1210_3225Metric, F.Cu at (288.5, 55.0)
- added C112: 47uC, Capacitor_THT:CP_Radial_D5.0mm_P2.00mm, F.Cu at (296.9, 54.0)
- added C115: 100nC, Capacitor_SMD:C_0805_2012Metric, F.Cu at (292.4, 45.3)
- added C116: 100nC, Capacitor_SMD:C_0805_2012Metric, F.Cu at (292.4, 48.4)
- added C60: 100nC, Capacitor_SMD:C_0805_2012Metric, F.Cu at (264.9, 45.3)
- added C61: 100nC, Capacitor_SMD:C_0805_2012Metric, F.Cu at (264.9, 97.6)
- added C62: 10uC, Capacitor_SMD:C_1210_3225Metric, F.Cu at (261.1, 110.2)
- added C63: 100nC, Capacitor_SMD:C_0805_2012Metric, F.Cu at (264.9, 48.4)
- added C64: 47uC, Capacitor_THT:CP_Radial_D5.0mm_P2.00mm, F.Cu at (269.5, 109.2)
- added C65: 100nC, Capacitor_SMD:C_0805_2012Metric, F.Cu at (240.8, 45.3)
- added C66: 100nC, Capacitor_SMD:C_0805_2012Metric, F.Cu at (240.8, 48.4)
- added C67: 100nC, Capacitor_SMD:C_0805_2012Metric, F.Cu at (264.9, 100.6)
- added C68: 100nC, Capacitor_SMD:C_0805_2012Metric, F.Cu at (264.9, 103.6)
- added C69: 100nC, Capacitor_SMD:C_0805_2012Metric, F.Cu at (228.4, 77.6)
- added C70: 100nC, Capacitor_SMD:C_0805_2012Metric, F.Cu at (228.4, 80.6)
- added C71: 100nC, Capacitor_SMD:C_0805_2012Metric, F.Cu at (228.4, 83.6)
- added C72: 100nC, Capacitor_SMD:C_0805_2012Metric, F.Cu at (228.4, 86.6)
- added C73: 100pC, Capacitor_SMD:C_0805_2012Metric, F.Cu at (228.4, 89.7)
- added C74: 100pC, Capacitor_SMD:C_0805_2012Metric, F.Cu at (228.4, 92.7)
- added C75: 100nC, Capacitor_SMD:C_0805_2012Metric, F.Cu at (232.9, 77.6)
- added C77: 100nC, Capacitor_SMD:C_0805_2012Metric, F.Cu at (232.9, 80.6)
- added C78: 100nC, Capacitor_SMD:C_0805_2012Metric, F.Cu at (232.9, 83.6)
- added C79: 10uC, Capacitor_SMD:C_1210_3225Metric, F.Cu at (229.0, 96.3)
- added C80: 47uC, Capacitor_THT:CP_Radial_D5.0mm_P2.00mm, F.Cu at (237.4, 95.3)
- added C83: 100nC, Capacitor_SMD:C_0805_2012Metric, F.Cu at (232.9, 86.6)
- added C84: 100nC, Capacitor_SMD:C_0805_2012Metric, F.Cu at (232.9, 89.7)
- added C85: 100nC, Capacitor_SMD:C_0805_2012Metric, F.Cu at (260.5, 63.9)
- added C86: 100nC, Capacitor_SMD:C_0805_2012Metric, F.Cu at (260.5, 66.9)
- added C87: 100nC, Capacitor_SMD:C_0805_2012Metric, F.Cu at (260.5, 70.0)
- added C88: 100nC, Capacitor_SMD:C_0805_2012Metric, F.Cu at (260.5, 73.0)
- added C89: 100pC, Capacitor_SMD:C_0805_2012Metric, F.Cu at (260.5, 76.0)
- added C90: 100pC, Capacitor_SMD:C_0805_2012Metric, F.Cu at (260.5, 79.0)
- added C91: 100nC, Capacitor_SMD:C_0805_2012Metric, F.Cu at (264.9, 63.9)
- added C93: 100nC, Capacitor_SMD:C_0805_2012Metric, F.Cu at (264.9, 66.9)
- added C94: 100nC, Capacitor_SMD:C_0805_2012Metric, F.Cu at (264.9, 70.0)
- added C95: 10uC, Capacitor_SMD:C_1210_3225Metric, F.Cu at (261.1, 82.6)
- added C96: 47uC, Capacitor_THT:CP_Radial_D5.0mm_P2.00mm, F.Cu at (269.5, 81.6)
- added C99: 100nC, Capacitor_SMD:C_0805_2012Metric, F.Cu at (264.9, 73.0)
- added J19: Motor Connector, Connector_JST:JST_PH_B6B-PH-K_1x06_P2.00mm_Vertical, F.Cu at (238.1, 78.8)
- added J22: Motor Connector, Connector_JST:JST_PH_B6B-PH-K_1x06_P2.00mm_Vertical, F.Cu at (270.1, 65.2)
- added J25: Motor Connector, Connector_JST:JST_PH_B6B-PH-K_1x06_P2.00mm_Vertical, F.Cu at (297.6, 37.5)
- added L5: 10uL, Inductor_SMD:L_0805_2012Metric, F.Cu at (248.7, 88.7)
- added L6: 10uL, Inductor_SMD:L_0805_2012Metric, F.Cu at (280.8, 75.0)
- added L7: 10uL, Inductor_SMD:L_0805_2012Metric, F.Cu at (308.2, 47.4)
- added L8: 10uL, Inductor_SMD:L_0805_2012Metric, F.Cu at (245.2, 67.4)
- added R39: 1kR, Resistor_SMD:R_0805_2012Metric, F.Cu at (244.2, 84.1)
- added R40: 1kR, Resistor_SMD:R_0805_2012Metric, F.Cu at (244.2, 87.1)
- added R41: 10kR, Resistor_SMD:R_0805_2012Metric, F.Cu at (244.2, 90.0)
- added R42: 10kR, Resistor_SMD:R_0805_2012Metric, F.Cu at (244.2, 93.0)
- added R43: 150mR, Resistor_SMD:R_1206_3216Metric, F.Cu at (229.0, 100.1)
- added R48: 1kR, Resistor_SMD:R_0805_2012Metric, F.Cu at (276.3, 70.5)
- added R49: 1kR, Resistor_SMD:R_0805_2012Metric, F.Cu at (276.3, 73.4)
- added R50: 10kR, Resistor_SMD:R_0805_2012Metric, F.Cu at (276.3, 76.4)
- added R51: 10kR, Resistor_SMD:R_0805_2012Metric, F.Cu at (276.3, 79.3)
- added R52: 150mR, Resistor_SMD:R_1206_3216Metric, F.Cu at (261.1, 86.4)
- added R57: 1kR, Resistor_SMD:R_0805_2012Metric, F.Cu at (303.7, 42.8)
- added R58: 1kR, Resistor_SMD:R_0805_2012Metric, F.Cu at (303.7, 45.8)
- added R59: 10kR, Resistor_SMD:R_0805_2012Metric, F.Cu at (303.7, 48.7)
- added R60: 10kR, Resistor_SMD:R_0805_2012Metric, F.Cu at (303.7, 51.7)
- added R61: 150mR, Resistor_SMD:R_1206_3216Metric, F.Cu at (288.5, 58.8)
- added U29: 74AHC2G08, Package_SO:TSSOP-8_3x3mm_P0.65mm, F.Cu at (270.6, 103.6)
- added U30: DRV8870DDA, Package_SO:Texas_HTSOP-8-1EP_3.9x4.9mm_P1.27mm_EP2.95x4.9mm_Mask2.4x3.1mm_ThermalVias, F.Cu at (278.8, 111.8)
- added U31: INA180A1, Package_TO_SOT_SMD:SOT-23-5, F.Cu at (281.1, 99.0)
- added U33: 74AHC2G125, Package_SO:TSSOP-8_3x3mm_P0.65mm, F.Cu at (238.6, 85.0)
- added U34: 74AHC2G08, Package_SO:TSSOP-8_3x3mm_P0.65mm, F.Cu at (270.6, 48.4)
- added U39: 74AHC2G08, Package_SO:TSSOP-8_3x3mm_P0.65mm, F.Cu at (238.6, 89.7)
- added U40: DRV8870DDA, Package_SO:Texas_HTSOP-8-1EP_3.9x4.9mm_P1.27mm_EP2.95x4.9mm_Mask2.4x3.1mm_ThermalVias, F.Cu at (246.8, 97.8)
- added U41: INA180A1, Package_TO_SOT_SMD:SOT-23-5, F.Cu at (249.0, 85.1)
- added U43: 74AHC2G125, Package_SO:TSSOP-8_3x3mm_P0.65mm, F.Cu at (270.6, 71.3)
- added U47: 74AHC2G08, Package_SO:TSSOP-8_3x3mm_P0.65mm, F.Cu at (270.6, 76.0)
- added U48: DRV8870DDA, Package_SO:Texas_HTSOP-8-1EP_3.9x4.9mm_P1.27mm_EP2.95x4.9mm_Mask2.4x3.1mm_ThermalVias, F.Cu at (278.8, 84.1)
- added U49: INA180A1, Package_TO_SOT_SMD:SOT-23-5, F.Cu at (281.1, 71.4)
- added U51: 74AHC2G125, Package_SO:TSSOP-8_3x3mm_P0.65mm, F.Cu at (298.1, 43.7)
- added U55: 74AHC2G08, Package_SO:TSSOP-8_3x3mm_P0.65mm, F.Cu at (298.1, 48.4)
- added U56: DRV8870DDA, Package_SO:Texas_HTSOP-8-1EP_3.9x4.9mm_P1.27mm_EP2.95x4.9mm_Mask2.4x3.1mm_ThermalVias, F.Cu at (306.2, 56.5)
- added U57: INA180A1, Package_TO_SOT_SMD:SOT-23-5, F.Cu at (308.5, 43.8)
- C22, C45: value 10uC -> 100nC; footprint Capacitor_SMD:C_1210_3225Metric -> Capacitor_SMD:C_0805_2012Metric
- C25, C48: value 47uC -> 100nC; footprint Capacitor_THT:CP_Radial_D5.0mm_P2.00mm -> Capacitor_SMD:C_0805_2012Metric
- C29: value 100nC -> 10uC; footprint Capacitor_SMD:C_0805_2012Metric -> Capacitor_SMD:C_1210_3225Metric
- C30: value 100nC -> 47uC; footprint Capacitor_SMD:C_0805_2012Metric -> Capacitor_THT:CP_Radial_D5.0mm_P2.00mm
- C46, C47: value 100pC -> 100nC
- C49, C50: value 100nC -> 100pC
- R18, R19, R27, R28: value 10kR -> 1kR
- R20, R21, R29, R30: value 1kR -> 10kR
- U12: value INA180A1 -> MCP6S26; footprint Package_TO_SOT_SMD:SOT-23-5 -> Package_SO:SOIC-14_3.9x8.7mm_P1.27mm
- U15: value 74AHC2G125 -> 74AHC2G08
- U16: value 74AHC2G08 -> DRV8870DDA; footprint Package_SO:TSSOP-8_3x3mm_P0.65mm -> Package_SO:Texas_HTSOP-8-1EP_3.9x4.9mm_P1.27mm_EP2.95x4.9mm_Mask2.4x3.1mm_ThermalVias
- U17: value 74AHC14 -> INA180A1; footprint Package_SO:TSSOP-14_4.4x5mm_P0.65mm -> Package_TO_SOT_SMD:SOT-23-5
- U19: value INA180A1 -> 74AHC2G125; footprint Package_TO_SOT_SMD:SOT-23-5 -> Package_SO:TSSOP-8_3x3mm_P0.65mm
- U9: value 74AHC2G08 -> 74AHC2G125
- moved U17 87.4 mm to (308.5, 71.4)
- moved R27 81.9 mm to (276.3, 98.1)
- moved R28 81.9 mm to (276.3, 101.0)
- moved R29 81.9 mm to (276.3, 104.0)
- moved R30 81.9 mm to (276.3, 106.9)
- moved U7 80.0 mm to (281.1, 43.8)
- moved C43 76.6 mm to (292.4, 73.0)
- moved C44 76.6 mm to (292.4, 76.0)
- moved C36 75.4 mm to (304.9, 114.3)
- moved C37 75.4 mm to (304.9, 117.3)
- moved C38 75.4 mm to (304.9, 120.3)
- moved C39 75.4 mm to (304.9, 123.3)
- moved C40 75.4 mm to (304.9, 126.3)
- moved U14 75.4 mm to (312.4, 118.8)
- moved R37 74.4 mm to (228.4, 117.0)
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Connections:
- net /Motor Control/EN_ENC_MOTOR1 renamed /Motor Control/H-bridge #1/~{ENABLE_ENCODER}
- C20 pad 1: Net-(U11-VREF) -> +5V
- C21 pad 1: +12V -> +5V
- C22 pad 1: +12V -> +5V
- C25 pad 1: +12V -> +5V
- C26 pad 1: +5V -> Net-(C26-Pad1)
- C27 pad 1: Net-(U12-V+) -> Net-(U16-VREF)
- C28 pad 1: +5V -> +12V
- C29 pad 1: Net-(C29-Pad1) -> +12V
- C30 pad 1: Net-(C30-Pad1) -> +12V
- C41 pad 1: +5V -> Net-(C41-Pad1)
- C42 pad 1: +5V -> Net-(C42-Pad1)
- C43 pad 1: Net-(U18-VREF) -> Net-(U17-V+)
- C44 pad 1: +12V -> +5V
- C45 pad 1: +12V -> +5V
- C46 pad 1: Net-(C46-Pad1) -> +5V
- C47 pad 1: Net-(C47-Pad1) -> +5V
- C48 pad 1: +12V -> +5V
- C49 pad 1: +5V -> Net-(C49-Pad1)
- C50 pad 1: Net-(U19-V+) -> Net-(C50-Pad1)
- C53 pad 1: Net-(C53-Pad1) -> Net-(U30-VREF)
- J12 pad 5: /Motor Control/H-bridge #1/ENCODER_A -> /*5
- J12 pad 6: /Motor Control/H-bridge #1/ENCODER_B -> /*4
- J15 pad 1: /Motor Control/H-bridge #3/MOTOR+ -> /Motor Control/H-bridge #4/MOTOR+
- J15 pad 2: /Motor Control/H-bridge #3/MOTOR- -> /Motor Control/H-bridge #4/MOTOR-
- J15 pad 5: /Motor Control/H-bridge #1/ENCODER_A -> /*5
- J15 pad 6: /Motor Control/H-bridge #1/ENCODER_B -> /*4
- J9 pad 5: /Motor Control/H-bridge #1/ENCODER_A -> /*7
- J9 pad 6: /Motor Control/H-bridge #1/ENCODER_B -> /*6
- L2 pad 2: Net-(U12-V+) -> Net-(U17-V+)
- L3 pad 2: Net-(U19-V+) -> Net-(U31-V+)
- R11 pad 2: /Motor Control/H-bridge #1/ENCODER_A -> /*7
- R12 pad 2: /Motor Control/H-bridge #1/ENCODER_B -> /*6
- R18 pad 1: +5V -> Net-(C23-Pad1)
- R18 pad 2: Net-(U11-VREF) -> /*5
- R19 pad 1: Net-(U11-VREF) -> Net-(C24-Pad1)
- R19 pad 2: GND -> /*4
- R20 pad 1: Net-(C23-Pad1) -> +5V
- R20 pad 2: /Motor Control/H-bridge #1/ENCODER_A -> Net-(U16-VREF)
- R21 pad 1: Net-(C24-Pad1) -> Net-(U16-VREF)
- R21 pad 2: /Motor Control/H-bridge #1/ENCODER_B -> GND
- R22 pad 2: Net-(U11-ISEN) -> Net-(U16-ISEN)
- R23 pad 1: Net-(C29-Pad1) -> Net-(C26-Pad1)
- R24 pad 1: Net-(C30-Pad1) -> Net-(J13-Pin_1)
- R24 pad 2: Net-(J14-Pin_1) -> +5V
- R25 pad 1: Net-(J13-Pin_1) -> Net-(C41-Pad1)
- R25 pad 2: +5V -> Net-(J14-Pin_1)
- R26 pad 1: Net-(J14-Pin_1) -> Net-(C42-Pad1)
- R26 pad 2: +5V -> Net-(J16-Pin_1)
- R27 pad 1: +5V -> Net-(C49-Pad1)
- R27 pad 2: Net-(U18-VREF) -> /*5
- R28 pad 1: Net-(U18-VREF) -> Net-(C50-Pad1)
- R28 pad 2: GND -> /*4
- R29 pad 1: Net-(C46-Pad1) -> +5V
- R29 pad 2: /Motor Control/H-bridge #1/ENCODER_A -> Net-(U30-VREF)
- R30 pad 1: Net-(C47-Pad1) -> Net-(U30-VREF)
- R30 pad 2: /Motor Control/H-bridge #1/ENCODER_B -> GND
- R31 pad 2: Net-(U18-ISEN) -> Net-(U30-ISEN)
- R32 pad 2: Net-(J16-Pin_1) -> Net-(J17-Pin_1)
- R33 pad 1: Net-(C53-Pad1) -> Net-(J14-Pin_1)
- R33 pad 2: Net-(J17-Pin_1) -> +5V
- U12 pad 1: /Motor Control/CURRENT2 -> /A1
- U12 pad 2: GND -> /Motor Control/CURRENT_M1A
- U12 pad 3: Net-(U11-ISEN) -> /Motor Control/CURRENT_M1B
- U12 pad 4: GND -> /Motor Control/CURRENT_M2A
- U12 pad 5: Net-(U12-V+) -> /Motor Control/CURRENT_M2B
- U15 pad 1: /Motor Control/EN_ENC_MOTOR3 -> Net-(U15-Pad1)
- U15 pad 2: Net-(U15-Pad2) -> /EN_M1B
- U15 pad 3: /Motor Control/H-bridge #1/ENCODER_A -> /Motor Control/H-bridge #2/IN2
- U15 pad 6: /Motor Control/H-bridge #1/ENCODER_B -> /EN_M1B
- U15 pad 7: /Motor Control/EN_ENC_MOTOR3 -> /Motor Control/H-bridge #2/IN1
- U16 pad 1: /Motor Control/EN_MOTOR3 -> GND
- U16 pad 2: /Motor Control/PWM1 -> /Motor Control/H-bridge #2/IN2
- U16 pad 3: Net-(U18-IN2) -> /Motor Control/H-bridge #2/IN1
- U16 pad 4: GND -> Net-(U16-VREF)
- U16 pad 5: /Motor Control/EN_MOTOR3 -> +12V
- U16 pad 6: /Motor Control/PWM2 -> /Motor Control/H-bridge #2/MOTOR+
- U16 pad 7: Net-(U18-IN1) -> Net-(U16-ISEN)
- U16 pad 8: +5V -> /Motor Control/H-bridge #2/MOTOR-
- U17 pad 1: Net-(C47-Pad1) -> /Motor Control/CURRENT_M1B
- U17 pad 2: Net-(U17-Pad2) -> GND
- U17 pad 3: Net-(U17-Pad2) -> Net-(U16-ISEN)
- U17 pad 4: Net-(U15-Pad2) -> GND
- U17 pad 5: Net-(C52-Pad1) -> Net-(U17-V+)
- U19 pad 1: /Motor Control/CURRENT3 -> /Motor Control/H-bridge #4/~{ENABLE_ENCODER}
- U19 pad 2: GND -> unconnected-(U19-Pad2)
- U19 pad 3: Net-(U18-ISEN) -> /*5
- U19 pad 5: Net-(U19-V+) -> unconnected-(U19-Pad5)
- U2 pad 13: /LED00 -> /EN_M1A
- U2 pad 14: /LED01 -> /EN_M1B
- U2 pad 15: /LED02 -> /EN_M2A
- U2 pad 16: /LED03 -> /EN_M2B
- U2 pad 17: unconnected-(U2-IO1_4-Pad17) -> /EN_M3A
- U2 pad 18: unconnected-(U2-IO1_5-Pad18) -> /EN_M3B
- U2 pad 19: unconnected-(U2-IO1_6-Pad19) -> /F/~{R}_MA
- U2 pad 20: unconnected-(U2-IO1_7-Pad20) -> /F/~{R}_MB
- U2 pad 22: /SCL/A5 -> /SCL/21
- U2 pad 23: /SDA/A4 -> /SDA/20
- U23 pad 11: /51 -> Net-(U12-SO)
- U23 pad 2: /Motor Control/CURRENT1 -> /Motor Control/CURRENT_M1A
- U23 pad 3: /Motor Control/CURRENT2 -> /Motor Control/CURRENT_M1B
- U23 pad 4: /Motor Control/CURRENT3 -> /Motor Control/CURRENT_M2A
- U23 pad 5: GND -> /Motor Control/CURRENT_M2B
- U23 pad 6: GND -> /Motor Control/CURRENT_M3A
- U23 pad 7: GND -> /Motor Control/CURRENT_M3B
- U3 pad 2: Net-(U3-Pad2) -> unconnected-(U3-Pad2)
- U3 pad 3: /Motor Control/H-bridge #1/ENCODER_A -> /*7
- U3 pad 5: Net-(U3-Pad5) -> unconnected-(U3-Pad5)
- U3 pad 6: /Motor Control/H-bridge #1/ENCODER_B -> /*6
- U5 pad 1: Net-(C11-Pad1) -> Net-(C52-Pad1)
- U5 pad 10: Net-(U5-Pad10) -> /LIM_SW02
- U5 pad 11: Net-(C10-Pad1) -> Net-(C26-Pad1)
- U5 pad 12: Net-(U3-Pad5) -> /LIM_SW03
- U5 pad 13: Net-(U5-Pad10) -> Net-(C41-Pad1)
- U5 pad 2: Net-(U5-Pad2) -> /LIM_SW05
- U5 pad 3: Net-(U5-Pad2) -> Net-(C42-Pad1)
- U5 pad 4: Net-(U3-Pad2) -> /LIM_SW04
- U6 pad 2: Net-(U6-IN2) -> /Motor Control/H-bridge #1/IN2
- U6 pad 3: Net-(U6-IN1) -> /Motor Control/H-bridge #1/IN1
- U7 pad 1: /Motor Control/CURRENT1 -> /Motor Control/CURRENT_M1A
- U9 pad 1: /Motor Control/EN_MOTOR2 -> /Motor Control/H-bridge #2/~{ENABLE_ENCODER}
- U9 pad 2: /Motor Control/PWM1 -> unconnected-(U9-Pad2)
- U9 pad 3: Net-(U11-IN2) -> /*5
- U9 pad 5: /Motor Control/EN_MOTOR2 -> unconnected-(U9-Pad5)
- U9 pad 6: /Motor Control/PWM2 -> /*4
- U9 pad 7: Net-(U11-IN1) -> /Motor Control/H-bridge #2/~{ENABLE_ENCODER}

Commit message: Progressed ECAD.
Parts:
- moved C2 17.9 mm to (236.9, 95.9)
- moved C33 17.9 mm to (274.9, 107.9)
- moved C35 17.9 mm to (274.9, 113.9)
- moved C38 17.9 mm to (291.9, 107.9)
- moved C40 17.9 mm to (291.9, 113.9)
- moved C45 17.9 mm to (247.5, 79.2)
- moved C47 17.9 mm to (247.5, 85.2)
- moved C50 17.9 mm to (247.5, 94.3)
- moved C51 17.9 mm to (251.9, 79.2)
- moved C61 17.9 mm to (251.9, 85.2)
- moved C71 17.9 mm to (215.4, 71.3)
- moved C74 17.9 mm to (215.4, 80.3)
- moved C78 17.9 mm to (219.9, 71.3)
- moved C79 17.9 mm to (216.0, 83.9)
- moved J15 17.9 mm to (257.1, 80.4)
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