File: ECAD/BDCMotorControlShieldMega/rs232_interface.kicad_sch (KiCad schematic)
At the start: 7 parts, among them U4 SP213

Commit message: Progressed ECAD.
Parts:
- removed L1: 10uL, Inductor_SMD:L_0805_2012Metric, symbol Device:L
- renumbered C11 to C28, C12 to C29, C13 to C30, C14 to C31, C15 to C32, U4 to U13
Connections:
- net +5VD is gone; now on net +5V: C32.1, U13.11 (VCC)
Other:
- moved on the sheet: C32

Commit message: Progressed ECAD.
Parts:
- renumbered C28 to C31, C29 to C32, C30 to C33, C31 to C34, C32 to C35

Commit message: Progressed ECAD.
Parts:
- U13: Status OK -> (none)
Changed lines of the file:
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@@
 			)
 		)
-		(property "Status" "OK"
+		(property "Status" ""
 			(at 175.26 100.33 0)
 			(effects

Commit message: Progressed ECAD.
Parts:
- U13: Status (none) -> OK
Changed lines of the file:
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@@
 			)
 		)
-		(property "Status" ""
+		(property "Status" "OK"
 			(at 175.26 100.33 0)
 			(effects

Commit message: Progressed ECAD.
Parts:
- C31, C32, C33, C34: MPN C0805F104K5RACAUTO -> (none)
- C35: footprint Capacitor_SMD:C_0805_2012Metric -> Capacitor_SMD:C_0603_1608Metric; MPN C0805F104K5RACAUTO -> (none)
Changed lines of the file:
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@@
 			)
 		)
-		(property "Datasheet" "https://www.lcsc.com/datasheet/lcsc_datasheet_2304140030_KEMET-C0805F104K5RACAUTO_C141162.pdf"
+		(property "Datasheet" ""
 			(at 104.14 88.9 0)
 			(effects
@@
 			)
 		)
-		(property "MPN" "C0805F104K5RACAUTO"
+		(property "MPN" ""
 			(at 104.14 88.9 0)
 			(effects
@@
 			)
 		)
-		(property "Footprint" "Capacitor_SMD:C_0805_2012Metric"
+		(property "Footprint" "Capacitor_SMD:C_0603_1608Metric"
 			(at 176.2252 60.96 0)
 			(effects
@@
 			)
 		)
-		(property "Datasheet" "https://www.lcsc.com/datasheet/lcsc_datasheet_2304140030_KEMET-C0805F104K5RACAUTO_C141162.pdf"
+		(property "Datasheet" ""
 			(at 175.26 57.15 0)
 			(effects
@@
 			)
 		)
-		(property "MPN" "C0805F104K5RACAUTO"
+		(property "MPN" ""
 			(at 175.26 57.15 0)
 			(effects
@@
 			)
 		)
-		(property "Datasheet" "https://www.lcsc.com/datasheet/lcsc_datasheet_2304140030_KEMET-C0805F104K5RACAUTO_C141162.pdf"
+		(property "Datasheet" ""
 			(at 87.63 88.9 0)
 			(effects
@@
 			)
 		)
-		(property "MPN" "C0805F104K5RACAUTO"
+		(property "MPN" ""
 			(at 87.63 88.9 0)
 			(effects
@@
 			)
 		)
-		(property "Datasheet" "https://www.lcsc.com/datasheet/lcsc_datasheet_2304140030_KEMET-C0805F104K5RACAUTO_C141162.pdf"
+		(property "Datasheet" ""
 			(at 104.14 111.76 0)
 			(effects
@@
 			)
 		)
-		(property "MPN" "C0805F104K5RACAUTO"
+		(property "MPN" ""
 			(at 104.14 111.76 0)
 			(effects
@@
 			)
 		)
-		(property "Datasheet" "https://www.lcsc.com/datasheet/lcsc_datasheet_2304140030_KEMET-C0805F104K5RACAUTO_C141162.pdf"
+		(property "Datasheet" ""
 			(at 87.63 111.76 0)
 			(effects
@@
 			)
 		)
-		(property "MPN" "C0805F104K5RACAUTO"
+		(property "MPN" ""
 			(at 87.63 111.76 0)
 			(effects

Commit message: Progressed ECAD.
Parts:
- removed U13: SP213, Package_SO:SSOP-28_5.3x10.2mm_P0.65mm, symbol Interface_UART_custom:MAX213
- added U24: SP3243E, Package_SO:TSSOP-28_4.4x9.7mm_P0.65mm, symbol Interface_UART_custom:SP3243E
- C31, C32, C33, C34: value 100nC -> 330nC
- C35: footprint Capacitor_SMD:C_0603_1608Metric -> Capacitor_SMD:C_0805_2012Metric
Connections:
- net +5V: now also U24.26 (VCC); no longer C34.1
- net C1+: now also U24.28 (C1+)
- net C1-: now also U24.24 (C1-)
- net C2+: now also U24.1 (C2+)
- net C2-: now also U24.2 (C2-)
- net CTS: now also U24.19 (R1OUT)
- net CTS_LINE: now also U24.4 (R1IN)
- net DCD: now also U24.17 (R3OUT)
- net DCD_LINE: now also U24.6 (R3IN)
- net DSR: now also U24.16 (R4OUT)
- net DSR_LINE: now also U24.7 (R4IN)
- net DTR: now also U24.14 (T1IN)
- net DTR_LINE: now also U24.9 (T1OUT)
- net GND: now also C34.2, U24.25 (GND)
- net RI: now also U24.18 (R2OUT)
- net RI_LINE: now also U24.5 (R2IN)
- net RTS: now also U24.12 (T3IN)
- net RTS_LINE: now also U24.11 (T3OUT)
- net RX: now also U24.15 (R5OUT)
- net RX_LINE: now also U24.8 (R5IN)
- net TX: now also U24.13 (T2IN)
- net TX_LINE: now also U24.10 (T2OUT)
- net V+: now also C34.1, U24.27 (V+); no longer C34.2
- net V-: now also U24.3 (V-)
- new net ~{SHUTDOWN}: U24.22 (~{SHUTDOWN}), U24.23 (~{ONLINE})
- new net ~{STATUS}: U24.21 (~{STATUS})
- no-connect marks 2 -> 1
Other:
- note removed: "6.3V"
- note removed: "Imax = 6mA"
- moved on the sheet: C31, C32, C33, C34, C35
