File: ECAD/BDCMotorController/BDCMotorController.kicad_sch (KiCad schematic)
At the start: 2 parts

Commit message: Progressed ECAD.
Other:
- sheet ADC conditioning ports: added none; removed ADC_VREF
Changed lines of the file:
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@@
 	(text "Used I2C Addresses\nMotor control I/O expander: 0b0100 000\nDigital Potentiometer: 0b0101 100\nDigital Potentiometer: 0b0101 110\nSerial ports I/O expander: 0b0100 111\nSerial ports I/O expander: 0b0100 110"
 		(exclude_from_sim no)
-		(at 146.812 119.126 0)
+		(at 197.612 150.622 0)
 		(effects
 			(font
@@
 	(text "(ADC0)    PF0\n(ADC1)    PF1"
 		(exclude_from_sim no)
-		(at 121.666 60.96 0)
+		(at 121.666 60.706 0)
 		(effects
 			(font
@@
 			(width 0)
 			(type solid)
-		)
-	)
-	(wire
-		(pts
-			(xy 137.16 66.04) (xy 147.32 66.04)
-		)
-		(stroke
-			(width 0)
-			(type default)
 		)
 	)
@@
 	(label "50"
 		(at 201.93 53.34 0)
-		(effects
-			(font
-				(size 1.27 1.27)
-			)
-			(justify left bottom)
-		)
-	)
-	(label "AREF"
-		(at 137.16 66.04 0)
 		(effects
 			(font
@@
 	(sheet
 		(at 147.32 57.15)
-		(size 26.67 11.43)
+		(size 26.67 7.62)
 		(exclude_from_sim no)
 		(in_bom yes)
@@
 		)
 		(property "Sheetfile" "adc_input.kicad_sch"
-			(at 147.32 69.1646 0)
+			(at 147.32 65.3546 0)
 			(effects
 				(font
@@
 		(pin "VA1_OUT" output
 			(at 147.32 62.23 180)
-			(effects
-				(font
-					(size 1.27 1.27)
-				)
-				(justify left)
-			)
-		)
-		(pin "ADC_VREF" output
-			(at 147.32 66.04 180)
 			(effects
 				(font
@@
 	)
 	(sheet
-		(at 34.29 83.82)
-		(size 27.94 7.62)
+		(at 90.17 22.86)
+		(size 27.94 111.76)
 		(exclude_from_sim no)
 		(in_bom yes)
@@
 		)
 		(property "Sheetname" "MCU"
-			(at 34.29 83.1084 0)
+			(at 90.17 22.1484 0)
 			(effects
 				(font
@@
 		)
 		(property "Sheetfile" "mcu.kicad_sch"
-			(at 34.29 92.0246 0)
+			(at 90.17 135.2046 0)
 			(effects
 				(font
@@
 	)
 	(sheet
-		(at 35.56 104.14)
+		(at 33.02 73.66)
 		(size 24.13 13.97)
 		(exclude_from_sim no)
@@
 		)
 		(property "Sheetname" "USB"
-			(at 35.56 103.4284 0)
+			(at 33.02 72.9484 0)
 			(effects
 				(font
@@
 		)
 		(property "Sheetfile" "usb.kicad_sch"
-			(at 35.56 118.6946 0)
-			(effects
-				(font
+			(at 33.02 88.2146 0)
+			(effects
+				(font

Commit message: Progressed ECAD.
Other:
- sheet MCU ports: added ADC0, ADC1, MISO, MOSI, OC1A, OC1C, RXD1, RXD2, RXD3, SCK, SCL, SDA, SS, TXD1, TXD2, TXD3; removed none
- sheet USB ports: added RX, TX, ~{MCU_RESET}, ~{USB_ON}; removed none

Commit message: Progressed ECAD.
Parts:
- removed C1: 10uC, Capacitor_SMD:C_1210_3225Metric, symbol Device:C
- removed C2: 100nC, Capacitor_SMD:C_0805_2012Metric, symbol Device:C
Other:
- sheet MCU ports: added ICP4, PCINT16, PCINT17, PCINT18, PK4, PK5, PK6, PK7, RXD0, TXD0, ~{RESET}, ~{SS}, ~{USB_ON}; removed SS
- note added: "Use OC1B for internal ADC trigger"
- note removed: "(ADC0) PF0 (ADC1) PF1"
- note removed: "(OC1A) PB5 (OC1C) PB7 ((OC1B) PB6 for internal ADC trigger) Any 4 digital input pins. Will be pooled in FW. (SCK) PB1 (MOSI) PB2 (MISO) PB3 (SS) PB0 (SCL) PD0 (SDA) PD1 (PCINT10) PJ1"
- note removed: "(RXD1) PD2 (TXD1) PD3 (RXD2) PH0 (TXD2) PH1 (SCL) PD0 (SDA) PD1 (PCINT9) PJ0"
- note removed: "Power supply decoupling"

Commit message: Progressed ECAD.
Changed lines of the file:
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@@
 	(sheet
 		(at 107.95 34.29)
-		(size 27.94 106.68)
+		(size 27.94 100.33)
 		(exclude_from_sim no)
 		(in_bom yes)
@@
 		)
 		(property "Sheetfile" "mcu.kicad_sch"
-			(at 107.95 141.5546 0)
+			(at 107.95 135.2046 0)
 			(effects
 				(font

Commit message: Progressed ECAD.
Other:
- added sheet LCD (lcd.kicad_sch)
- sheet MCU ports: added INT5, INT6, INT7, PF4, PF5, PF6, PF7, PK0, PK1, PK2, PK3, PL5, PL6, PL7; removed PCINT16, PCINT17, PCINT18

Commit message: Progressed ECAD.
Other:
- sheet ADC conditioning ports: added VA0_CLIPPING, VA1_CLIPPING; removed none
- sheet MCU ports: added INT4, PCINT12, PCINT13, PCINT14, PCINT15; removed ~{USB_ON}
- sheet Motor Control ports: added ENCODER_A_TOGGLE, ENCODER_B_TOGGLE; removed none

Commit message: Progressed ECAD.
Other:
- sheet Motor Control ports: added ENCODER_MA_TOGGLE, ENCODER_MB_TOGGLE; removed ENCODER_A_TOGGLE, ENCODER_B_TOGGLE
Changed lines of the file:
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@@
 			)
 		)
-		(pin "ENCODER_A_TOGGLE" output
+		(pin "ENCODER_MA_TOGGLE" output
 			(at 170.18 43.18 180)
 			(effects
@@
 			)
 		)
-		(pin "ENCODER_B_TOGGLE" output
+		(pin "ENCODER_MB_TOGGLE" output
 			(at 170.18 45.72 180)
 			(effects

Commit message: Progressed ECAD.
Connections:
- no-connect marks 0 -> 2
Other:
- sheet ADC conditioning ports: added none; removed VA0_CLIPPING, VA1_CLIPPING
