File: ECAD/BDCMotorController/h_bridge.kicad_sch (KiCad schematic)
At the start: 25 parts, among them J1 Motor Connector, U1 74AHC2G125, U2 74AHC00, U3 74AHC00, U4 74AHC1G17, U5 DRV8870DDA, U6 74AHC1G17, U7 INA180A1

Commit message: Progressed ECAD.
Parts:
- renumbered C3 to C1, C12 to C10, C13 to C11, C14 to C12, C15 to C13, C4 to C2, C5 to C3, C6 to C4, C7 to C5, C8 to C6, C9 to C7, C10 to C8, C11 to C9
Connections:
- net +12V renamed VDC

Commit message: Progressed ECAD.
Parts:
- removed J1: Motor Connector, Connector_JST:JST_PH_B6B-PH-K_1x06_P2.00mm_Vertical, symbol Connector_Generic:Conn_01x06
- added J1: Screw_Terminal_01x06, TerminalBlock_Phoenix:TerminalBlock_Phoenix_MPT-0,5-6-2.54_1x06_P2.54mm_Horizontal, symbol Connector:Screw_Terminal_01x06
Connections:
- net +5V: now also J1.3 (Pin_3)
- net ENCODER_A: now also J1.5 (Pin_5)
- net ENCODER_B: now also J1.6 (Pin_6)
- net GND: now also J1.4 (Pin_4)
- net MOTOR+: now also J1.1 (Pin_1)
- net MOTOR-: now also J1.2 (Pin_2)

Commit message: Progressed ECAD.
Parts:
- C1, C11, C13, C2, C4, C5, C6, C7, C8: Status OK -> (none)
- C10: footprint Capacitor_THT:CP_Radial_D5.0mm_P2.00mm -> Capacitor_SMD:C_1210_3225Metric; MPN 35YXJ47M5X11 -> GRM32ER61C476KE15L
- R1, R3: MPN AC0805FR-7W1KL -> (none)
Changed lines of the file:
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@@
 			)
 		)
-		(property "Status" "OK"
+		(property "Status" ""
 			(at 30.48 133.35 0)
 			(effects
@@
 			)
 		)
-		(property "Status" "OK"
+		(property "Status" ""
 			(at 130.81 62.23 0)
 			(effects
@@
 			)
 		)
-		(property "Datasheet" "https://datasheet.lcsc.com/lcsc/2010202005_YAGEO-AC0805FR-7W1KL_C727989.pdf"
+		(property "Datasheet" ""
 			(at 264.16 133.35 0)
 			(effects
@@
 			)
 		)
-		(property "MPN" "AC0805FR-7W1KL"
+		(property "MPN" ""
 			(at 264.16 133.35 90)
 			(effects
@@
 			)
 		)
-		(property "Status" "OK"
+		(property "Status" ""
 			(at 254 52.07 0)
 			(effects
@@
 			)
 		)
-		(property "Status" "OK"
+		(property "Status" ""
 			(at 264.16 52.07 0)
 			(effects
@@
 			)
 		)
-		(property "Status" "OK"
+		(property "Status" ""
 			(at 167.64 143.51 0)
 			(effects
@@
 			)
 		)
-		(property "Datasheet" "https://datasheet.lcsc.com/lcsc/1912111437_Taiyo-Yuden-UMK325AB7106KM-T_C386167.pdf"
+		(property "Datasheet" ""
 			(at 204.47 91.44 0)
 			(effects
@@
 			)
 		)
-		(property "Status" "OK"
+		(property "Status" ""
 			(at 185.42 68.58 0)
 			(effects
@@
 			)
 		)
-		(property "Status" "OK"
+		(property "Status" ""
 			(at 180.34 143.51 0)
 			(effects
@@
 			)
 		)
-		(property "Footprint" "Capacitor_THT:CP_Radial_D5.0mm_P2.00mm"
+		(property "Footprint" "Capacitor_SMD:C_1210_3225Metric"
 			(at 218.1352 95.25 0)
 			(effects
@@
 			)
 		)
-		(property "Datasheet" "https://datasheet.lcsc.com/lcsc/1809192224_Rubycon-35YXJ47M5X11_C88761.pdf"
+		(property "Datasheet" "https://www.lcsc.com/datasheet/lcsc_datasheet_2212021100_Murata-Electronics-GRM32ER61C476KE15L_C77101.pdf"
 			(at 217.17 91.44 0)
 			(effects
@@
 			)
 		)
-		(property "MPN" "35YXJ47M5X11"
+		(property "MPN" "GRM32ER61C476KE15L"
 			(at 217.17 91.44 0)
 			(effects
@@
 			)
 		)
-		(property "Status" "OK"
+		(property "Status" ""
 			(at 190.5 91.44 0)
 			(effects
@@
 			)
 		)
-		(property "Datasheet" "https://datasheet.lcsc.com/lcsc/2010202005_YAGEO-AC0805FR-7W1KL_C727989.pdf"
+		(property "Datasheet" ""
 			(at 142.24 133.35 0)
 			(effects
@@
 			)
 		)
-		(property "MPN" "AC0805FR-7W1KL"
+		(property "MPN" ""
 			(at 142.24 133.35 90)
 			(effects
@@
 			)
 		)
-		(property "Status" "OK"
+		(property "Status" ""
 			(at 156.21 62.23 0)
 			(effects

Commit message: Progressed ECAD.
Parts:
- R1, R3: Status OK -> (none)
Changed lines of the file:
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@@
 			)
 		)
-		(property "Status" "OK"
+		(property "Status" ""
 			(at 264.16 133.35 90)
 			(effects
@@
 			)
 		)
-		(property "Status" "OK"
+		(property "Status" ""
 			(at 142.24 133.35 90)
 			(effects

Commit message: Progressed ECAD.
Parts:
- removed C13: 100nC, Capacitor_SMD:C_0805_2012Metric, symbol Device:C

Commit message: Progressed ECAD.
Parts:
- removed L1: 10uL, Inductor_SMD:L_0805_2012Metric, symbol Device:L
Connections:
- net +5V: now also C11.1, U7.5 (V+)
