File: ECAD/BDCMotorController/power.kicad_sch (KiCad schematic)
At the start: 26 parts, among them J16 DC, U63 TPS561208DDCR, U64 TLV75801PDBVR, U65 LM2776

Commit message: Progressed ECAD.
Parts:
- removed D11: CMS30I30A, Diode_SMD:D_SOD-128, symbol Device:D_Schottky
- added C116: 10uC, Capacitor_SMD:C_1210_3225Metric, symbol Device:C
- added C118: 100nC, Capacitor_SMD:C_0805_2012Metric, symbol Device:C
- renumbered C117 to C115, C118 to C117, D12 to D11
Connections:
- net +5V: now also C116.1, C118.1
- net GND: now also C116.2, C118.2
- net VDC: now also J16.1
Other:
- note added: "Power supply decoupling"

Commit message: Progressed ECAD.
Other:
- note removed: "Power supply decoupling"
- moved on the sheet: C115, C116, C117, C118, C119

Commit message: Progressed ECAD.
Parts:
- renumbered C116 to C115, C118 to C116, C115 to C117, C117 to C118, C120 to C119, C119 to C120, R59 to R57, R60 to R58, R61 to R59, R62 to R60, R63 to R61

Commit message: Progressed ECAD.
Parts:
- renumbered C115 to C116, C116 to C117, C117 to C118, C118 to C119, C119 to C120, C120 to C121, C121 to C122, C122 to C123, C123 to C124, C124 to C125, C125 to C126, C126 to C127, C127 to C128, C128 to C129, C129 to C130, C130 to C131, U63 to U64, U64 to U65, U65 to U66

Commit message: Progressed ECAD.
Parts:
- renumbered J16 to J12

Commit message: Progressed ECAD.
Parts:
- renumbered C116 to C115, C117 to C116, C118 to C117, C119 to C118, C120 to C119, C121 to C120, C122 to C121, C123 to C122, C124 to C123, C125 to C124, C126 to C125, C127 to C126, C128 to C127, C129 to C128, C130 to C129, C131 to C130, D11 to D9, U64 to U63, U65 to U64, U66 to U65

Commit message: Progressed ECAD.
Parts:
- C116: Status OK -> (none)
- C117, C118, C119, C120, C125, C127: MPN C0805F104K5RACAUTO -> (none); Status OK -> (none)
- R57: MPN RC0805JR-0710KL -> (none); Status OK -> (none)
- R59, R61: MPN RT0805BRD0710KL -> (none); Status OK -> (none)
Changed lines of the file:
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@@
 	(wire
 		(pts
-			(xy 156.21 100.33) (xy 158.75 100.33)
+			(xy 154.94 100.33) (xy 158.75 100.33)
 		)
 		(stroke
@@
 	(wire
 		(pts
-			(xy 156.21 93.98) (xy 156.21 100.33)
+			(xy 154.94 93.98) (xy 154.94 100.33)
 		)
 		(stroke
@@
 	(wire
 		(pts
-			(xy 153.67 93.98) (xy 156.21 93.98)
+			(xy 153.67 93.98) (xy 154.94 93.98)
 		)
 		(stroke
@@
 			)
 		)
-		(property "Datasheet" "https://www.lcsc.com/datasheet/lcsc_datasheet_2304140030_KEMET-C0805F104K5RACAUTO_C141162.pdf"
+		(property "Datasheet" ""
 			(at 158.75 40.64 0)
 			(effects
@@
 			)
 		)
-		(property "Status" "OK"
+		(property "Status" ""
 			(at 158.75 40.64 0)
 			(effects
@@
 			)
 		)
-		(property "MPN" "C0805F104K5RACAUTO"
+		(property "MPN" ""
 			(at 158.75 40.64 0)
 			(effects
@@
 			)
 		)
-		(property "Datasheet" "https://www.lcsc.com/datasheet/lcsc_datasheet_2304140030_KEMET-C0805F104K5RACAUTO_C141162.pdf"
+		(property "Datasheet" ""
 			(at 83.82 45.72 0)
 			(effects
@@
 			)
 		)
-		(property "Status" "OK"
+		(property "Status" ""
 			(at 83.82 45.72 0)
 			(effects
@@
 			)
 		)
-		(property "MPN" "C0805F104K5RACAUTO"
+		(property "MPN" ""
 			(at 83.82 45.72 0)
 			(effects
@@
 			)
 		)
-		(property "Datasheet" "https://www.lcsc.com/datasheet/lcsc_datasheet_1810171610_YAGEO-RC0805JR-0710KL_C100047.pdf"
+		(property "Datasheet" ""
 			(at 128.27 45.72 0)
 			(effects
@@
 			)
 		)
-		(property "Status" "OK"
+		(property "Status" ""
 			(at 128.27 45.72 0)
 			(effects
@@
 			)
 		)
-		(property "MPN" "RC0805JR-0710KL"
+		(property "MPN" ""
 			(at 128.27 45.72 0)
 			(effects
@@
 			)
 		)
-		(property "Status" "OK"
+		(property "Status" ""
 			(at 44.45 176.53 0)
 			(effects
@@
 			)
 		)
-		(property "Datasheet" "https://datasheet.lcsc.com/lcsc/1912111437_Taiyo-Yuden-UMK325AB7106KM-T_C386167.pdf"
+		(property "Datasheet" ""
 			(at 30.48 176.53 0)
 			(effects
@@
 			)
 		)
-		(property "Datasheet" "https://www.lcsc.com/datasheet/lcsc_datasheet_2304140030_KEMET-C0805F104K5RACAUTO_C141162.pdf"
+		(property "Datasheet" ""
 			(at 90.17 176.53 0)
 			(effects
@@
 			)
 		)
-		(property "Status" "OK"
+		(property "Status" ""
 			(at 90.17 176.53 0)
 			(effects
@@
 			)
 		)
-		(property "MPN" "C0805F104K5RACAUTO"
+		(property "MPN" ""
 			(at 90.17 176.53 0)
 			(effects
@@
 			)
 		)
-		(property "Datasheet" "https://www.lcsc.com/datasheet/lcsc_datasheet_2304140030_KEMET-C0805F104K5RACAUTO_C141162.pdf"
+		(property "Datasheet" ""
 			(at 74.93 176.53 0)
 			(effects
@@
 			)
 		)
-		(property "Status" "OK"
+		(property "Status" ""
 			(at 74.93 176.53 0)
 			(effects
@@
 			)
 		)
-		(property "MPN" "C0805F104K5RACAUTO"
+		(property "MPN" ""
 			(at 74.93 176.53 0)
 			(effects
@@
 			)
 		)
-		(property "Datasheet" "https://www.lcsc.com/datasheet/lcsc_datasheet_2304140030_KEMET-C0805F104K5RACAUTO_C141162.pdf"
+		(property "Datasheet" ""
 			(at 173.99 96.52 0)
 			(effects
@@
 			)
 		)
-		(property "Status" "OK"
+		(property "Status" ""
 			(at 173.99 96.52 0)
 			(effects
@@
 			)
 		)
-		(property "MPN" "C0805F104K5RACAUTO"
+		(property "MPN" ""
 			(at 173.99 96.52 0)
 			(effects
@@
 			)
 		)
-		(property "Datasheet" "https://www.lcsc.com/datasheet/lcsc_datasheet_2304140030_YAGEO-RT0805BRD0710KL_C110775.pdf"
+		(property "Datasheet" ""
 			(at 158.75 105.41 0)
 			(effects
@@
 			)
 		)
-		(property "Status" "OK"
+		(property "Status" ""
 			(at 158.75 105.41 0)
 			(effects
@@
 			)
 		)
-		(property "MPN" "RT0805BRD0710KL"
+		(property "MPN" ""
 			(at 158.75 105.41 0)
 			(effects
@@
 			)
 		)
-		(property "Datasheet" "https://www.lcsc.com/datasheet/lcsc_datasheet_2304140030_KEMET-C0805F104K5RACAUTO_C141162.pdf"
+		(property "Datasheet" ""
 			(at 59.69 176.53 0)
 			(effects
@@
 			)
 		)
-		(property "Status" "OK"
+		(property "Status" ""
 			(at 59.69 176.53 0)
 			(effects
@@
 			)
 		)
-		(property "MPN" "C0805F104K5RACAUTO"
+		(property "MPN" ""
 			(at 59.69 176.53 0)
 			(effects
@@
 			)
 		)
-		(property "Datasheet" "https://www.lcsc.com/datasheet/lcsc_datasheet_2304140030_YAGEO-RT0805BRD0710KL_C110775.pdf"
+		(property "Datasheet" ""
 			(at 190.5 58.42 0)
 			(effects
@@
 			)
 		)
-		(property "Status" "OK"
+		(property "Status" ""
 			(at 190.5 58.42 0)
 			(effects
@@
 			)
 		)
-		(property "MPN" "RT0805BRD0710KL"
+		(property "MPN" ""
 			(at 190.5 58.42 0)
 			(effects

Commit message: Progressed ECAD.
Parts:
- renumbered C115 to C110, C116 to C111, C117 to C112, C118 to C113, C119 to C114, C120 to C115, C121 to C116, C122 to C117, C123 to C118, C124 to C119, C125 to C120, C126 to C121, C127 to C122, C128 to C123, C129 to C124, C130 to C125, D9 to D11, L9 to L1, R57 to R59, R58 to R60, R59 to R61, R60 to R62, R61 to R63
