File: ECAD/BDCMotorController/lcd.kicad_sch (KiCad schematic)
At the start: 1 part

Commit message: Progressed ECAD.
Parts:
- removed DS1: WC1602A, Display:WC1602A, symbol Display_Character:WC1602A
- added H1, H2, H3, H4: MountingHole, MountingHole:MountingHole_3.2mm_M3, symbol Mechanical:MountingHole
- added J18: Conn_01x16, Connector_PinHeader_2.54mm:PinHeader_1x16_P2.54mm_Vertical, symbol Connector_Generic:Conn_01x16
- added U34: MCP4431, Package_SO:TSSOP-20_4.4x6.5mm_P0.65mm, symbol Potentiometer_Digital:MCP4431-xxxx-ST
Connections:
- net +5V: now also J18.2 (Pin_2), U34.1 (P3A)
- net DB0: now also J18.7 (Pin_7)
- net DB1: now also J18.8 (Pin_8)
- net DB2: now also J18.9 (Pin_9)
- net DB3: now also J18.10 (Pin_10)
- net DB4: now also J18.11 (Pin_11)
- net DB5: now also J18.12 (Pin_12)
- net DB6: now also J18.13 (Pin_13)
- net DB7: now also J18.14 (Pin_14)
- net E: now also J18.6 (Pin_6)
- net GND: now also J18.1 (Pin_1), U34.18 (P2B), U34.3 (P3B)
- net RS: now also J18.4 (Pin_4)
- net R~{W}: now also J18.5 (Pin_5)
- new net LED_A: J18.15 (Pin_15)
- new net LED_K: J18.16 (Pin_16)
- new net Vo: J18.3 (Pin_3), U34.2 (P3W)
- no-connect marks 0 -> 2

Commit message: Progressed ECAD.
Parts:
- removed U34: MCP4431, Package_SO:TSSOP-20_4.4x6.5mm_P0.65mm, symbol Potentiometer_Digital:MCP4431-xxxx-ST
- added C150: 100nC, Capacitor_SMD:C_0805_2012Metric, symbol Device:C
- added RV1, RV2: R_Potentiometer, symbol Device:R_Potentiometer
- added U75: LM317_TO-252, Package_TO_SOT_SMD:TO-252-2, symbol Regulator_Linear:LM317_TO-252
- renumbered J18 to J14
Connections:
- net LED_K is gone; now on net GND: J14.16 (Pin_16)
- net +5V: now also RV2.3
- net GND: now also C150.2, RV2.1
- net Vo: now also RV2.2
- net LED_A renamed BL_LED
- net BL_LED: now also RV1.3, U75.1 (ADJ)
- new net: RV1.1, RV1.2, U75.2 (VO)
- new net VDC: C150.1, U75.3 (VI)
- no-connect marks 2 -> 0
Other:
- note added: "I_{LIM} = 1.2/R I_{LIM} = 125 mA"
- moved on the sheet: H1, H2, H3, H4, J14

Commit message: Progressed ECAD.
Parts:
- added R78: 10R, symbol Device:R
- RV1: value R_Potentiometer -> 200R; footprint (none) -> Potentiometer_THT:Potentiometer_Bourns_3296X_Horizontal; MPN (none) -> 3296X-1-201LF
- RV2: value R_Potentiometer -> 10kR; footprint (none) -> Potentiometer_THT:Potentiometer_Bourns_3296X_Horizontal; MPN (none) -> 3296X-1-103LF
Connections:
- net BL_LED: now also RV1.2
- new net: R78.1, U75.2 (VO)
- new net: R78.2, RV1.1
Other:
- note added: "I_{LIM} = 1.25/R I_{LCD LIM} = 125 mA I_{MAX} = 125 mA I_{MIN} = 6 mA"
- note removed: "I_{LIM} = 1.2/R I_{LIM} = 125 mA"
- moved on the sheet: C150, RV1, U75

Commit message: Progressed ECAD.
Parts:
- R70: renamed from R78; footprint (none) -> Resistor_SMD:R_0805_2012Metric
- renumbered C150 to C149, U75 to U74
Other:
- note added: "I_{LCD MAX} = 125 mA I_{LIM} = 1.25/R I_{MAX} = 125 mA I_{MIN} = 6 mA"
- note removed: "I_{LIM} = 1.25/R I_{LCD LIM} = 125 mA I_{MAX} = 125 mA I_{MIN} = 6 mA"
Changed lines of the file:
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@@
 	(generator_version "9.0")
 	(paper "A4")
-	(text "I_{LIM} = 1.25/R\nI_{LCD LIM} = 125 mA\nI_{MAX} = 125 mA\nI_{MIN} = 6 mA"
+	(text "I_{LCD MAX} = 125 mA\nI_{LIM} = 1.25/R\nI_{MAX} = 125 mA\nI_{MIN} = 6 mA"
 		(exclude_from_sim no)
 		(at 103.632 89.662 0)
@@
 		(dnp no)
 		(fields_autoplaced yes)
-		(property "Reference" "#PWR0457"
+		(property "Reference" "#PWR0451"
 			(at 135.89 82.55 0)
 			(effects
@@
 			(project "BDCMotorController"
 				(path "/e63e39d7-6ac0-4ffd-8aa3-1841a4541b55/cd796a32-6854-439f-8a8a-358ee712a355"
-					(reference "#PWR0457")
+					(reference "#PWR0451")
 					(unit 1)
 				)
@@
 		(dnp no)
 		(fields_autoplaced yes)
-		(property "Reference" "#PWR0456"
+		(property "Reference" "#PWR0450"
 			(at 135.89 72.39 0)
 			(effects
@@
 			(project "BDCMotorController"
 				(path "/e63e39d7-6ac0-4ffd-8aa3-1841a4541b55/cd796a32-6854-439f-8a8a-358ee712a355"
-					(reference "#PWR0456")
+					(reference "#PWR0450")
 					(unit 1)
 				)
@@
 		(dnp no)
 		(fields_autoplaced yes)
-		(property "Reference" "U75"
+		(property "Reference" "U74"
 			(at 102.87 96.52 0)
 			(effects
@@
 			(project ""
 				(path "/e63e39d7-6ac0-4ffd-8aa3-1841a4541b55/cd796a32-6854-439f-8a8a-358ee712a355"
-					(reference "U75")
+					(reference "U74")
 					(unit 1)
 				)
@@
 		(dnp no)
 		(fields_autoplaced yes)
-		(property "Reference" "#PWR0454"
+		(property "Reference" "#PWR0448"
 			(at 78.74 105.41 0)
 			(effects
@@
 			(project "BDCMotorController"
 				(path "/e63e39d7-6ac0-4ffd-8aa3-1841a4541b55/cd796a32-6854-439f-8a8a-358ee712a355"
-					(reference "#PWR0454")
+					(reference "#PWR0448")
 					(unit 1)
 				)
@@
 		(dnp no)
 		(fields_autoplaced yes)
-		(property "Reference" "#PWR0458"
+		(property "Reference" "#PWR0452"
 			(at 151.13 113.03 0)
 			(effects
@@
 			(project "BDCMotorController"
 				(path "/e63e39d7-6ac0-4ffd-8aa3-1841a4541b55/cd796a32-6854-439f-8a8a-358ee712a355"
-					(reference "#PWR0458")
+					(reference "#PWR0452")
 					(unit 1)
 				)
@@
 		(dnp no)
 		(fields_autoplaced yes)
-		(property "Reference" "R78"
+		(property "Reference" "R70"
 			(at 114.3 96.52 90)
 			(effects
@@
 			)
 		)
-		(property "Footprint" ""
+		(property "Footprint" "Resistor_SMD:R_0805_2012Metric"
 			(at 114.3 104.648 90)
 			(effects
@@
 			(project ""
 				(path "/e63e39d7-6ac0-4ffd-8aa3-1841a4541b55/cd796a32-6854-439f-8a8a-358ee712a355"
-					(reference "R78")
+					(reference "R70")
 					(unit 1)
 				)
@@
 		(dnp no)
 		(fields_autoplaced yes)
-		(property "Reference" "#PWR0455"
+		(property "Reference" "#PWR0449"
 			(at 85.09 118.11 0)
 			(effects
@@
 			(project "BDCMotorController"
 				(path "/e63e39d7-6ac0-4ffd-8aa3-1841a4541b55/cd796a32-6854-439f-8a8a-358ee712a355"
-					(reference "#PWR0455")
+					(reference "#PWR0449")
 					(unit 1)
 				)
@@
 		(dnp no)
 		(fields_autoplaced yes)
-		(property "Reference" "#PWR0459"
+		(property "Reference" "#PWR0453"
 			(at 146.05 67.31 0)
 			(effects
@@
 			(project "BDCMotorController"
 				(path "/e63e39d7-6ac0-4ffd-8aa3-1841a4541b55/cd796a32-6854-439f-8a8a-358ee712a355"
-					(reference "#PWR0459")
+					(reference "#PWR0453")
 					(unit 1)
 				)
@@
 		(on_board yes)
 		(dnp no)
-		(property "Reference" "C150"
+		(property "Reference" "C149"
 			(at 92.964 106.68 0)
 			(effects
@@
 			(project "BDCMotorController"
 				(path "/e63e39d7-6ac0-4ffd-8aa3-1841a4541b55/cd796a32-6854-439f-8a8a-358ee712a355"
-					(reference "C150")
+					(reference "C149")
 					(unit 1)
 				)
@@
 		(on_board yes)
 		(dnp no)
-		(property "Reference" "#PWR0460"
+		(property "Reference" "#PWR0454"
 			(at 156.21 69.85 0)
 			(effects
@@
 			(project "BDCMotorController"
 				(path "/e63e39d7-6ac0-4ffd-8aa3-1841a4541b55/cd796a32-6854-439f-8a8a-358ee712a355"
-					(reference "#PWR0460")
+					(reference "#PWR0454")
 					(unit 1)
 				)

Commit message: Progressed ECAD.
Parts:
- C149: Status OK -> (none)
Changed lines of the file:
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@@
 			)
 		)
-		(property "Status" "OK"
+		(property "Status" ""
 			(at 85.09 107.95 0)
 			(effects

Commit message: Progressed ECAD.
Parts:
- renumbered C149 to C142, R70 to R72
Changed lines of the file:
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@@
 		(dnp no)
 		(fields_autoplaced yes)
-		(property "Reference" "#PWR0451"
+		(property "Reference" "#PWR0457"
 			(at 135.89 82.55 0)
 			(effects
@@
 			(project "BDCMotorController"
 				(path "/e63e39d7-6ac0-4ffd-8aa3-1841a4541b55/cd796a32-6854-439f-8a8a-358ee712a355"
-					(reference "#PWR0451")
+					(reference "#PWR0457")
 					(unit 1)
 				)
@@
 		(dnp no)
 		(fields_autoplaced yes)
-		(property "Reference" "#PWR0450"
+		(property "Reference" "#PWR0456"
 			(at 135.89 72.39 0)
 			(effects
@@
 			(project "BDCMotorController"
 				(path "/e63e39d7-6ac0-4ffd-8aa3-1841a4541b55/cd796a32-6854-439f-8a8a-358ee712a355"
-					(reference "#PWR0450")
+					(reference "#PWR0456")
 					(unit 1)
 				)
@@
 		(dnp no)
 		(fields_autoplaced yes)
-		(property "Reference" "#PWR0448"
+		(property "Reference" "#PWR0454"
 			(at 78.74 105.41 0)
 			(effects
@@
 			(project "BDCMotorController"
 				(path "/e63e39d7-6ac0-4ffd-8aa3-1841a4541b55/cd796a32-6854-439f-8a8a-358ee712a355"
-					(reference "#PWR0448")
+					(reference "#PWR0454")
 					(unit 1)
 				)
@@
 		(dnp no)
 		(fields_autoplaced yes)
-		(property "Reference" "#PWR0452"
+		(property "Reference" "#PWR0458"
 			(at 151.13 113.03 0)
 			(effects
@@
 			(project "BDCMotorController"
 				(path "/e63e39d7-6ac0-4ffd-8aa3-1841a4541b55/cd796a32-6854-439f-8a8a-358ee712a355"
-					(reference "#PWR0452")
+					(reference "#PWR0458")
 					(unit 1)
 				)
@@
 		(dnp no)
 		(fields_autoplaced yes)
-		(property "Reference" "R70"
+		(property "Reference" "R72"
 			(at 114.3 96.52 90)
 			(effects
@@
 			(project ""
 				(path "/e63e39d7-6ac0-4ffd-8aa3-1841a4541b55/cd796a32-6854-439f-8a8a-358ee712a355"
-					(reference "R70")
+					(reference "R72")
 					(unit 1)
 				)
@@
 		(dnp no)
 		(fields_autoplaced yes)
-		(property "Reference" "#PWR0449"
+		(property "Reference" "#PWR0455"
 			(at 85.09 118.11 0)
 			(effects
@@
 			(project "BDCMotorController"
 				(path "/e63e39d7-6ac0-4ffd-8aa3-1841a4541b55/cd796a32-6854-439f-8a8a-358ee712a355"
-					(reference "#PWR0449")
+					(reference "#PWR0455")
 					(unit 1)
 				)
@@
 		(dnp no)
 		(fields_autoplaced yes)
-		(property "Reference" "#PWR0453"
+		(property "Reference" "#PWR0459"
 			(at 146.05 67.31 0)
 			(effects
@@
 			(project "BDCMotorController"
 				(path "/e63e39d7-6ac0-4ffd-8aa3-1841a4541b55/cd796a32-6854-439f-8a8a-358ee712a355"
-					(reference "#PWR0453")
+					(reference "#PWR0459")
 					(unit 1)
 				)
@@
 		(on_board yes)
 		(dnp no)
-		(property "Reference" "C149"
+		(property "Reference" "C142"
 			(at 92.964 106.68 0)
 			(effects
@@
 			(project "BDCMotorController"
 				(path "/e63e39d7-6ac0-4ffd-8aa3-1841a4541b55/cd796a32-6854-439f-8a8a-358ee712a355"
-					(reference "C149")
+					(reference "C142")
 					(unit 1)
 				)
@@
 		(on_board yes)
 		(dnp no)
-		(property "Reference" "#PWR0454"
+		(property "Reference" "#PWR0460"
 			(at 156.21 69.85 0)
 			(effects
@@
 			(project "BDCMotorController"
 				(path "/e63e39d7-6ac0-4ffd-8aa3-1841a4541b55/cd796a32-6854-439f-8a8a-358ee712a355"
-					(reference "#PWR0454")
-					(unit 1)
-				)
+					(reference "#PWR0460")
+					(unit 1)
+				)

Commit message: Progressed ECAD.
Parts:
- renumbered R72 to R65
Changed lines of the file:
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@@
 		(dnp no)
 		(fields_autoplaced yes)
-		(property "Reference" "#PWR0457"
+		(property "Reference" "#PWR0450"
 			(at 135.89 82.55 0)
 			(effects
@@
 			(project "BDCMotorController"
 				(path "/e63e39d7-6ac0-4ffd-8aa3-1841a4541b55/cd796a32-6854-439f-8a8a-358ee712a355"
-					(reference "#PWR0457")
+					(reference "#PWR0450")
 					(unit 1)
 				)
@@
 		(dnp no)
 		(fields_autoplaced yes)
-		(property "Reference" "#PWR0456"
+		(property "Reference" "#PWR0449"
 			(at 135.89 72.39 0)
 			(effects
@@
 			(project "BDCMotorController"
 				(path "/e63e39d7-6ac0-4ffd-8aa3-1841a4541b55/cd796a32-6854-439f-8a8a-358ee712a355"
-					(reference "#PWR0456")
+					(reference "#PWR0449")
 					(unit 1)
 				)
@@
 		(dnp no)
 		(fields_autoplaced yes)
-		(property "Reference" "#PWR0454"
+		(property "Reference" "#PWR0447"
 			(at 78.74 105.41 0)
 			(effects
@@
 			(project "BDCMotorController"
 				(path "/e63e39d7-6ac0-4ffd-8aa3-1841a4541b55/cd796a32-6854-439f-8a8a-358ee712a355"
-					(reference "#PWR0454")
+					(reference "#PWR0447")
 					(unit 1)
 				)
@@
 		(dnp no)
 		(fields_autoplaced yes)
-		(property "Reference" "#PWR0458"
+		(property "Reference" "#PWR0451"
 			(at 151.13 113.03 0)
 			(effects
@@
 			(project "BDCMotorController"
 				(path "/e63e39d7-6ac0-4ffd-8aa3-1841a4541b55/cd796a32-6854-439f-8a8a-358ee712a355"
-					(reference "#PWR0458")
+					(reference "#PWR0451")
 					(unit 1)
 				)
@@
 		(dnp no)
 		(fields_autoplaced yes)
-		(property "Reference" "R72"
+		(property "Reference" "R65"
 			(at 114.3 96.52 90)
 			(effects
@@
 			(project ""
 				(path "/e63e39d7-6ac0-4ffd-8aa3-1841a4541b55/cd796a32-6854-439f-8a8a-358ee712a355"
-					(reference "R72")
+					(reference "R65")
 					(unit 1)
 				)
@@
 		(dnp no)
 		(fields_autoplaced yes)
-		(property "Reference" "#PWR0455"
+		(property "Reference" "#PWR0448"
 			(at 85.09 118.11 0)
 			(effects
@@
 			(project "BDCMotorController"
 				(path "/e63e39d7-6ac0-4ffd-8aa3-1841a4541b55/cd796a32-6854-439f-8a8a-358ee712a355"
-					(reference "#PWR0455")
+					(reference "#PWR0448")
 					(unit 1)
 				)
@@
 		(dnp no)
 		(fields_autoplaced yes)
-		(property "Reference" "#PWR0459"
+		(property "Reference" "#PWR0452"
 			(at 146.05 67.31 0)
 			(effects
@@
 			(project "BDCMotorController"
 				(path "/e63e39d7-6ac0-4ffd-8aa3-1841a4541b55/cd796a32-6854-439f-8a8a-358ee712a355"
-					(reference "#PWR0459")
+					(reference "#PWR0452")
 					(unit 1)
 				)
@@
 		(on_board yes)
 		(dnp no)
-		(property "Reference" "#PWR0460"
+		(property "Reference" "#PWR0453"
 			(at 156.21 69.85 0)
 			(effects
@@
 			(project "BDCMotorController"
 				(path "/e63e39d7-6ac0-4ffd-8aa3-1841a4541b55/cd796a32-6854-439f-8a8a-358ee712a355"
-					(reference "#PWR0460")
-					(unit 1)
-				)
+					(reference "#PWR0453")
+					(unit 1)
+				)
