File: ECAD/BDCMotorController/lim_sw.kicad_sch (KiCad schematic)
At the start: 36 parts, among them J10 Limit switch, J11 Limit switch, J12 Limit switch, J13 Limit switch, J14 Limit switch, J15 Limit switch, U52 74AHC1G17, U53 74AHC1G17, U54 74AHC1G17, U55 74AHC1G17, U56 74AHC1G17, U57 74AHC1G17

Commit message: Progressed ECAD.
Parts:
- renumbered C102 to C100, C103 to C101, C104 to C102, C105 to C103, C106 to C104, C107 to C105, C108 to C106, C109 to C107, C110 to C108, C111 to C109, C100 to C98, C101 to C99

Commit message: Progressed ECAD.
Parts:
- renumbered R30 to R28, R31 to R29, R32 to R30, R33 to R31, R34 to R32, R35 to R33, R36 to R34, R37 to R35, R38 to R36, R39 to R37, R40 to R38, R41 to R39

Commit message: Progressed ECAD.
Parts:
- removed J10, J11, J12, J13, J14, J15: Limit switch, Connector_JST:JST_PH_B2B-PH-K_1x02_P2.00mm_Vertical, symbol Connector_Generic:Conn_01x02
- added J10, J11: Screw_Terminal_01x06, TerminalBlock_Phoenix:TerminalBlock_Phoenix_MPT-0,5-6-2.54_1x06_P2.54mm_Horizontal, symbol Connector:Screw_Terminal_01x06
Connections:
- net GND: now also J10.2 (Pin_2), J10.4 (Pin_4), J10.6 (Pin_6), J11.2 (Pin_2), J11.4 (Pin_4), J11.6 (Pin_6)
- net LIM5: now reaches R35.2, R38.1
- net LIM5: now also J11.3 (Pin_3)
- net LIM6: now reaches R36.2, R39.1
- net LIM6: now also J11.5 (Pin_5)
- net LIM3: now reaches R30.2, R33.1
- net LIM3: now also J10.5 (Pin_5)
- net LIM4: now reaches R34.2, R37.1
- net LIM4: now also J11.1 (Pin_1)
- net LIM2: now reaches R29.2, R32.1
- net LIM2: now also J10.3 (Pin_3)
- net LIM1: now reaches R28.2, R31.1
- net LIM1: now also J10.1 (Pin_1)

Commit message: Progressed ECAD.
Parts:
- C100, C101, C102, C103, C104, C105, C106, C107, C108, C109, C98, C99: Status OK -> (none)
- R28, R29, R30, R31, R32, R33, R34, R35, R36, R37, R38, R39: MPN RC0805JR-0710KL -> (none); Status OK -> (none)
Changed lines of the file:
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@@
 			)
 		)
-		(property "Status" "OK"
+		(property "Status" ""
 			(at 46.99 59.69 0)
 			(effects
@@
 			)
 		)
-		(property "Status" "OK"
+		(property "Status" ""
 			(at 166.37 123.19 0)
 			(effects
@@
 			)
 		)
-		(property "Status" "OK"
+		(property "Status" ""
 			(at 166.37 59.69 0)
 			(effects
@@
 			)
 		)
-		(property "Datasheet" "https://www.lcsc.com/datasheet/lcsc_datasheet_1810171610_YAGEO-RC0805JR-0710KL_C100047.pdf"
+		(property "Datasheet" ""
 			(at 220.98 59.69 0)
 			(effects
@@
 			)
 		)
-		(property "MPN" "RC0805JR-0710KL"
+		(property "MPN" ""
 			(at 220.98 59.69 90)
 			(effects
@@
 			)
 		)
-		(property "Status" "OK"
+		(property "Status" ""
 			(at 220.98 59.69 90)
 			(effects
@@
 			)
 		)
-		(property "Status" "OK"
+		(property "Status" ""
 			(at 166.37 90.17 0)
 			(effects
@@
 			)
 		)
-		(property "Status" "OK"
+		(property "Status" ""
 			(at 46.99 123.19 0)
 			(effects
@@
 			)
 		)
-		(property "Datasheet" "https://www.lcsc.com/datasheet/lcsc_datasheet_1810171610_YAGEO-RC0805JR-0710KL_C100047.pdf"
+		(property "Datasheet" ""
 			(at 101.6 91.44 0)
 			(effects
@@
 			)
 		)
-		(property "MPN" "RC0805JR-0710KL"
+		(property "MPN" ""
 			(at 101.6 91.44 90)
 			(effects
@@
 			)
 		)
-		(property "Status" "OK"
+		(property "Status" ""
 			(at 101.6 91.44 90)
 			(effects
@@
 			)
 		)
-		(property "Status" "OK"
+		(property "Status" ""
 			(at 90.17 128.27 0)
 			(effects
@@
 			)
 		)
-		(property "Datasheet" "https://www.lcsc.com/datasheet/lcsc_datasheet_1810171610_YAGEO-RC0805JR-0710KL_C100047.pdf"
+		(property "Datasheet" ""
 			(at 110.49 118.11 0)
 			(effects
@@
 			)
 		)
-		(property "MPN" "RC0805JR-0710KL"
+		(property "MPN" ""
 			(at 110.49 118.11 0)
 			(effects
@@
 			)
 		)
-		(property "Status" "OK"
+		(property "Status" ""
 			(at 110.49 118.11 0)
 			(effects
@@
 			)
 		)
-		(property "Datasheet" "https://www.lcsc.com/datasheet/lcsc_datasheet_1810171610_YAGEO-RC0805JR-0710KL_C100047.pdf"
+		(property "Datasheet" ""
 			(at 110.49 86.36 0)
 			(effects
@@
 			)
 		)
-		(property "MPN" "RC0805JR-0710KL"
+		(property "MPN" ""
 			(at 110.49 86.36 0)
 			(effects
@@
 			)
 		)
-		(property "Status" "OK"
+		(property "Status" ""
 			(at 110.49 86.36 0)
 			(effects
@@
 			)
 		)
-		(property "Datasheet" "https://www.lcsc.com/datasheet/lcsc_datasheet_1810171610_YAGEO-RC0805JR-0710KL_C100047.pdf"
+		(property "Datasheet" ""
 			(at 101.6 59.69 0)
 			(effects
@@
 			)
 		)
-		(property "MPN" "RC0805JR-0710KL"
+		(property "MPN" ""
 			(at 101.6 59.69 90)
 			(effects
@@
 			)
 		)
-		(property "Status" "OK"
+		(property "Status" ""
 			(at 101.6 59.69 90)
 			(effects
@@
 			)
 		)
-		(property "Datasheet" "https://www.lcsc.com/datasheet/lcsc_datasheet_1810171610_YAGEO-RC0805JR-0710KL_C100047.pdf"
+		(property "Datasheet" ""
 			(at 229.87 86.36 0)
 			(effects
@@
 			)
 		)
-		(property "MPN" "RC0805JR-0710KL"
+		(property "MPN" ""
 			(at 229.87 86.36 0)
 			(effects
@@
 			)
 		)
-		(property "Status" "OK"
+		(property "Status" ""
 			(at 229.87 86.36 0)
 			(effects
@@
 			)
 		)
-		(property "Status" "OK"
+		(property "Status" ""
 			(at 90.17 96.52 0)
 			(effects
@@
 			)
 		)
-		(property "Datasheet" "https://www.lcsc.com/datasheet/lcsc_datasheet_1810171610_YAGEO-RC0805JR-0710KL_C100047.pdf"
+		(property "Datasheet" ""
 			(at 101.6 123.19 0)
 			(effects
@@
 			)
 		)
-		(property "MPN" "RC0805JR-0710KL"
+		(property "MPN" ""
 			(at 101.6 123.19 90)
 			(effects
@@
 			)
 		)
-		(property "Status" "OK"
+		(property "Status" ""
 			(at 101.6 123.19 90)
 			(effects
@@
 			)
 		)
-		(property "Datasheet" "https://www.lcsc.com/datasheet/lcsc_datasheet_1810171610_YAGEO-RC0805JR-0710KL_C100047.pdf"
+		(property "Datasheet" ""
 			(at 229.87 54.61 0)
 			(effects
@@
 			)
 		)
-		(property "MPN" "RC0805JR-0710KL"
+		(property "MPN" ""
 			(at 229.87 54.61 0)
 			(effects
@@
 			)
 		)
-		(property "Status" "OK"
+		(property "Status" ""
 			(at 229.87 54.61 0)
 			(effects
@@
 			)
 		)
-		(property "Status" "OK"
+		(property "Status" ""
 			(at 90.17 64.77 0)
 			(effects
@@
 			)
 		)
-		(property "Status" "OK"
+		(property "Status" ""
 			(at 209.55 96.52 0)
 			(effects
@@
 			)
 		)
-		(property "Status" "OK"
+		(property "Status" ""
 			(at 209.55 128.27 0)
 			(effects
@@
 			)
 		)
-		(property "Status" "OK"
+		(property "Status" ""
 			(at 209.55 64.77 0)
 			(effects
@@
 			)
 		)
-		(property "Datasheet" "https://www.lcsc.com/datasheet/lcsc_datasheet_1810171610_YAGEO-RC0805JR-0710KL_C100047.pdf"
+		(property "Datasheet" ""
 			(at 229.87 118.11 0)
 			(effects
@@
 			)
 		)
-		(property "MPN" "RC0805JR-0710KL"
+		(property "MPN" ""
 			(at 229.87 118.11 0)
 			(effects
@@
 			)
 		)
-		(property "Status" "OK"
+		(property "Status" ""
 			(at 229.87 118.11 0)
 			(effects
@@
 			)
 		)
-		(property "Status" "OK"
+		(property "Status" ""
 			(at 46.99 91.44 0)
 			(effects
@@
 			)
 		)
-		(property "Datasheet" "https://www.lcsc.com/datasheet/lcsc_datasheet_1810171610_YAGEO-RC0805JR-0710KL_C100047.pdf"
+		(property "Datasheet" ""
 			(at 110.49 54.61 0)
 			(effects
@@
 			)
 		)
-		(property "MPN" "RC0805JR-0710KL"
+		(property "MPN" ""
 			(at 110.49 54.61 0)
 			(effects
@@
 			)
 		)
-		(property "Status" "OK"
+		(property "Status" ""
 			(at 110.49 54.61 0)
 			(effects
@@
 			)
 		)
-		(property "Datasheet" "https://www.lcsc.com/datasheet/lcsc_datasheet_1810171610_YAGEO-RC0805JR-0710KL_C100047.pdf"
+		(property "Datasheet" ""
 			(at 220.98 123.19 0)
 			(effects
@@
 			)
 		)
-		(property "MPN" "RC0805JR-0710KL"
+		(property "MPN" ""
 			(at 220.98 123.19 90)
 			(effects
@@
 			)
 		)
-		(property "Status" "OK"
+		(property "Status" ""
 			(at 220.98 123.19 90)
 			(effects
@@
 			)
 		)
-		(property "Datasheet" "https://www.lcsc.com/datasheet/lcsc_datasheet_1810171610_YAGEO-RC0805JR-0710KL_C100047.pdf"
+		(property "Datasheet" ""
 			(at 220.98 91.44 0)
 			(effects
@@
 			)
 		)
-		(property "MPN" "RC0805JR-0710KL"
+		(property "MPN" ""
 			(at 220.98 91.44 90)
 			(effects
@@
 			)
 		)
-		(property "Status" "OK"
+		(property "Status" ""
 			(at 220.98 91.44 90)
 			(effects

Commit message: Progressed ECAD.
Parts:
- renumbered C108 to C100, C109 to C101, C98 to C90, C99 to C91, C100 to C92, C101 to C93, C102 to C94, C103 to C95, C104 to C96, C105 to C97, C106 to C98, C107 to C99, R28 to R30, R29 to R31, R30 to R32, R31 to R33, R32 to R34, R33 to R35, R34 to R36, R35 to R37, R36 to R38, R37 to R39, R38 to R40, R39 to R41

Commit message: Progressed ECAD.
Parts:
- renumbered R30 to R23, R31 to R24, R32 to R25, R33 to R26, R34 to R27, R35 to R28, R36 to R29, R37 to R30, R38 to R31, R39 to R32, R40 to R33, R41 to R34

Commit message: Progressed ECAD.
Parts:
- renumbered C90 to C65, C91 to C66, C92 to C67, C93 to C68, C94 to C69, C95 to C70, C96 to C71, C97 to C72, C98 to C73, C99 to C74, C100 to C75, C101 to C76, J10 to J8, J11 to J9, R23 to R17, R24 to R18, R25 to R19, R26 to R20, R27 to R21, R28 to R22, R29 to R23, R30 to R24, R31 to R25, R32 to R26, R33 to R27, R34 to R28, U52 to U37, U53 to U38, U54 to U39, U55 to U40, U56 to U41, U57 to U42
