File: ECAD/BDCMotorController/adc_input.kicad_sch (KiCad schematic)
At the start: 23 parts, among them U60 LM4040DBZ-3.0, U61 AD8648, U62 AD8648

Commit message: Progressed ECAD.
Parts:
- C112, C113, C114: Status OK -> (none)
- R42: MPN AC0805FR-7W1KL -> (none)
Changed lines of the file:
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@@
 			)
 		)
-		(property "Status" "OK"
+		(property "Status" ""
 			(at 115.57 179.07 0)
 			(effects
@@
 			)
 		)
-		(property "Datasheet" "~"
+		(property "Datasheet" ""
 			(at 260.35 82.55 0)
 			(effects
@@
 			)
 		)
-		(property "Datasheet" "~"
+		(property "Datasheet" ""
 			(at 208.28 57.15 0)
 			(effects
@@
 			)
 		)
-		(property "Datasheet" "~"
+		(property "Datasheet" ""
 			(at 77.47 138.43 0)
 			(effects
@@
 			)
 		)
-		(property "Datasheet" "~"
+		(property "Datasheet" ""
 			(at 105.41 88.9 0)
 			(effects
@@
 			)
 		)
-		(property "Datasheet" "~"
+		(property "Datasheet" ""
 			(at 53.34 73.66 0)
 			(effects
@@
 			)
 		)
-		(property "Datasheet" "~"
+		(property "Datasheet" ""
 			(at 53.34 67.31 0)
 			(effects
@@
 			)
 		)
-		(property "Status" "OK"
+		(property "Status" ""
 			(at 87.63 179.07 0)
 			(effects
@@
 			)
 		)
-		(property "Datasheet" "~"
+		(property "Datasheet" ""
 			(at 243.84 88.9 0)
 			(effects
@@
 			)
 		)
-		(property "Datasheet" "~"
+		(property "Datasheet" ""
 			(at 191.77 73.66 0)
 			(effects
@@
 			)
 		)
-		(property "Datasheet" "~"
+		(property "Datasheet" ""
 			(at 243.84 82.55 0)
 			(effects
@@
 			)
 		)
-		(property "Datasheet" "~"
+		(property "Datasheet" ""
 			(at 191.77 67.31 0)
 			(effects
@@
 			)
 		)
-		(property "Datasheet" "~"
+		(property "Datasheet" ""
 			(at 91.44 132.08 0)
 			(effects
@@
 			)
 		)
-		(property "Datasheet" "~"
+		(property "Datasheet" ""
 			(at 121.92 82.55 0)
 			(effects
@@
 			)
 		)
-		(property "Datasheet" "https://datasheet.lcsc.com/lcsc/2010202005_YAGEO-AC0805FR-7W1KL_C727989.pdf"
+		(property "Datasheet" ""
 			(at 31.75 134.62 0)
 			(effects
@@
 			)
 		)
-		(property "MPN" "AC0805FR-7W1KL"
+		(property "MPN" ""
 			(at 31.75 134.62 0)
 			(effects
@@
 			)
 		)
-		(property "Datasheet" "~"
+		(property "Datasheet" ""
 			(at 105.41 82.55 0)
 			(effects
@@
 			)
 		)
-		(property "Status" "OK"
+		(property "Status" ""
 			(at 54.61 142.24 0)
 			(effects
@@
 			)
 		)
-		(property "Datasheet" "~"
+		(property "Datasheet" ""
 			(at 69.85 57.15 0)
 			(effects

Commit message: Progressed ECAD.
Parts:
- R42: Status OK -> (none)
Changed lines of the file:
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@@
 			)
 		)
-		(property "Status" "OK"
+		(property "Status" ""
 			(at 31.75 134.62 0)
 			(effects

Commit message: Progressed ECAD.
Parts:
- added C13, C26: 100nC, Capacitor_SMD:C_0805_2012Metric, symbol Device:C
Connections:
- net +5V: now also C13.1, C26.1; no longer C113.1, C114.1
- net GND: now also C113.1, C114.1, C13.2, C26.2
Other:
- moved on the sheet: C113, C114, U61E, U62E

Commit message: Progressed ECAD.
Parts:
- renumbered C13 to C105, C112 to C106, C113 to C107, C26 to C108, C114 to C109, D8 to D10, D7 to D9, R42 to R44, R43 to R45, R44 to R46, R45 to R47, R46 to R48, R47 to R49, R48 to R50, R49 to R51, R50 to R52, R51 to R53, R52 to R54, R53 to R55, R54 to R56, R55 to R57, R56 to R58

Commit message: Progressed ECAD.
Parts:
- renumbered D9 to D1, D10 to D2, R44 to R37, R45 to R38, R46 to R39, R47 to R40, R48 to R41, R49 to R42, R50 to R43, R51 to R44, R52 to R45, R53 to R46, R54 to R47, R55 to R48, R56 to R49, R57 to R50, R58 to R51

Commit message: Progressed ECAD.
Parts:
- R38, R39, R40, R41, R42, R43, R44, R45, R46, R47, R48, R49, R50, R51: value 1kR -> 10kR
Changed lines of the file:
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@@
 			)
 		)
-		(property "Value" "1kR"
+		(property "Value" "10kR"
 			(at 260.35 78.74 90)
 			(effects
@@
 			)
 		)
-		(property "Value" "1kR"
+		(property "Value" "10kR"
 			(at 208.28 54.61 90)
 			(effects
@@
 			)
 		)
-		(property "Value" "1kR"
+		(property "Value" "10kR"
 			(at 77.47 134.62 90)
 			(effects
@@
 			)
 		)
-		(property "Value" "1kR"
+		(property "Value" "10kR"
 			(at 105.41 91.44 90)
 			(effects
@@
 			)
 		)
-		(property "Value" "1kR"
+		(property "Value" "10kR"
 			(at 53.34 76.2 90)
 			(effects
@@
 			)
 		)
-		(property "Value" "1kR"
+		(property "Value" "10kR"
 			(at 53.34 63.5 90)
 			(effects
@@
 			)
 		)
-		(property "Value" "1kR"
+		(property "Value" "10kR"
 			(at 243.84 91.44 90)
 			(effects
@@
 			)
 		)
-		(property "Value" "1kR"
+		(property "Value" "10kR"
 			(at 191.77 76.2 90)
 			(effects
@@
 			)
 		)
-		(property "Value" "1kR"
+		(property "Value" "10kR"
 			(at 243.84 80.01 90)
 			(effects
@@
 			)
 		)
-		(property "Value" "1kR"
+		(property "Value" "10kR"
 			(at 191.77 63.5 90)
 			(effects
@@
 			)
 		)
-		(property "Value" "1kR"
+		(property "Value" "10kR"
 			(at 91.44 129.54 90)
 			(effects
@@
 			)
 		)
-		(property "Value" "1kR"
+		(property "Value" "10kR"
 			(at 121.92 78.74 90)
 			(effects
@@
 			)
 		)
-		(property "Value" "1kR"
+		(property "Value" "10kR"
 			(at 105.41 80.01 90)
 			(effects
@@
 			)
 		)
-		(property "Value" "1kR"
+		(property "Value" "10kR"
 			(at 69.85 54.61 90)
 			(effects

Commit message: Progressed ECAD.
Parts:
- renumbered C105 to C80, C106 to C81, C107 to C82, C108 to C83, C109 to C84, R37 to R31, R38 to R32, R39 to R33, R40 to R34, R41 to R35, R42 to R36, R43 to R37, R44 to R38, R45 to R39, R46 to R40, R47 to R41, R48 to R42, R49 to R43, R50 to R44, R51 to R45, U60 to U45, U61 to U46, U62 to U47
