File: ECAD/BDCMotorController/motor_control.kicad_sch (KiCad schematic)
At the start: 15 parts, among them U33 MCP4431, U34 MCP4431, U35 PCA9555PW, U36 MCP6S26, U37 MCP6S26

Commit message: Progressed ECAD.
Parts:
- removed C69, C71: 100nC, Capacitor_SMD:C_0805_2012Metric, symbol Device:C
Other:
- moved on the sheet: C68, C70, L5, L6

Commit message: Progressed ECAD.
Parts:
- removed L5, L6: 10uL, Inductor_SMD:L_0805_2012Metric, symbol Device:L
- renumbered C65 to C61, C66 to C62, C67 to C63, C68 to C64, C70 to C65, R21 to R23
Connections:
- net +5V: now also C64.1, C65.1, U36.14 (V_{DD}), U37.14 (V_{DD})

Commit message: Progressed ECAD.
Parts:
- added R16: 10kR, Resistor_SMD:R_0805_2012Metric, symbol Device:R
- renumbered R23 to R15
Connections:
- net GND: now also R16.2
- net PGA_SO: now also R16.1; no longer U37.12 (SO)
- no-connect marks 4 -> 5

Commit message: Progressed ECAD.
Other:
- note added: "The SO is on the MCP6S26 is only used for daisy chain multiple units. No read commans are available, so not useful to connect back to the MCU."
Changed lines of the file:
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@@
+		)
+	)
+	(text "The SO is on the MCP6S26 is only used for daisy chain multiple units.\nNo read commans are available, so not useful to connect back to the MCU.\n"
+		(exclude_from_sim no)
+		(at 226.314 157.988 0)
+		(effects
+			(font
+				(size 1.27 1.27)
+			)
 		)
 	)

Commit message: Progressed ECAD.
Parts:
- removed C62: 100nC, Capacitor_SMD:C_0805_2012Metric, symbol Device:C
- removed U34: MCP4431, Package_SO:TSSOP-20_4.4x6.5mm_P0.65mm, symbol Potentiometer_Digital:MCP4431-xxxx-ST
Connections:
- net CURRENT_M3A is gone; now on net GND: U36.6 (CH4), U37.6 (CH4)
- net CURRENT_M3B is gone; now on net GND: U36.7 (CH5), U37.7 (CH5)
- net EN_M3A renamed POT_~{RESET}
- net POT_~{RESET}: now also U33.15 (~{RESET})
- net EN_M3B: no longer names the net of U35.18 (IO1_5)
- net POT1_~{RESET}: no longer names the net of U35.10 (IO0_6)
- net POT1_~{RESET}: no longer U33.15 (~{RESET})
- net POT2_~{RESET}: no longer names the net of U35.11 (IO0_7)
- no-connect marks 5 -> 4
Other:
- removed sheet H-bridge #5
- removed sheet H-bridge #6
- note added: "The SO pin on the MCP6S26 is only used for daisy chain multiple such units. No read commans are available, so not useful to connect back to the MCU."
- note removed: "I2C Address: 0101 110"
- note removed: "The SO is on the MCP6S26 is only used for daisy chain multiple units. No read commans are available, so not useful to connect back to the MCU."
- moved on the sheet: C61, C63, C64, C65, R15, R16, U33E, U35, U36, U37

Commit message: Progressed ECAD.
Parts:
- renumbered C63 to C62, C64 to C63, C65 to C64, U35 to U34, U36 to U35, U37 to U36

Commit message: Progressed ECAD.
Parts:
- removed U33: MCP4431, Package_SO:TSSOP-20_4.4x6.5mm_P0.65mm, symbol Potentiometer_Digital:MCP4431-xxxx-ST
- added U68: MCP4451, Package_SO:TSSOP-20_4.4x6.5mm_P0.65mm, symbol Potentiometer_Digital:MCP4451-xxxx-ST
Connections:
- net +5V: now also U68.1 (P3A), U68.10 (P1A), U68.11 (P0A), U68.17 (VDD), U68.20 (P2A)
- net GND: now also U68.13 (P0B), U68.16 (A1), U68.18 (P2B), U68.3 (P3B), U68.4 (HVC/A0), U68.7 (VSS), U68.8 (P1B)
- net POT_~{RESET}: now also U68.15 (~{RESET})
- net SCL: now also U68.5 (SCL)
- net SDA: now also U68.6 (SDA)
- net VREF_M1A: now also U68.12 (P0W)
- net VREF_M1B: now also U68.9 (P1W)
- net VREF_M2A: now also U68.19 (P2W)
- net VREF_M2B: now also U68.2 (P3W)
