File: ECAD/BDCMotorController/BDCMotorController.kicad_pcb (KiCad board)
At the start: 2 copper layers, 150 x 80.5 mm, 370 parts, among them J1 Screw_Terminal_01x06, J10 Screw_Terminal_01x06, J11 Screw_Terminal_01x06, J12 DC, J13 USB_B, J14 Conn_01x16, J15 ICSP, J2 Screw_Terminal_01x06, J3 Screw_Terminal_01x06, J4 Screw_Terminal_01x06, J5 DE9_Pins_MountingHoles, J6 DE9_Pins_MountingHoles, J7 DE9_Pins_MountingHoles, J8 Screw_Terminal_01x06, J9 Screw_Terminal_01x06, Q1 BC847, SW1 SW_Push, U1 74AHC2G125, U10 74AHC00, U11 74AHC1G17, U12 DRV8870DDA, U13 74AHC1G17, U14 INA180A1, U15 SP3243E, U16 SP3243E, U17 74AHC2G125, U18 74AHC00, U19 74AHC00, U2 74AHC00, U20 74AHC1G17, U21 DRV8870DDA, U22 74AHC1G17, U23 INA180A1, U24 74AHC2G125, U25 74AHC00, U26 74AHC00, U27 74AHC1G17, U28 DRV8870DDA, U29 74AHC1G17, U3 74AHC00, U30 INA180A1, U31 PCA9555PW, U32 PCA9555PW, U33 MCP4431, U34 MCP4431, U35 PCA9555PW, U36 MCP6S26, U37 MCP6S26, U38 74AHC2G125, U39 74AHC00, U4 74AHC1G17, U40 74AHC00, U41 74AHC1G17, U42 DRV8870DDA, U43 74AHC1G17, U44 INA180A1, U45 74AHC2G125, U46 74AHC00, U47 74AHC00, U48 74AHC1G17, U49 DRV8870DDA, U5 DRV8870DDA, U50 74AHC1G17, U51 INA180A1, U52 74AHC1G17, U53 74AHC1G17, U54 74AHC1G17, U55 74AHC1G17, U56 74AHC1G17, U57 74AHC1G17, U58 74AHC1G17, U59 IRM-H6xxT, U6 74AHC1G17, U60 LM4040DBZ-3.0, U61 AD8648, U63 AD8648, U64 TPS561208DDCR, U65 TLV75801PDBVR, U66 LM2776, U67 SP3243E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

Commit message: Progressed ECAD.
Parts:
- removed C167: 100nC, Capacitor_SMD:C_0805_2012Metric
- removed D14: LED, LED_SMD:LED_0805_2012Metric
- removed D15: 4148, Diode_SMD:D_SOD-123
- removed U83: 74AHC00, Package_SO:TSSOP-14_4.4x5mm_P0.65mm
- added C113: 100nC, Capacitor_SMD:C_0805_2012Metric, F.Cu at (-89.3, 116.3)
- added D10: LED, LED_SMD:LED_0805_2012Metric, F.Cu at (-55.7, 79.2)
- added D7: BAV99, Package_TO_SOT_SMD:SOT-23, F.Cu at (-75.9, 109.7)
- added D8: BAV99, Package_TO_SOT_SMD:SOT-23, F.Cu at (-75.9, 114.3)
- added D9: CMS30I30A, Diode_SMD:D_SOD-128, F.Cu at (-107.5, 50.1)
- added R78: 1kR, Resistor_SMD:R_0805_2012Metric, F.Cu at (-30.6, 102.4)
- added U62: AD8648, Package_SO:TSSOP-14_4.4x5mm_P0.65mm, F.Cu at (-73.9, 104.0)
- C115: value 100nC -> 10uC; footprint Capacitor_SMD:C_0805_2012Metric -> Capacitor_SMD:C_1210_3225Metric
- C116: value 10uC -> 100nC; footprint Capacitor_SMD:C_1210_3225Metric -> Capacitor_SMD:C_0805_2012Metric
- C121: value 100nC -> 10uC
- C122: value 10uC -> 2.2uC
- C123: value 2.2uC -> 10uC
- C124: value 10uC -> 1uC
- C125: value 1uC -> 100nC
- C126: value 100nC -> 2.2uC
- C127: value 2.2uC -> 100nC
- C128, C139, C156: value 100nC -> 13pC
- C129: value 13pC -> 10uC
- C130: value 10uC -> 47uC; footprint Capacitor_SMD:C_0805_2012Metric -> Capacitor_SMD:C_1210_3225Metric
- C131: value 47uC -> 100nC; footprint Capacitor_SMD:C_1210_3225Metric -> Capacitor_SMD:C_0805_2012Metric
- C132: value 100nC -> 330nC
- C136: value 330nC -> 4n7C
- C137: value 4n7C -> 100nC
- C141, C157, C160: value 13pC -> 100nC
- C142: value 100nC -> 10uC; footprint Capacitor_SMD:C_0805_2012Metric -> Capacitor_SMD:C_1206_3216Metric
- C143: value 10uC -> 100nC; footprint Capacitor_SMD:C_1206_3216Metric -> Capacitor_SMD:C_0805_2012Metric
- C146, C164: value 100nC -> 100pC
- C148, C166: value 100pC -> 100nC
- C158: value 100nC -> 4n7C
- C159: value 4n7C -> 13pC
- D11: value CMS30I30A -> LED; footprint Diode_SMD:D_SOD-128 -> LED_SMD:LED_0805_2012Metric
- D13: value LED -> 4148; footprint LED_SMD:LED_0805_2012Metric -> Diode_SMD:D_SOD-123
- R70: value 1kR -> 10R
- R71: value 10kR -> 1kR
- R72: value 100kR -> 10kR
- R73: value 10kR -> 100kR
- R76: value 1kR -> 10kR
- RV1: value 10R -> 200R
- U63: value AD8648 -> TPS561208DDCR; footprint Package_SO:TSSOP-14_4.4x5mm_P0.65mm -> Package_TO_SOT_SMD:SOT-23-6
- U64: value TPS561208DDCR -> TLV75801PDBVR; footprint Package_TO_SOT_SMD:SOT-23-6 -> Package_TO_SOT_SMD:SOT-23-5
- U65: value TLV75801PDBVR -> LM2776; footprint Package_TO_SOT_SMD:SOT-23-5 -> Package_TO_SOT_SMD:SOT-23-6
- U66: value LM2776 -> SP3243E; footprint Package_TO_SOT_SMD:SOT-23-6 -> Package_SO:TSSOP-28_4.4x9.7mm_P0.65mm
- U67: value SP3243E -> USBLC6-2SC6; footprint Package_SO:TSSOP-28_4.4x9.7mm_P0.65mm -> Package_TO_SOT_SMD:SOT-23-6
- U68: value USBLC6-2SC6 -> FT232RN; footprint Package_TO_SOT_SMD:SOT-23-6 -> Package_SO:SSOP-28_5.3x10.2mm_P0.65mm
- U69: value FT232RN -> 74AHC00; footprint Package_SO:SSOP-28_5.3x10.2mm_P0.65mm -> Package_SO:TSSOP-14_4.4x5mm_P0.65mm
- U71, U80: value 74AHC00 -> 74AHC1G17; footprint Package_SO:TSSOP-14_4.4x5mm_P0.65mm -> Package_TO_SOT_SMD:SC-74A-5_1.55x2.9mm_P0.95mm
- U73, U82: value 74AHC1G17 -> 74AHC00; footprint Package_TO_SOT_SMD:SC-74A-5_1.55x2.9mm_P0.95mm -> Package_SO:TSSOP-14_4.4x5mm_P0.65mm
- U74: value 74AHC00 -> LM317_TO-252; footprint Package_SO:TSSOP-14_4.4x5mm_P0.65mm -> Package_TO_SOT_SMD:TO-252-2
- U75: value LM317_TO-252 -> ATmega2560-16A; footprint Package_TO_SOT_SMD:TO-252-2 -> Package_QFP:TQFP-100_14x14mm_P0.5mm
- U76: value ATmega2560-16A -> 74AHC573; footprint Package_QFP:TQFP-100_14x14mm_P0.5mm -> Package_SO:TSSOP-20_4.4x6.5mm_P0.65mm
- U77: value 74AHC573 -> AS7C4096A; footprint Package_SO:TSSOP-20_4.4x6.5mm_P0.65mm -> Package_SO:TSOP-II-44_10.16x18.41mm_P0.8mm
- U78: value AS7C4096A -> 74AHC00; footprint Package_SO:TSOP-II-44_10.16x18.41mm_P0.8mm -> Package_SO:TSSOP-14_4.4x5mm_P0.65mm
- moved U51 412.8 mm to (-62.0, 57.2)
- moved C93 408.7 mm to (-61.7, 61.5)
- moved R26 404.2 mm to (-44.1, 47.6)
- moved U48 399.7 mm to (-44.2, 39.1)
- moved U50 399.7 mm to (-44.2, 43.7)
- moved U49 397.4 mm to (-50.9, 53.2)
- moved U46 396.3 mm to (-51.3, 40.0)
- moved U47 396.3 mm to (-51.3, 46.6)
- moved L8 392.0 mm to (-42.0, 57.9)
- moved C85 392.0 mm to (-62.3, 38.2)
- moved C86 392.0 mm to (-62.3, 41.2)
- moved C87 392.0 mm to (-62.3, 44.2)
- moved C88 392.0 mm to (-62.3, 47.2)
- moved C89 392.0 mm to (-62.3, 50.3)
- moved C90 392.0 mm to (-62.3, 53.3)
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Connections:
- C115 pad 2: -5V -> GND
- C117 pad 1: +5V -> GND
- C117 pad 2: GND -> +5V
- C119 pad 2: +5V -> VDC
- C120 pad 2: VDC -> +5V
- C121 pad 1: GND -> VDC
- C121 pad 2: +5V -> GND
- C122 pad 1: VDC -> +5V
- C123 pad 1: +5V -> VDC
- C124 pad 1: VDC -> Net-(U65-C1+)
- C124 pad 2: GND -> Net-(U65-C1-)
- C125 pad 1: Net-(U66-C1+) -> Net-(U63-BOOT)
- C125 pad 2: Net-(U66-C1-) -> Net-(U63-SW)
- C126 pad 1: Net-(U64-BOOT) -> -5V
- C126 pad 2: Net-(U64-SW) -> GND
- C127 pad 1: -5V -> +5V
- C127 pad 2: GND -> Net-(U64-FB)
- C128 pad 1: +5V -> /Power/5V5
- C128 pad 2: Net-(U65-FB) -> Net-(U63-FB)
- C129 pad 1: /Power/5V5 -> +5V
- C129 pad 2: Net-(U64-FB) -> GND
- C130 pad 1: +5V -> /Power/5V5
- C131 pad 1: /Power/5V5 -> +5V
- C132 pad 1: +5V -> /Serial ports/RS232 Interface #3/C1+
- C132 pad 2: GND -> /Serial ports/RS232 Interface #3/C1-
- C133 pad 1: /Serial ports/RS232 Interface #3/C1+ -> /Serial ports/RS232 Interface #3/V-
- C133 pad 2: /Serial ports/RS232 Interface #3/C1- -> GND
- C134 pad 1: /Serial ports/RS232 Interface #3/V- -> /Serial ports/RS232 Interface #3/C2+
- C134 pad 2: GND -> /Serial ports/RS232 Interface #3/C2-
- C135 pad 1: /Serial ports/RS232 Interface #3/C2+ -> /Serial ports/RS232 Interface #3/V+
- C135 pad 2: /Serial ports/RS232 Interface #3/C2- -> GND
- C136 pad 1: /Serial ports/RS232 Interface #3/V+ -> Net-(J13-Shield)
- C137 pad 1: Net-(J13-Shield) -> VBUS
- C138 pad 1: VBUS -> Net-(U68-3V3OUT)
- C139 pad 1: Net-(U69-3V3OUT) -> /USB/USBP
- C140 pad 1: /USB/USBP -> /USB/USBM
- C141 pad 1: /USB/USBM -> +5V
- C143 pad 1: +5V -> Net-(U68-DTR)
- C143 pad 2: GND -> /MCU/~{RESET}
- C144 pad 1: Net-(U69-DTR) -> +5V
- C144 pad 2: /MCU/~{RESET} -> GND
- C146 pad 1: +5V -> Net-(C146-Pad1)
- C148 pad 1: Net-(C148-Pad1) -> +5V
- C149 pad 1: +5V -> VDC
- C150 pad 1: VDC -> +5V
- C155 pad 1: +5V -> +5VA
- C156 pad 1: +5VA -> /MCU/XTAL2
- C157 pad 1: /MCU/XTAL2 -> +3VADC
- C158 pad 1: +3VADC -> /MCU/~{RESET}
- C159 pad 1: /MCU/~{RESET} -> /MCU/XTAL1
- C160 pad 1: /MCU/XTAL1 -> +5V
- C164 pad 1: +5V -> Net-(C164-Pad1)
- C166 pad 1: Net-(C166-Pad1) -> +5V
- D11 pad 1: /Power/5V5 -> Net-(D11-K)
- D13 pad 1: Net-(D13-K) -> +5V
- D13 pad 2: +5V -> /MCU/~{RESET}
- L9 pad 1: Net-(U64-SW) -> Net-(U63-SW)
- R51 pad 1: Net-(D9-A) -> Net-(U62A--)
- R52 pad 1: Net-(D9-A) -> Net-(U62A--)
- R53 pad 2: Net-(D9-A) -> Net-(U62A--)
- R54 pad 1: Net-(U63B--) -> Net-(U62B--)
- R55 pad 2: Net-(U63B--) -> Net-(U62B--)
- R56 pad 2: Net-(U63B--) -> Net-(U62B--)
- R57 pad 2: Net-(U64-EN) -> Net-(U63-EN)
- R58 pad 2: Net-(U65-FB) -> Net-(U64-FB)
- R59 pad 1: Net-(U65-FB) -> Net-(U64-FB)
- R60 pad 2: Net-(U64-FB) -> Net-(U63-FB)
- R61 pad 1: Net-(U64-FB) -> Net-(U63-FB)
- R65 pad 2: Net-(D12-K) -> Net-(D10-K)
- R66 pad 2: Net-(D13-K) -> Net-(D11-K)
- R68 pad 1: Net-(C147-Pad1) -> Net-(C146-Pad1)
- R69 pad 1: Net-(C148-Pad1) -> Net-(C147-Pad1)
- R70 pad 1: Net-(Q1-C) -> Net-(U74-VO)
- R70 pad 2: Net-(D14-K) -> Net-(R70-Pad2)
- R71 pad 1: +5V -> Net-(Q1-C)
- R71 pad 2: /MCU/~{RESET} -> Net-(D12-K)
- R72 pad 1: /MCU/XTAL2 -> +5V
- R72 pad 2: /MCU/XTAL1 -> /MCU/~{RESET}
- R73 pad 1: Net-(Q1-B) -> /MCU/XTAL2
- R73 pad 2: /MCU/LED_IND -> /MCU/XTAL1
- R74 pad 1: +5V -> Net-(Q1-B)
- R74 pad 2: /MCU/SDA -> /MCU/LED_IND
- R75 pad 2: /MCU/SCL -> /MCU/SDA
- R76 pad 1: Net-(C165-Pad1) -> +5V
- R76 pad 2: /Motor Control/H-bridge #1/ENCODER_A -> /MCU/SCL
- R77 pad 1: Net-(C166-Pad1) -> Net-(C164-Pad1)
- R77 pad 2: /Motor Control/H-bridge #1/ENCODER_B -> /Motor Control/H-bridge #1/ENCODER_A
- RV1 pad 1: Net-(U75-VO) -> Net-(R70-Pad2)
- RV1 pad 2: Net-(U75-VO) -> /LCD/BL_LED
- U63 pad 1: Net-(D10-A) -> GND
- U63 pad 2: Net-(D9-A) -> Net-(U63-SW)
- U63 pad 3: GND -> VDC
- U63 pad 4: +5V -> Net-(U63-FB)
- U63 pad 5: GND -> Net-(U63-EN)
- U63 pad 6: Net-(U63B--) -> Net-(U63-BOOT)
- U64 pad 1: GND -> /Power/5V5
- U64 pad 2: Net-(U64-SW) -> GND
- U64 pad 3: VDC -> /Power/5V5
- U64 pad 5: Net-(U64-EN) -> +5V
- U65 pad 1: /Power/5V5 -> -5V
- U65 pad 3: /Power/5V5 -> +5V
- U65 pad 4: Net-(U65-FB) -> +5V
- U65 pad 5: +5V -> Net-(U65-C1+)
- U66 pad 1: -5V -> /Serial ports/RS232 Interface #3/C2+
- U66 pad 2: GND -> /Serial ports/RS232 Interface #3/C2-
- U66 pad 3: +5V -> /Serial ports/RS232 Interface #3/V-
- U66 pad 4: +5V -> /Serial ports/CTS_LINE3
- U66 pad 5: Net-(U66-C1+) -> /Serial ports/RI_LINE3
- U66 pad 6: Net-(U66-C1-) -> /Serial ports/DCD_LINE3
- U67 pad 1: /Serial ports/RS232 Interface #3/C2+ -> Net-(J13-D+)
- U67 pad 2: /Serial ports/RS232 Interface #3/C2- -> GND
- U67 pad 3: /Serial ports/RS232 Interface #3/V- -> Net-(J13-D-)
- U67 pad 4: /Serial ports/CTS_LINE3 -> /USB/USBM
- U67 pad 5: /Serial ports/RI_LINE3 -> VBUS
- U67 pad 6: /Serial ports/DCD_LINE3 -> /USB/USBP
- U68 pad 1: Net-(J13-D+) -> /MCU/RXD0
- U68 pad 2: GND -> Net-(U68-DTR)
- U68 pad 3: Net-(J13-D-) -> unconnected-(U68-RTS-Pad3)
- U68 pad 4: /USB/USBM -> +5V
- U68 pad 5: VBUS -> /MCU/TXD0
- U68 pad 6: /USB/USBP -> unconnected-(U68-RI-Pad6)
- U69 pad 1: /MCU/RXD0 -> /Motor Control/H-bridge #2/ENCODER_A
- U69 pad 10: unconnected-(U69-DCD-Pad10) -> Net-(U69-Pad10)
- U69 pad 11: unconnected-(U69-CTS-Pad11) -> Net-(U69-Pad11)
- U69 pad 12: unconnected-(U69-CBUS4-Pad12) -> /Motor Control/H-bridge #2/ENCODER_A
- U69 pad 13: unconnected-(U69-CBUS2-Pad13) -> Net-(U69-Pad10)
- U69 pad 14: /MCU/PCINT15 -> +5V
- U69 pad 2: Net-(U69-DTR) -> Net-(U69-Pad2)
- U69 pad 3: unconnected-(U69-RTS-Pad3) -> Net-(U69-Pad10)
- U69 pad 4: +5V -> Net-(U69-Pad11)
- U69 pad 5: /MCU/TXD0 -> Net-(U69-Pad5)
- U69 pad 6: unconnected-(U69-RI-Pad6) -> Net-(U69-Pad6)
- U69 pad 8: (no net) -> Net-(U69-Pad5)
- U69 pad 9: unconnected-(U69-DCR-Pad9) -> Net-(U69-Pad2)
- U70 pad 1: /Motor Control/H-bridge #2/ENCODER_A -> /Motor Control/H-bridge #2/ENCODER_B
- U70 pad 12: /Motor Control/H-bridge #2/ENCODER_A -> /Motor Control/H-bridge #2/ENCODER_B
- U71 pad 1: /Motor Control/H-bridge #2/ENCODER_B -> unconnected-(U71-NC-Pad1)
- U71 pad 2: Net-(U71-Pad2) -> Net-(C146-Pad1)
- U71 pad 3: Net-(U71-Pad10) -> GND
- U71 pad 4: Net-(U71-Pad11) -> Net-(U69-Pad2)
- U71 pad 5: Net-(U71-Pad5) -> +5V
- U73 pad 1: unconnected-(U73-NC-Pad1) -> GND
- U73 pad 2: Net-(C148-Pad1) -> GND
- U73 pad 3: GND -> unconnected-(U73-Pad3)
- U73 pad 4: Net-(U71-Pad2) -> Net-(U73-Pad11)
- U73 pad 5: +5V -> Net-(U73-Pad5)
- U74 pad 1: GND -> /LCD/BL_LED
- U74 pad 2: GND -> Net-(U74-VO)
- U74 pad 3: unconnected-(U74-Pad3) -> VDC
- U75 pad 1: /LCD/BL_LED -> unconnected-(U75-PG5-Pad1)
- U75 pad 2: Net-(U75-VO) -> /MCU/RXD0
- U75 pad 3: VDC -> /MCU/TXD0
- U76 pad 1: unconnected-(U76-PG5-Pad1) -> /MCU/~{XMEM_EN}
- U76 pad 10: +5V -> GND
- U76 pad 11: GND -> /MCU/XMEM_ALE
- U76 pad 12: /MCU/RXD2 -> Net-(U76-Q7)
- U76 pad 13: /MCU/TXD2 -> Net-(U76-Q6)
- U76 pad 14: unconnected-(U76-PH2-Pad14) -> Net-(U76-Q5)
- U76 pad 15: unconnected-(U76-PH3-Pad15) -> Net-(U76-Q4)
- U76 pad 16: unconnected-(U76-PH4-Pad16) -> Net-(U76-Q3)
- U76 pad 17: unconnected-(U76-PH5-Pad17) -> Net-(U76-Q2)
- U76 pad 18: /MCU/LED_IND -> Net-(U76-Q1)
- U76 pad 19: /MCU/~{SS} -> Net-(U76-Q0)
- U76 pad 2: /MCU/RXD0 -> /MCU/XMEM_AD0
- U76 pad 20: /MCU/SCK -> +5V
- U76 pad 3: /MCU/TXD0 -> /MCU/XMEM_AD1
- U76 pad 4: unconnected-(U76-PE2-Pad4) -> /MCU/XMEM_AD2
- U76 pad 5: unconnected-(U76-PE3-Pad5) -> /MCU/XMEM_AD3
- U76 pad 6: /MCU/INT4 -> /MCU/XMEM_AD4
- U76 pad 7: /MCU/INT5 -> /MCU/XMEM_AD5
- U76 pad 8: /MCU/INT6 -> /MCU/XMEM_AD6
- U76 pad 9: /MCU/INT7 -> /MCU/XMEM_AD7
- U77 pad 1: /MCU/~{XMEM_EN} -> unconnected-(U77-NC-Pad1)
- U77 pad 10: GND -> /MCU/XMEM_AD1
- U77 pad 11: /MCU/XMEM_ALE -> +5V
- U77 pad 12: Net-(U77-Q7) -> GND
- U77 pad 13: Net-(U77-Q6) -> /MCU/XMEM_AD2
- U77 pad 14: Net-(U77-Q5) -> /MCU/XMEM_AD3
- U77 pad 15: Net-(U77-Q4) -> /MCU/XMEM_~{WR}
- U77 pad 16: Net-(U77-Q3) -> Net-(U76-Q5)
- U77 pad 17: Net-(U77-Q2) -> Net-(U76-Q6)
- U77 pad 18: Net-(U77-Q1) -> Net-(U76-Q7)
- U77 pad 19: Net-(U77-Q0) -> /MCU/XMEM_A08
- U77 pad 2: /MCU/XMEM_AD0 -> unconnected-(U77-NC-Pad2)
- U77 pad 20: +5V -> /MCU/XMEM_A09
- U77 pad 3: /MCU/XMEM_AD1 -> Net-(U76-Q0)
- U77 pad 4: /MCU/XMEM_AD2 -> Net-(U76-Q1)
- U77 pad 5: /MCU/XMEM_AD3 -> Net-(U76-Q2)
- U77 pad 6: /MCU/XMEM_AD4 -> Net-(U76-Q3)
- U77 pad 7: /MCU/XMEM_AD5 -> Net-(U76-Q4)
- U77 pad 8: /MCU/XMEM_AD6 -> /MCU/~{XMEM_EN}
- U77 pad 9: /MCU/XMEM_AD7 -> /MCU/XMEM_AD0
- U78 pad 1: unconnected-(U78-NC-Pad1) -> /Motor Control/H-bridge #1/ENCODER_A
- U78 pad 10: /MCU/XMEM_AD1 -> Net-(U78-Pad10)
- U78 pad 11: +5V -> Net-(U78-Pad11)
- U78 pad 12: GND -> /Motor Control/H-bridge #1/ENCODER_A
- U78 pad 13: /MCU/XMEM_AD2 -> Net-(U78-Pad10)
- U78 pad 14: /MCU/XMEM_AD3 -> +5V
- U78 pad 2: unconnected-(U78-NC-Pad2) -> Net-(U78-Pad2)
- U78 pad 3: Net-(U77-Q0) -> Net-(U78-Pad10)
- U78 pad 4: Net-(U77-Q1) -> Net-(U78-Pad11)
- U78 pad 5: Net-(U77-Q2) -> Net-(U78-Pad5)
- U78 pad 6: Net-(U77-Q3) -> Net-(U78-Pad6)
- U78 pad 7: Net-(U77-Q4) -> GND
- U78 pad 8: /MCU/~{XMEM_EN} -> Net-(U78-Pad5)
- U78 pad 9: /MCU/XMEM_AD0 -> Net-(U78-Pad2)
- U79 pad 1: /Motor Control/H-bridge #1/ENCODER_A -> /Motor Control/H-bridge #1/ENCODER_B
- U79 pad 12: /Motor Control/H-bridge #1/ENCODER_A -> /Motor Control/H-bridge #1/ENCODER_B
- U80 pad 1: /Motor Control/H-bridge #1/ENCODER_B -> unconnected-(U80-NC-Pad1)
- U80 pad 2: Net-(U80-Pad2) -> Net-(C164-Pad1)
- U80 pad 3: Net-(U80-Pad10) -> GND
- U80 pad 4: Net-(U80-Pad11) -> Net-(U78-Pad2)
- U80 pad 5: Net-(U80-Pad5) -> +5V
- U82 pad 1: unconnected-(U82-NC-Pad1) -> GND
- U82 pad 2: Net-(C166-Pad1) -> GND
- U82 pad 3: GND -> unconnected-(U82-Pad3)
- U82 pad 4: Net-(U80-Pad2) -> Net-(U82-Pad11)
- U82 pad 5: +5V -> Net-(U82-Pad5)

Commit message: Progressed ECAD.
Parts:
- C10, C23, C46, C59, C81, C94: footprint Capacitor_THT:CP_Radial_D5.0mm_P2.00mm -> Capacitor_SMD:C_1210_3225Metric
- C142: footprint Capacitor_SMD:C_1206_3216Metric -> Capacitor_SMD:C_1210_3225Metric
- R15, R16, R17, R18, R19, R20: footprint Resistor_SMD:R_0805_2012Metric_Pad1.20x1.40mm_HandSolder -> Resistor_SMD:R_0805_2012Metric
- moved C11 213.0 mm to (46.5, 183.0)
- moved C13 206.4 mm to (46.5, 180.5)
- moved U7 201.1 mm to (41.8, 181.1)
- moved C8 198.5 mm to (26.0, 177.0)
- moved R2 194.2 mm to (35.5, 181.0), turned to 90 degrees
- moved L1 194.1 mm to (46.5, 185.0)
- moved C10 188.3 mm to (23.0, 187.5)
- moved C9 187.2 mm to (25.5, 181.0)
- moved U5 187.2 mm to (34.8, 173.8), turned to -90 degrees
- moved C1 172.6 mm to (25.4, 138.3)
- moved C12 172.6 mm to (29.9, 147.3)
- moved C2 172.6 mm to (25.4, 141.3)
- moved C3 172.6 mm to (25.4, 144.3)
- moved C4 172.6 mm to (25.4, 147.3)
- moved C5 172.6 mm to (25.4, 150.3)
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
Commit message: Progressed ECAD.
Parts:
- removed C1, C100, C101, C102, C103, C104, C105, C106, C107, C108, C109, C11, C110, C112, C113, C114, C116, C117, C118, C119, C120, C125, C127, C13, C131, C137, C138, C14, C141, C143, C144, C145, C148, C149, C15, C150, C151, C152, C153, C154, C155, C157, C160, C161, C162, C163, C166, C17, C18, C19, C2, C20, C21, C24, C26, C27, C32, C37, C38, C4, C40, C41, C42, C43, C44, C47, C49, C5, C50, C51, C53, C54, C55, C56, C57, C6, C60, C62, C63, C64, C65, C66, C67, C68, C69, C7, C70, C71, C72, C73, C75, C76, C77, C78, C79, C8, C82, C84, C85, C86, C88, C89, C90, C91, C92, C95, C97, C98, C99: 100nC, Capacitor_SMD:C_0805_2012Metric
- removed C10, C130, C23, C46, C59, C81, C94: 47uC, Capacitor_SMD:C_1210_3225Metric
- removed C111: 4.7uC, Capacitor_SMD:C_0805_2012Metric
- removed C115, C142, C22, C45, C58, C80, C9, C93: 10uC, Capacitor_SMD:C_1210_3225Metric
- removed C12, C146, C147, C16, C164, C165, C25, C3, C39, C48, C52, C61, C74, C83, C87, C96: 100pC, Capacitor_SMD:C_0805_2012Metric
- removed C121, C123, C129: 10uC, Capacitor_SMD:C_0805_2012Metric
- removed C122, C126: 2.2uC, Capacitor_SMD:C_0805_2012Metric
- removed C124: 1uC, Capacitor_SMD:C_0805_2012Metric
- removed C128, C139, C140, C156, C159: 13pC, Capacitor_SMD:C_0805_2012Metric
- removed C132, C133, C134, C135, C28, C29, C30, C31, C33, C34, C35, C36: 330nC, Capacitor_SMD:C_0805_2012Metric
- removed C136, C158: 4n7C, Capacitor_SMD:C_0805_2012Metric
- removed D1, D10, D11, D12, D2, D3, D4, D5, D6: LED, LED_SMD:LED_0805_2012Metric
- removed D13: 4148, Diode_SMD:D_SOD-123
- removed D7, D8: BAV99, Package_TO_SOT_SMD:SOT-23
- removed D9: CMS30I30A, Diode_SMD:D_SOD-128
- removed H1, H2, H3, H4: MountingHole, MountingHole:MountingHole_3.2mm_M3
- removed J1, J10, J11, J2, J3, J4, J8, J9: Screw_Terminal_01x06, TerminalBlock_Phoenix:TerminalBlock_Phoenix_MPT-0,5-6-2.54_1x06_P2.54mm_Horizontal
- removed J12: DC, Connector_BarrelJack:BarrelJack_Horizontal
- removed J13: USB_B, Connector_USB:USB_B_TE_5787834_Vertical
- removed J14: Conn_01x16, Connector_PinHeader_2.54mm:PinHeader_1x16_P2.54mm_Vertical
- removed J15: ICSP, Connector_PinHeader_2.54mm:PinHeader_2x03_P2.54mm_Vertical
- removed J5, J6, J7: DE9_Pins_MountingHoles, Connector_Dsub:DSUB-9_Pins_Vertical_P2.77x2.84mm_MountingHoles
- removed L1, L10, L2, L3, L4, L5, L6, L7, L8: 10uL, Inductor_SMD:L_0805_2012Metric
- removed L9: 4u7L, Inductor_SMD:L_1008_2520Metric
- removed Q1: BC847, Package_TO_SOT_SMD:SOT-23
- removed R1, R10, R12, R15, R16, R17, R18, R19, R20, R22, R24, R25, R27, R3, R4, R42, R43, R44, R45, R46, R47, R48, R49, R50, R51, R52, R53, R54, R55, R56, R6, R65, R66, R68, R69, R7, R71, R77, R78, R9: 1kR, Resistor_SMD:R_0805_2012Metric
- removed R11, R2, R23, R26, R5, R8: 150mR, Resistor_SMD:R_1206_3216Metric
- removed R13, R14, R21, R28, R29, R30, R31, R32, R33, R34, R35, R36, R37, R38, R39, R41, R57, R59, R61, R64, R67, R72, R74, R75, R76: 10kR, Resistor_SMD:R_0805_2012Metric
- removed R40: 160R, Resistor_SMD:R_0805_2012Metric
- removed R58: 80k6R, Resistor_SMD:R_0805_2012Metric
- removed R60: 61k9R, Resistor_SMD:R_0805_2012Metric
- removed R62: 1MR, Resistor_SMD:R_0805_2012Metric
- removed R63: 4k7R, Resistor_SMD:R_0805_2012Metric
- removed R70: 10R, Resistor_SMD:R_0805_2012Metric
- removed R73: 100kR, Resistor_SMD:R_0805_2012Metric
- removed RV1: 200R, Potentiometer_THT:Potentiometer_Bourns_3296X_Horizontal
- removed RV2: 10kR, Potentiometer_THT:Potentiometer_Bourns_3296X_Horizontal
- removed SW1: SW_Push, Button_Switch_THT:SW_PUSH_6mm_H13mm
- removed U1, U17, U24, U38, U45, U8: 74AHC2G125, Package_SO:TSSOP-8_3x3mm_P0.65mm
- removed U10, U18, U19, U2, U25, U26, U3, U39, U40, U46, U47, U69, U70, U73, U78, U79, U82, U9: 74AHC00, Package_SO:TSSOP-14_4.4x5mm_P0.65mm
- removed U11, U13, U20, U22, U27, U29, U4, U41, U43, U48, U50, U52, U53, U54, U55, U56, U57, U58, U6, U71, U72, U80, U81: 74AHC1G17, Package_TO_SOT_SMD:SC-74A-5_1.55x2.9mm_P0.95mm
- removed U12, U21, U28, U42, U49, U5: DRV8870DDA, Package_SO:Texas_HTSOP-8-1EP_3.9x4.9mm_P1.27mm_EP2.95x4.9mm_Mask2.4x3.1mm_ThermalVias
- removed U14, U23, U30, U44, U51, U7: INA180A1, Package_TO_SOT_SMD:SOT-23-5
- removed U15, U16, U66: SP3243E, Package_SO:TSSOP-28_4.4x9.7mm_P0.65mm
- removed U31, U32, U35: PCA9555PW, Package_SO:TSSOP-24_4.4x7.8mm_P0.65mm
- removed U33, U34: MCP4431, Package_SO:TSSOP-20_4.4x6.5mm_P0.65mm
- removed U36, U37: MCP6S26, Package_SO:SOIC-14_3.9x8.7mm_P1.27mm
- removed U59: IRM-H6xxT, OptoDevice:Everlight_IRM-H6xxT
- removed U60: LM4040DBZ-3.0, Package_TO_SOT_SMD:SOT-23
- removed U61, U62: AD8648, Package_SO:TSSOP-14_4.4x5mm_P0.65mm
- removed U63: TPS561208DDCR, Package_TO_SOT_SMD:SOT-23-6
- removed U64: TLV75801PDBVR, Package_TO_SOT_SMD:SOT-23-5
- removed U65: LM2776, Package_TO_SOT_SMD:SOT-23-6
- removed U67: USBLC6-2SC6, Package_TO_SOT_SMD:SOT-23-6
- removed U68: FT232RN, Package_SO:SSOP-28_5.3x10.2mm_P0.65mm
- removed U74: LM317_TO-252, Package_TO_SOT_SMD:TO-252-2
- removed U75: ATmega2560-16A, Package_QFP:TQFP-100_14x14mm_P0.5mm
- removed U76: 74AHC573, Package_SO:TSSOP-20_4.4x6.5mm_P0.65mm
- removed U77: AS7C4096A, Package_SO:TSOP-II-44_10.16x18.41mm_P0.8mm
- removed Y1: 16MHz, Crystal:Crystal_SMD_3225-4Pin_3.2x2.5mm

Commit message: Progressed ECAD.
Parts:
- added ?: , , F.Cu at (96.5, 104.1)
- added C1: 100nC, Capacitor_SMD:C_0805_2012Metric, F.Cu at (-44.5, 244.1)
- added C10: 47uC, Capacitor_SMD:C_1210_3225Metric, F.Cu at (-35.0, 266.6)
- added C100: 47uC, Capacitor_SMD:C_1210_3225Metric, F.Cu at (46.4, 33.4)
- added C101: 100nC, Capacitor_SMD:C_0805_2012Metric, F.Cu at (45.5, 134.8)
- added C102: 330nC, Capacitor_SMD:C_0805_2012Metric, F.Cu at (45.5, 137.8)
- added C103: 330nC, Capacitor_SMD:C_0805_2012Metric, F.Cu at (45.5, 140.8)
- added C104: 330nC, Capacitor_SMD:C_0805_2012Metric, F.Cu at (45.5, 143.8)
- added C105: 330nC, Capacitor_SMD:C_0805_2012Metric, F.Cu at (45.5, 146.8)
- added C106: 100nC, Capacitor_SMD:C_0805_2012Metric, F.Cu at (-6.20, 67.2)
- added C107: 100nC, Capacitor_SMD:C_0805_2012Metric, F.Cu at (-6.20, 70.2)
- added C108: 13pC, Capacitor_SMD:C_0805_2012Metric, F.Cu at (-6.20, 73.2)
- added C109: 13pC, Capacitor_SMD:C_0805_2012Metric, F.Cu at (-6.20, 76.2)
- added C11: 100nC, Capacitor_SMD:C_0805_2012Metric, F.Cu at (-40.0, 253.1)
- added C110: 100nC, Capacitor_SMD:C_0805_2012Metric, F.Cu at (-6.20, 79.3)
- added C111: 10uC, Capacitor_SMD:C_0805_2012Metric, F.Cu at (-6.20, 82.3)
- added C112: 100nC, Capacitor_SMD:C_0805_2012Metric, F.Cu at (-61.7, 126.5)
- added C113: 100pC, Capacitor_SMD:C_0805_2012Metric, F.Cu at (-61.7, 129.5)
- added C114: 100pC, Capacitor_SMD:C_0805_2012Metric, F.Cu at (-61.7, 132.5)
- added C115: 100nC, Capacitor_SMD:C_0805_2012Metric, F.Cu at (-61.7, 135.5)
- added C116: 100nC, Capacitor_SMD:C_0805_2012Metric, F.Cu at (-61.7, 138.5)
- added C117: 100nC, Capacitor_SMD:C_0805_2012Metric, F.Cu at (6.34, 125.9)
- added C118: 100nC, Capacitor_SMD:C_0805_2012Metric, F.Cu at (-3.07, 38.5)
- added C119: 100nC, Capacitor_SMD:C_0805_2012Metric, F.Cu at (-3.07, 41.5)
- added C12: 100pC, Capacitor_SMD:C_0805_2012Metric, F.Cu at (-40.0, 256.1)
- added C120: 100nC, Capacitor_SMD:C_0805_2012Metric, F.Cu at (-3.07, 44.5)
- added C121: 100nC, Capacitor_SMD:C_0805_2012Metric, F.Cu at (-3.07, 47.5)
- added C122: 100nC, Capacitor_SMD:C_0805_2012Metric, F.Cu at (-3.07, 50.5)
- added C123: 13pC, Capacitor_SMD:C_0805_2012Metric, F.Cu at (-3.07, 53.5)
- added C124: 100nC, Capacitor_SMD:C_0805_2012Metric, F.Cu at (30.0, 67.2)
- added C125: 100nC, Capacitor_SMD:C_0805_2012Metric, F.Cu at (1.38, 38.5)
- added C126: 100nC, Capacitor_SMD:C_0805_2012Metric, F.Cu at (1.38, 41.5)
- added C127: 100pC, Capacitor_SMD:C_0805_2012Metric, F.Cu at (30.0, 70.2)
- added C128: 100pC, Capacitor_SMD:C_0805_2012Metric, F.Cu at (30.0, 73.2)
- added C129: 13pC, Capacitor_SMD:C_0805_2012Metric, F.Cu at (1.38, 44.5)
- added C13: 100nC, Capacitor_SMD:C_0805_2012Metric, F.Cu at (56.7, 231.7)
- added C130: 100nC, Capacitor_SMD:C_0805_2012Metric, F.Cu at (30.0, 76.2)
- added C131: 100nC, Capacitor_SMD:C_0805_2012Metric, F.Cu at (1.38, 47.5)
- added C132: 100nC, Capacitor_SMD:C_0805_2012Metric, F.Cu at (30.0, 79.3)
- added C133: 100nC, Capacitor_SMD:C_0805_2012Metric, F.Cu at (1.38, 50.5)
- added C14: 100nC, Capacitor_SMD:C_0805_2012Metric, F.Cu at (56.7, 234.7)
- added C15: 100pC, Capacitor_SMD:C_0805_2012Metric, F.Cu at (56.7, 237.7)
- added C16: 100nC, Capacitor_SMD:C_0805_2012Metric, F.Cu at (56.7, 240.8)
- added C17: 100nC, Capacitor_SMD:C_0805_2012Metric, F.Cu at (56.7, 243.8)
- added C18: 100nC, Capacitor_SMD:C_0805_2012Metric, F.Cu at (56.7, 246.8)
- added C19: 100nC, Capacitor_SMD:C_0805_2012Metric, F.Cu at (61.2, 231.7)
- added C2: 100nC, Capacitor_SMD:C_0805_2012Metric, F.Cu at (-44.5, 247.1)
- added C20: 100nC, Capacitor_SMD:C_0805_2012Metric, F.Cu at (61.2, 234.7)
- added C21: 10uC, Capacitor_SMD:C_0805_2012Metric, F.Cu at (61.2, 237.7)
- added C22: 47uC, Capacitor_SMD:C_1210_3225Metric, F.Cu at (66.2, 254.3)
- added C23: 100nC, Capacitor_SMD:C_0805_2012Metric, F.Cu at (61.2, 240.8)
- added C24: 100pC, Capacitor_SMD:C_0805_2012Metric, F.Cu at (61.2, 243.8)
- added C25: 100nC, Capacitor_SMD:C_0805_2012Metric, F.Cu at (45.5, 117.8)
- added C26: 330nC, Capacitor_SMD:C_0805_2012Metric, F.Cu at (45.5, 120.8)
- added C27: 330nC, Capacitor_SMD:C_0805_2012Metric, F.Cu at (45.5, 123.8)
- added C28: 330nC, Capacitor_SMD:C_0805_2012Metric, F.Cu at (45.5, 126.8)
- added C29: 330nC, Capacitor_SMD:C_0805_2012Metric, F.Cu at (45.5, 129.8)
- added C3: 100pC, Capacitor_SMD:C_0805_2012Metric, F.Cu at (-44.5, 250.1)
- added C30: 100nC, Capacitor_SMD:C_0805_2012Metric, F.Cu at (45.6, 96.0)
- added C31: 330nC, Capacitor_SMD:C_0805_2012Metric, F.Cu at (45.6, 99.1)
- added C32: 330nC, Capacitor_SMD:C_0805_2012Metric, F.Cu at (45.6, 102.1)
- added C33: 330nC, Capacitor_SMD:C_0805_2012Metric, F.Cu at (45.6, 105.1)
- added C34: 330nC, Capacitor_SMD:C_0805_2012Metric, F.Cu at (45.6, 108.1)
- added C35: 100nC, Capacitor_SMD:C_0805_2012Metric, F.Cu at (108.0, 231.3)
- added C36: 100nC, Capacitor_SMD:C_0805_2012Metric, F.Cu at (108.0, 234.3)
- added C37: 100pC, Capacitor_SMD:C_0805_2012Metric, F.Cu at (108.0, 237.3)
- added C38: 100nC, Capacitor_SMD:C_0805_2012Metric, F.Cu at (108.0, 240.4)
- added C39: 100nC, Capacitor_SMD:C_0805_2012Metric, F.Cu at (108.0, 243.4)
- added C4: 100nC, Capacitor_SMD:C_0805_2012Metric, F.Cu at (-44.5, 253.1)
- added C40: 100nC, Capacitor_SMD:C_0805_2012Metric, F.Cu at (108.0, 246.4)
- added C41: 100nC, Capacitor_SMD:C_0805_2012Metric, F.Cu at (112.5, 231.3)
- added C42: 100nC, Capacitor_SMD:C_0805_2012Metric, F.Cu at (112.5, 234.3)
- added C43: 10uC, Capacitor_SMD:C_0805_2012Metric, F.Cu at (112.5, 237.3)
- added C44: 47uC, Capacitor_SMD:C_1210_3225Metric, F.Cu at (117.5, 253.9)
- added C45: 100nC, Capacitor_SMD:C_0805_2012Metric, F.Cu at (112.5, 240.4)
- added C46: 100pC, Capacitor_SMD:C_0805_2012Metric, F.Cu at (112.5, 243.4)
- added C47: 100nC, Capacitor_SMD:C_0805_2012Metric, F.Cu at (157.7, 232.1)
- added C48: 100nC, Capacitor_SMD:C_0805_2012Metric, F.Cu at (157.7, 235.1)
- added C49: 100pC, Capacitor_SMD:C_0805_2012Metric, F.Cu at (157.7, 238.1)
- added C5: 100nC, Capacitor_SMD:C_0805_2012Metric, F.Cu at (-44.5, 256.1)
- added C50: 100nC, Capacitor_SMD:C_0805_2012Metric, F.Cu at (157.7, 241.1)
- added C51: 100nC, Capacitor_SMD:C_0805_2012Metric, F.Cu at (157.7, 244.1)
- added C52: 100nC, Capacitor_SMD:C_0805_2012Metric, F.Cu at (157.7, 247.2)
- added C53: 100nC, Capacitor_SMD:C_0805_2012Metric, F.Cu at (162.1, 232.1)
- added C54: 100nC, Capacitor_SMD:C_0805_2012Metric, F.Cu at (162.1, 235.1)
- added C55: 10uC, Capacitor_SMD:C_0805_2012Metric, F.Cu at (162.1, 238.1)
- added C56: 47uC, Capacitor_SMD:C_1210_3225Metric, F.Cu at (167.2, 254.7)
- added C57: 100nC, Capacitor_SMD:C_0805_2012Metric, F.Cu at (162.1, 241.1)
- added C58: 100pC, Capacitor_SMD:C_0805_2012Metric, F.Cu at (162.1, 244.1)
- added C59: 100nC, Capacitor_SMD:C_0805_2012Metric, F.Cu at (-37.6, 29.5)
- added C6: 100nC, Capacitor_SMD:C_0805_2012Metric, F.Cu at (-44.5, 259.1)
- added C60: 100nC, Capacitor_SMD:C_0805_2012Metric, F.Cu at (-37.6, 32.5)
- added C61: 100nC, Capacitor_SMD:C_0805_2012Metric, F.Cu at (20.9, 96.0)
- added C62: 100nC, Capacitor_SMD:C_0805_2012Metric, F.Cu at (20.9, 99.1)
- added C63: 100nC, Capacitor_SMD:C_0805_2012Metric, F.Cu at (20.9, 102.1)
- added C64: 100nC, Capacitor_SMD:C_0805_2012Metric, F.Cu at (20.9, 105.1)
- added C65: 100nC, Capacitor_SMD:C_0805_2012Metric, F.Cu at (-65.0, 84.2)
- added C66: 100nC, Capacitor_SMD:C_0805_2012Metric, F.Cu at (-65.0, 87.3)
- added C67: 100nC, Capacitor_SMD:C_0805_2012Metric, F.Cu at (-65.0, 90.3)
- added C68: 100nC, Capacitor_SMD:C_0805_2012Metric, F.Cu at (-65.0, 93.3)
- added C69: 100nC, Capacitor_SMD:C_0805_2012Metric, F.Cu at (-60.6, 84.2)
- added C7: 100nC, Capacitor_SMD:C_0805_2012Metric, F.Cu at (-40.0, 244.1)
- added C70: 100nC, Capacitor_SMD:C_0805_2012Metric, F.Cu at (-60.6, 87.3)
- added C71: 100nC, Capacitor_SMD:C_0805_2012Metric, F.Cu at (-60.6, 90.3)
- added C72: 100nC, Capacitor_SMD:C_0805_2012Metric, F.Cu at (-60.6, 93.3)
- added C73: 100nC, Capacitor_SMD:C_0805_2012Metric, F.Cu at (-56.1, 84.2)
- added C74: 100nC, Capacitor_SMD:C_0805_2012Metric, F.Cu at (-56.1, 87.3)
- added C75: 100nC, Capacitor_SMD:C_0805_2012Metric, F.Cu at (-56.1, 90.3)
- added C76: 100nC, Capacitor_SMD:C_0805_2012Metric, F.Cu at (-56.1, 93.3)
- added C77: 100nC, Capacitor_SMD:C_0805_2012Metric, F.Cu at (41.9, 67.2)
- added C78: 2.2uC, Capacitor_SMD:C_0805_2012Metric, F.Cu at (41.9, 70.2)
- added C79: 2.2uC, Capacitor_SMD:C_0805_2012Metric, F.Cu at (41.9, 73.2)
- added C8: 100nC, Capacitor_SMD:C_0805_2012Metric, F.Cu at (-40.0, 247.1)
- added C80: 100nC, Capacitor_SMD:C_0805_2012Metric, F.Cu at (39.1, 131.2)
- added C81: 100nC, Capacitor_SMD:C_0805_2012Metric, F.Cu at (39.1, 134.2)
- added C82: 100nC, Capacitor_SMD:C_0805_2012Metric, F.Cu at (39.1, 137.2)
- added C83: 100nC, Capacitor_SMD:C_0805_2012Metric, F.Cu at (39.1, 140.2)
- added C84: 100nC, Capacitor_SMD:C_0805_2012Metric, F.Cu at (39.1, 143.2)
- added C85: 10uC, Capacitor_SMD:C_0805_2012Metric, F.Cu at (18.7, 20.1)
- added C86: 100nC, Capacitor_SMD:C_0805_2012Metric, F.Cu at (18.7, 23.1)
- added C87: 100nC, Capacitor_SMD:C_0805_2012Metric, F.Cu at (18.7, 26.1)
- added C88: 100nC, Capacitor_SMD:C_0805_2012Metric, F.Cu at (18.7, 29.1)
- added C89: 100nC, Capacitor_SMD:C_0805_2012Metric, F.Cu at (18.7, 32.1)
- added C9: 10uC, Capacitor_SMD:C_0805_2012Metric, F.Cu at (-40.0, 250.1)
- added C90: 100nC, Capacitor_SMD:C_0805_2012Metric, F.Cu at (18.7, 35.2)
- added C91: 2.2uC, Capacitor_SMD:C_0805_2012Metric, F.Cu at (23.1, 20.1)
- added C92: 10uC, Capacitor_SMD:C_0805_2012Metric, F.Cu at (23.1, 23.1)
- added C93: 10uC, Capacitor_SMD:C_0805_2012Metric, F.Cu at (23.1, 26.1)
- added C94: 1uC, Capacitor_SMD:C_0805_2012Metric, F.Cu at (23.1, 29.1)
- added C95: 100nC, Capacitor_SMD:C_0805_2012Metric, F.Cu at (23.1, 32.1)
- added C96: 2.2uC, Capacitor_SMD:C_0805_2012Metric, F.Cu at (23.1, 35.2)
- added C97: 100nC, Capacitor_SMD:C_0805_2012Metric, F.Cu at (27.6, 20.1)
- added C98: 13pC, Capacitor_SMD:C_0805_2012Metric, F.Cu at (27.6, 23.1)
- added C99: 10uC, Capacitor_SMD:C_0805_2012Metric, F.Cu at (27.6, 26.1)
- added D1: BAV99, Package_TO_SOT_SMD:SOT-23, F.Cu at (34.4, 131.9)
- added D2: BAV99, Package_TO_SOT_SMD:SOT-23, F.Cu at (34.4, 136.4)
- added D3: SMAJ16CA, Diode_SMD:D_SMA, F.Cu at (46.0, 45.3)
- added D4: BZX84C10, Package_TO_SOT_SMD:SOT-23, F.Cu at (46.0, 37.7)
- added D5: CMS30I30A, Diode_SMD:D_SOD-128, F.Cu at (45.7, 49.6)
- added D6: 4148, Diode_SMD:D_SOD-123, F.Cu at (6.52, 51.7)
- added H1: MountingHole, MountingHole:MountingHole_3.2mm_M3, F.Cu at (0.14, 98.5)
- added H2: MountingHole, MountingHole:MountingHole_3.2mm_M3, F.Cu at (0.14, 106.5)
- added H3: MountingHole, MountingHole:MountingHole_3.2mm_M3, F.Cu at (0.14, 114.4)
- added H4: MountingHole, MountingHole:MountingHole_3.2mm_M3, F.Cu at (0.14, 122.4)
- added J1: Screw_Terminal_01x06, TerminalBlock_Phoenix:TerminalBlock_Phoenix_MPT-0,5-6-2.54_1x06_P2.54mm_Horizontal, F.Cu at (94.0, 109.2)
- added J10: DC, Connector_BarrelJack:BarrelJack_Horizontal, F.Cu at (44.3, 24.0)
- added J11: USB_B, Connector_USB:USB_B_TE_5787834_Vertical, F.Cu at (5.55, 70.8)
- added J12: Conn_01x16, Connector_PinHeader_2.54mm:PinHeader_1x16_P2.54mm_Vertical, F.Cu at (-6.13, 96.8)
- added J13: ICSP, Connector_PinHeader_2.54mm:PinHeader_2x03_P2.54mm_Vertical, F.Cu at (5.51, 28.9)
- added J2: Screw_Terminal_01x06, TerminalBlock_Phoenix:TerminalBlock_Phoenix_MPT-0,5-6-2.54_1x06_P2.54mm_Horizontal, F.Cu at (65.9, 234.3)
- added J3: Screw_Terminal_01x06, TerminalBlock_Phoenix:TerminalBlock_Phoenix_MPT-0,5-6-2.54_1x06_P2.54mm_Horizontal, F.Cu at (117.2, 233.9)
- added J4: Screw_Terminal_01x06, TerminalBlock_Phoenix:TerminalBlock_Phoenix_MPT-0,5-6-2.54_1x06_P2.54mm_Horizontal, F.Cu at (166.9, 234.7)
- added J5: DE9_Pins_MountingHoles, Connector_Dsub:DSUB-9_Pins_Vertical_P2.77x2.84mm_MountingHoles, F.Cu at (-61.8, 24.9)
- added J6: DE9_Pins_MountingHoles, Connector_Dsub:DSUB-9_Pins_Vertical_P2.77x2.84mm_MountingHoles, F.Cu at (-61.8, 40.0)
- added J7: DE9_Pins_MountingHoles, Connector_Dsub:DSUB-9_Pins_Vertical_P2.77x2.84mm_MountingHoles, F.Cu at (-61.8, 55.0)
- added J8: Screw_Terminal_01x06, TerminalBlock_Phoenix:TerminalBlock_Phoenix_MPT-0,5-6-2.54_1x06_P2.54mm_Horizontal, F.Cu at (-64.7, 69.8)
- added J9: Screw_Terminal_01x06, TerminalBlock_Phoenix:TerminalBlock_Phoenix_MPT-0,5-6-2.54_1x06_P2.54mm_Horizontal, F.Cu at (-64.7, 78.4)
- added L1: 4u7L, Inductor_SMD:L_Vishay_IHLP-4040, F.Cu at (36.7, 37.1)
- added L2: 10uL, Inductor_SMD:L_1210_3225Metric, F.Cu at (11.7, 47.6)
- added Q1: QM6015D, Package_TO_SOT_SMD:TO-252-2, F.Cu at (36.7, 47.2)
- added Q2: BC847, Package_TO_SOT_SMD:SOT-23, F.Cu at (6.57, 117.7)
- added Q3: IRLML5203, Package_TO_SOT_SMD:SOT-23, F.Cu at (6.57, 122.2)
- added R1: 1kR, Resistor_SMD:R_0805_2012Metric, F.Cu at (-21.4, 259.2)
- added R10: 1kR, Resistor_SMD:R_0805_2012Metric, F.Cu at (180.8, 247.2)
- added R11: 150mR, Resistor_SMD:R_1206_3216Metric, F.Cu at (158.3, 255.0)
- added R12: 1kR, Resistor_SMD:R_0805_2012Metric, F.Cu at (180.8, 250.2)
- added R13: 10kR, Resistor_SMD:R_0805_2012Metric, F.Cu at (-33.1, 29.4)
- added R14: 10kR, Resistor_SMD:R_0805_2012Metric, F.Cu at (-33.1, 32.4)
- added R15: 10kR, Resistor_SMD:R_0805_2012Metric, F.Cu at (20.9, 108.1)
- added R16: 10kR, Resistor_SMD:R_0805_2012Metric, F.Cu at (20.9, 111.0)
- added R17: 10kR, Resistor_SMD:R_0805_2012Metric, F.Cu at (-51.7, 84.2)
- added R18: 10kR, Resistor_SMD:R_0805_2012Metric, F.Cu at (-51.7, 87.2)
- added R19: 10kR, Resistor_SMD:R_0805_2012Metric, F.Cu at (-51.7, 90.1)
- added R2: 150mR, Resistor_SMD:R_1206_3216Metric, F.Cu at (96.5, 100.5)
- added R20: 10kR, Resistor_SMD:R_0805_2012Metric, F.Cu at (-51.7, 93.1)
- added R21: 10kR, Resistor_SMD:R_0805_2012Metric, F.Cu at (-47.3, 84.2)
- added R22: 10kR, Resistor_SMD:R_0805_2012Metric, F.Cu at (-47.3, 87.2)
- added R23: 10kR, Resistor_SMD:R_0805_2012Metric, F.Cu at (-47.3, 90.1)
- added R24: 10kR, Resistor_SMD:R_0805_2012Metric, F.Cu at (-47.3, 93.1)
- added R25: 10kR, Resistor_SMD:R_0805_2012Metric, F.Cu at (-42.9, 84.2)
- added R26: 10kR, Resistor_SMD:R_0805_2012Metric, F.Cu at (-42.9, 87.2)
- added R27: 10kR, Resistor_SMD:R_0805_2012Metric, F.Cu at (-42.9, 90.1)
- added R28: 10kR, Resistor_SMD:R_0805_2012Metric, F.Cu at (-42.9, 93.1)
- added R29: 160R, Resistor_SMD:R_0805_2012Metric, F.Cu at (46.3, 73.7)
- added R3: 1kR, Resistor_SMD:R_0805_2012Metric, F.Cu at (-21.4, 262.1)
- added R30: 10kR, Resistor_SMD:R_0805_2012Metric, F.Cu at (46.3, 76.7)
- added R31: 1kR, Resistor_SMD:R_0805_2012Metric, F.Cu at (20.9, 117.7)
- added R32: 10kR, Resistor_SMD:R_0805_2012Metric, F.Cu at (20.9, 120.7)
- added R33: 10kR, Resistor_SMD:R_0805_2012Metric, F.Cu at (20.9, 123.6)
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Routing:
- added copper zone on F.Cu, net /Motor Control/H-bridge #1/MOTOR+
- added copper zone on F.Cu, net /Motor Control/H-bridge #1/MOTOR-
- added copper zone on F.Cu, net GND
Other:
- copper layers 2 -> 4

Commit message: Progressed ECAD.
Parts:
- added ?: , , F.Cu at (90.8, 106.0)
- moved C11 214.2 mm to (110.7, 101.0)
- moved C10 204.0 mm to (86.1, 102.4), turned to 180 degrees
- moved C9 197.0 mm to (86.4, 98.9), turned to 180 degrees
- moved C8 197.0 mm to (86.6, 96.1), turned to 180 degrees
- moved U5 2.37 mm to (95.9, 93.0)
- moved U7 1.65 mm to (102.9, 102.0), turned to -90 degrees
- moved R2 0.19 mm to (96.5, 100.3)
Routing:
- net Net-(U5-ISEN): track 0.00 -> 8.19 mm, vias 0 -> 2
- added copper zone on F.Cu, net Net-(U5-ISEN)
- added copper zone on B.Cu, net VDC
- added copper zone on F.Cu, net VDC

Commit message: Update BDCMotorController.kicad_pcb
Parts:
- moved C10 2.84 mm to (88.9, 102.9)
- moved C9 2.65 mm to (88.9, 99.7)
- moved C8 2.50 mm to (88.9, 97.2)
Changed lines of the file:
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@@
 	(footprint "Capacitor_SMD:C_0805_2012Metric"
 		(layer "F.Cu")
-		(at 86.36 98.933 180)
+		(at 88.9 99.695 180)
 		(descr "Capacitor SMD 0805 (2012 Metric), square (rectangular) end terminal, IPC-7351 nominal, (Body size source: IPC-SM-782 page 76, https://www.pcb-3d.com/wordpress/wp-content/uploads/ipc-sm-782a_amendment_1_and_2.pdf, https://docs.google.com/spreadsheets/d/1BsfQQcO9C6DZCsRaXUlFlo91Tg2WpOkGARC1WS5S8t0/edit?usp=sharing), generated with kicad-footprint-generator")
 		(tags "capacitor")
@@
 	(footprint "Capacitor_SMD:C_0805_2012Metric"
 		(layer "F.Cu")
-		(at 86.614 96.139 180)
+		(at 88.9 97.155 180)
 		(descr "Capacitor SMD 0805 (2012 Metric), square (rectangular) end terminal, IPC-7351 nominal, (Body size source: IPC-SM-782 page 76, https://www.pcb-3d.com/wordpress/wp-content/uploads/ipc-sm-782a_amendment_1_and_2.pdf, https://docs.google.com/spreadsheets/d/1BsfQQcO9C6DZCsRaXUlFlo91Tg2WpOkGARC1WS5S8t0/edit?usp=sharing), generated with kicad-footprint-generator")
 		(tags "capacitor")
@@
 	(footprint "Capacitor_SMD:C_1210_3225Metric"
 		(layer "F.Cu")
-		(at 86.106 102.362 180)
+		(at 88.9 102.87 180)
 		(descr "Capacitor SMD 1210 (3225 Metric), square (rectangular) end terminal, IPC-7351 nominal, (Body size source: IPC-SM-782 page 76, https://www.pcb-3d.com/wordpress/wp-content/uploads/ipc-sm-782a_amendment_1_and_2.pdf), generated with kicad-footprint-generator")
 		(tags "capacitor")
@@
 		(polygon
 			(pts
+				(xy 97.79 105.664) (xy 97.79 105.156) (xy 94.996 105.156) (xy 94.996 105.664)
+			)
+		)
+	)
+	(zone
+		(net 0)
+		(net_name "")
+		(layer "F.Cu")
+		(hatch edge 0.5)
+		(connect_pads yes
+			(clearance 0)
+		)
+		(min_thickness 0.25)
+		(filled_areas_thickness no)
+		(keepout
+			(tracks allowed)
+			(vias allowed)
+			(pads allowed)
+			(copperpour not_allowed)
+			(footprints allowed)
+		)
+		(placement
+			(enabled no)
+			(sheetname "")
+		)
+		(fill
+			(thermal_gap 0.5)
+			(thermal_bridge_width 0.5)
+		)
+		(polygon
+			(pts
 				(xy 100.076 110.744) (xy 100.584 110.744) (xy 100.584 97.536) (xy 100.076 97.536)
 			)
@@
 			(thermal_gap 0.5)
 			(thermal_bridge_width 0.5)
-			(smoothing fillet)
-			(radius 1)
 		)
 		(polygon
@@
 		(polygon
 			(pts
-				(xy 95.25 101.6) (xy 97.79 101.6) (xy 97.79 105.41) (xy 95.25 105.41)
+				(xy 95.25 101.6) (xy 97.79 101.6) (xy 97.79 104.14) (xy 95.25 104.14)
 			)
 		)
@@
 		(polygon
 			(pts
-				(xy 97.536 105.156) (xy 98.044 105.156) (xy 98.044 98.044) (xy 97.536 98.044)
+				(xy 97.536 105.664) (xy 98.044 105.664) (xy 98.044 98.044) (xy 97.536 98.044)
 			)
 		)

Commit message: Progressed ECAD.
Parts:
- C11, U7: moved to B.Cu
- moved C11 7.88 mm to (103.0, 99.5), turned to 90 degrees
- moved U7 4.18 mm to (99.5, 99.5), turned to 0 degrees
- moved C9 1.20 mm to (89.9, 99.1)
- moved C10 1.14 mm to (89.4, 101.9)
- moved C8 1.09 mm to (89.9, 96.8)
- moved ? 0.90 mm to (91.4, 106.7)
Routing:
- net Net-(U5-ISEN): track 8.19 -> 1.34 mm, vias 2 -> 1

Commit message: Update BDCMotorController.kicad_pcb
Parts:
- added ?: , , F.Cu at (88.9, 104.1)
- moved C1 250.8 mm to (93.9, 34.8)
- moved C12 250.8 mm to (98.4, 46.9)
- moved C2 250.8 mm to (93.9, 37.9)
- moved C3 250.8 mm to (93.9, 40.9)
- moved C4 250.8 mm to (93.9, 43.9)
- moved C5 250.8 mm to (93.9, 46.9)
- moved C6 250.8 mm to (93.9, 49.9)
- moved C7 250.8 mm to (98.4, 34.8)
- moved R1 250.8 mm to (117.0, 50.0)
- moved R3 250.8 mm to (117.0, 52.9)
- moved U1 250.8 mm to (95.2, 53.7)
- moved U2 250.8 mm to (105.0, 45.3)
- moved U4 250.8 mm to (112.1, 50.9)
- moved U6 250.8 mm to (112.1, 55.5)
- moved U3 250.8 mm to (105.0, 52.0)
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